File: hardware/68040pc.kicad_pcb (KiCad board)
At the start: 4 copper layers, 221 x 243.8 mm, 23 parts, among them J1 EXP, J13 DIN-5_180degree, J14 Mini-DIN-6, J15 COM1, J16 COM2, J17 LPT, J2 EXP, J3 EXP, J4 EXP, J5 EXP, J6 EXP, J7 EXP, J8 EXP, P8 Conn_01x06, P9 Conn_01x06, U1 68LC040, U2 ICE40HX4K-TQ144, U3 SN74ALVC164245, U4 SN74ALVC164245

Commit message: reconfigure expansion slot schematic
Parts:
- added C3: 0.1u, Capacitor_SMD:C_0603_1608Metric, F.Cu at (247.2, 279.0)
- added D1: LTST-C191KGKT, LED_SMD:LED_0603_1608Metric, F.Cu at (251.3, 285.8)
- added R1: 2.2K, Resistor_SMD:R_0603_1608Metric, F.Cu at (247.2, 281.5)
- added R2: 10K, Resistor_SMD:R_0603_1608Metric, F.Cu at (247.2, 284.0)
- added R3: 10K, Resistor_SMD:R_0603_1608Metric, F.Cu at (247.2, 286.5)
- added U5: W25Q32JVSSIM, Package_SO:SOIC-8_5.23x5.23mm_P1.27mm, F.Cu at (254.4, 281.1)
- moved U3 0.08 mm to (238.8, 236.2)
Connections:
- J1 pad A12: unconnected-(J1-PadA12) -> /Expansion/A1
- J1 pad A13: unconnected-(J1-PadA13) -> /Expansion/A3
- J1 pad A14: unconnected-(J1-PadA14) -> /Expansion/A5
- J1 pad A15: unconnected-(J1-PadA15) -> /Expansion/A7
- J1 pad A16: unconnected-(J1-PadA16) -> /Expansion/A9
- J1 pad A17: unconnected-(J1-PadA17) -> /Expansion/A11
- J1 pad A18: unconnected-(J1-PadA18) -> /Expansion/A13
- J1 pad A19: unconnected-(J1-PadA19) -> /Expansion/A15
- J1 pad A20: unconnected-(J1-PadA20) -> /Expansion/A17
- J1 pad A21: unconnected-(J1-PadA21) -> /Expansion/A19
- J1 pad B17: unconnected-(J1-PadB17) -> /Expansion/A0
- J1 pad B18: unconnected-(J1-PadB18) -> /Expansion/A20
- J1 pad B19: unconnected-(J1-PadB19) -> /Expansion/A21
- J1 pad B20: unconnected-(J1-PadB20) -> /Expansion/A22
- J1 pad B21: unconnected-(J1-PadB21) -> /Expansion/A23
- J1 pad B22: unconnected-(J1-PadB22) -> /Expansion/A24
- J1 pad B23: unconnected-(J1-PadB23) -> /Expansion/A25
- J1 pad B24: unconnected-(J1-PadB24) -> /Expansion/A26
- J1 pad B25: unconnected-(J1-PadB25) -> /Expansion/A27
- J1 pad B26: unconnected-(J1-PadB26) -> /Expansion/A28
- J1 pad B27: unconnected-(J1-PadB27) -> /Expansion/A29
- J1 pad B28: unconnected-(J1-PadB28) -> /Expansion/A30
- J1 pad B29: unconnected-(J1-PadB29) -> /Expansion/A31
- J1 pad C12: unconnected-(J1-PadC12) -> /Expansion/A2
- J1 pad C13: unconnected-(J1-PadC13) -> /Expansion/A4
- J1 pad C14: unconnected-(J1-PadC14) -> /Expansion/A6
- J1 pad C15: unconnected-(J1-PadC15) -> /Expansion/A8
- J1 pad C16: unconnected-(J1-PadC16) -> /Expansion/A10
- J1 pad C17: unconnected-(J1-PadC17) -> /Expansion/A12
- J1 pad C18: unconnected-(J1-PadC18) -> /Expansion/A14
- J1 pad C19: unconnected-(J1-PadC19) -> /Expansion/A16
- J1 pad C20: unconnected-(J1-PadC20) -> /Expansion/A18
- J2 pad A12: unconnected-(J2-PadA12) -> /Expansion/A1
- J2 pad A13: unconnected-(J2-PadA13) -> /Expansion/A3
- J2 pad A14: unconnected-(J2-PadA14) -> /Expansion/A5
- J2 pad A15: unconnected-(J2-PadA15) -> /Expansion/A7
- J2 pad A16: unconnected-(J2-PadA16) -> /Expansion/A9
- J2 pad A17: unconnected-(J2-PadA17) -> /Expansion/A11
- J2 pad A18: unconnected-(J2-PadA18) -> /Expansion/A13
- J2 pad A19: unconnected-(J2-PadA19) -> /Expansion/A15
- J2 pad A20: unconnected-(J2-PadA20) -> /Expansion/A17
- J2 pad A21: unconnected-(J2-PadA21) -> /Expansion/A19
- J2 pad B17: unconnected-(J2-PadB17) -> /Expansion/A0
- J2 pad B18: unconnected-(J2-PadB18) -> /Expansion/A20
- J2 pad B19: unconnected-(J2-PadB19) -> /Expansion/A21
- J2 pad B20: unconnected-(J2-PadB20) -> /Expansion/A22
- J2 pad B21: unconnected-(J2-PadB21) -> /Expansion/A23
- J2 pad B22: unconnected-(J2-PadB22) -> /Expansion/A24
- J2 pad B23: unconnected-(J2-PadB23) -> /Expansion/A25
- J2 pad B24: unconnected-(J2-PadB24) -> /Expansion/A26
- J2 pad B25: unconnected-(J2-PadB25) -> /Expansion/A27
- J2 pad B26: unconnected-(J2-PadB26) -> /Expansion/A28
- J2 pad B27: unconnected-(J2-PadB27) -> /Expansion/A29
- J2 pad B28: unconnected-(J2-PadB28) -> /Expansion/A30
- J2 pad B29: unconnected-(J2-PadB29) -> /Expansion/A31
- J2 pad C12: unconnected-(J2-PadC12) -> /Expansion/A2
- J2 pad C13: unconnected-(J2-PadC13) -> /Expansion/A4
- J2 pad C14: unconnected-(J2-PadC14) -> /Expansion/A6
- J2 pad C15: unconnected-(J2-PadC15) -> /Expansion/A8
- J2 pad C16: unconnected-(J2-PadC16) -> /Expansion/A10
- J2 pad C17: unconnected-(J2-PadC17) -> /Expansion/A12
- J2 pad C18: unconnected-(J2-PadC18) -> /Expansion/A14
- J2 pad C19: unconnected-(J2-PadC19) -> /Expansion/A16
- J2 pad C20: unconnected-(J2-PadC20) -> /Expansion/A18
- J3 pad A10: unconnected-(J3-PadA10) -> /Expansion/D14
- J3 pad A12: unconnected-(J3-PadA12) -> /Expansion/A1
- J3 pad A13: unconnected-(J3-PadA13) -> /Expansion/A3
- J3 pad A14: unconnected-(J3-PadA14) -> /Expansion/A5
- J3 pad A15: unconnected-(J3-PadA15) -> /Expansion/A7
- J3 pad A16: unconnected-(J3-PadA16) -> /Expansion/A9
- J3 pad A17: unconnected-(J3-PadA17) -> /Expansion/A11
- J3 pad A18: unconnected-(J3-PadA18) -> /Expansion/A13
- J3 pad A19: unconnected-(J3-PadA19) -> /Expansion/A15
- J3 pad A20: unconnected-(J3-PadA20) -> /Expansion/A17
- J3 pad A21: unconnected-(J3-PadA21) -> /Expansion/A19
- J3 pad A3: unconnected-(J3-PadA3) -> /Expansion/D0
- J3 pad A4: unconnected-(J3-PadA4) -> /Expansion/D2
- J3 pad A5: unconnected-(J3-PadA5) -> /Expansion/D4
- J3 pad A6: unconnected-(J3-PadA6) -> /Expansion/D6
- J3 pad A7: unconnected-(J3-PadA7) -> /Expansion/D8
- J3 pad A8: unconnected-(J3-PadA8) -> /Expansion/D10
- J3 pad A9: unconnected-(J3-PadA9) -> /Expansion/D12
- J3 pad B1: unconnected-(J3-PadB1) -> /Expansion/D16
- J3 pad B10: unconnected-(J3-PadB10) -> /Expansion/D25
- J3 pad B11: unconnected-(J3-PadB11) -> /Expansion/D26
- J3 pad B12: unconnected-(J3-PadB12) -> /Expansion/D27
- J3 pad B13: unconnected-(J3-PadB13) -> /Expansion/D28
- J3 pad B14: unconnected-(J3-PadB14) -> /Expansion/D29
- J3 pad B15: unconnected-(J3-PadB15) -> /Expansion/D30
- J3 pad B16: unconnected-(J3-PadB16) -> /Expansion/D31
- J3 pad B17: unconnected-(J3-PadB17) -> /Expansion/A0
- J3 pad B18: unconnected-(J3-PadB18) -> /Expansion/A20
- J3 pad B19: unconnected-(J3-PadB19) -> /Expansion/A21
- J3 pad B2: unconnected-(J3-PadB2) -> /Expansion/D17
- J3 pad B20: unconnected-(J3-PadB20) -> /Expansion/A22
- J3 pad B21: unconnected-(J3-PadB21) -> /Expansion/A23
- J3 pad B22: unconnected-(J3-PadB22) -> /Expansion/A24
- J3 pad B23: unconnected-(J3-PadB23) -> /Expansion/A25
- J3 pad B24: unconnected-(J3-PadB24) -> /Expansion/A26
- J3 pad B25: unconnected-(J3-PadB25) -> /Expansion/A27
- J3 pad B26: unconnected-(J3-PadB26) -> /Expansion/A28
- J3 pad B27: unconnected-(J3-PadB27) -> /Expansion/A29
- J3 pad B28: unconnected-(J3-PadB28) -> /Expansion/A30
- J3 pad B29: unconnected-(J3-PadB29) -> /Expansion/A31
- J3 pad B3: unconnected-(J3-PadB3) -> /Expansion/D18
- J3 pad B4: unconnected-(J3-PadB4) -> /Expansion/D19
- J3 pad B5: unconnected-(J3-PadB5) -> /Expansion/D20
- J3 pad B6: unconnected-(J3-PadB6) -> /Expansion/D21
- J3 pad B7: unconnected-(J3-PadB7) -> /Expansion/D22
- J3 pad B8: unconnected-(J3-PadB8) -> /Expansion/D23
- J3 pad B9: unconnected-(J3-PadB9) -> /Expansion/D24
- J3 pad C10: unconnected-(J3-PadC10) -> /Expansion/D15
- J3 pad C12: unconnected-(J3-PadC12) -> /Expansion/A2
- J3 pad C13: unconnected-(J3-PadC13) -> /Expansion/A4
- J3 pad C14: unconnected-(J3-PadC14) -> /Expansion/A6
- J3 pad C15: unconnected-(J3-PadC15) -> /Expansion/A8
- J3 pad C16: unconnected-(J3-PadC16) -> /Expansion/A10
- J3 pad C17: unconnected-(J3-PadC17) -> /Expansion/A12
- J3 pad C18: unconnected-(J3-PadC18) -> /Expansion/A14
- J3 pad C19: unconnected-(J3-PadC19) -> /Expansion/A16
- J3 pad C20: unconnected-(J3-PadC20) -> /Expansion/A18
- J3 pad C3: unconnected-(J3-PadC3) -> /Expansion/D1
- J3 pad C4: unconnected-(J3-PadC4) -> /Expansion/D3
- J3 pad C5: unconnected-(J3-PadC5) -> /Expansion/D5
- J3 pad C6: unconnected-(J3-PadC6) -> /Expansion/D7
- J3 pad C7: unconnected-(J3-PadC7) -> /Expansion/D9
- J3 pad C8: unconnected-(J3-PadC8) -> /Expansion/D11
- J3 pad C9: unconnected-(J3-PadC9) -> /Expansion/D13
- J4 pad A10: unconnected-(J4-PadA10) -> /Expansion/D14
- J4 pad A12: unconnected-(J4-PadA12) -> /Expansion/A1
- J4 pad A13: unconnected-(J4-PadA13) -> /Expansion/A3
- J4 pad A14: unconnected-(J4-PadA14) -> /Expansion/A5
- J4 pad A15: unconnected-(J4-PadA15) -> /Expansion/A7
- J4 pad A16: unconnected-(J4-PadA16) -> /Expansion/A9
- J4 pad A17: unconnected-(J4-PadA17) -> /Expansion/A11
- J4 pad A18: unconnected-(J4-PadA18) -> /Expansion/A13
- J4 pad A19: unconnected-(J4-PadA19) -> /Expansion/A15
- J4 pad A20: unconnected-(J4-PadA20) -> /Expansion/A17
- J4 pad A21: unconnected-(J4-PadA21) -> /Expansion/A19
- J4 pad A3: unconnected-(J4-PadA3) -> /Expansion/D0
- J4 pad A4: unconnected-(J4-PadA4) -> /Expansion/D2
- J4 pad A5: unconnected-(J4-PadA5) -> /Expansion/D4
- J4 pad A6: unconnected-(J4-PadA6) -> /Expansion/D6
- J4 pad A7: unconnected-(J4-PadA7) -> /Expansion/D8
- J4 pad A8: unconnected-(J4-PadA8) -> /Expansion/D10
- J4 pad A9: unconnected-(J4-PadA9) -> /Expansion/D12
- J4 pad B1: unconnected-(J4-PadB1) -> /Expansion/D16
- J4 pad B10: unconnected-(J4-PadB10) -> /Expansion/D25
- J4 pad B11: unconnected-(J4-PadB11) -> /Expansion/D26
- J4 pad B12: unconnected-(J4-PadB12) -> /Expansion/D27
- J4 pad B13: unconnected-(J4-PadB13) -> /Expansion/D28
- J4 pad B14: unconnected-(J4-PadB14) -> /Expansion/D29
- J4 pad B15: unconnected-(J4-PadB15) -> /Expansion/D30
- J4 pad B16: unconnected-(J4-PadB16) -> /Expansion/D31
- J4 pad B17: unconnected-(J4-PadB17) -> /Expansion/A0
- J4 pad B18: unconnected-(J4-PadB18) -> /Expansion/A20
- J4 pad B19: unconnected-(J4-PadB19) -> /Expansion/A21
- J4 pad B2: unconnected-(J4-PadB2) -> /Expansion/D17
- J4 pad B20: unconnected-(J4-PadB20) -> /Expansion/A22
- J4 pad B21: unconnected-(J4-PadB21) -> /Expansion/A23
- J4 pad B22: unconnected-(J4-PadB22) -> /Expansion/A24
- J4 pad B23: unconnected-(J4-PadB23) -> /Expansion/A25
- J4 pad B24: unconnected-(J4-PadB24) -> /Expansion/A26
- J4 pad B25: unconnected-(J4-PadB25) -> /Expansion/A27
- J4 pad B26: unconnected-(J4-PadB26) -> /Expansion/A28
- J4 pad B27: unconnected-(J4-PadB27) -> /Expansion/A29
- J4 pad B28: unconnected-(J4-PadB28) -> /Expansion/A30
- J4 pad B29: unconnected-(J4-PadB29) -> /Expansion/A31
- J4 pad B3: unconnected-(J4-PadB3) -> /Expansion/D18
- J4 pad B4: unconnected-(J4-PadB4) -> /Expansion/D19
- J4 pad B5: unconnected-(J4-PadB5) -> /Expansion/D20
- J4 pad B6: unconnected-(J4-PadB6) -> /Expansion/D21
- J4 pad B7: unconnected-(J4-PadB7) -> /Expansion/D22
- J4 pad B8: unconnected-(J4-PadB8) -> /Expansion/D23
- J4 pad B9: unconnected-(J4-PadB9) -> /Expansion/D24
- J4 pad C10: unconnected-(J4-PadC10) -> /Expansion/D15
- J4 pad C12: unconnected-(J4-PadC12) -> /Expansion/A2
- J4 pad C13: unconnected-(J4-PadC13) -> /Expansion/A4
- J4 pad C14: unconnected-(J4-PadC14) -> /Expansion/A6
- J4 pad C15: unconnected-(J4-PadC15) -> /Expansion/A8
- J4 pad C16: unconnected-(J4-PadC16) -> /Expansion/A10
- J4 pad C17: unconnected-(J4-PadC17) -> /Expansion/A12
- J4 pad C18: unconnected-(J4-PadC18) -> /Expansion/A14
- J4 pad C19: unconnected-(J4-PadC19) -> /Expansion/A16
- J4 pad C20: unconnected-(J4-PadC20) -> /Expansion/A18
- J4 pad C3: unconnected-(J4-PadC3) -> /Expansion/D1
- J4 pad C4: unconnected-(J4-PadC4) -> /Expansion/D3
- J4 pad C5: unconnected-(J4-PadC5) -> /Expansion/D5
- J4 pad C6: unconnected-(J4-PadC6) -> /Expansion/D7
- J4 pad C7: unconnected-(J4-PadC7) -> /Expansion/D9
- J4 pad C8: unconnected-(J4-PadC8) -> /Expansion/D11
- J4 pad C9: unconnected-(J4-PadC9) -> /Expansion/D13
- J5 pad A10: unconnected-(J5-PadA10) -> /Expansion/D14
- J5 pad A12: unconnected-(J5-PadA12) -> /Expansion/A1
- J5 pad A13: unconnected-(J5-PadA13) -> /Expansion/A3
- J5 pad A14: unconnected-(J5-PadA14) -> /Expansion/A5
- J5 pad A15: unconnected-(J5-PadA15) -> /Expansion/A7
- J5 pad A16: unconnected-(J5-PadA16) -> /Expansion/A9
- J5 pad A17: unconnected-(J5-PadA17) -> /Expansion/A11
- J5 pad A18: unconnected-(J5-PadA18) -> /Expansion/A13
- J5 pad A19: unconnected-(J5-PadA19) -> /Expansion/A15
- J5 pad A20: unconnected-(J5-PadA20) -> /Expansion/A17
- J5 pad A21: unconnected-(J5-PadA21) -> /Expansion/A19
- J5 pad A3: unconnected-(J5-PadA3) -> /Expansion/D0
- J5 pad A4: unconnected-(J5-PadA4) -> /Expansion/D2
- J5 pad A5: unconnected-(J5-PadA5) -> /Expansion/D4
- J5 pad A6: unconnected-(J5-PadA6) -> /Expansion/D6
- J5 pad A7: unconnected-(J5-PadA7) -> /Expansion/D8
- J5 pad A8: unconnected-(J5-PadA8) -> /Expansion/D10
- J5 pad A9: unconnected-(J5-PadA9) -> /Expansion/D12
- J5 pad B1: unconnected-(J5-PadB1) -> /Expansion/D16
- J5 pad B10: unconnected-(J5-PadB10) -> /Expansion/D25
- J5 pad B11: unconnected-(J5-PadB11) -> /Expansion/D26
- J5 pad B12: unconnected-(J5-PadB12) -> /Expansion/D27
- J5 pad B13: unconnected-(J5-PadB13) -> /Expansion/D28
- J5 pad B14: unconnected-(J5-PadB14) -> /Expansion/D29
- J5 pad B15: unconnected-(J5-PadB15) -> /Expansion/D30
- J5 pad B16: unconnected-(J5-PadB16) -> /Expansion/D31
- J5 pad B17: unconnected-(J5-PadB17) -> /Expansion/A0
- J5 pad B18: unconnected-(J5-PadB18) -> /Expansion/A20
- J5 pad B19: unconnected-(J5-PadB19) -> /Expansion/A21
- J5 pad B2: unconnected-(J5-PadB2) -> /Expansion/D17
- J5 pad B20: unconnected-(J5-PadB20) -> /Expansion/A22
- J5 pad B21: unconnected-(J5-PadB21) -> /Expansion/A23
- J5 pad B22: unconnected-(J5-PadB22) -> /Expansion/A24
- J5 pad B23: unconnected-(J5-PadB23) -> /Expansion/A25
- J5 pad B24: unconnected-(J5-PadB24) -> /Expansion/A26
- J5 pad B25: unconnected-(J5-PadB25) -> /Expansion/A27
- J5 pad B26: unconnected-(J5-PadB26) -> /Expansion/A28
- J5 pad B27: unconnected-(J5-PadB27) -> /Expansion/A29
- J5 pad B28: unconnected-(J5-PadB28) -> /Expansion/A30
- J5 pad B29: unconnected-(J5-PadB29) -> /Expansion/A31
- J5 pad B3: unconnected-(J5-PadB3) -> /Expansion/D18
- J5 pad B4: unconnected-(J5-PadB4) -> /Expansion/D19
- J5 pad B5: unconnected-(J5-PadB5) -> /Expansion/D20
- J5 pad B6: unconnected-(J5-PadB6) -> /Expansion/D21
- J5 pad B7: unconnected-(J5-PadB7) -> /Expansion/D22
- J5 pad B8: unconnected-(J5-PadB8) -> /Expansion/D23
- J5 pad B9: unconnected-(J5-PadB9) -> /Expansion/D24
- J5 pad C10: unconnected-(J5-PadC10) -> /Expansion/D15
- J5 pad C12: unconnected-(J5-PadC12) -> /Expansion/A2
- J5 pad C13: unconnected-(J5-PadC13) -> /Expansion/A4
- J5 pad C14: unconnected-(J5-PadC14) -> /Expansion/A6
- J5 pad C15: unconnected-(J5-PadC15) -> /Expansion/A8
- J5 pad C16: unconnected-(J5-PadC16) -> /Expansion/A10
- J5 pad C17: unconnected-(J5-PadC17) -> /Expansion/A12
- J5 pad C18: unconnected-(J5-PadC18) -> /Expansion/A14
- J5 pad C19: unconnected-(J5-PadC19) -> /Expansion/A16
- J5 pad C20: unconnected-(J5-PadC20) -> /Expansion/A18
- J5 pad C3: unconnected-(J5-PadC3) -> /Expansion/D1
- J5 pad C4: unconnected-(J5-PadC4) -> /Expansion/D3
- J5 pad C5: unconnected-(J5-PadC5) -> /Expansion/D5
- J5 pad C6: unconnected-(J5-PadC6) -> /Expansion/D7
- J5 pad C7: unconnected-(J5-PadC7) -> /Expansion/D9
- J5 pad C8: unconnected-(J5-PadC8) -> /Expansion/D11
- J5 pad C9: unconnected-(J5-PadC9) -> /Expansion/D13
- J6 pad A10: unconnected-(J6-PadA10) -> /Expansion/D14
- J6 pad A12: unconnected-(J6-PadA12) -> /Expansion/A1
- J6 pad A13: unconnected-(J6-PadA13) -> /Expansion/A3
- J6 pad A14: unconnected-(J6-PadA14) -> /Expansion/A5
- J6 pad A15: unconnected-(J6-PadA15) -> /Expansion/A7
- J6 pad A16: unconnected-(J6-PadA16) -> /Expansion/A9
- J6 pad A17: unconnected-(J6-PadA17) -> /Expansion/A11
- J6 pad A18: unconnected-(J6-PadA18) -> /Expansion/A13
- J6 pad A19: unconnected-(J6-PadA19) -> /Expansion/A15
- J6 pad A20: unconnected-(J6-PadA20) -> /Expansion/A17
- J6 pad A21: unconnected-(J6-PadA21) -> /Expansion/A19
- J6 pad A3: unconnected-(J6-PadA3) -> /Expansion/D0
- J6 pad A4: unconnected-(J6-PadA4) -> /Expansion/D2
- J6 pad A5: unconnected-(J6-PadA5) -> /Expansion/D4
- J6 pad A6: unconnected-(J6-PadA6) -> /Expansion/D6
- J6 pad A7: unconnected-(J6-PadA7) -> /Expansion/D8
- J6 pad A8: unconnected-(J6-PadA8) -> /Expansion/D10
- J6 pad A9: unconnected-(J6-PadA9) -> /Expansion/D12
- J6 pad B1: unconnected-(J6-PadB1) -> /Expansion/D16
- J6 pad B10: unconnected-(J6-PadB10) -> /Expansion/D25
- J6 pad B11: unconnected-(J6-PadB11) -> /Expansion/D26
- J6 pad B12: unconnected-(J6-PadB12) -> /Expansion/D27
- J6 pad B13: unconnected-(J6-PadB13) -> /Expansion/D28
- J6 pad B14: unconnected-(J6-PadB14) -> /Expansion/D29
- J6 pad B15: unconnected-(J6-PadB15) -> /Expansion/D30
- J6 pad B16: unconnected-(J6-PadB16) -> /Expansion/D31
- J6 pad B17: unconnected-(J6-PadB17) -> /Expansion/A0
- J6 pad B18: unconnected-(J6-PadB18) -> /Expansion/A20
- J6 pad B19: unconnected-(J6-PadB19) -> /Expansion/A21
- J6 pad B2: unconnected-(J6-PadB2) -> /Expansion/D17
- J6 pad B20: unconnected-(J6-PadB20) -> /Expansion/A22
- J6 pad B21: unconnected-(J6-PadB21) -> /Expansion/A23
- J6 pad B22: unconnected-(J6-PadB22) -> /Expansion/A24
- J6 pad B23: unconnected-(J6-PadB23) -> /Expansion/A25
- J6 pad B24: unconnected-(J6-PadB24) -> /Expansion/A26
- J6 pad B25: unconnected-(J6-PadB25) -> /Expansion/A27
- J6 pad B26: unconnected-(J6-PadB26) -> /Expansion/A28
- J6 pad B27: unconnected-(J6-PadB27) -> /Expansion/A29
- J6 pad B28: unconnected-(J6-PadB28) -> /Expansion/A30
- J6 pad B29: unconnected-(J6-PadB29) -> /Expansion/A31
- J6 pad B3: unconnected-(J6-PadB3) -> /Expansion/D18
- J6 pad B4: unconnected-(J6-PadB4) -> /Expansion/D19
- J6 pad B5: unconnected-(J6-PadB5) -> /Expansion/D20
- J6 pad B6: unconnected-(J6-PadB6) -> /Expansion/D21
- J6 pad B7: unconnected-(J6-PadB7) -> /Expansion/D22
- J6 pad B8: unconnected-(J6-PadB8) -> /Expansion/D23
- J6 pad B9: unconnected-(J6-PadB9) -> /Expansion/D24
- J6 pad C10: unconnected-(J6-PadC10) -> /Expansion/D15
- J6 pad C12: unconnected-(J6-PadC12) -> /Expansion/A2
- J6 pad C13: unconnected-(J6-PadC13) -> /Expansion/A4
- J6 pad C14: unconnected-(J6-PadC14) -> /Expansion/A6
- J6 pad C15: unconnected-(J6-PadC15) -> /Expansion/A8
- J6 pad C16: unconnected-(J6-PadC16) -> /Expansion/A10
- J6 pad C17: unconnected-(J6-PadC17) -> /Expansion/A12
- J6 pad C18: unconnected-(J6-PadC18) -> /Expansion/A14
- J6 pad C19: unconnected-(J6-PadC19) -> /Expansion/A16
- J6 pad C20: unconnected-(J6-PadC20) -> /Expansion/A18
- J6 pad C3: unconnected-(J6-PadC3) -> /Expansion/D1
- J6 pad C4: unconnected-(J6-PadC4) -> /Expansion/D3
- J6 pad C5: unconnected-(J6-PadC5) -> /Expansion/D5
- J6 pad C6: unconnected-(J6-PadC6) -> /Expansion/D7
- J6 pad C7: unconnected-(J6-PadC7) -> /Expansion/D9
- J6 pad C8: unconnected-(J6-PadC8) -> /Expansion/D11
- J6 pad C9: unconnected-(J6-PadC9) -> /Expansion/D13
- J7 pad A10: unconnected-(J7-PadA10) -> /Expansion/D14
- J7 pad A12: unconnected-(J7-PadA12) -> /Expansion/A1
- J7 pad A13: unconnected-(J7-PadA13) -> /Expansion/A3
- J7 pad A14: unconnected-(J7-PadA14) -> /Expansion/A5
- J7 pad A15: unconnected-(J7-PadA15) -> /Expansion/A7
- J7 pad A16: unconnected-(J7-PadA16) -> /Expansion/A9
- J7 pad A17: unconnected-(J7-PadA17) -> /Expansion/A11
- J7 pad A18: unconnected-(J7-PadA18) -> /Expansion/A13
- J7 pad A19: unconnected-(J7-PadA19) -> /Expansion/A15
- J7 pad A20: unconnected-(J7-PadA20) -> /Expansion/A17
- J7 pad A21: unconnected-(J7-PadA21) -> /Expansion/A19
- J7 pad A3: unconnected-(J7-PadA3) -> /Expansion/D0
- J7 pad A4: unconnected-(J7-PadA4) -> /Expansion/D2
- J7 pad A5: unconnected-(J7-PadA5) -> /Expansion/D4
- J7 pad A6: unconnected-(J7-PadA6) -> /Expansion/D6
- J7 pad A7: unconnected-(J7-PadA7) -> /Expansion/D8
- J7 pad A8: unconnected-(J7-PadA8) -> /Expansion/D10
- J7 pad A9: unconnected-(J7-PadA9) -> /Expansion/D12
- J7 pad B1: unconnected-(J7-PadB1) -> /Expansion/D16
- J7 pad B10: unconnected-(J7-PadB10) -> /Expansion/D25
- J7 pad B11: unconnected-(J7-PadB11) -> /Expansion/D26
- J7 pad B12: unconnected-(J7-PadB12) -> /Expansion/D27
- J7 pad B13: unconnected-(J7-PadB13) -> /Expansion/D28
- J7 pad B14: unconnected-(J7-PadB14) -> /Expansion/D29
- J7 pad B15: unconnected-(J7-PadB15) -> /Expansion/D30
- J7 pad B16: unconnected-(J7-PadB16) -> /Expansion/D31
- J7 pad B17: unconnected-(J7-PadB17) -> /Expansion/A0
- J7 pad B18: unconnected-(J7-PadB18) -> /Expansion/A20
- J7 pad B19: unconnected-(J7-PadB19) -> /Expansion/A21
- J7 pad B2: unconnected-(J7-PadB2) -> /Expansion/D17
- J7 pad B20: unconnected-(J7-PadB20) -> /Expansion/A22
- J7 pad B21: unconnected-(J7-PadB21) -> /Expansion/A23
- J7 pad B22: unconnected-(J7-PadB22) -> /Expansion/A24
- J7 pad B23: unconnected-(J7-PadB23) -> /Expansion/A25
- J7 pad B24: unconnected-(J7-PadB24) -> /Expansion/A26
- J7 pad B25: unconnected-(J7-PadB25) -> /Expansion/A27
- J7 pad B26: unconnected-(J7-PadB26) -> /Expansion/A28
- J7 pad B27: unconnected-(J7-PadB27) -> /Expansion/A29
- J7 pad B28: unconnected-(J7-PadB28) -> /Expansion/A30
- J7 pad B29: unconnected-(J7-PadB29) -> /Expansion/A31
- J7 pad B3: unconnected-(J7-PadB3) -> /Expansion/D18
- J7 pad B4: unconnected-(J7-PadB4) -> /Expansion/D19
- J7 pad B5: unconnected-(J7-PadB5) -> /Expansion/D20
- J7 pad B6: unconnected-(J7-PadB6) -> /Expansion/D21
- J7 pad B7: unconnected-(J7-PadB7) -> /Expansion/D22
- J7 pad B8: unconnected-(J7-PadB8) -> /Expansion/D23
- J7 pad B9: unconnected-(J7-PadB9) -> /Expansion/D24
- J7 pad C10: unconnected-(J7-PadC10) -> /Expansion/D15
- J7 pad C12: unconnected-(J7-PadC12) -> /Expansion/A2
- J7 pad C13: unconnected-(J7-PadC13) -> /Expansion/A4
- J7 pad C14: unconnected-(J7-PadC14) -> /Expansion/A6
- J7 pad C15: unconnected-(J7-PadC15) -> /Expansion/A8
- J7 pad C16: unconnected-(J7-PadC16) -> /Expansion/A10
- J7 pad C17: unconnected-(J7-PadC17) -> /Expansion/A12
- J7 pad C18: unconnected-(J7-PadC18) -> /Expansion/A14
- J7 pad C19: unconnected-(J7-PadC19) -> /Expansion/A16
- J7 pad C20: unconnected-(J7-PadC20) -> /Expansion/A18
- J7 pad C3: unconnected-(J7-PadC3) -> /Expansion/D1
- J7 pad C4: unconnected-(J7-PadC4) -> /Expansion/D3
- J7 pad C5: unconnected-(J7-PadC5) -> /Expansion/D5
- J7 pad C6: unconnected-(J7-PadC6) -> /Expansion/D7
- J7 pad C7: unconnected-(J7-PadC7) -> /Expansion/D9
- J7 pad C8: unconnected-(J7-PadC8) -> /Expansion/D11
- J7 pad C9: unconnected-(J7-PadC9) -> /Expansion/D13
- J8 pad A10: unconnected-(J8-PadA10) -> /Expansion/D14
- J8 pad A12: unconnected-(J8-PadA12) -> /Expansion/A1
- J8 pad A13: unconnected-(J8-PadA13) -> /Expansion/A3
- J8 pad A14: unconnected-(J8-PadA14) -> /Expansion/A5
- J8 pad A15: unconnected-(J8-PadA15) -> /Expansion/A7
- J8 pad A16: unconnected-(J8-PadA16) -> /Expansion/A9
- J8 pad A17: unconnected-(J8-PadA17) -> /Expansion/A11
- J8 pad A18: unconnected-(J8-PadA18) -> /Expansion/A13
- J8 pad A19: unconnected-(J8-PadA19) -> /Expansion/A15
- J8 pad A20: unconnected-(J8-PadA20) -> /Expansion/A17
- J8 pad A21: unconnected-(J8-PadA21) -> /Expansion/A19
- J8 pad A3: unconnected-(J8-PadA3) -> /Expansion/D0
- J8 pad A4: unconnected-(J8-PadA4) -> /Expansion/D2
- J8 pad A5: unconnected-(J8-PadA5) -> /Expansion/D4
- J8 pad A6: unconnected-(J8-PadA6) -> /Expansion/D6
- J8 pad A7: unconnected-(J8-PadA7) -> /Expansion/D8
- J8 pad A8: unconnected-(J8-PadA8) -> /Expansion/D10
- J8 pad A9: unconnected-(J8-PadA9) -> /Expansion/D12
- J8 pad B1: unconnected-(J8-PadB1) -> /Expansion/D16
- J8 pad B10: unconnected-(J8-PadB10) -> /Expansion/D25
- J8 pad B11: unconnected-(J8-PadB11) -> /Expansion/D26
- J8 pad B12: unconnected-(J8-PadB12) -> /Expansion/D27
- J8 pad B13: unconnected-(J8-PadB13) -> /Expansion/D28
- J8 pad B14: unconnected-(J8-PadB14) -> /Expansion/D29
- J8 pad B15: unconnected-(J8-PadB15) -> /Expansion/D30
- J8 pad B16: unconnected-(J8-PadB16) -> /Expansion/D31
- J8 pad B17: unconnected-(J8-PadB17) -> /Expansion/A0
- J8 pad B18: unconnected-(J8-PadB18) -> /Expansion/A20
- J8 pad B19: unconnected-(J8-PadB19) -> /Expansion/A21
- J8 pad B2: unconnected-(J8-PadB2) -> /Expansion/D17
- J8 pad B20: unconnected-(J8-PadB20) -> /Expansion/A22
- J8 pad B21: unconnected-(J8-PadB21) -> /Expansion/A23
- J8 pad B22: unconnected-(J8-PadB22) -> /Expansion/A24
- J8 pad B23: unconnected-(J8-PadB23) -> /Expansion/A25
- J8 pad B24: unconnected-(J8-PadB24) -> /Expansion/A26
- J8 pad B25: unconnected-(J8-PadB25) -> /Expansion/A27
- J8 pad B26: unconnected-(J8-PadB26) -> /Expansion/A28
- J8 pad B27: unconnected-(J8-PadB27) -> /Expansion/A29
- J8 pad B28: unconnected-(J8-PadB28) -> /Expansion/A30
- J8 pad B29: unconnected-(J8-PadB29) -> /Expansion/A31
- J8 pad B3: unconnected-(J8-PadB3) -> /Expansion/D18
- J8 pad B4: unconnected-(J8-PadB4) -> /Expansion/D19
- J8 pad B5: unconnected-(J8-PadB5) -> /Expansion/D20
- J8 pad B6: unconnected-(J8-PadB6) -> /Expansion/D21
- J8 pad B7: unconnected-(J8-PadB7) -> /Expansion/D22
- J8 pad B8: unconnected-(J8-PadB8) -> /Expansion/D23
- J8 pad B9: unconnected-(J8-PadB9) -> /Expansion/D24
- J8 pad C10: unconnected-(J8-PadC10) -> /Expansion/D15
- J8 pad C12: unconnected-(J8-PadC12) -> /Expansion/A2
- J8 pad C13: unconnected-(J8-PadC13) -> /Expansion/A4
- J8 pad C14: unconnected-(J8-PadC14) -> /Expansion/A6
- J8 pad C15: unconnected-(J8-PadC15) -> /Expansion/A8
- J8 pad C16: unconnected-(J8-PadC16) -> /Expansion/A10
- J8 pad C17: unconnected-(J8-PadC17) -> /Expansion/A12
- J8 pad C18: unconnected-(J8-PadC18) -> /Expansion/A14
- J8 pad C19: unconnected-(J8-PadC19) -> /Expansion/A16
- J8 pad C20: unconnected-(J8-PadC20) -> /Expansion/A18
- J8 pad C3: unconnected-(J8-PadC3) -> /Expansion/D1
- J8 pad C4: unconnected-(J8-PadC4) -> /Expansion/D3
- J8 pad C5: unconnected-(J8-PadC5) -> /Expansion/D5
- J8 pad C6: unconnected-(J8-PadC6) -> /Expansion/D7
- J8 pad C7: unconnected-(J8-PadC7) -> /Expansion/D9
- J8 pad C8: unconnected-(J8-PadC8) -> /Expansion/D11
- J8 pad C9: unconnected-(J8-PadC9) -> /Expansion/D13
- U1 pad A1: /Memory/A31 -> /Expansion/A31
- U1 pad A10: /Memory/D12 -> /Expansion/D12
- U1 pad A11: /Memory/D13 -> /Expansion/D13
- U1 pad A12: /Memory/D14 -> /Expansion/D14
- U1 pad A13: /Memory/D15 -> /Expansion/D15
- U1 pad A14: /Memory/D17 -> /Expansion/D17
- U1 pad A15: /Memory/D19 -> /Expansion/D19
- U1 pad A16: /Memory/D20 -> /Expansion/D20
- U1 pad A17: /Memory/D21 -> /Expansion/D21
- U1 pad A18: /Memory/D24 -> /Expansion/D24
- U1 pad A2: /Memory/D3 -> /Expansion/D3
- U1 pad A3: /Memory/D4 -> /Expansion/D4
- U1 pad A4: /Memory/D5 -> /Expansion/D5
- U1 pad A5: /Memory/D6 -> /Expansion/D6
- U1 pad A6: /Memory/D7 -> /Expansion/D7
- U1 pad A7: /Memory/D9 -> /Expansion/D9
- U1 pad A8: /Memory/D10 -> /Expansion/D10
- U1 pad A9: /Memory/D11 -> /Expansion/D11
- U1 pad B1: /Memory/A29 -> /Expansion/A29
- U1 pad B11: /Memory/D16 -> /Expansion/D16
- U1 pad B12: /Memory/D18 -> /Expansion/D18
- U1 pad B16: /Memory/D22 -> /Expansion/D22
- U1 pad B18: /Memory/D26 -> /Expansion/D26
- U1 pad B3: /Memory/D1 -> /Expansion/D1
- U1 pad B7: /Memory/D8 -> /Expansion/D8
- U1 pad C1: /Memory/A27 -> /Expansion/A27
- U1 pad C15: /Memory/D23 -> /Expansion/D23
- U1 pad C16: /Memory/D25 -> /Expansion/D25
- U1 pad C18: /Memory/D28 -> /Expansion/D28
- U1 pad C3: /Memory/D0 -> /Expansion/D0
- U1 pad C4: /Memory/D2 -> /Expansion/D2
- U1 pad D1: /Memory/A24 -> /Expansion/A24
- U1 pad D16: /Memory/D27 -> /Expansion/D27
- U1 pad D18: /Memory/D31 -> /Expansion/D31
- U1 pad D3: /Memory/A30 -> /Expansion/A30
- U1 pad E1: /Memory/A22 -> /Expansion/A22
- U1 pad E16: /Memory/D29 -> /Expansion/D29
- U1 pad E17: /Memory/D30 -> /Expansion/D30
- U1 pad E18: /Memory/A8 -> /Expansion/A8
- U1 pad E2: /Memory/A26 -> /Expansion/A26
- U1 pad E3: /Memory/A28 -> /Expansion/A28
- U1 pad F1: /Memory/A21 -> /Expansion/A21
- U1 pad F16: /Memory/A9 -> /Expansion/A9
- U1 pad F18: /Memory/A7 -> /Expansion/A7
- U1 pad F3: /Memory/A25 -> /Expansion/A25
- U1 pad G1: /Memory/A20 -> /Expansion/A20
- U1 pad G16: /Memory/A6 -> /Expansion/A6
- U1 pad G18: /Memory/A5 -> /Expansion/A5
- U1 pad G3: /Memory/A23 -> /Expansion/A23
- U1 pad H1: /Memory/A18 -> /Expansion/A18
- U1 pad H18: /Memory/A4 -> /Expansion/A4
- U1 pad J1: /Memory/A17 -> /Expansion/A17
- U1 pad J17: /Memory/A2 -> /Expansion/A2
- U1 pad J18: /Memory/A3 -> /Expansion/A3
- U1 pad J2: /Memory/A19 -> /Expansion/A19
- U1 pad K1: /Memory/A15 -> /Expansion/A15
- U1 pad K18: /Memory/A1 -> /Expansion/A1
- U1 pad K2: /Memory/A16 -> /Expansion/A16
- U1 pad L1: /Memory/A14 -> /Expansion/A14
- U1 pad L18: /Memory/A0 -> /Expansion/A0
- U1 pad M1: /Memory/A13 -> /Expansion/A13
- U1 pad N1: /Memory/A12 -> /Expansion/A12
- U1 pad N3: /Memory/A11 -> /Expansion/A11
- U1 pad P1: /Memory/A10 -> /Expansion/A10
- U2 pad 101: /Memory/A10 -> /Expansion/A10
- U2 pad 102: /Memory/A11 -> /Expansion/A11
- U2 pad 104: /Memory/A12 -> /Expansion/A12
- U2 pad 105: /Memory/A13 -> /Expansion/A13
- U2 pad 106: /Memory/A14 -> /Expansion/A14
- U2 pad 107: /Memory/A15 -> /Expansion/A15
- U2 pad 110: /Memory/A16 -> /Expansion/A16
- U2 pad 112: /Memory/A17 -> /Expansion/A17
- U2 pad 113: /Memory/A18 -> /Expansion/A18
- U2 pad 114: /Memory/A19 -> /Expansion/A19
- U2 pad 115: /Memory/A20 -> /Expansion/A20
- U2 pad 116: /Memory/A21 -> /Expansion/A21
- U2 pad 117: /Memory/A22 -> /Expansion/A22
- U2 pad 118: /Memory/A23 -> /Expansion/A23
- U2 pad 119: /Memory/A24 -> /Expansion/A24
- U2 pad 120: /Memory/A25 -> /Expansion/A25
- U2 pad 121: /Memory/A26 -> /Expansion/A26
- U2 pad 122: /Memory/A27 -> /Expansion/A27
- U2 pad 124: /Memory/A28 -> /Expansion/A28
- U2 pad 125: /Memory/A29 -> /Expansion/A29
- U2 pad 128: /Memory/A30 -> /Expansion/A30
- U2 pad 129: /Memory/A31 -> /Expansion/A31
- U2 pad 65: unconnected-(U2E-CDONE-Pad65) -> /Memory/CDONE
- U2 pad 67: unconnected-(U2E-IOB_105_SDO-Pad67) -> /Memory/FLASH_MOSI
- U2 pad 68: unconnected-(U2E-IOB_106_SDI-Pad68) -> /Memory/FLASH_MISO
- U2 pad 70: unconnected-(U2E-IOB_107_SCK-Pad70) -> /Memory/FLASH_SCK
- U2 pad 71: unconnected-(U2E-IOB_108_SS-Pad71) -> /Memory/FLASH_SS
- U2 pad 88: /Memory/A0 -> /Expansion/A0
- U2 pad 90: /Memory/A1 -> /Expansion/A1
- U2 pad 91: /Memory/A2 -> /Expansion/A2
- U2 pad 93: /Memory/A3 -> /Expansion/A3
- U2 pad 94: /Memory/A4 -> /Expansion/A4
- U2 pad 95: /Memory/A5 -> /Expansion/A5
- U2 pad 96: /Memory/A6 -> /Expansion/A6
- U2 pad 97: /Memory/A7 -> /Expansion/A7
- U2 pad 98: /Memory/A8 -> /Expansion/A8
- U2 pad 99: /Memory/A9 -> /Expansion/A9
- U3 pad 1: unconnected-(U3A-1DIR-Pad1) -> /Memory/DRAM_BUF_DIR
- U3 pad 10: unconnected-(U3B-GND-Pad10) -> GND
- U3 pad 11: /Memory/D6 -> /Expansion/D6
- U3 pad 12: /Memory/D7 -> /Expansion/D7
- U3 pad 13: /Memory/D8 -> /Expansion/D8
- U3 pad 14: /Memory/D9 -> /Expansion/D9
- U3 pad 15: unconnected-(U3B-GND-Pad15) -> GND
- U3 pad 16: /Memory/D10 -> /Expansion/D10
- U3 pad 17: /Memory/D11 -> /Expansion/D11
- U3 pad 18: unconnected-(U3B-VCCB-Pad18) -> +5V
- U3 pad 19: /Memory/D12 -> /Expansion/D12
- U3 pad 2: /Memory/D0 -> /Expansion/D0
- U3 pad 20: /Memory/D13 -> /Expansion/D13
- U3 pad 21: unconnected-(U3B-GND-Pad21) -> GND
- U3 pad 22: /Memory/D14 -> /Expansion/D14
- U3 pad 23: /Memory/D15 -> /Expansion/D15
- U3 pad 24: unconnected-(U3A-2DIR-Pad24) -> /Memory/DRAM_BUF_DIR
- U3 pad 25: unconnected-(U3A-*2OE-Pad25) -> /Memory/DRAM_BUF_~{OE}
- U3 pad 28: unconnected-(U3B-GND-Pad28) -> GND
- U3 pad 3: /Memory/D1 -> /Expansion/D1
- U3 pad 31: unconnected-(U3B-VCCA-Pad31) -> +3V3
- U3 pad 34: unconnected-(U3B-GND-Pad34) -> GND
- U3 pad 39: unconnected-(U3B-GND-Pad39) -> GND
- U3 pad 4: unconnected-(U3B-GND-Pad4) -> GND
- U3 pad 42: unconnected-(U3B-VCCA-Pad42) -> +3V3
- U3 pad 45: unconnected-(U3B-GND-Pad45) -> GND
- U3 pad 48: unconnected-(U3A-*1OE-Pad48) -> /Memory/DRAM_BUF_~{OE}
- U3 pad 5: /Memory/D2 -> /Expansion/D2
- U3 pad 6: /Memory/D3 -> /Expansion/D3
- U3 pad 7: unconnected-(U3B-VCCB-Pad7) -> +5V
- U3 pad 8: /Memory/D4 -> /Expansion/D4
- U3 pad 9: /Memory/D5 -> /Expansion/D5
- U4 pad 1: unconnected-(U4A-1DIR-Pad1) -> /Memory/DRAM_BUF_DIR
- U4 pad 10: unconnected-(U4B-GND-Pad10) -> GND
- U4 pad 11: /Memory/D22 -> /Expansion/D22
- U4 pad 12: /Memory/D23 -> /Expansion/D23
- U4 pad 13: /Memory/D24 -> /Expansion/D24
- U4 pad 14: /Memory/D25 -> /Expansion/D25
- U4 pad 15: unconnected-(U4B-GND-Pad15) -> GND
- U4 pad 16: /Memory/D26 -> /Expansion/D26
- U4 pad 17: /Memory/D27 -> /Expansion/D27
- U4 pad 18: unconnected-(U4B-VCCB-Pad18) -> +5V
- U4 pad 19: /Memory/D28 -> /Expansion/D28
- U4 pad 2: /Memory/D16 -> /Expansion/D16
- U4 pad 20: /Memory/D29 -> /Expansion/D29
- U4 pad 21: unconnected-(U4B-GND-Pad21) -> GND
- U4 pad 22: /Memory/D30 -> /Expansion/D30
- U4 pad 23: /Memory/D31 -> /Expansion/D31
- U4 pad 24: unconnected-(U4A-2DIR-Pad24) -> /Memory/DRAM_BUF_DIR
- U4 pad 25: unconnected-(U4A-*2OE-Pad25) -> /Memory/DRAM_BUF_~{OE}
- U4 pad 28: unconnected-(U4B-GND-Pad28) -> GND
- U4 pad 3: /Memory/D17 -> /Expansion/D17
- U4 pad 31: unconnected-(U4B-VCCA-Pad31) -> +3V3
- U4 pad 34: unconnected-(U4B-GND-Pad34) -> GND
- U4 pad 39: unconnected-(U4B-GND-Pad39) -> GND
- U4 pad 4: unconnected-(U4B-GND-Pad4) -> GND
- U4 pad 42: unconnected-(U4B-VCCA-Pad42) -> +3V3
- U4 pad 45: unconnected-(U4B-GND-Pad45) -> GND
- U4 pad 48: unconnected-(U4A-*1OE-Pad48) -> /Memory/DRAM_BUF_~{OE}
- U4 pad 5: /Memory/D18 -> /Expansion/D18
- U4 pad 6: /Memory/D19 -> /Expansion/D19
- U4 pad 7: unconnected-(U4B-VCCB-Pad7) -> +5V
- U4 pad 8: /Memory/D20 -> /Expansion/D20
- U4 pad 9: /Memory/D21 -> /Expansion/D21
