File: hardware/68040pc.kicad_pcb (KiCad board)
At the start: 4 copper layers, 221 x 243.8 mm, 29 parts, among them J1 EXP, J13 DIN-5_180degree, J14 Mini-DIN-6, J15 COM1, J16 COM2, J17 LPT, J2 EXP, J3 EXP, J4 EXP, J5 EXP, J6 EXP, J7 EXP, J8 EXP, P8 Conn_01x06, P9 Conn_01x06, U1 68LC040, U2 ICE40HX4K-TQ144, U3 SN74ALVC164245, U4 SN74ALVC164245, U5 W25Q32JVSSIM

Commit message: updates
Parts:
- added RN1: R_Network04_US, Resistor_THT:R_Array_SIP5, F.Cu at (85.7, 201.9)
- added RN2: R_Network04_US, Resistor_THT:R_Array_SIP5, F.Cu at (167.0, 201.9)
- added RN3: 10k, Resistor_THT:R_Array_SIP5, F.Cu at (90.1, 270.8)
- added RN4: 10k, Resistor_THT:R_Array_SIP5, F.Cu at (90.1, 275.1)
- added RN5: 10k, Resistor_THT:R_Array_SIP5, F.Cu at (90.1, 279.5)
- added RN6: 10k, Resistor_THT:R_Array_SIP5, F.Cu at (90.1, 283.8)
- added U10: 74HC165, Package_SO:SOIC-16_3.9x9.9mm_P1.27mm, F.Cu at (319.4, 214.6)
- added U11: 74HC245, Package_SO:SOIC-20W_7.5x12.8mm_P1.27mm, F.Cu at (143.5, 223.3)
- added U12: 74HC245, Package_SO:SOIC-20W_7.5x12.8mm_P1.27mm, F.Cu at (158.1, 223.3)
- added U13: 74HC245, Package_SO:SOIC-20W_7.5x12.8mm_P1.27mm, F.Cu at (172.7, 223.3)
- added U14: 74HC245, Package_SO:SOIC-20W_7.5x12.8mm_P1.27mm, F.Cu at (187.3, 223.3)
- added U6: 74LS32, Package_SO:SOIC-14_3.9x8.7mm_P1.27mm, F.Cu at (106.0, 205.7)
- added U7: 74LS32, Package_SO:SOIC-14_3.9x8.7mm_P1.27mm, F.Cu at (187.3, 205.7)
- added U8: LTC6905xS5-133, Package_TO_SOT_SMD:TSOT-23-5, F.Cu at (109.3, 271.6)
- added U9: 74HC165, Package_SO:SOIC-16_3.9x9.9mm_P1.27mm, F.Cu at (310.4, 214.6)
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- renumbered J8 to J1, J7 to J2, J6 to J3, J3 to J5, J5 to J6, J2 to J7, J1 to J8
Connections:
- net /PWR_GD renamed /Power/PWR_GOOD
- J1 pad A1: unconnected-(J8-PadA1) -> GND
- J1 pad A10: /Expansion/D14 -> /Expansion/ExpansionSlot8/D14
- J1 pad A11: unconnected-(J8-PadA11) -> GND
- J1 pad A12: /Expansion/A1 -> /Expansion/ExpansionSlot8/A1
- J1 pad A13: /Expansion/A3 -> /Expansion/ExpansionSlot8/A3
- J1 pad A14: /Expansion/A5 -> /Expansion/ExpansionSlot8/A5
- J1 pad A15: /Expansion/A7 -> /Expansion/ExpansionSlot8/A7
- J1 pad A16: /Expansion/A9 -> /Expansion/ExpansionSlot8/A9
- J1 pad A17: /Expansion/A11 -> /Expansion/ExpansionSlot8/A11
- J1 pad A18: /Expansion/A13 -> /Expansion/ExpansionSlot8/A13
- J1 pad A19: /Expansion/A15 -> /Expansion/ExpansionSlot8/A15
- J1 pad A2: unconnected-(J8-PadA2) -> /Expansion/ExpansionSlot8/~{CFG_{IN}}
- J1 pad A20: /Expansion/A17 -> /Expansion/ExpansionSlot8/A17
- J1 pad A21: /Expansion/A19 -> /Expansion/ExpansionSlot8/A19
- J1 pad A24: unconnected-(J8-PadA24) -> +5V
- J1 pad A3: /Expansion/D0 -> /Expansion/ExpansionSlot8/D0
- J1 pad A31: unconnected-(J8-PadA31) -> +12V
- J1 pad A32: unconnected-(J8-PadA32) -> GND
- J1 pad A4: /Expansion/D2 -> /Expansion/ExpansionSlot8/D2
- J1 pad A5: /Expansion/D4 -> /Expansion/ExpansionSlot8/D4
- J1 pad A6: /Expansion/D6 -> /Expansion/ExpansionSlot8/D6
- J1 pad A7: /Expansion/D8 -> /Expansion/ExpansionSlot8/D8
- J1 pad A8: /Expansion/D10 -> /Expansion/ExpansionSlot8/D10
- J1 pad A9: /Expansion/D12 -> /Expansion/ExpansionSlot8/D12
- J1 pad B1: /Expansion/D16 -> /Expansion/ExpansionSlot8/D16
- J1 pad B10: /Expansion/D25 -> /Expansion/ExpansionSlot8/D25
- J1 pad B11: /Expansion/D26 -> /Expansion/ExpansionSlot8/D26
- J1 pad B12: /Expansion/D27 -> /Expansion/ExpansionSlot8/D27
- J1 pad B13: /Expansion/D28 -> /Expansion/ExpansionSlot8/D28
- J1 pad B14: /Expansion/D29 -> /Expansion/ExpansionSlot8/D29
- J1 pad B15: /Expansion/D30 -> /Expansion/ExpansionSlot8/D30
- J1 pad B16: /Expansion/D31 -> /Expansion/ExpansionSlot8/D31
- J1 pad B17: /Expansion/A0 -> /Expansion/ExpansionSlot8/A0
- J1 pad B18: /Expansion/A20 -> /Expansion/ExpansionSlot8/A20
- J1 pad B19: /Expansion/A21 -> /Expansion/ExpansionSlot8/A21
- J1 pad B2: /Expansion/D17 -> /Expansion/ExpansionSlot8/D17
- J1 pad B20: /Expansion/A22 -> /Expansion/ExpansionSlot8/A22
- J1 pad B21: /Expansion/A23 -> /Expansion/ExpansionSlot8/A23
- J1 pad B22: /Expansion/A24 -> /Expansion/ExpansionSlot8/A24
- J1 pad B23: /Expansion/A25 -> /Expansion/ExpansionSlot8/A25
- J1 pad B24: /Expansion/A26 -> /Expansion/ExpansionSlot8/A26
- J1 pad B25: /Expansion/A27 -> /Expansion/ExpansionSlot8/A27
- J1 pad B26: /Expansion/A28 -> /Expansion/ExpansionSlot8/A28
- J1 pad B27: /Expansion/A29 -> /Expansion/ExpansionSlot8/A29
- J1 pad B28: /Expansion/A30 -> /Expansion/ExpansionSlot8/A30
- J1 pad B29: /Expansion/A31 -> /Expansion/ExpansionSlot8/A31
- J1 pad B3: /Expansion/D18 -> /Expansion/ExpansionSlot8/D18
- J1 pad B31: unconnected-(J8-PadB31) -> /Expansion/ExpansionSlot8/BCLK
- J1 pad B32: unconnected-(J8-PadB32) -> GND
- J1 pad B4: /Expansion/D19 -> /Expansion/ExpansionSlot8/D19
- J1 pad B5: /Expansion/D20 -> /Expansion/ExpansionSlot8/D20
- J1 pad B6: /Expansion/D21 -> /Expansion/ExpansionSlot8/D21
- J1 pad B7: /Expansion/D22 -> /Expansion/ExpansionSlot8/D22
- J1 pad B8: /Expansion/D23 -> /Expansion/ExpansionSlot8/D23
- J1 pad B9: /Expansion/D24 -> /Expansion/ExpansionSlot8/D24
- J1 pad C1: unconnected-(J8-PadC1) -> +5V
- J1 pad C10: /Expansion/D15 -> /Expansion/ExpansionSlot8/D15
- J1 pad C11: unconnected-(J8-PadC11) -> GND
- J1 pad C12: /Expansion/A2 -> /Expansion/ExpansionSlot8/A2
- J1 pad C13: /Expansion/A4 -> /Expansion/ExpansionSlot8/A4
- J1 pad C14: /Expansion/A6 -> /Expansion/ExpansionSlot8/A6
- J1 pad C15: /Expansion/A8 -> /Expansion/ExpansionSlot8/A8
- J1 pad C16: /Expansion/A10 -> /Expansion/ExpansionSlot8/A10
- J1 pad C17: /Expansion/A12 -> /Expansion/ExpansionSlot8/A12
- J1 pad C18: /Expansion/A14 -> /Expansion/ExpansionSlot8/A14
- J1 pad C19: /Expansion/A16 -> /Expansion/ExpansionSlot8/A16
- J1 pad C2: unconnected-(J8-PadC2) -> /Expansion/ExpansionSlot8/~{CFG_{OUT}}
- J1 pad C20: /Expansion/A18 -> /Expansion/ExpansionSlot8/A18
- J1 pad C24: unconnected-(J8-PadC24) -> GND
- J1 pad C3: /Expansion/D1 -> /Expansion/ExpansionSlot8/D1
- J1 pad C30: unconnected-(J8-PadC30) -> +3V3
- J1 pad C31: unconnected-(J8-PadC31) -> +12V
- J1 pad C32: unconnected-(J8-PadC32) -> GND
- J1 pad C4: /Expansion/D3 -> /Expansion/ExpansionSlot8/D3
- J1 pad C5: /Expansion/D5 -> /Expansion/ExpansionSlot8/D5
- J1 pad C6: /Expansion/D7 -> /Expansion/ExpansionSlot8/D7
- J1 pad C7: /Expansion/D9 -> /Expansion/ExpansionSlot8/D9
- J1 pad C8: /Expansion/D11 -> /Expansion/ExpansionSlot8/D11
- J1 pad C9: /Expansion/D13 -> /Expansion/ExpansionSlot8/D13
- J2 pad A1: unconnected-(J7-PadA1) -> GND
- J2 pad A10: /Expansion/D14 -> /Expansion/ExpansionSlot7/D14
- J2 pad A11: unconnected-(J7-PadA11) -> GND
- J2 pad A12: /Expansion/A1 -> /Expansion/ExpansionSlot7/A1
- J2 pad A13: /Expansion/A3 -> /Expansion/ExpansionSlot7/A3
- J2 pad A14: /Expansion/A5 -> /Expansion/ExpansionSlot7/A5
- J2 pad A15: /Expansion/A7 -> /Expansion/ExpansionSlot7/A7
- J2 pad A16: /Expansion/A9 -> /Expansion/ExpansionSlot7/A9
- J2 pad A17: /Expansion/A11 -> /Expansion/ExpansionSlot7/A11
- J2 pad A18: /Expansion/A13 -> /Expansion/ExpansionSlot7/A13
- J2 pad A19: /Expansion/A15 -> /Expansion/ExpansionSlot7/A15
- J2 pad A2: unconnected-(J7-PadA2) -> /Expansion/ExpansionSlot7/~{CFG_{IN}}
- J2 pad A20: /Expansion/A17 -> /Expansion/ExpansionSlot7/A17
- J2 pad A21: /Expansion/A19 -> /Expansion/ExpansionSlot7/A19
- J2 pad A24: unconnected-(J7-PadA24) -> +5V
- J2 pad A3: /Expansion/D0 -> /Expansion/ExpansionSlot7/D0
- J2 pad A31: unconnected-(J7-PadA31) -> +12V
- J2 pad A32: unconnected-(J7-PadA32) -> GND
- J2 pad A4: /Expansion/D2 -> /Expansion/ExpansionSlot7/D2
- J2 pad A5: /Expansion/D4 -> /Expansion/ExpansionSlot7/D4
- J2 pad A6: /Expansion/D6 -> /Expansion/ExpansionSlot7/D6
- J2 pad A7: /Expansion/D8 -> /Expansion/ExpansionSlot7/D8
- J2 pad A8: /Expansion/D10 -> /Expansion/ExpansionSlot7/D10
- J2 pad A9: /Expansion/D12 -> /Expansion/ExpansionSlot7/D12
- J2 pad B1: /Expansion/D16 -> /Expansion/ExpansionSlot7/D16
- J2 pad B10: /Expansion/D25 -> /Expansion/ExpansionSlot7/D25
- J2 pad B11: /Expansion/D26 -> /Expansion/ExpansionSlot7/D26
- J2 pad B12: /Expansion/D27 -> /Expansion/ExpansionSlot7/D27
- J2 pad B13: /Expansion/D28 -> /Expansion/ExpansionSlot7/D28
- J2 pad B14: /Expansion/D29 -> /Expansion/ExpansionSlot7/D29
- J2 pad B15: /Expansion/D30 -> /Expansion/ExpansionSlot7/D30
- J2 pad B16: /Expansion/D31 -> /Expansion/ExpansionSlot7/D31
- J2 pad B17: /Expansion/A0 -> /Expansion/ExpansionSlot7/A0
- J2 pad B18: /Expansion/A20 -> /Expansion/ExpansionSlot7/A20
- J2 pad B19: /Expansion/A21 -> /Expansion/ExpansionSlot7/A21
- J2 pad B2: /Expansion/D17 -> /Expansion/ExpansionSlot7/D17
- J2 pad B20: /Expansion/A22 -> /Expansion/ExpansionSlot7/A22
- J2 pad B21: /Expansion/A23 -> /Expansion/ExpansionSlot7/A23
- J2 pad B22: /Expansion/A24 -> /Expansion/ExpansionSlot7/A24
- J2 pad B23: /Expansion/A25 -> /Expansion/ExpansionSlot7/A25
- J2 pad B24: /Expansion/A26 -> /Expansion/ExpansionSlot7/A26
- J2 pad B25: /Expansion/A27 -> /Expansion/ExpansionSlot7/A27
- J2 pad B26: /Expansion/A28 -> /Expansion/ExpansionSlot7/A28
- J2 pad B27: /Expansion/A29 -> /Expansion/ExpansionSlot7/A29
- J2 pad B28: /Expansion/A30 -> /Expansion/ExpansionSlot7/A30
- J2 pad B29: /Expansion/A31 -> /Expansion/ExpansionSlot7/A31
- J2 pad B3: /Expansion/D18 -> /Expansion/ExpansionSlot7/D18
- J2 pad B31: unconnected-(J7-PadB31) -> /Expansion/ExpansionSlot7/BCLK
- J2 pad B32: unconnected-(J7-PadB32) -> GND
- J2 pad B4: /Expansion/D19 -> /Expansion/ExpansionSlot7/D19
- J2 pad B5: /Expansion/D20 -> /Expansion/ExpansionSlot7/D20
- J2 pad B6: /Expansion/D21 -> /Expansion/ExpansionSlot7/D21
- J2 pad B7: /Expansion/D22 -> /Expansion/ExpansionSlot7/D22
- J2 pad B8: /Expansion/D23 -> /Expansion/ExpansionSlot7/D23
- J2 pad B9: /Expansion/D24 -> /Expansion/ExpansionSlot7/D24
- J2 pad C1: unconnected-(J7-PadC1) -> +5V
- J2 pad C10: /Expansion/D15 -> /Expansion/ExpansionSlot7/D15
- J2 pad C11: unconnected-(J7-PadC11) -> GND
- J2 pad C12: /Expansion/A2 -> /Expansion/ExpansionSlot7/A2
- J2 pad C13: /Expansion/A4 -> /Expansion/ExpansionSlot7/A4
- J2 pad C14: /Expansion/A6 -> /Expansion/ExpansionSlot7/A6
- J2 pad C15: /Expansion/A8 -> /Expansion/ExpansionSlot7/A8
- J2 pad C16: /Expansion/A10 -> /Expansion/ExpansionSlot7/A10
- J2 pad C17: /Expansion/A12 -> /Expansion/ExpansionSlot7/A12
- J2 pad C18: /Expansion/A14 -> /Expansion/ExpansionSlot7/A14
- J2 pad C19: /Expansion/A16 -> /Expansion/ExpansionSlot7/A16
- J2 pad C2: unconnected-(J7-PadC2) -> /Expansion/ExpansionSlot7/~{CFG_{OUT}}
- J2 pad C20: /Expansion/A18 -> /Expansion/ExpansionSlot7/A18
- J2 pad C24: unconnected-(J7-PadC24) -> GND
- J2 pad C3: /Expansion/D1 -> /Expansion/ExpansionSlot7/D1
- J2 pad C30: unconnected-(J7-PadC30) -> +3V3
- J2 pad C31: unconnected-(J7-PadC31) -> +12V
- J2 pad C32: unconnected-(J7-PadC32) -> GND
- J2 pad C4: /Expansion/D3 -> /Expansion/ExpansionSlot7/D3
- J2 pad C5: /Expansion/D5 -> /Expansion/ExpansionSlot7/D5
- J2 pad C6: /Expansion/D7 -> /Expansion/ExpansionSlot7/D7
- J2 pad C7: /Expansion/D9 -> /Expansion/ExpansionSlot7/D9
- J2 pad C8: /Expansion/D11 -> /Expansion/ExpansionSlot7/D11
- J2 pad C9: /Expansion/D13 -> /Expansion/ExpansionSlot7/D13
- J3 pad A1: unconnected-(J6-PadA1) -> GND
- J3 pad A10: /Expansion/D14 -> /Expansion/ExpansionSlot6/D14
- J3 pad A11: unconnected-(J6-PadA11) -> GND
- J3 pad A12: /Expansion/A1 -> /Expansion/ExpansionSlot6/A1
- J3 pad A13: /Expansion/A3 -> /Expansion/ExpansionSlot6/A3
- J3 pad A14: /Expansion/A5 -> /Expansion/ExpansionSlot6/A5
- J3 pad A15: /Expansion/A7 -> /Expansion/ExpansionSlot6/A7
- J3 pad A16: /Expansion/A9 -> /Expansion/ExpansionSlot6/A9
- J3 pad A17: /Expansion/A11 -> /Expansion/ExpansionSlot6/A11
- J3 pad A18: /Expansion/A13 -> /Expansion/ExpansionSlot6/A13
- J3 pad A19: /Expansion/A15 -> /Expansion/ExpansionSlot6/A15
- J3 pad A2: unconnected-(J6-PadA2) -> /Expansion/ExpansionSlot6/~{CFG_{IN}}
- J3 pad A20: /Expansion/A17 -> /Expansion/ExpansionSlot6/A17
- J3 pad A21: /Expansion/A19 -> /Expansion/ExpansionSlot6/A19
- J3 pad A24: unconnected-(J6-PadA24) -> +5V
- J3 pad A3: /Expansion/D0 -> /Expansion/ExpansionSlot6/D0
- J3 pad A31: unconnected-(J6-PadA31) -> +12V
- J3 pad A32: unconnected-(J6-PadA32) -> GND
- J3 pad A4: /Expansion/D2 -> /Expansion/ExpansionSlot6/D2
- J3 pad A5: /Expansion/D4 -> /Expansion/ExpansionSlot6/D4
- J3 pad A6: /Expansion/D6 -> /Expansion/ExpansionSlot6/D6
- J3 pad A7: /Expansion/D8 -> /Expansion/ExpansionSlot6/D8
- J3 pad A8: /Expansion/D10 -> /Expansion/ExpansionSlot6/D10
- J3 pad A9: /Expansion/D12 -> /Expansion/ExpansionSlot6/D12
- J3 pad B1: /Expansion/D16 -> /Expansion/ExpansionSlot6/D16
- J3 pad B10: /Expansion/D25 -> /Expansion/ExpansionSlot6/D25
- J3 pad B11: /Expansion/D26 -> /Expansion/ExpansionSlot6/D26
- J3 pad B12: /Expansion/D27 -> /Expansion/ExpansionSlot6/D27
- J3 pad B13: /Expansion/D28 -> /Expansion/ExpansionSlot6/D28
- J3 pad B14: /Expansion/D29 -> /Expansion/ExpansionSlot6/D29
- J3 pad B15: /Expansion/D30 -> /Expansion/ExpansionSlot6/D30
- J3 pad B16: /Expansion/D31 -> /Expansion/ExpansionSlot6/D31
- J3 pad B17: /Expansion/A0 -> /Expansion/ExpansionSlot6/A0
- J3 pad B18: /Expansion/A20 -> /Expansion/ExpansionSlot6/A20
- J3 pad B19: /Expansion/A21 -> /Expansion/ExpansionSlot6/A21
- J3 pad B2: /Expansion/D17 -> /Expansion/ExpansionSlot6/D17
- J3 pad B20: /Expansion/A22 -> /Expansion/ExpansionSlot6/A22
- J3 pad B21: /Expansion/A23 -> /Expansion/ExpansionSlot6/A23
- J3 pad B22: /Expansion/A24 -> /Expansion/ExpansionSlot6/A24
- J3 pad B23: /Expansion/A25 -> /Expansion/ExpansionSlot6/A25
- J3 pad B24: /Expansion/A26 -> /Expansion/ExpansionSlot6/A26
- J3 pad B25: /Expansion/A27 -> /Expansion/ExpansionSlot6/A27
- J3 pad B26: /Expansion/A28 -> /Expansion/ExpansionSlot6/A28
- J3 pad B27: /Expansion/A29 -> /Expansion/ExpansionSlot6/A29
- J3 pad B28: /Expansion/A30 -> /Expansion/ExpansionSlot6/A30
- J3 pad B29: /Expansion/A31 -> /Expansion/ExpansionSlot6/A31
- J3 pad B3: /Expansion/D18 -> /Expansion/ExpansionSlot6/D18
- J3 pad B31: unconnected-(J6-PadB31) -> /Expansion/ExpansionSlot6/BCLK
- J3 pad B32: unconnected-(J6-PadB32) -> GND
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Routing:
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
Commit message: updates
Parts:
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Connections:
- net /Expansion/ExpansionSlot1/D0 renamed /Expansion/ExpansionSlot1/EXD0
- net /Expansion/ExpansionSlot1/D1 renamed /Expansion/ExpansionSlot1/EXD1
- net /Expansion/ExpansionSlot1/D10 renamed /Expansion/ExpansionSlot1/EXD10
- net /Expansion/ExpansionSlot1/D11 renamed /Expansion/ExpansionSlot1/EXD11
- net /Expansion/ExpansionSlot1/D12 renamed /Expansion/ExpansionSlot1/EXD12
- net /Expansion/ExpansionSlot1/D13 renamed /Expansion/ExpansionSlot1/EXD13
- net /Expansion/ExpansionSlot1/D14 renamed /Expansion/ExpansionSlot1/EXD14
- net /Expansion/ExpansionSlot1/D15 renamed /Expansion/ExpansionSlot1/EXD15
- net /Expansion/ExpansionSlot1/D16 renamed /Expansion/ExpansionSlot1/EXD16
- net /Expansion/ExpansionSlot1/D17 renamed /Expansion/ExpansionSlot1/EXD17
- net /Expansion/ExpansionSlot1/D18 renamed /Expansion/ExpansionSlot1/EXD18
- net /Expansion/ExpansionSlot1/D19 renamed /Expansion/ExpansionSlot1/EXD19
- net /Expansion/ExpansionSlot1/D2 renamed /Expansion/ExpansionSlot1/EXD2
- net /Expansion/ExpansionSlot1/D20 renamed /Expansion/ExpansionSlot1/EXD20
- net /Expansion/ExpansionSlot1/D21 renamed /Expansion/ExpansionSlot1/EXD21
- net /Expansion/ExpansionSlot1/D22 renamed /Expansion/ExpansionSlot1/EXD22
- net /Expansion/ExpansionSlot1/D23 renamed /Expansion/ExpansionSlot1/EXD23
- net /Expansion/ExpansionSlot1/D24 renamed /Expansion/ExpansionSlot1/EXD24
- net /Expansion/ExpansionSlot1/D25 renamed /Expansion/ExpansionSlot1/EXD25
- net /Expansion/ExpansionSlot1/D26 renamed /Expansion/ExpansionSlot1/EXD26
- net /Expansion/ExpansionSlot1/D27 renamed /Expansion/ExpansionSlot1/EXD27
- net /Expansion/ExpansionSlot1/D28 renamed /Expansion/ExpansionSlot1/EXD28
- net /Expansion/ExpansionSlot1/D29 renamed /Expansion/ExpansionSlot1/EXD29
- net /Expansion/ExpansionSlot1/D3 renamed /Expansion/ExpansionSlot1/EXD3
- net /Expansion/ExpansionSlot1/D30 renamed /Expansion/ExpansionSlot1/EXD30
- net /Expansion/ExpansionSlot1/D31 renamed /Expansion/ExpansionSlot1/EXD31
- net /Expansion/ExpansionSlot1/D4 renamed /Expansion/ExpansionSlot1/EXD4
- net /Expansion/ExpansionSlot1/D5 renamed /Expansion/ExpansionSlot1/EXD5
- net /Expansion/ExpansionSlot1/D6 renamed /Expansion/ExpansionSlot1/EXD6
- net /Expansion/ExpansionSlot1/D7 renamed /Expansion/ExpansionSlot1/EXD7
- net /Expansion/ExpansionSlot1/D8 renamed /Expansion/ExpansionSlot1/EXD8
- net /Expansion/ExpansionSlot1/D9 renamed /Expansion/ExpansionSlot1/EXD9
- net /Expansion/ExpansionSlot2/A0 renamed /Expansion/ExpansionSlot2/EXA0
- net /Expansion/ExpansionSlot2/A1 renamed /Expansion/ExpansionSlot2/EXA1
- net /Expansion/ExpansionSlot2/A10 renamed /Expansion/ExpansionSlot2/EXA10
- net /Expansion/ExpansionSlot2/A11 renamed /Expansion/ExpansionSlot2/EXA11
- net /Expansion/ExpansionSlot2/A12 renamed /Expansion/ExpansionSlot2/EXA12
- net /Expansion/ExpansionSlot2/A13 renamed /Expansion/ExpansionSlot2/EXA13
- net /Expansion/ExpansionSlot2/A14 renamed /Expansion/ExpansionSlot2/EXA14
- net /Expansion/ExpansionSlot2/A15 renamed /Expansion/ExpansionSlot2/EXA15
- net /Expansion/ExpansionSlot2/A16 renamed /Expansion/ExpansionSlot2/EXA16
- net /Expansion/ExpansionSlot2/A17 renamed /Expansion/ExpansionSlot2/EXA17
- net /Expansion/ExpansionSlot2/A18 renamed /Expansion/ExpansionSlot2/EXA18
- net /Expansion/ExpansionSlot2/A19 renamed /Expansion/ExpansionSlot2/EXA19
- net /Expansion/ExpansionSlot2/A2 renamed /Expansion/ExpansionSlot2/EXA2
- net /Expansion/ExpansionSlot2/A20 renamed /Expansion/ExpansionSlot2/EXA20
- net /Expansion/ExpansionSlot2/A21 renamed /Expansion/ExpansionSlot2/EXA21
- net /Expansion/ExpansionSlot2/A22 renamed /Expansion/ExpansionSlot2/EXA22
- net /Expansion/ExpansionSlot2/A23 renamed /Expansion/ExpansionSlot2/EXA23
- net /Expansion/ExpansionSlot2/A24 renamed /Expansion/ExpansionSlot2/EXA24
- net /Expansion/ExpansionSlot2/A25 renamed /Expansion/ExpansionSlot2/EXA25
- net /Expansion/ExpansionSlot2/A26 renamed /Expansion/ExpansionSlot2/EXA26
- net /Expansion/ExpansionSlot2/A27 renamed /Expansion/ExpansionSlot2/EXA27
- net /Expansion/ExpansionSlot2/A28 renamed /Expansion/ExpansionSlot2/EXA28
- net /Expansion/ExpansionSlot2/A29 renamed /Expansion/ExpansionSlot2/EXA29
- net /Expansion/ExpansionSlot2/A3 renamed /Expansion/ExpansionSlot2/EXA3
- net /Expansion/ExpansionSlot2/A30 renamed /Expansion/ExpansionSlot2/EXA30
- net /Expansion/ExpansionSlot2/A31 renamed /Expansion/ExpansionSlot2/EXA31
- net /Expansion/ExpansionSlot2/A4 renamed /Expansion/ExpansionSlot2/EXA4
- net /Expansion/ExpansionSlot2/A5 renamed /Expansion/ExpansionSlot2/EXA5
- net /Expansion/ExpansionSlot2/A6 renamed /Expansion/ExpansionSlot2/EXA6
- net /Expansion/ExpansionSlot2/A7 renamed /Expansion/ExpansionSlot2/EXA7
- net /Expansion/ExpansionSlot2/A8 renamed /Expansion/ExpansionSlot2/EXA8
- net /Expansion/ExpansionSlot2/A9 renamed /Expansion/ExpansionSlot2/EXA9
- net /Expansion/ExpansionSlot2/D0 renamed /Expansion/ExpansionSlot2/EXD0
- net /Expansion/ExpansionSlot2/D1 renamed /Expansion/ExpansionSlot2/EXD1
- net /Expansion/ExpansionSlot2/D10 renamed /Expansion/ExpansionSlot2/EXD10
- net /Expansion/ExpansionSlot2/D11 renamed /Expansion/ExpansionSlot2/EXD11
- net /Expansion/ExpansionSlot2/D12 renamed /Expansion/ExpansionSlot2/EXD12
- net /Expansion/ExpansionSlot2/D13 renamed /Expansion/ExpansionSlot2/EXD13
- net /Expansion/ExpansionSlot2/D14 renamed /Expansion/ExpansionSlot2/EXD14
- net /Expansion/ExpansionSlot2/D15 renamed /Expansion/ExpansionSlot2/EXD15
- net /Expansion/ExpansionSlot2/D16 renamed /Expansion/ExpansionSlot2/EXD16
- net /Expansion/ExpansionSlot2/D17 renamed /Expansion/ExpansionSlot2/EXD17
- net /Expansion/ExpansionSlot2/D18 renamed /Expansion/ExpansionSlot2/EXD18
- net /Expansion/ExpansionSlot2/D19 renamed /Expansion/ExpansionSlot2/EXD19
- net /Expansion/ExpansionSlot2/D2 renamed /Expansion/ExpansionSlot2/EXD2
- net /Expansion/ExpansionSlot2/D20 renamed /Expansion/ExpansionSlot2/EXD20
- net /Expansion/ExpansionSlot2/D21 renamed /Expansion/ExpansionSlot2/EXD21
- net /Expansion/ExpansionSlot2/D22 renamed /Expansion/ExpansionSlot2/EXD22
- net /Expansion/ExpansionSlot2/D23 renamed /Expansion/ExpansionSlot2/EXD23
- net /Expansion/ExpansionSlot2/D24 renamed /Expansion/ExpansionSlot2/EXD24
- net /Expansion/ExpansionSlot2/D25 renamed /Expansion/ExpansionSlot2/EXD25
- net /Expansion/ExpansionSlot2/D26 renamed /Expansion/ExpansionSlot2/EXD26
- net /Expansion/ExpansionSlot2/D27 renamed /Expansion/ExpansionSlot2/EXD27
- net /Expansion/ExpansionSlot2/D28 renamed /Expansion/ExpansionSlot2/EXD28
- net /Expansion/ExpansionSlot2/D29 renamed /Expansion/ExpansionSlot2/EXD29
- net /Expansion/ExpansionSlot2/D3 renamed /Expansion/ExpansionSlot2/EXD3
- net /Expansion/ExpansionSlot2/D30 renamed /Expansion/ExpansionSlot2/EXD30
- net /Expansion/ExpansionSlot2/D31 renamed /Expansion/ExpansionSlot2/EXD31
- net /Expansion/ExpansionSlot2/D4 renamed /Expansion/ExpansionSlot2/EXD4
- net /Expansion/ExpansionSlot2/D5 renamed /Expansion/ExpansionSlot2/EXD5
- net /Expansion/ExpansionSlot2/D6 renamed /Expansion/ExpansionSlot2/EXD6
- net /Expansion/ExpansionSlot2/D7 renamed /Expansion/ExpansionSlot2/EXD7
- net /Expansion/ExpansionSlot2/D8 renamed /Expansion/ExpansionSlot2/EXD8
- net /Expansion/ExpansionSlot2/D9 renamed /Expansion/ExpansionSlot2/EXD9
- net /Expansion/ExpansionSlot3/A0 renamed /Expansion/ExpansionSlot3/EXA0
- net /Expansion/ExpansionSlot3/A1 renamed /Expansion/ExpansionSlot3/EXA1
- net /Expansion/ExpansionSlot3/A10 renamed /Expansion/ExpansionSlot3/EXA10
- net /Expansion/ExpansionSlot3/A11 renamed /Expansion/ExpansionSlot3/EXA11
- net /Expansion/ExpansionSlot3/A12 renamed /Expansion/ExpansionSlot3/EXA12
- net /Expansion/ExpansionSlot3/A13 renamed /Expansion/ExpansionSlot3/EXA13
- net /Expansion/ExpansionSlot3/A14 renamed /Expansion/ExpansionSlot3/EXA14
- net /Expansion/ExpansionSlot3/A15 renamed /Expansion/ExpansionSlot3/EXA15
- net /Expansion/ExpansionSlot3/A16 renamed /Expansion/ExpansionSlot3/EXA16
- net /Expansion/ExpansionSlot3/A17 renamed /Expansion/ExpansionSlot3/EXA17
- net /Expansion/ExpansionSlot3/A18 renamed /Expansion/ExpansionSlot3/EXA18
- net /Expansion/ExpansionSlot3/A19 renamed /Expansion/ExpansionSlot3/EXA19
- net /Expansion/ExpansionSlot3/A2 renamed /Expansion/ExpansionSlot3/EXA2
- net /Expansion/ExpansionSlot3/A20 renamed /Expansion/ExpansionSlot3/EXA20
- net /Expansion/ExpansionSlot3/A21 renamed /Expansion/ExpansionSlot3/EXA21
- net /Expansion/ExpansionSlot3/A22 renamed /Expansion/ExpansionSlot3/EXA22
- net /Expansion/ExpansionSlot3/A23 renamed /Expansion/ExpansionSlot3/EXA23
- net /Expansion/ExpansionSlot3/A24 renamed /Expansion/ExpansionSlot3/EXA24
- net /Expansion/ExpansionSlot3/A25 renamed /Expansion/ExpansionSlot3/EXA25
- net /Expansion/ExpansionSlot3/A26 renamed /Expansion/ExpansionSlot3/EXA26
- net /Expansion/ExpansionSlot3/A27 renamed /Expansion/ExpansionSlot3/EXA27
- net /Expansion/ExpansionSlot3/A28 renamed /Expansion/ExpansionSlot3/EXA28
- net /Expansion/ExpansionSlot3/A29 renamed /Expansion/ExpansionSlot3/EXA29
- net /Expansion/ExpansionSlot3/A3 renamed /Expansion/ExpansionSlot3/EXA3
- net /Expansion/ExpansionSlot3/A30 renamed /Expansion/ExpansionSlot3/EXA30
- net /Expansion/ExpansionSlot3/A31 renamed /Expansion/ExpansionSlot3/EXA31
- net /Expansion/ExpansionSlot3/A4 renamed /Expansion/ExpansionSlot3/EXA4
- net /Expansion/ExpansionSlot3/A5 renamed /Expansion/ExpansionSlot3/EXA5
- net /Expansion/ExpansionSlot3/A6 renamed /Expansion/ExpansionSlot3/EXA6
- net /Expansion/ExpansionSlot3/A7 renamed /Expansion/ExpansionSlot3/EXA7
- net /Expansion/ExpansionSlot3/A8 renamed /Expansion/ExpansionSlot3/EXA8
- net /Expansion/ExpansionSlot3/A9 renamed /Expansion/ExpansionSlot3/EXA9
- net /Expansion/ExpansionSlot3/D0 renamed /Expansion/ExpansionSlot3/EXD0
- net /Expansion/ExpansionSlot3/D1 renamed /Expansion/ExpansionSlot3/EXD1
- net /Expansion/ExpansionSlot3/D10 renamed /Expansion/ExpansionSlot3/EXD10
- net /Expansion/ExpansionSlot3/D11 renamed /Expansion/ExpansionSlot3/EXD11
- net /Expansion/ExpansionSlot3/D12 renamed /Expansion/ExpansionSlot3/EXD12
- net /Expansion/ExpansionSlot3/D13 renamed /Expansion/ExpansionSlot3/EXD13
- net /Expansion/ExpansionSlot3/D14 renamed /Expansion/ExpansionSlot3/EXD14
- net /Expansion/ExpansionSlot3/D15 renamed /Expansion/ExpansionSlot3/EXD15
- net /Expansion/ExpansionSlot3/D16 renamed /Expansion/ExpansionSlot3/EXD16
- net /Expansion/ExpansionSlot3/D17 renamed /Expansion/ExpansionSlot3/EXD17
- net /Expansion/ExpansionSlot3/D18 renamed /Expansion/ExpansionSlot3/EXD18
- net /Expansion/ExpansionSlot3/D19 renamed /Expansion/ExpansionSlot3/EXD19
- net /Expansion/ExpansionSlot3/D2 renamed /Expansion/ExpansionSlot3/EXD2
- net /Expansion/ExpansionSlot3/D20 renamed /Expansion/ExpansionSlot3/EXD20
- net /Expansion/ExpansionSlot3/D21 renamed /Expansion/ExpansionSlot3/EXD21
- net /Expansion/ExpansionSlot3/D22 renamed /Expansion/ExpansionSlot3/EXD22
- net /Expansion/ExpansionSlot3/D23 renamed /Expansion/ExpansionSlot3/EXD23
- net /Expansion/ExpansionSlot3/D24 renamed /Expansion/ExpansionSlot3/EXD24
- net /Expansion/ExpansionSlot3/D25 renamed /Expansion/ExpansionSlot3/EXD25
- net /Expansion/ExpansionSlot3/D26 renamed /Expansion/ExpansionSlot3/EXD26
- net /Expansion/ExpansionSlot3/D27 renamed /Expansion/ExpansionSlot3/EXD27
- net /Expansion/ExpansionSlot3/D28 renamed /Expansion/ExpansionSlot3/EXD28
- net /Expansion/ExpansionSlot3/D29 renamed /Expansion/ExpansionSlot3/EXD29
- net /Expansion/ExpansionSlot3/D3 renamed /Expansion/ExpansionSlot3/EXD3
- net /Expansion/ExpansionSlot3/D30 renamed /Expansion/ExpansionSlot3/EXD30
- net /Expansion/ExpansionSlot3/D31 renamed /Expansion/ExpansionSlot3/EXD31
- net /Expansion/ExpansionSlot3/D4 renamed /Expansion/ExpansionSlot3/EXD4
- net /Expansion/ExpansionSlot3/D5 renamed /Expansion/ExpansionSlot3/EXD5
- net /Expansion/ExpansionSlot3/D6 renamed /Expansion/ExpansionSlot3/EXD6
- net /Expansion/ExpansionSlot3/D7 renamed /Expansion/ExpansionSlot3/EXD7
- net /Expansion/ExpansionSlot3/D8 renamed /Expansion/ExpansionSlot3/EXD8
- net /Expansion/ExpansionSlot3/D9 renamed /Expansion/ExpansionSlot3/EXD9
- net /Expansion/ExpansionSlot4/A0 renamed /Expansion/ExpansionSlot4/EXA0
- net /Expansion/ExpansionSlot4/A1 renamed /Expansion/ExpansionSlot4/EXA1
- net /Expansion/ExpansionSlot4/A10 renamed /Expansion/ExpansionSlot4/EXA10
- net /Expansion/ExpansionSlot4/A11 renamed /Expansion/ExpansionSlot4/EXA11
- net /Expansion/ExpansionSlot4/A12 renamed /Expansion/ExpansionSlot4/EXA12
- net /Expansion/ExpansionSlot4/A13 renamed /Expansion/ExpansionSlot4/EXA13
- net /Expansion/ExpansionSlot4/A14 renamed /Expansion/ExpansionSlot4/EXA14
- net /Expansion/ExpansionSlot4/A15 renamed /Expansion/ExpansionSlot4/EXA15
- net /Expansion/ExpansionSlot4/A16 renamed /Expansion/ExpansionSlot4/EXA16
- net /Expansion/ExpansionSlot4/A17 renamed /Expansion/ExpansionSlot4/EXA17
- net /Expansion/ExpansionSlot4/A18 renamed /Expansion/ExpansionSlot4/EXA18
- net /Expansion/ExpansionSlot4/A19 renamed /Expansion/ExpansionSlot4/EXA19
- net /Expansion/ExpansionSlot4/A2 renamed /Expansion/ExpansionSlot4/EXA2
- net /Expansion/ExpansionSlot4/A20 renamed /Expansion/ExpansionSlot4/EXA20
- net /Expansion/ExpansionSlot4/A21 renamed /Expansion/ExpansionSlot4/EXA21
- net /Expansion/ExpansionSlot4/A22 renamed /Expansion/ExpansionSlot4/EXA22
- net /Expansion/ExpansionSlot4/A23 renamed /Expansion/ExpansionSlot4/EXA23
- net /Expansion/ExpansionSlot4/A24 renamed /Expansion/ExpansionSlot4/EXA24
- net /Expansion/ExpansionSlot4/A25 renamed /Expansion/ExpansionSlot4/EXA25
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Routing:
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
Commit message: updates
Parts:
- added C1: C, Capacitor_SMD:C_0603_1608Metric, F.Cu at (283.1, 312.9)
- added C2: C, Capacitor_SMD:C_0603_1608Metric, F.Cu at (283.1, 315.4)
- added R4: 10k, Resistor_SMD:R_0603_1608Metric, F.Cu at (316.0, 292.3)
- added R5: 10k, Capacitor_SMD:C_0603_1608Metric, F.Cu at (316.0, 294.8)
- added U15: SN74ALVC164245, Package_SO:TSSOP-48_6.1x12.5mm_P0.5mm, F.Cu at (222.9, 247.7)
- added U16: SN74ALVC164245, Package_SO:TSSOP-48_6.1x12.5mm_P0.5mm, F.Cu at (212.1, 258.5)
- added U17: SN74ALVC164245, Package_SO:TSSOP-48_6.1x12.5mm_P0.5mm, F.Cu at (214.0, 278.2)
- added U18: SN74ALVC164245, Package_SO:TSSOP-48_6.1x12.5mm_P0.5mm, F.Cu at (224.7, 289.0)
- added U19: 74HC245, Package_SO:SOIC-20W_7.5x12.8mm_P1.27mm, F.Cu at (160.0, 231.1)
- added U20: 74HC245, Package_SO:SOIC-20W_7.5x12.8mm_P1.27mm, F.Cu at (175.3, 231.1)
- added U21: 74HC245, Package_SO:SOIC-20W_7.5x12.8mm_P1.27mm, F.Cu at (190.5, 231.1)
- added U22: 74HC245, Package_SO:SOIC-20W_7.5x12.8mm_P1.27mm, F.Cu at (205.7, 231.1)
- added U23: PCF8584, Package_SO:SOIC-20W_7.5x12.8mm_P1.27mm, F.Cu at (104.1, 287.0)
- added U24: ~, Package_LCC:PLCC-68_SMD-Socket, F.Cu at (116.8, 261.6)
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Connections:
- J1 pad A10: /Expansion/ExpansionSlot8/EXD14 -> /Expansion/EXD14
- J1 pad A12: /Expansion/ExpansionSlot8/EXA1 -> /Expansion/EXA1
- J1 pad A13: /Expansion/ExpansionSlot8/EXA3 -> /Expansion/EXA3
- J1 pad A14: /Expansion/ExpansionSlot8/EXA5 -> /Expansion/EXA5
- J1 pad A15: /Expansion/ExpansionSlot8/EXA7 -> /Expansion/EXA7
- J1 pad A16: /Expansion/ExpansionSlot8/EXA9 -> /Expansion/EXA9
- J1 pad A17: /Expansion/ExpansionSlot8/EXA11 -> /Expansion/EXA11
- J1 pad A18: /Expansion/ExpansionSlot8/EXA13 -> /Expansion/EXA13
- J1 pad A19: /Expansion/ExpansionSlot8/EXA15 -> /Expansion/EXA15
- J1 pad A20: /Expansion/ExpansionSlot8/EXA17 -> /Expansion/EXA17
- J1 pad A21: /Expansion/ExpansionSlot8/EXA19 -> /Expansion/EXA19
- J1 pad A3: /Expansion/ExpansionSlot8/EXD0 -> /Expansion/EXD0
- J1 pad A4: /Expansion/ExpansionSlot8/EXD2 -> /Expansion/EXD2
- J1 pad A5: /Expansion/ExpansionSlot8/EXD4 -> /Expansion/EXD4
- J1 pad A6: /Expansion/ExpansionSlot8/EXD6 -> /Expansion/EXD6
- J1 pad A7: /Expansion/ExpansionSlot8/EXD8 -> /Expansion/EXD8
- J1 pad A8: /Expansion/ExpansionSlot8/EXD10 -> /Expansion/EXD10
- J1 pad A9: /Expansion/ExpansionSlot8/EXD12 -> /Expansion/EXD12
- J1 pad B1: /Expansion/ExpansionSlot8/EXD16 -> /Expansion/EXD16
- J1 pad B10: /Expansion/ExpansionSlot8/EXD25 -> /Expansion/EXD25
- J1 pad B11: /Expansion/ExpansionSlot8/EXD26 -> /Expansion/EXD26
- J1 pad B12: /Expansion/ExpansionSlot8/EXD27 -> /Expansion/EXD27
- J1 pad B13: /Expansion/ExpansionSlot8/EXD28 -> /Expansion/EXD28
- J1 pad B14: /Expansion/ExpansionSlot8/EXD29 -> /Expansion/EXD29
- J1 pad B15: /Expansion/ExpansionSlot8/EXD30 -> /Expansion/EXD30
- J1 pad B16: /Expansion/ExpansionSlot8/EXD31 -> /Expansion/EXD31
- J1 pad B17: /Expansion/ExpansionSlot8/EXA0 -> /Expansion/EXA0
- J1 pad B18: /Expansion/ExpansionSlot8/EXA20 -> /Expansion/EXA20
- J1 pad B19: /Expansion/ExpansionSlot8/EXA21 -> /Expansion/EXA21
- J1 pad B2: /Expansion/ExpansionSlot8/EXD17 -> /Expansion/EXD17
- J1 pad B20: /Expansion/ExpansionSlot8/EXA22 -> /Expansion/EXA22
- J1 pad B21: /Expansion/ExpansionSlot8/EXA23 -> /Expansion/EXA23
- J1 pad B22: /Expansion/ExpansionSlot8/EXA24 -> /Expansion/EXA24
- J1 pad B23: /Expansion/ExpansionSlot8/EXA25 -> /Expansion/EXA25
- J1 pad B24: /Expansion/ExpansionSlot8/EXA26 -> /Expansion/EXA26
- J1 pad B25: /Expansion/ExpansionSlot8/EXA27 -> /Expansion/EXA27
- J1 pad B26: /Expansion/ExpansionSlot8/EXA28 -> /Expansion/EXA28
- J1 pad B27: /Expansion/ExpansionSlot8/EXA29 -> /Expansion/EXA29
- J1 pad B28: /Expansion/ExpansionSlot8/EXA30 -> /Expansion/EXA30
- J1 pad B29: /Expansion/ExpansionSlot8/EXA31 -> /Expansion/EXA31
- J1 pad B3: /Expansion/ExpansionSlot8/EXD18 -> /Expansion/EXD18
- J1 pad B4: /Expansion/ExpansionSlot8/EXD19 -> /Expansion/EXD19
- J1 pad B5: /Expansion/ExpansionSlot8/EXD20 -> /Expansion/EXD20
- J1 pad B6: /Expansion/ExpansionSlot8/EXD21 -> /Expansion/EXD21
- J1 pad B7: /Expansion/ExpansionSlot8/EXD22 -> /Expansion/EXD22
- J1 pad B8: /Expansion/ExpansionSlot8/EXD23 -> /Expansion/EXD23
- J1 pad B9: /Expansion/ExpansionSlot8/EXD24 -> /Expansion/EXD24
- J1 pad C10: /Expansion/ExpansionSlot8/EXD15 -> /Expansion/EXD15
- J1 pad C12: /Expansion/ExpansionSlot8/EXA2 -> /Expansion/EXA2
- J1 pad C13: /Expansion/ExpansionSlot8/EXA4 -> /Expansion/EXA4
- J1 pad C14: /Expansion/ExpansionSlot8/EXA6 -> /Expansion/EXA6
- J1 pad C15: /Expansion/ExpansionSlot8/EXA8 -> /Expansion/EXA8
- J1 pad C16: /Expansion/ExpansionSlot8/EXA10 -> /Expansion/EXA10
- J1 pad C17: /Expansion/ExpansionSlot8/EXA12 -> /Expansion/EXA12
- J1 pad C18: /Expansion/ExpansionSlot8/EXA14 -> /Expansion/EXA14
- J1 pad C19: /Expansion/ExpansionSlot8/EXA16 -> /Expansion/EXA16
- J1 pad C20: /Expansion/ExpansionSlot8/EXA18 -> /Expansion/EXA18
- J1 pad C3: /Expansion/ExpansionSlot8/EXD1 -> /Expansion/EXD1
- J1 pad C4: /Expansion/ExpansionSlot8/EXD3 -> /Expansion/EXD3
- J1 pad C5: /Expansion/ExpansionSlot8/EXD5 -> /Expansion/EXD5
- J1 pad C6: /Expansion/ExpansionSlot8/EXD7 -> /Expansion/EXD7
- J1 pad C7: /Expansion/ExpansionSlot8/EXD9 -> /Expansion/EXD9
- J1 pad C8: /Expansion/ExpansionSlot8/EXD11 -> /Expansion/EXD11
- J1 pad C9: /Expansion/ExpansionSlot8/EXD13 -> /Expansion/EXD13
- J2 pad A10: /Expansion/ExpansionSlot7/EXD14 -> /Expansion/EXD14
- J2 pad A12: /Expansion/ExpansionSlot7/EXA1 -> /Expansion/EXA1
- J2 pad A13: /Expansion/ExpansionSlot7/EXA3 -> /Expansion/EXA3
- J2 pad A14: /Expansion/ExpansionSlot7/EXA5 -> /Expansion/EXA5
- J2 pad A15: /Expansion/ExpansionSlot7/EXA7 -> /Expansion/EXA7
- J2 pad A16: /Expansion/ExpansionSlot7/EXA9 -> /Expansion/EXA9
- J2 pad A17: /Expansion/ExpansionSlot7/EXA11 -> /Expansion/EXA11
- J2 pad A18: /Expansion/ExpansionSlot7/EXA13 -> /Expansion/EXA13
- J2 pad A19: /Expansion/ExpansionSlot7/EXA15 -> /Expansion/EXA15
- J2 pad A20: /Expansion/ExpansionSlot7/EXA17 -> /Expansion/EXA17
- J2 pad A21: /Expansion/ExpansionSlot7/EXA19 -> /Expansion/EXA19
- J2 pad A3: /Expansion/ExpansionSlot7/EXD0 -> /Expansion/EXD0
- J2 pad A4: /Expansion/ExpansionSlot7/EXD2 -> /Expansion/EXD2
- J2 pad A5: /Expansion/ExpansionSlot7/EXD4 -> /Expansion/EXD4
- J2 pad A6: /Expansion/ExpansionSlot7/EXD6 -> /Expansion/EXD6
- J2 pad A7: /Expansion/ExpansionSlot7/EXD8 -> /Expansion/EXD8
- J2 pad A8: /Expansion/ExpansionSlot7/EXD10 -> /Expansion/EXD10
- J2 pad A9: /Expansion/ExpansionSlot7/EXD12 -> /Expansion/EXD12
- J2 pad B1: /Expansion/ExpansionSlot7/EXD16 -> /Expansion/EXD16
- J2 pad B10: /Expansion/ExpansionSlot7/EXD25 -> /Expansion/EXD25
- J2 pad B11: /Expansion/ExpansionSlot7/EXD26 -> /Expansion/EXD26
- J2 pad B12: /Expansion/ExpansionSlot7/EXD27 -> /Expansion/EXD27
- J2 pad B13: /Expansion/ExpansionSlot7/EXD28 -> /Expansion/EXD28
- J2 pad B14: /Expansion/ExpansionSlot7/EXD29 -> /Expansion/EXD29
- J2 pad B15: /Expansion/ExpansionSlot7/EXD30 -> /Expansion/EXD30
- J2 pad B16: /Expansion/ExpansionSlot7/EXD31 -> /Expansion/EXD31
- J2 pad B17: /Expansion/ExpansionSlot7/EXA0 -> /Expansion/EXA0
- J2 pad B18: /Expansion/ExpansionSlot7/EXA20 -> /Expansion/EXA20
- J2 pad B19: /Expansion/ExpansionSlot7/EXA21 -> /Expansion/EXA21
- J2 pad B2: /Expansion/ExpansionSlot7/EXD17 -> /Expansion/EXD17
- J2 pad B20: /Expansion/ExpansionSlot7/EXA22 -> /Expansion/EXA22
- J2 pad B21: /Expansion/ExpansionSlot7/EXA23 -> /Expansion/EXA23
- J2 pad B22: /Expansion/ExpansionSlot7/EXA24 -> /Expansion/EXA24
- J2 pad B23: /Expansion/ExpansionSlot7/EXA25 -> /Expansion/EXA25
- J2 pad B24: /Expansion/ExpansionSlot7/EXA26 -> /Expansion/EXA26
- J2 pad B25: /Expansion/ExpansionSlot7/EXA27 -> /Expansion/EXA27
- J2 pad B26: /Expansion/ExpansionSlot7/EXA28 -> /Expansion/EXA28
- J2 pad B27: /Expansion/ExpansionSlot7/EXA29 -> /Expansion/EXA29
- J2 pad B28: /Expansion/ExpansionSlot7/EXA30 -> /Expansion/EXA30
- J2 pad B29: /Expansion/ExpansionSlot7/EXA31 -> /Expansion/EXA31
- J2 pad B3: /Expansion/ExpansionSlot7/EXD18 -> /Expansion/EXD18
- J2 pad B4: /Expansion/ExpansionSlot7/EXD19 -> /Expansion/EXD19
- J2 pad B5: /Expansion/ExpansionSlot7/EXD20 -> /Expansion/EXD20
- J2 pad B6: /Expansion/ExpansionSlot7/EXD21 -> /Expansion/EXD21
- J2 pad B7: /Expansion/ExpansionSlot7/EXD22 -> /Expansion/EXD22
- J2 pad B8: /Expansion/ExpansionSlot7/EXD23 -> /Expansion/EXD23
- J2 pad B9: /Expansion/ExpansionSlot7/EXD24 -> /Expansion/EXD24
- J2 pad C10: /Expansion/ExpansionSlot7/EXD15 -> /Expansion/EXD15
- J2 pad C12: /Expansion/ExpansionSlot7/EXA2 -> /Expansion/EXA2
- J2 pad C13: /Expansion/ExpansionSlot7/EXA4 -> /Expansion/EXA4
- J2 pad C14: /Expansion/ExpansionSlot7/EXA6 -> /Expansion/EXA6
- J2 pad C15: /Expansion/ExpansionSlot7/EXA8 -> /Expansion/EXA8
- J2 pad C16: /Expansion/ExpansionSlot7/EXA10 -> /Expansion/EXA10
- J2 pad C17: /Expansion/ExpansionSlot7/EXA12 -> /Expansion/EXA12
- J2 pad C18: /Expansion/ExpansionSlot7/EXA14 -> /Expansion/EXA14
- J2 pad C19: /Expansion/ExpansionSlot7/EXA16 -> /Expansion/EXA16
- J2 pad C20: /Expansion/ExpansionSlot7/EXA18 -> /Expansion/EXA18
- J2 pad C3: /Expansion/ExpansionSlot7/EXD1 -> /Expansion/EXD1
- J2 pad C4: /Expansion/ExpansionSlot7/EXD3 -> /Expansion/EXD3
- J2 pad C5: /Expansion/ExpansionSlot7/EXD5 -> /Expansion/EXD5
- J2 pad C6: /Expansion/ExpansionSlot7/EXD7 -> /Expansion/EXD7
- J2 pad C7: /Expansion/ExpansionSlot7/EXD9 -> /Expansion/EXD9
- J2 pad C8: /Expansion/ExpansionSlot7/EXD11 -> /Expansion/EXD11
- J2 pad C9: /Expansion/ExpansionSlot7/EXD13 -> /Expansion/EXD13
- J3 pad A10: /Expansion/ExpansionSlot6/EXD14 -> /Expansion/EXD14
- J3 pad A12: /Expansion/ExpansionSlot6/EXA1 -> /Expansion/EXA1
- J3 pad A13: /Expansion/ExpansionSlot6/EXA3 -> /Expansion/EXA3
- J3 pad A14: /Expansion/ExpansionSlot6/EXA5 -> /Expansion/EXA5
- J3 pad A15: /Expansion/ExpansionSlot6/EXA7 -> /Expansion/EXA7
- J3 pad A16: /Expansion/ExpansionSlot6/EXA9 -> /Expansion/EXA9
- J3 pad A17: /Expansion/ExpansionSlot6/EXA11 -> /Expansion/EXA11
- J3 pad A18: /Expansion/ExpansionSlot6/EXA13 -> /Expansion/EXA13
- J3 pad A19: /Expansion/ExpansionSlot6/EXA15 -> /Expansion/EXA15
- J3 pad A20: /Expansion/ExpansionSlot6/EXA17 -> /Expansion/EXA17
- J3 pad A21: /Expansion/ExpansionSlot6/EXA19 -> /Expansion/EXA19
- J3 pad A3: /Expansion/ExpansionSlot6/EXD0 -> /Expansion/EXD0
- J3 pad A4: /Expansion/ExpansionSlot6/EXD2 -> /Expansion/EXD2
- J3 pad A5: /Expansion/ExpansionSlot6/EXD4 -> /Expansion/EXD4
- J3 pad A6: /Expansion/ExpansionSlot6/EXD6 -> /Expansion/EXD6
- J3 pad A7: /Expansion/ExpansionSlot6/EXD8 -> /Expansion/EXD8
- J3 pad A8: /Expansion/ExpansionSlot6/EXD10 -> /Expansion/EXD10
- J3 pad A9: /Expansion/ExpansionSlot6/EXD12 -> /Expansion/EXD12
- J3 pad B1: /Expansion/ExpansionSlot6/EXD16 -> /Expansion/EXD16
- J3 pad B10: /Expansion/ExpansionSlot6/EXD25 -> /Expansion/EXD25
- J3 pad B11: /Expansion/ExpansionSlot6/EXD26 -> /Expansion/EXD26
- J3 pad B12: /Expansion/ExpansionSlot6/EXD27 -> /Expansion/EXD27
- J3 pad B13: /Expansion/ExpansionSlot6/EXD28 -> /Expansion/EXD28
- J3 pad B14: /Expansion/ExpansionSlot6/EXD29 -> /Expansion/EXD29
- J3 pad B15: /Expansion/ExpansionSlot6/EXD30 -> /Expansion/EXD30
- J3 pad B16: /Expansion/ExpansionSlot6/EXD31 -> /Expansion/EXD31
- J3 pad B17: /Expansion/ExpansionSlot6/EXA0 -> /Expansion/EXA0
- J3 pad B18: /Expansion/ExpansionSlot6/EXA20 -> /Expansion/EXA20
- J3 pad B19: /Expansion/ExpansionSlot6/EXA21 -> /Expansion/EXA21
- J3 pad B2: /Expansion/ExpansionSlot6/EXD17 -> /Expansion/EXD17
- J3 pad B20: /Expansion/ExpansionSlot6/EXA22 -> /Expansion/EXA22
- J3 pad B21: /Expansion/ExpansionSlot6/EXA23 -> /Expansion/EXA23
- J3 pad B22: /Expansion/ExpansionSlot6/EXA24 -> /Expansion/EXA24
- J3 pad B23: /Expansion/ExpansionSlot6/EXA25 -> /Expansion/EXA25
- J3 pad B24: /Expansion/ExpansionSlot6/EXA26 -> /Expansion/EXA26
- J3 pad B25: /Expansion/ExpansionSlot6/EXA27 -> /Expansion/EXA27
- J3 pad B26: /Expansion/ExpansionSlot6/EXA28 -> /Expansion/EXA28
- J3 pad B27: /Expansion/ExpansionSlot6/EXA29 -> /Expansion/EXA29
- J3 pad B28: /Expansion/ExpansionSlot6/EXA30 -> /Expansion/EXA30
- J3 pad B29: /Expansion/ExpansionSlot6/EXA31 -> /Expansion/EXA31
- J3 pad B3: /Expansion/ExpansionSlot6/EXD18 -> /Expansion/EXD18
- J3 pad B4: /Expansion/ExpansionSlot6/EXD19 -> /Expansion/EXD19
- J3 pad B5: /Expansion/ExpansionSlot6/EXD20 -> /Expansion/EXD20
- J3 pad B6: /Expansion/ExpansionSlot6/EXD21 -> /Expansion/EXD21
- J3 pad B7: /Expansion/ExpansionSlot6/EXD22 -> /Expansion/EXD22
- J3 pad B8: /Expansion/ExpansionSlot6/EXD23 -> /Expansion/EXD23
- J3 pad B9: /Expansion/ExpansionSlot6/EXD24 -> /Expansion/EXD24
- J3 pad C10: /Expansion/ExpansionSlot6/EXD15 -> /Expansion/EXD15
- J3 pad C12: /Expansion/ExpansionSlot6/EXA2 -> /Expansion/EXA2
- J3 pad C13: /Expansion/ExpansionSlot6/EXA4 -> /Expansion/EXA4
- J3 pad C14: /Expansion/ExpansionSlot6/EXA6 -> /Expansion/EXA6
- J3 pad C15: /Expansion/ExpansionSlot6/EXA8 -> /Expansion/EXA8
- J3 pad C16: /Expansion/ExpansionSlot6/EXA10 -> /Expansion/EXA10
- J3 pad C17: /Expansion/ExpansionSlot6/EXA12 -> /Expansion/EXA12
- J3 pad C18: /Expansion/ExpansionSlot6/EXA14 -> /Expansion/EXA14
- J3 pad C19: /Expansion/ExpansionSlot6/EXA16 -> /Expansion/EXA16
- J3 pad C20: /Expansion/ExpansionSlot6/EXA18 -> /Expansion/EXA18
- J3 pad C3: /Expansion/ExpansionSlot6/EXD1 -> /Expansion/EXD1
- J3 pad C4: /Expansion/ExpansionSlot6/EXD3 -> /Expansion/EXD3
- J3 pad C5: /Expansion/ExpansionSlot6/EXD5 -> /Expansion/EXD5
- J3 pad C6: /Expansion/ExpansionSlot6/EXD7 -> /Expansion/EXD7
- J3 pad C7: /Expansion/ExpansionSlot6/EXD9 -> /Expansion/EXD9
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Routing:
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