File: hardware/68040pc.kicad_pcb (KiCad board)
At the start: 4 copper layers, 221 x 243.8 mm, 58 parts, among them J1 EXP, J13 DIN-5_180degree, J14 Mini-DIN-6, J15 COM1, J16 COM2, J17 LPT, J2 EXP, J3 EXP, J4 EXP, J5 EXP, J6 EXP, J7 EXP, J8 EXP, P8 Conn_01x06, P9 Conn_01x06, U1 68LC040, U10 74HC165, U11 74HC245, U12 74HC245, U13 74HC245, U14 74HC245, U15 SN74ALVC164245, U16 SN74ALVC164245, U17 SN74ALVC164245, U18 SN74ALVC164245, U19 74HC245, U2 ICE40HX4K-TQ144, U20 74HC245, U21 74HC245, U22 74HC245, U23 PCF8584, U3 SN74ALVC164245, U4 SN74ALVC164245, U5 W25Q32JVSSIM, U6 74LS32, U7 74LS32, U8 LTC6905xS5-133, U9 74HC165

Commit message: begin work on a simpler first draft board
Parts:
- removed C1, C2: C, Capacitor_SMD:C_0603_1608Metric
- removed the J1 at (220.4, 189.0)
- removed J10, J11, J12: ~, 68040:SIMM-72
- removed J13: DIN-5_180degree, 68040:DIN5-180
- removed J14: Mini-DIN-6, 68040:Mini-DIN6
- removed J15: COM1, Connector_PinHeader_2.54mm:PinHeader_2x05_P2.54mm_Vertical
- removed J16: COM2, Connector_PinHeader_2.54mm:PinHeader_2x05_P2.54mm_Vertical
- removed J17: LPT, Connector_PinHeader_2.54mm:PinHeader_2x13_P2.54mm_Vertical
- removed J5, J6, J7, J8: EXP, 68040:EXP
- removed RN3, RN4, RN5, RN6: 10k, Resistor_THT:R_Array_SIP5
- removed U20, U21, U22: 74HC245, Package_SO:SOIC-20W_7.5x12.8mm_P1.27mm
- added C4: .1uF, Capacitor_SMD:C_0603_1608Metric, F.Cu at (193.0, 102.7)
- added J3: EXP, 68040:EXP, F.Cu at (194.3, 237.5)
- RN2: value R_Network04_US -> 10k
- U10: value 74HC165 -> 74HC245; footprint Package_SO:SOIC-16_3.9x9.9mm_P1.27mm -> Package_SO:SOIC-20W_7.5x12.8mm_P1.27mm
- U17: value SN74ALVC164245 -> W25Q32JVSSIM; footprint Package_SO:TSSOP-48_6.1x12.5mm_P0.5mm -> Package_SO:SOIC-8_5.23x5.23mm_P1.27mm
- U2: value ICE40HX4K-TQ144 -> SN74ALVC164245; footprint Package_QFP:TQFP-144_20x20mm_P0.5mm -> Package_SO:TSSOP-48_6.1x12.5mm_P0.5mm
- U5: value W25Q32JVSSIM -> ICE40HX4K-TQ144; footprint Package_SO:SOIC-8_5.23x5.23mm_P1.27mm -> Package_QFP:TQFP-144_20x20mm_P0.5mm
- U6, U7: value 74LS32 -> 74HC245; footprint Package_SO:SOIC-14_3.9x8.7mm_P1.27mm -> Package_SO:SOIC-20W_7.5x12.8mm_P1.27mm
- U9: value 74HC165 -> 74LS32; footprint Package_SO:SOIC-16_3.9x9.9mm_P1.27mm -> Package_SO:SOIC-14_3.9x8.7mm_P1.27mm
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- renumbered J3 to J1, J4 to J2, J2 to J4
Connections:
- D1 pad 2: /Memory/CDONE -> /FPGA/CDONE
- J1 pad A2: /Expansion/ExpansionSlot6/~{CFG_{IN}} -> /Expansion/ExpansionSlot4/~{CFG_{IN}}
- J1 pad B31: /Expansion/ExpansionSlot6/BCLK -> /Expansion/ExpansionSlot4/BCLK
- J1 pad C2: /Expansion/ExpansionSlot6/~{CFG_{OUT}} -> /Expansion/ExpansionSlot4/~{CFG_{OUT}}
- J2 pad A2: /Expansion/ExpansionSlot5/~{CFG_{IN}} -> /Expansion/ExpansionSlot1/~{CFG_{IN}}
- J2 pad B31: /Expansion/ExpansionSlot5/BCLK -> /Expansion/ExpansionSlot1/BCLK
- J2 pad C2: /Expansion/ExpansionSlot5/~{CFG_{OUT}} -> /Expansion/ExpansionSlot1/~{CFG_{OUT}}
- J4 pad A2: /Expansion/ExpansionSlot7/~{CFG_{IN}} -> /Expansion/ExpansionSlot3/~{CFG_{IN}}
- J4 pad B31: /Expansion/ExpansionSlot7/BCLK -> /Expansion/ExpansionSlot3/BCLK
- J4 pad C2: /Expansion/ExpansionSlot7/~{CFG_{OUT}} -> /Expansion/ExpansionSlot3/~{CFG_{OUT}}
- J9 pad 12: /Memory/DRAM_A0 -> /FPGA/DRAM_A0
- J9 pad 13: /Memory/DRAM_A1 -> /FPGA/DRAM_A1
- J9 pad 14: /Memory/DRAM_A2 -> /FPGA/DRAM_A2
- J9 pad 15: /Memory/DRAM_A3 -> /FPGA/DRAM_A3
- J9 pad 16: /Memory/DRAM_A4 -> /FPGA/DRAM_A4
- J9 pad 17: /Memory/DRAM_A5 -> /FPGA/DRAM_A5
- J9 pad 18: /Memory/DRAM_A6 -> /FPGA/DRAM_A6
- J9 pad 19: /Memory/DRAM_A10 -> /FPGA/DRAM_A10
- J9 pad 28: /Memory/DRAM_A7 -> /FPGA/DRAM_A7
- J9 pad 29: /Memory/DRAM_A11 -> /FPGA/DRAM_A11
- J9 pad 31: /Memory/DRAM_A8 -> /FPGA/DRAM_A8
- J9 pad 32: /Memory/DRAM_A9 -> /FPGA/DRAM_A9
- J9 pad 33: /Memory/~{RAS3} -> /FPGA/~{RAS3}
- J9 pad 34: /Memory/~{RAS2} -> /FPGA/~{RAS2}
- J9 pad 40: /Memory/~{CAS_A0} -> /FPGA/~{CAS_A0}
- J9 pad 41: /Memory/~{CAS_A2} -> /FPGA/~{CAS_A2}
- J9 pad 42: /Memory/~{CAS_A3} -> /FPGA/~{CAS_A3}
- J9 pad 43: /Memory/~{CAS_A1} -> /FPGA/~{CAS_A1}
- J9 pad 44: /Memory/~{RAS0} -> /FPGA/~{RAS0}
- J9 pad 45: /Memory/~{RAS1} -> /FPGA/~{RAS1}
- J9 pad 67: /Memory/PD_{A}1 -> /FPGA/PD_{A}1
- J9 pad 68: /Memory/PD_{A}2 -> /FPGA/PD_{A}2
- J9 pad 69: /Memory/PD_{A}3 -> /FPGA/PD_{A}3
- J9 pad 70: /Memory/PD_{A}4 -> /FPGA/PD_{A}4
- R1 pad 1: /Memory/CDONE -> /FPGA/CDONE
- R2 pad 1: /Memory/FLASH_SS -> /FPGA/FLASH_SS
- R3 pad 1: /Memory/FLASH_SCK -> /FPGA/FLASH_SCK
- RN2 pad 1: GND -> +3V3
- RN2 pad 2: /Expansion/ExpansionSlot8/~{CFG_{OUT}} -> /FPGA/PD_{A}4
- RN2 pad 3: /Expansion/ExpansionSlot7/~{CFG_{OUT}} -> /FPGA/PD_{A}3
- RN2 pad 4: /Expansion/ExpansionSlot6/~{CFG_{OUT}} -> /FPGA/PD_{A}2
- RN2 pad 5: /Expansion/ExpansionSlot5/~{CFG_{OUT}} -> /FPGA/PD_{A}1
- U10 pad 1: /Memory/RAMPDSR_SH/~{LD} -> /Expansion/EXDIR
- U10 pad 10: Net-(U10-DS) -> GND
- U10 pad 11: /Memory/PD_{C}1 -> /Expansion/EXA15
- U10 pad 12: /Memory/PD_{C}2 -> /Expansion/EXA14
- U10 pad 13: /Memory/PD_{C}3 -> /Expansion/EXA13
- U10 pad 14: /Memory/PD_{C}4 -> /Expansion/EXA12
- U10 pad 15: GND -> /Expansion/EXA11
- U10 pad 16: +3V3 -> /Expansion/EXA10
- U10 pad 2: /Memory/RAMPDSR_CLK -> /Expansion/A8
- U10 pad 3: /Memory/PD_{D}1 -> /Expansion/A9
- U10 pad 4: /Memory/PD_{D}2 -> /Expansion/A10
- U10 pad 5: /Memory/PD_{D}3 -> /Expansion/A11
- U10 pad 6: /Memory/PD_{D}4 -> /Expansion/A12
- U10 pad 7: unconnected-(U10-~{Q7}-Pad7) -> /Expansion/A13
- U10 pad 8: GND -> /Expansion/A14
- U10 pad 9: /Memory/RAMPDSR_D_{OUT} -> /Expansion/A15
- U11 pad 1: /Expansion/EXDIR -> unconnected-(U11-A->B-Pad1)
- U11 pad 11: /Expansion/EXA7 -> /Expansion/EXD15
- U11 pad 12: /Expansion/EXA6 -> /Expansion/EXD14
- U11 pad 13: /Expansion/EXA5 -> /Expansion/EXD13
- U11 pad 14: /Expansion/EXA4 -> /Expansion/EXD12
- U11 pad 15: /Expansion/EXA3 -> /Expansion/EXD11
- U11 pad 16: /Expansion/EXA2 -> /Expansion/EXD10
- U11 pad 17: /Expansion/EXA1 -> /Expansion/EXD9
- U11 pad 18: /Expansion/EXA0 -> /Expansion/EXD8
- U11 pad 2: /Expansion/A0 -> /Expansion/D8
- U11 pad 3: /Expansion/A1 -> /Expansion/D9
- U11 pad 4: /Expansion/A2 -> /Expansion/D10
- U11 pad 5: /Expansion/A3 -> /Expansion/D11
- U11 pad 6: /Expansion/A4 -> /Expansion/D12
- U11 pad 7: /Expansion/A5 -> /Expansion/D13
- U11 pad 8: /Expansion/A6 -> /Expansion/D14
- U11 pad 9: /Expansion/A7 -> /Expansion/D15
- U12 pad 11: /Expansion/EXA15 -> /Expansion/EXA23
- U12 pad 12: /Expansion/EXA14 -> /Expansion/EXA22
- U12 pad 13: /Expansion/EXA13 -> /Expansion/EXA21
- U12 pad 14: /Expansion/EXA12 -> /Expansion/EXA20
- U12 pad 15: /Expansion/EXA11 -> /Expansion/EXA19
- U12 pad 16: /Expansion/EXA10 -> /Expansion/EXA18
- U12 pad 17: /Expansion/EXA9 -> /Expansion/EXA17
- U12 pad 18: /Expansion/EXA8 -> /Expansion/EXA16
- U12 pad 2: /Expansion/A8 -> /Expansion/A16
- U12 pad 3: /Expansion/A9 -> /Expansion/A17
- U12 pad 4: /Expansion/A10 -> /Expansion/A18
- U12 pad 5: /Expansion/A11 -> /Expansion/A19
- U12 pad 6: /Expansion/A12 -> /Expansion/A20
- U12 pad 7: /Expansion/A13 -> /Expansion/A21
- U12 pad 8: /Expansion/A14 -> /Expansion/A22
- U12 pad 9: /Expansion/A15 -> /Expansion/A23
- U13 pad 1: /Expansion/EXDIR -> unconnected-(U13-A->B-Pad1)
- U13 pad 11: /Expansion/EXA23 -> /Expansion/EXD23
- U13 pad 12: /Expansion/EXA22 -> /Expansion/EXD22
- U13 pad 13: /Expansion/EXA21 -> /Expansion/EXD21
- U13 pad 14: /Expansion/EXA20 -> /Expansion/EXD20
- U13 pad 15: /Expansion/EXA19 -> /Expansion/EXD19
- U13 pad 16: /Expansion/EXA18 -> /Expansion/EXD18
- U13 pad 17: /Expansion/EXA17 -> /Expansion/EXD17
- U13 pad 18: /Expansion/EXA16 -> /Expansion/EXD16
- U13 pad 2: /Expansion/A16 -> /Expansion/D16
- U13 pad 3: /Expansion/A17 -> /Expansion/D17
- U13 pad 4: /Expansion/A18 -> /Expansion/D18
- U13 pad 5: /Expansion/A19 -> /Expansion/D19
- U13 pad 6: /Expansion/A20 -> /Expansion/D20
- U13 pad 7: /Expansion/A21 -> /Expansion/D21
- U13 pad 8: /Expansion/A22 -> /Expansion/D22
- U13 pad 9: /Expansion/A23 -> /Expansion/D23
- U15 pad 10: unconnected-(U15B-GND-Pad10) -> GND
- U15 pad 11: /Expansion/A6 -> /Expansion/D22
- U15 pad 12: /Expansion/A7 -> /Expansion/D23
- U15 pad 13: /Expansion/A8 -> /Expansion/D24
- U15 pad 14: /Expansion/A9 -> /Expansion/D25
- U15 pad 15: unconnected-(U15B-GND-Pad15) -> GND
- U15 pad 16: /Expansion/A10 -> /Expansion/D26
- U15 pad 17: /Expansion/A11 -> /Expansion/D27
- U15 pad 18: unconnected-(U15B-VCCB-Pad18) -> +5V
- U15 pad 19: /Expansion/A12 -> /Expansion/D28
- U15 pad 2: /Expansion/A0 -> /Expansion/D16
- U15 pad 20: /Expansion/A13 -> /Expansion/D29
- U15 pad 21: unconnected-(U15B-GND-Pad21) -> GND
- U15 pad 22: /Expansion/A14 -> /Expansion/D30
- U15 pad 23: /Expansion/A15 -> /Expansion/D31
- U15 pad 26: /Memory/FPGA_A15 -> /FPGA/FPGA_D31
- U15 pad 27: /Memory/FPGA_A14 -> /FPGA/FPGA_D30
- U15 pad 28: unconnected-(U15B-GND-Pad28) -> GND
- U15 pad 29: /Memory/FPGA_A13 -> /FPGA/FPGA_D29
- U15 pad 3: /Expansion/A1 -> /Expansion/D17
- U15 pad 30: /Memory/FPGA_A12 -> /FPGA/FPGA_D28
- U15 pad 31: unconnected-(U15B-VCCA-Pad31) -> +3V3
- U15 pad 32: /Memory/FPGA_A11 -> /FPGA/FPGA_D27
- U15 pad 33: /Memory/FPGA_A10 -> /FPGA/FPGA_D26
- U15 pad 34: unconnected-(U15B-GND-Pad34) -> GND
- U15 pad 35: /Memory/FPGA_A9 -> /FPGA/FPGA_D25
- U15 pad 36: /Memory/FPGA_A8 -> /FPGA/FPGA_D24
- U15 pad 37: /Memory/FPGA_A7 -> /FPGA/FPGA_D23
- U15 pad 38: /Memory/FPGA_A6 -> /FPGA/FPGA_D22
- U15 pad 39: unconnected-(U15B-GND-Pad39) -> GND
- U15 pad 4: unconnected-(U15B-GND-Pad4) -> GND
- U15 pad 40: /Memory/FPGA_A5 -> /FPGA/FPGA_D21
- U15 pad 41: /Memory/FPGA_A4 -> /FPGA/FPGA_D20
- U15 pad 42: unconnected-(U15B-VCCA-Pad42) -> +3V3
- U15 pad 43: /Memory/FPGA_A3 -> /FPGA/FPGA_D19
- U15 pad 44: /Memory/FPGA_A2 -> /FPGA/FPGA_D18
- U15 pad 45: unconnected-(U15B-GND-Pad45) -> GND
- U15 pad 46: /Memory/FPGA_A1 -> /FPGA/FPGA_D17
- U15 pad 47: /Memory/FPGA_A0 -> /FPGA/FPGA_D16
- U15 pad 5: /Expansion/A2 -> /Expansion/D18
- U15 pad 6: /Expansion/A3 -> /Expansion/D19
- U15 pad 7: unconnected-(U15B-VCCB-Pad7) -> +5V
- U15 pad 8: /Expansion/A4 -> /Expansion/D20
- U15 pad 9: /Expansion/A5 -> /Expansion/D21
- U16 pad 10: unconnected-(U16B-GND-Pad10) -> GND
- U16 pad 11: /Expansion/A25 -> /Expansion/A6
- U16 pad 12: /Expansion/A24 -> /Expansion/A7
- U16 pad 13: /Expansion/A23 -> /Expansion/A8
- U16 pad 14: /Expansion/A22 -> /Expansion/A9
- U16 pad 15: unconnected-(U16B-GND-Pad15) -> GND
- U16 pad 16: /Expansion/A21 -> /Expansion/A10
- U16 pad 17: /Expansion/A20 -> /Expansion/A11
- U16 pad 18: unconnected-(U16B-VCCB-Pad18) -> +5V
- U16 pad 19: /Expansion/A19 -> /Expansion/A12
- U16 pad 2: /Expansion/A31 -> /Expansion/A0
- U16 pad 20: /Expansion/A18 -> /Expansion/A13
- U16 pad 21: unconnected-(U16B-GND-Pad21) -> GND
- U16 pad 22: /Expansion/A17 -> /Expansion/A14
- U16 pad 23: /Expansion/A16 -> /Expansion/A15
- U16 pad 26: /Memory/FPGA_A16 -> /FPGA/FPGA_A15
- U16 pad 27: /Memory/FPGA_A17 -> /FPGA/FPGA_A14
- U16 pad 28: unconnected-(U16B-GND-Pad28) -> GND
- U16 pad 29: /Memory/FPGA_A18 -> /FPGA/FPGA_A13
- U16 pad 3: /Expansion/A30 -> /Expansion/A1
- U16 pad 30: /Memory/FPGA_A19 -> /FPGA/FPGA_A12
- U16 pad 31: unconnected-(U16B-VCCA-Pad31) -> +3V3
- U16 pad 32: /Memory/FPGA_A20 -> /FPGA/FPGA_A11
- U16 pad 33: /Memory/FPGA_A21 -> /FPGA/FPGA_A10
- U16 pad 34: unconnected-(U16B-GND-Pad34) -> GND
- U16 pad 35: /Memory/FPGA_A22 -> /FPGA/FPGA_A9
- U16 pad 36: /Memory/FPGA_A23 -> /FPGA/FPGA_A8
- U16 pad 37: /Memory/FPGA_A24 -> /FPGA/FPGA_A7
- U16 pad 38: /Memory/FPGA_A25 -> /FPGA/FPGA_A6
- U16 pad 39: unconnected-(U16B-GND-Pad39) -> GND
- U16 pad 4: unconnected-(U16B-GND-Pad4) -> GND
- U16 pad 40: /Memory/FPGA_A26 -> /FPGA/FPGA_A5
- U16 pad 41: /Memory/FPGA_A27 -> /FPGA/FPGA_A4
- U16 pad 42: unconnected-(U16B-VCCA-Pad42) -> +3V3
- U16 pad 43: /Memory/FPGA_A28 -> /FPGA/FPGA_A3
- U16 pad 44: /Memory/FPGA_A29 -> /FPGA/FPGA_A2
- U16 pad 45: unconnected-(U16B-GND-Pad45) -> GND
- U16 pad 46: /Memory/FPGA_A30 -> /FPGA/FPGA_A1
- U16 pad 47: /Memory/FPGA_A31 -> /FPGA/FPGA_A0
- U16 pad 5: /Expansion/A29 -> /Expansion/A2
- U16 pad 6: /Expansion/A28 -> /Expansion/A3
- U16 pad 7: unconnected-(U16B-VCCB-Pad7) -> +5V
- U16 pad 8: /Expansion/A27 -> /Expansion/A4
- U16 pad 9: /Expansion/A26 -> /Expansion/A5
- U17 pad 1: unconnected-(U17A-1DIR-Pad1) -> /FPGA/FLASH_SS
- U17 pad 2: /Expansion/D0 -> /FPGA/FLASH_MISO
- U17 pad 3: /Expansion/D1 -> unconnected-(U17-IO2-Pad3)
- U17 pad 4: unconnected-(U17B-GND-Pad4) -> GND
- U17 pad 5: /Expansion/D2 -> /FPGA/FLASH_MOSI
- U17 pad 6: /Expansion/D3 -> /FPGA/FLASH_SCK
- U17 pad 8: /Expansion/D4 -> +3V3
- U18 pad 10: unconnected-(U18B-GND-Pad10) -> GND
- U18 pad 11: /Expansion/D22 -> /Expansion/A25
- U18 pad 12: /Expansion/D23 -> /Expansion/A24
- U18 pad 13: /Expansion/D24 -> /Expansion/A23
- U18 pad 14: /Expansion/D25 -> /Expansion/A22
- U18 pad 15: unconnected-(U18B-GND-Pad15) -> GND
- U18 pad 16: /Expansion/D26 -> /Expansion/A21
- U18 pad 17: /Expansion/D27 -> /Expansion/A20
- U18 pad 18: unconnected-(U18B-VCCB-Pad18) -> +5V
- U18 pad 19: /Expansion/D28 -> /Expansion/A19
- U18 pad 2: /Expansion/D16 -> /Expansion/A31
- U18 pad 20: /Expansion/D29 -> /Expansion/A18
- U18 pad 21: unconnected-(U18B-GND-Pad21) -> GND
- U18 pad 22: /Expansion/D30 -> /Expansion/A17
- U18 pad 23: /Expansion/D31 -> /Expansion/A16
- U18 pad 26: /Memory/FPGA_D31 -> /FPGA/FPGA_A16
- U18 pad 27: /Memory/FPGA_D30 -> /FPGA/FPGA_A17
- U18 pad 28: unconnected-(U18B-GND-Pad28) -> GND
- U18 pad 29: /Memory/FPGA_D29 -> /FPGA/FPGA_A18
- U18 pad 3: /Expansion/D17 -> /Expansion/A30
- U18 pad 30: /Memory/FPGA_D28 -> /FPGA/FPGA_A19
- U18 pad 31: unconnected-(U18B-VCCA-Pad31) -> +3V3
- U18 pad 32: /Memory/FPGA_D27 -> /FPGA/FPGA_A20
- U18 pad 33: /Memory/FPGA_D26 -> /FPGA/FPGA_A21
- U18 pad 34: unconnected-(U18B-GND-Pad34) -> GND
- U18 pad 35: /Memory/FPGA_D25 -> /FPGA/FPGA_A22
- U18 pad 36: /Memory/FPGA_D24 -> /FPGA/FPGA_A23
- U18 pad 37: /Memory/FPGA_D23 -> /FPGA/FPGA_A24
- U18 pad 38: /Memory/FPGA_D22 -> /FPGA/FPGA_A25
- U18 pad 39: unconnected-(U18B-GND-Pad39) -> GND
- U18 pad 4: unconnected-(U18B-GND-Pad4) -> GND
- U18 pad 40: /Memory/FPGA_D21 -> /FPGA/FPGA_A26
- U18 pad 41: /Memory/FPGA_D20 -> /FPGA/FPGA_A27
- U18 pad 42: unconnected-(U18B-VCCA-Pad42) -> +3V3
- U18 pad 43: /Memory/FPGA_D19 -> /FPGA/FPGA_A28
- U18 pad 44: /Memory/FPGA_D18 -> /FPGA/FPGA_A29
- U18 pad 45: unconnected-(U18B-GND-Pad45) -> GND
- U18 pad 46: /Memory/FPGA_D17 -> /FPGA/FPGA_A30
- U18 pad 47: /Memory/FPGA_D16 -> /FPGA/FPGA_A31
- U18 pad 5: /Expansion/D18 -> /Expansion/A29
- U18 pad 6: /Expansion/D19 -> /Expansion/A28
- U18 pad 7: unconnected-(U18B-VCCB-Pad7) -> +5V
- U18 pad 8: /Expansion/D20 -> /Expansion/A27
- U18 pad 9: /Expansion/D21 -> /Expansion/A26
- U19 pad 11: /Expansion/EXD7 -> /Expansion/EXD31
- U19 pad 12: /Expansion/EXD6 -> /Expansion/EXD30
- U19 pad 13: /Expansion/EXD5 -> /Expansion/EXD29
- U19 pad 14: /Expansion/EXD4 -> /Expansion/EXD28
- U19 pad 15: /Expansion/EXD3 -> /Expansion/EXD27
- U19 pad 16: /Expansion/EXD2 -> /Expansion/EXD26
- U19 pad 17: /Expansion/EXD1 -> /Expansion/EXD25
- U19 pad 18: /Expansion/EXD0 -> /Expansion/EXD24
- U19 pad 2: /Expansion/D0 -> /Expansion/D24
- U19 pad 3: /Expansion/D1 -> /Expansion/D25
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Routing:
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- added copper zone on In1.Cu, net GND
- added copper zone on In2.Cu, net GND
Other:
- board size 221 x 243.8 mm -> 159.8 x 203.2 mm

Commit message: updates
Parts:
- added C1: C, Capacitor_SMD:C_0603_1608Metric, F.Cu at (106.2, 17.0)
- added C2: C, Capacitor_SMD:C_0603_1608Metric, F.Cu at (106.2, 19.5)
- added J13: DIN-5_180degree, 68040:DIN5-180, F.Cu at (107.4, -24.4)
- added J14: Mini-DIN-6, 68040:Mini-DIN6, F.Cu at (94.7, -1.07)
- added J15: COM1, Connector_PinHeader_2.54mm:PinHeader_2x05_P2.54mm_Vertical, F.Cu at (92.2, 6.40)
- added J16: COM2, Connector_PinHeader_2.54mm:PinHeader_2x05_P2.54mm_Vertical, F.Cu at (99.3, 6.40)
- added J17: LPT, Connector_PinHeader_2.54mm:PinHeader_2x13_P2.54mm_Vertical, F.Cu at (85.0, -29.1)
- added U20: 68681, Package_DIP:DIP-40_W15.24mm, F.Cu at (65.8, -29.4)
- added U21: ATmega8-16A, Package_QFP:TQFP-32_7x7mm_P0.8mm, F.Cu at (110.0, 9.90)
- added U22: IS61C5128AS-25TLI, Package_SO:TSOP-II-32_21.0x10.2mm_P1.27mm, F.Cu at (71.5, 34.0)
- added U25: IS61C5128AS-25TLI, Package_SO:TSOP-II-32_21.0x10.2mm_P1.27mm, F.Cu at (85.9, 34.0)
- added U26: iCE40HX8K-CT256(256-Ball_caBGA), 68040:256-Ball_caBGA(Pitch_0.80mm_Pad_0.40mm), F.Cu at (330.2, 101.6)
Connections:
- net /GND_{L} renamed /Processor/GND_{L}
- net /GND_{O} renamed /Processor/GND_{O}
- net /GND_{P} renamed /Processor/GND_{P}
- net /JS0 renamed /Processor/JS0
- net /PST0 renamed /Processor/PST0
- net /PST1 renamed /Processor/PST1
- net /PST2 renamed /Processor/PST2
- net /PST3 renamed /Processor/PST3
- net /SC0 renamed /Processor/SC0
- net /SC1 renamed /Processor/SC1
- net /SIZ0 renamed /Processor/SIZ0
- net /SIZ1 renamed /Processor/SIZ1
- net /TCK renamed /Processor/TCK
- net /TDI renamed /Processor/TDI
- net /TDO renamed /Processor/TDO
- net /TLN0 renamed /Processor/TLN0
- net /TLN1 renamed /Processor/TLN1
- net /TM0 renamed /Processor/TM0
- net /TM1 renamed /Processor/TM1
- net /TM2 renamed /Processor/TM2
- net /TMS renamed /Processor/TMS
- net /TT0 renamed /Processor/TT0
- net /TT1 renamed /Processor/TT1
- net /UPA0 renamed /Processor/UPA0
- net /UPA1 renamed /Processor/UPA1
- net /V_{CC}_{L} renamed /Processor/V_{CC}_{L}
- net /V_{CC}_{O} renamed /Processor/V_{CC}_{O}
- net /V_{CC}_{P} renamed /Processor/V_{CC}_{P}
- net /~{AVEC} renamed /Processor/~{AVEC}
- net /~{BB} renamed /Processor/~{BB}
- net /~{BG} renamed /Processor/~{BG}
- net /~{BR} renamed /Processor/~{BR}
- net /~{CDIS} renamed /Processor/~{CDIS}
- net /~{CIOUT} renamed /Processor/~{CIOUT}
- net /~{IPEND} renamed /Processor/~{IPEND}
- net /~{IPL0} renamed /Processor/~{IPL0}
- net /~{IPL1} renamed /Processor/~{IPL1}
- net /~{IPL2} renamed /Processor/~{IPL2}
- net /~{LOCKE} renamed /Processor/~{LOCKE}
- net /~{LOCK} renamed /Processor/~{LOCK}
- net /~{MDIS} renamed /Processor/~{MDIS}
- net /~{MI} renamed /Processor/~{MI}
- net /~{RSTI} renamed /Processor/~{RSTI}
- net /~{RSTO} renamed /Processor/~{RSTO}
- net /~{TIP} renamed /Processor/~{TIP}
- net /~{TSRT} renamed /Processor/~{TSRT}
- net /~{TS} renamed /Processor/~{TS}
- U1 pad A1: /Expansion/A31 -> /Processor/A31
- U1 pad A10: /D12 -> /Processor/D12
- U1 pad A11: /D13 -> /Processor/D13
- U1 pad A12: /D14 -> /Processor/D14
- U1 pad A13: /D15 -> /Processor/D15
- U1 pad A14: /D17 -> /Processor/D17
- U1 pad A15: /D19 -> /Processor/D19
- U1 pad A16: /D20 -> /Processor/D20
- U1 pad A17: /D21 -> /Processor/D21
- U1 pad A18: /D24 -> /Processor/D24
- U1 pad A2: /D3 -> /Processor/D3
- U1 pad A3: /D4 -> /Processor/D4
- U1 pad A4: /D5 -> /Processor/D5
- U1 pad A5: /D6 -> /Processor/D6
- U1 pad A6: /D7 -> /Processor/D7
- U1 pad A7: /D9 -> /Processor/D9
- U1 pad A8: /D10 -> /Processor/D10
- U1 pad A9: /D11 -> /Processor/D11
- U1 pad B1: /Expansion/A29 -> /Processor/A29
- U1 pad B11: /D16 -> /Processor/D16
- U1 pad B12: /D18 -> /Processor/D18
- U1 pad B16: /D22 -> /Processor/D22
- U1 pad B18: /D26 -> /Processor/D26
- U1 pad B3: /D1 -> /Processor/D1
- U1 pad B7: /D8 -> /Processor/D8
- U1 pad C1: /Expansion/A27 -> /Processor/A27
- U1 pad C15: /D23 -> /Processor/D23
- U1 pad C16: /D25 -> /Processor/D25
- U1 pad C18: /D28 -> /Processor/D28
- U1 pad C3: /D0 -> /Processor/D0
- U1 pad C4: /D2 -> /Processor/D2
- U1 pad D1: /Expansion/A24 -> /Processor/A24
- U1 pad D16: /D27 -> /Processor/D27
- U1 pad D18: /D31 -> /Processor/D31
- U1 pad D3: /Expansion/A30 -> /Processor/A30
- U1 pad E1: /Expansion/A22 -> /Processor/A22
- U1 pad E16: /D29 -> /Processor/D29
- U1 pad E17: /D30 -> /Processor/D30
- U1 pad E18: /Expansion/A8 -> /Processor/A8
- U1 pad E2: /Expansion/A26 -> /Processor/A26
- U1 pad E3: /Expansion/A28 -> /Processor/A28
- U1 pad F1: /Expansion/A21 -> /Processor/A21
- U1 pad F16: /Expansion/A9 -> /Processor/A9
- U1 pad F18: /Expansion/A7 -> /Processor/A7
- U1 pad F3: /Expansion/A25 -> /Processor/A25
- U1 pad G1: /Expansion/A20 -> /Processor/A20
- U1 pad G16: /Expansion/A6 -> /Processor/A6
- U1 pad G18: /Expansion/A5 -> /Processor/A5
- U1 pad G3: /Expansion/A23 -> /Processor/A23
- U1 pad H1: /Expansion/A18 -> /Processor/A18
- U1 pad H18: /Expansion/A4 -> /Processor/A4
- U1 pad J1: /Expansion/A17 -> /Processor/A17
- U1 pad J17: /Expansion/A2 -> /Processor/A2
- U1 pad J18: /Expansion/A3 -> /Processor/A3
- U1 pad J2: /Expansion/A19 -> /Processor/A19
- U1 pad K1: /Expansion/A15 -> /Processor/A15
- U1 pad K18: /Expansion/A1 -> /Processor/A1
- U1 pad K2: /Expansion/A16 -> /Processor/A16
- U1 pad L1: /Expansion/A14 -> /Processor/A14
- U1 pad L18: /Expansion/A0 -> /Processor/A0
- U1 pad M1: /Expansion/A13 -> /Processor/A13
- U1 pad N1: /Expansion/A12 -> /Processor/A12
- U1 pad N16: /R/~{W} -> /Processor/R/~{W}
- U1 pad N3: /Expansion/A11 -> /Processor/A11
- U1 pad P1: /Expansion/A10 -> /Processor/A10
- U1 pad R7: /BCLK -> /Processor/BCLK
- U1 pad R9: /PCLK -> /Processor/PCLK
- U15 pad 11: /Expansion/D22 -> /FPGA/D22
- U15 pad 12: /Expansion/D23 -> /FPGA/D23
- U15 pad 13: /Expansion/D24 -> /FPGA/D24
- U15 pad 14: /Expansion/D25 -> /FPGA/D25
- U15 pad 16: /Expansion/D26 -> /FPGA/D26
- U15 pad 17: /Expansion/D27 -> /FPGA/D27
- U15 pad 19: /Expansion/D28 -> /FPGA/D28
- U15 pad 2: /Expansion/D16 -> /FPGA/D16
- U15 pad 20: /Expansion/D29 -> /FPGA/D29
- U15 pad 22: /Expansion/D30 -> /FPGA/D30
- U15 pad 23: /Expansion/D31 -> /FPGA/D31
- U15 pad 3: /Expansion/D17 -> /FPGA/D17
- U15 pad 5: /Expansion/D18 -> /FPGA/D18
- U15 pad 6: /Expansion/D19 -> /FPGA/D19
- U15 pad 8: /Expansion/D20 -> /FPGA/D20
- U15 pad 9: /Expansion/D21 -> /FPGA/D21
- U16 pad 11: /Expansion/A6 -> /FPGA/A6
- U16 pad 12: /Expansion/A7 -> /FPGA/A7
- U16 pad 13: /Expansion/A8 -> /FPGA/A8
- U16 pad 14: /Expansion/A9 -> /FPGA/A9
- U16 pad 16: /Expansion/A10 -> /FPGA/A10
- U16 pad 17: /Expansion/A11 -> /FPGA/A11
- U16 pad 19: /Expansion/A12 -> /FPGA/A12
- U16 pad 2: /Expansion/A0 -> /FPGA/A0
- U16 pad 20: /Expansion/A13 -> /FPGA/A13
- U16 pad 22: /Expansion/A14 -> /FPGA/A14
- U16 pad 23: /Expansion/A15 -> /FPGA/A15
- U16 pad 3: /Expansion/A1 -> /FPGA/A1
- U16 pad 5: /Expansion/A2 -> /FPGA/A2
- U16 pad 6: /Expansion/A3 -> /FPGA/A3
- U16 pad 8: /Expansion/A4 -> /FPGA/A4
- U16 pad 9: /Expansion/A5 -> /FPGA/A5
- U18 pad 11: /Expansion/A25 -> /FPGA/A25
- U18 pad 12: /Expansion/A24 -> /FPGA/A24
- U18 pad 13: /Expansion/A23 -> /FPGA/A23
- U18 pad 14: /Expansion/A22 -> /FPGA/A22
- U18 pad 16: /Expansion/A21 -> /FPGA/A21
- U18 pad 17: /Expansion/A20 -> /FPGA/A20
- U18 pad 19: /Expansion/A19 -> /FPGA/A19
- U18 pad 2: /Expansion/A31 -> /FPGA/A31
- U18 pad 20: /Expansion/A18 -> /FPGA/A18
- U18 pad 22: /Expansion/A17 -> /FPGA/A17
- U18 pad 23: /Expansion/A16 -> /FPGA/A16
- U18 pad 3: /Expansion/A30 -> /FPGA/A30
- U18 pad 5: /Expansion/A29 -> /FPGA/A29
- U18 pad 6: /Expansion/A28 -> /FPGA/A28
- U18 pad 8: /Expansion/A27 -> /FPGA/A27
- U18 pad 9: /Expansion/A26 -> /FPGA/A26
- U2 pad 11: /Expansion/D6 -> /FPGA/D6
- U2 pad 12: /Expansion/D7 -> /FPGA/D7
- U2 pad 13: /Expansion/D8 -> /FPGA/D8
- U2 pad 14: /Expansion/D9 -> /FPGA/D9
- U2 pad 16: /Expansion/D10 -> /FPGA/D10
- U2 pad 17: /Expansion/D11 -> /FPGA/D11
- U2 pad 19: /Expansion/D12 -> /FPGA/D12
- U2 pad 2: /Expansion/D0 -> /FPGA/D0
- U2 pad 20: /Expansion/D13 -> /FPGA/D13
- U2 pad 22: /Expansion/D14 -> /FPGA/D14
- U2 pad 23: /Expansion/D15 -> /FPGA/D15
- U2 pad 3: /Expansion/D1 -> /FPGA/D1
- U2 pad 5: /Expansion/D2 -> /FPGA/D2
- U2 pad 6: /Expansion/D3 -> /FPGA/D3
- U2 pad 8: /Expansion/D4 -> /FPGA/D4
- U2 pad 9: /Expansion/D5 -> /FPGA/D5
- U24 pad 19: /Expansion/A1 -> /A1
- U24 pad 20: /Expansion/A0 -> /A0
- U3 pad 11: /Expansion/D11 -> /Memory/D11
- U3 pad 12: /Expansion/D27 -> /Memory/D27
- U3 pad 13: /Expansion/D12 -> /Memory/D12
- U3 pad 14: /Expansion/D28 -> /Memory/D28
- U3 pad 16: /Expansion/D29 -> /Memory/D29
- U3 pad 17: /Expansion/D13 -> /Memory/D13
- U3 pad 19: /Expansion/D30 -> /Memory/D30
- U3 pad 2: /Expansion/D8 -> /Memory/D8
- U3 pad 20: /Expansion/D14 -> /Memory/D14
- U3 pad 22: /Expansion/D31 -> /Memory/D31
- U3 pad 23: /Expansion/D15 -> /Memory/D15
- U3 pad 3: /Expansion/D24 -> /Memory/D24
- U3 pad 5: /Expansion/D9 -> /Memory/D9
- U3 pad 6: /Expansion/D25 -> /Memory/D25
- U3 pad 8: /Expansion/D10 -> /Memory/D10
- U3 pad 9: /Expansion/D26 -> /Memory/D26
- U4 pad 11: /Expansion/D3 -> /Memory/D3
- U4 pad 12: /Expansion/D19 -> /Memory/D19
- U4 pad 13: /Expansion/D4 -> /Memory/D4
- U4 pad 14: /Expansion/D20 -> /Memory/D20
- U4 pad 16: /Expansion/D5 -> /Memory/D5
- U4 pad 17: /Expansion/D21 -> /Memory/D21
- U4 pad 19: /Expansion/D6 -> /Memory/D6
- U4 pad 2: /Expansion/D0 -> /Memory/D0
- U4 pad 20: /Expansion/D22 -> /Memory/D22
- U4 pad 22: /Expansion/D7 -> /Memory/D7
- U4 pad 23: /Expansion/D23 -> /Memory/D23
- U4 pad 3: /Expansion/D16 -> /Memory/D16
- U4 pad 5: /Expansion/D1 -> /Memory/D1
- U4 pad 6: /Expansion/D17 -> /Memory/D17
- U4 pad 8: /Expansion/D2 -> /Memory/D2
- U4 pad 9: /Expansion/D18 -> /Memory/D18
- U5 pad 37: /FPGA/DRAM_A0 -> /FPGA/DRAM_A9
- U5 pad 38: /FPGA/DRAM_A1 -> /FPGA/DRAM_A8
- U5 pad 39: /FPGA/DRAM_A2 -> /FPGA/DRAM_A11
- U5 pad 41: /FPGA/DRAM_A3 -> /FPGA/DRAM_A7
- U5 pad 42: /FPGA/DRAM_A4 -> /FPGA/DRAM_A10
- U5 pad 43: /FPGA/DRAM_A5 -> /FPGA/DRAM_A6
- U5 pad 44: /FPGA/DRAM_A6 -> /FPGA/DRAM_A5
- U5 pad 45: /FPGA/DRAM_A10 -> /FPGA/DRAM_A4
- U5 pad 47: /FPGA/DRAM_A7 -> /FPGA/DRAM_A3
- U5 pad 48: /FPGA/DRAM_A11 -> /FPGA/DRAM_A2
- U5 pad 49: /FPGA/DRAM_A8 -> /FPGA/DRAM_A1
- U5 pad 52: /FPGA/DRAM_A9 -> /FPGA/DRAM_A0
Routing:
- net GND: track 1.91 -> 21.6 mm, vias 0 -> 16
- net unconnected-(U26C-CBSEL1/IOB_104/PIO2_45-PadP13): track 0.00 -> 4.57 mm
- net unconnected-(U26A-IOT_221/PIO0_45-PadC5): track 0.00 -> 4.29 mm
- net unconnected-(U26D-IOL_19B/PIO3_37-PadL3): track 0.00 -> 3.97 mm
- net unconnected-(U26B-IOR_142/PIO1_29-PadH14): track 0.00 -> 3.77 mm
- net unconnected-(U26B-IOR_134/PIO1_22-PadJ14): track 0.00 -> 3.77 mm
- net unconnected-(U26A-IOT_209/PIO0_34-PadC6): track 0.00 -> 3.77 mm
- net unconnected-(U26A-IOT_171/PIO0_03-PadB14): track 0.00 -> 3.77 mm
- net unconnected-(U26A-IOT_168/PIO0_00-PadC14): track 0.00 -> 3.77 mm
- net unconnected-(U26B-IOR_119/PIO1_10-PadL14): track 0.00 -> 3.77 mm
- net unconnected-(U26A-IOT_218/PIO0_42-PadA2): track 0.00 -> 3.33 mm
- net unconnected-(U26D-IOL_26A/PIO3_50-PadR1): track 0.00 -> 3.17 mm
- net unconnected-(U26C-IOB_71/PIO2_16-PadR6): track 0.00 -> 3.17 mm
- net unconnected-(U26C-IOB_55/PIO2_03-PadR2): track 0.00 -> 3.17 mm
- net unconnected-(U26C-IOB_102/PIO2_43-PadR16): track 0.00 -> 3.17 mm
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- added copper zone on In2.Cu, net +3.3V
Other:
- board size 159.8 x 203.2 mm -> 284.2 x 203.2 mm

Commit message: add interrupt logic, clean up modules
Parts:
- removed C1, C2: C, Capacitor_SMD:C_0603_1608Metric
- removed C4: .1uF, Capacitor_SMD:C_0603_1608Metric
- removed R4: 10k, Resistor_SMD:R_0603_1608Metric
- removed R5: 10k, Capacitor_SMD:C_0603_1608Metric
- removed RN1: R_Network04_US, Resistor_THT:R_Array_SIP5
- removed RN2: 10k, Resistor_THT:R_Array_SIP5
- removed U10, U11, U12, U13, U14, U19, U6, U7: 74HC245, Package_SO:SOIC-20W_7.5x12.8mm_P1.27mm
- removed U15, U16, U18: SN74ALVC164245, Package_SO:TSSOP-48_6.1x12.5mm_P0.5mm
- removed U17: W25Q32JVSSIM, Package_SO:SOIC-8_5.23x5.23mm_P1.27mm
- removed U20: 68681, Package_DIP:DIP-40_W15.24mm
- removed U21: ATmega8-16A, Package_QFP:TQFP-32_7x7mm_P0.8mm
- removed U22, U25: IS61C5128AS-25TLI, Package_SO:TSOP-II-32_21.0x10.2mm_P1.27mm
- removed U23: PCF8584, Package_SO:SOIC-20W_7.5x12.8mm_P1.27mm
- removed U24: ~, Package_LCC:PLCC-68_SMD-Socket
- removed U26: iCE40HX8K-CT256(256-Ball_caBGA), 68040:256-Ball_caBGA(Pitch_0.80mm_Pad_0.40mm)
- removed U8: LTC6905xS5-133, Package_TO_SOT_SMD:TSOT-23-5
- removed U9: 74LS32, Package_SO:SOIC-14_3.9x8.7mm_P1.27mm
- added J1: EXP, 68040:EXP, F.Cu at (78.1, 189.0)
- added J10: ~, 68040:SIMM-72, F.Cu at (247.7, 119.4)
- added J11: ~, 68040:SIMM-72, F.Cu at (259.1, 119.4)
- added J12: ~, 68040:SIMM-72, F.Cu at (270.5, 119.4)
- added J2: EXP, 68040:EXP, F.Cu at (98.4, 189.0)
- added J5: EXP, 68040:EXP, F.Cu at (118.8, 189.0)
- added J8: EXP, 68040:EXP, F.Cu at (220.4, 189.0)
- U2: value SN74ALVC164245 -> ICE40HX4K-TQ144; footprint Package_SO:TSSOP-48_6.1x12.5mm_P0.5mm -> Package_QFP:TQFP-144_20x20mm_P0.5mm
- U5: value ICE40HX4K-TQ144 -> W25Q32JVSSIM; footprint Package_QFP:TQFP-144_20x20mm_P0.5mm -> Package_SO:SOIC-8_5.23x5.23mm_P1.27mm
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- renumbered J2 to J4, J1 to J6, J4 to J7
Connections:
- net /Power/PWR_GOOD renamed /PWR_GD
- net /Processor/GND_{L} renamed /GND_{L}
- net /Processor/GND_{O} renamed /GND_{O}
- net /Processor/GND_{P} renamed /GND_{P}
- net /Processor/JS0 renamed /JS0
- net /Processor/PST0 renamed /PST0
- net /Processor/PST1 renamed /PST1
- net /Processor/PST2 renamed /PST2
- net /Processor/PST3 renamed /PST3
- net /Processor/SC0 renamed /SC0
- net /Processor/SC1 renamed /SC1
- net /Processor/TCK renamed /TCK
- net /Processor/TDI renamed /TDI
- net /Processor/TDO renamed /TDO
- net /Processor/TLN0 renamed /TLN0
- net /Processor/TLN1 renamed /TLN1
- net /Processor/TM0 renamed /TM0
- net /Processor/TM1 renamed /TM1
- net /Processor/TM2 renamed /TM2
- net /Processor/TMS renamed /TMS
- net /Processor/TT0 renamed /TT0
- net /Processor/TT1 renamed /TT1
- net /Processor/UPA0 renamed /UPA0
- net /Processor/UPA1 renamed /UPA1
- net /Processor/V_{CC}_{L} renamed /V_{CC}_{L}
- net /Processor/V_{CC}_{O} renamed /V_{CC}_{O}
- net /Processor/V_{CC}_{P} renamed /V_{CC}_{P}
- net /Processor/~{AVEC} renamed /~{AVEC}
- net /Processor/~{BB} renamed /~{BB}
- net /Processor/~{BG} renamed /~{BG}
- net /Processor/~{BR} renamed /~{BR}
- net /Processor/~{CDIS} renamed /~{CDIS}
- net /Processor/~{CIOUT} renamed /~{CIOUT}
- net /Processor/~{IPEND} renamed /~{IPEND}
- net /Processor/~{IPL0} renamed /~{IPL0}
- net /Processor/~{IPL1} renamed /~{IPL1}
- net /Processor/~{IPL2} renamed /~{IPL2}
- net /Processor/~{LOCKE} renamed /~{LOCKE}
- net /Processor/~{LOCK} renamed /~{LOCK}
- net /Processor/~{MDIS} renamed /~{MDIS}
- net /Processor/~{MI} renamed /~{MI}
- net /Processor/~{RSTI} renamed /~{RSTI}
- net /Processor/~{RSTO} renamed /~{RSTO}
- net /Processor/~{TIP} renamed /~{TIP}
- net /Processor/~{TSRT} renamed /~{TSRT}
- net /Processor/~{TS} renamed /~{TS}
- D1 pad 2: /FPGA/CDONE -> /Memory/CDONE
- J3 pad A1: GND -> unconnected-(J3-PadA1)
- J3 pad A10: /Expansion/EXD14 -> /Expansion/D14
- J3 pad A11: GND -> unconnected-(J3-PadA11)
- J3 pad A12: /Expansion/EXA1 -> /Expansion/A1
- J3 pad A13: /Expansion/EXA3 -> /Expansion/A3
- J3 pad A14: /Expansion/EXA5 -> /Expansion/A5
- J3 pad A15: /Expansion/EXA7 -> /Expansion/A7
- J3 pad A16: /Expansion/EXA9 -> /Expansion/A9
- J3 pad A17: /Expansion/EXA11 -> /Expansion/A11
- J3 pad A18: /Expansion/EXA13 -> /Expansion/A13
- J3 pad A19: /Expansion/EXA15 -> /Expansion/A15
- J3 pad A2: /Expansion/ExpansionSlot2/~{CFG_{IN}} -> unconnected-(J3-PadA2)
- J3 pad A20: /Expansion/EXA17 -> /Expansion/A17
- J3 pad A21: /Expansion/EXA19 -> /Expansion/A19
- J3 pad A24: +5V -> unconnected-(J3-PadA24)
- J3 pad A3: /Expansion/EXD0 -> /Expansion/D0
- J3 pad A31: +12V -> unconnected-(J3-PadA31)
- J3 pad A32: GND -> unconnected-(J3-PadA32)
- J3 pad A4: /Expansion/EXD2 -> /Expansion/D2
- J3 pad A5: /Expansion/EXD4 -> /Expansion/D4
- J3 pad A6: /Expansion/EXD6 -> /Expansion/D6
- J3 pad A7: /Expansion/EXD8 -> /Expansion/D8
- J3 pad A8: /Expansion/EXD10 -> /Expansion/D10
- J3 pad A9: /Expansion/EXD12 -> /Expansion/D12
- J3 pad B1: /Expansion/EXD16 -> /Expansion/D16
- J3 pad B10: /Expansion/EXD25 -> /Expansion/D25
- J3 pad B11: /Expansion/EXD26 -> /Expansion/D26
- J3 pad B12: /Expansion/EXD27 -> /Expansion/D27
- J3 pad B13: /Expansion/EXD28 -> /Expansion/D28
- J3 pad B14: /Expansion/EXD29 -> /Expansion/D29
- J3 pad B15: /Expansion/EXD30 -> /Expansion/D30
- J3 pad B16: /Expansion/EXD31 -> /Expansion/D31
- J3 pad B17: /Expansion/EXA0 -> /Expansion/A0
- J3 pad B18: /Expansion/EXA20 -> /Expansion/A20
- J3 pad B19: /Expansion/EXA21 -> /Expansion/A21
- J3 pad B2: /Expansion/EXD17 -> /Expansion/D17
- J3 pad B20: /Expansion/EXA22 -> /Expansion/A22
- J3 pad B21: /Expansion/EXA23 -> /Expansion/A23
- J3 pad B22: /Expansion/EXA24 -> /Expansion/A24
- J3 pad B23: /Expansion/EXA25 -> /Expansion/A25
- J3 pad B24: /Expansion/EXA26 -> /Expansion/A26
- J3 pad B25: /Expansion/EXA27 -> /Expansion/A27
- J3 pad B26: /Expansion/EXA28 -> /Expansion/A28
- J3 pad B27: /Expansion/EXA29 -> /Expansion/A29
- J3 pad B28: /Expansion/EXA30 -> /Expansion/A30
- J3 pad B29: /Expansion/EXA31 -> /Expansion/A31
- J3 pad B3: /Expansion/EXD18 -> /Expansion/D18
- J3 pad B31: /Expansion/ExpansionSlot2/BCLK -> unconnected-(J3-PadB31)
- J3 pad B32: GND -> unconnected-(J3-PadB32)
- J3 pad B4: /Expansion/EXD19 -> /Expansion/D19
- J3 pad B5: /Expansion/EXD20 -> /Expansion/D20
- J3 pad B6: /Expansion/EXD21 -> /Expansion/D21
- J3 pad B7: /Expansion/EXD22 -> /Expansion/D22
- J3 pad B8: /Expansion/EXD23 -> /Expansion/D23
- J3 pad B9: /Expansion/EXD24 -> /Expansion/D24
- J3 pad C1: +5V -> unconnected-(J3-PadC1)
- J3 pad C10: /Expansion/EXD15 -> /Expansion/D15
- J3 pad C11: GND -> unconnected-(J3-PadC11)
- J3 pad C12: /Expansion/EXA2 -> /Expansion/A2
- J3 pad C13: /Expansion/EXA4 -> /Expansion/A4
- J3 pad C14: /Expansion/EXA6 -> /Expansion/A6
- J3 pad C15: /Expansion/EXA8 -> /Expansion/A8
- J3 pad C16: /Expansion/EXA10 -> /Expansion/A10
- J3 pad C17: /Expansion/EXA12 -> /Expansion/A12
- J3 pad C18: /Expansion/EXA14 -> /Expansion/A14
- J3 pad C19: /Expansion/EXA16 -> /Expansion/A16
- J3 pad C2: /Expansion/ExpansionSlot2/~{CFG_{OUT}} -> unconnected-(J3-PadC2)
- J3 pad C20: /Expansion/EXA18 -> /Expansion/A18
- J3 pad C24: GND -> unconnected-(J3-PadC24)
- J3 pad C3: /Expansion/EXD1 -> /Expansion/D1
- J3 pad C30: +3V3 -> unconnected-(J3-PadC30)
- J3 pad C31: +12V -> unconnected-(J3-PadC31)
- J3 pad C32: GND -> unconnected-(J3-PadC32)
- J3 pad C4: /Expansion/EXD3 -> /Expansion/D3
- J3 pad C5: /Expansion/EXD5 -> /Expansion/D5
- J3 pad C6: /Expansion/EXD7 -> /Expansion/D7
- J3 pad C7: /Expansion/EXD9 -> /Expansion/D9
- J3 pad C8: /Expansion/EXD11 -> /Expansion/D11
- J3 pad C9: /Expansion/EXD13 -> /Expansion/D13
- J4 pad A1: GND -> unconnected-(J4-PadA1)
- J4 pad A10: /Expansion/EXD14 -> /Expansion/D14
- J4 pad A11: GND -> unconnected-(J4-PadA11)
- J4 pad A12: /Expansion/EXA1 -> /Expansion/A1
- J4 pad A13: /Expansion/EXA3 -> /Expansion/A3
- J4 pad A14: /Expansion/EXA5 -> /Expansion/A5
- J4 pad A15: /Expansion/EXA7 -> /Expansion/A7
- J4 pad A16: /Expansion/EXA9 -> /Expansion/A9
- J4 pad A17: /Expansion/EXA11 -> /Expansion/A11
- J4 pad A18: /Expansion/EXA13 -> /Expansion/A13
- J4 pad A19: /Expansion/EXA15 -> /Expansion/A15
- J4 pad A2: /Expansion/ExpansionSlot1/~{CFG_{IN}} -> unconnected-(J4-PadA2)
- J4 pad A20: /Expansion/EXA17 -> /Expansion/A17
- J4 pad A21: /Expansion/EXA19 -> /Expansion/A19
- J4 pad A24: +5V -> unconnected-(J4-PadA24)
- J4 pad A3: /Expansion/EXD0 -> /Expansion/D0
- J4 pad A31: +12V -> unconnected-(J4-PadA31)
- J4 pad A32: GND -> unconnected-(J4-PadA32)
- J4 pad A4: /Expansion/EXD2 -> /Expansion/D2
- J4 pad A5: /Expansion/EXD4 -> /Expansion/D4
- J4 pad A6: /Expansion/EXD6 -> /Expansion/D6
- J4 pad A7: /Expansion/EXD8 -> /Expansion/D8
- J4 pad A8: /Expansion/EXD10 -> /Expansion/D10
- J4 pad A9: /Expansion/EXD12 -> /Expansion/D12
- J4 pad B1: /Expansion/EXD16 -> /Expansion/D16
- J4 pad B10: /Expansion/EXD25 -> /Expansion/D25
- J4 pad B11: /Expansion/EXD26 -> /Expansion/D26
- J4 pad B12: /Expansion/EXD27 -> /Expansion/D27
- J4 pad B13: /Expansion/EXD28 -> /Expansion/D28
- J4 pad B14: /Expansion/EXD29 -> /Expansion/D29
- J4 pad B15: /Expansion/EXD30 -> /Expansion/D30
- J4 pad B16: /Expansion/EXD31 -> /Expansion/D31
- J4 pad B17: /Expansion/EXA0 -> /Expansion/A0
- J4 pad B18: /Expansion/EXA20 -> /Expansion/A20
- J4 pad B19: /Expansion/EXA21 -> /Expansion/A21
- J4 pad B2: /Expansion/EXD17 -> /Expansion/D17
- J4 pad B20: /Expansion/EXA22 -> /Expansion/A22
- J4 pad B21: /Expansion/EXA23 -> /Expansion/A23
- J4 pad B22: /Expansion/EXA24 -> /Expansion/A24
- J4 pad B23: /Expansion/EXA25 -> /Expansion/A25
- J4 pad B24: /Expansion/EXA26 -> /Expansion/A26
- J4 pad B25: /Expansion/EXA27 -> /Expansion/A27
- J4 pad B26: /Expansion/EXA28 -> /Expansion/A28
- J4 pad B27: /Expansion/EXA29 -> /Expansion/A29
- J4 pad B28: /Expansion/EXA30 -> /Expansion/A30
- J4 pad B29: /Expansion/EXA31 -> /Expansion/A31
- J4 pad B3: /Expansion/EXD18 -> /Expansion/D18
- J4 pad B31: /Expansion/ExpansionSlot1/BCLK -> unconnected-(J4-PadB31)
- J4 pad B32: GND -> unconnected-(J4-PadB32)
- J4 pad B4: /Expansion/EXD19 -> /Expansion/D19
- J4 pad B5: /Expansion/EXD20 -> /Expansion/D20
- J4 pad B6: /Expansion/EXD21 -> /Expansion/D21
- J4 pad B7: /Expansion/EXD22 -> /Expansion/D22
- J4 pad B8: /Expansion/EXD23 -> /Expansion/D23
- J4 pad B9: /Expansion/EXD24 -> /Expansion/D24
- J4 pad C1: +5V -> unconnected-(J4-PadC1)
- J4 pad C10: /Expansion/EXD15 -> /Expansion/D15
- J4 pad C11: GND -> unconnected-(J4-PadC11)
- J4 pad C12: /Expansion/EXA2 -> /Expansion/A2
- J4 pad C13: /Expansion/EXA4 -> /Expansion/A4
- J4 pad C14: /Expansion/EXA6 -> /Expansion/A6
- J4 pad C15: /Expansion/EXA8 -> /Expansion/A8
- J4 pad C16: /Expansion/EXA10 -> /Expansion/A10
- J4 pad C17: /Expansion/EXA12 -> /Expansion/A12
- J4 pad C18: /Expansion/EXA14 -> /Expansion/A14
- J4 pad C19: /Expansion/EXA16 -> /Expansion/A16
- J4 pad C2: /Expansion/ExpansionSlot1/~{CFG_{OUT}} -> unconnected-(J4-PadC2)
- J4 pad C20: /Expansion/EXA18 -> /Expansion/A18
- J4 pad C24: GND -> unconnected-(J4-PadC24)
- J4 pad C3: /Expansion/EXD1 -> /Expansion/D1
- J4 pad C30: +3V3 -> unconnected-(J4-PadC30)
- J4 pad C31: +12V -> unconnected-(J4-PadC31)
- J4 pad C32: GND -> unconnected-(J4-PadC32)
- J4 pad C4: /Expansion/EXD3 -> /Expansion/D3
- J4 pad C5: /Expansion/EXD5 -> /Expansion/D5
- J4 pad C6: /Expansion/EXD7 -> /Expansion/D7
- J4 pad C7: /Expansion/EXD9 -> /Expansion/D9
- J4 pad C8: /Expansion/EXD11 -> /Expansion/D11
- J4 pad C9: /Expansion/EXD13 -> /Expansion/D13
- J6 pad A1: GND -> unconnected-(J6-PadA1)
- J6 pad A10: /Expansion/EXD14 -> /Expansion/D14
- J6 pad A11: GND -> unconnected-(J6-PadA11)
- J6 pad A12: /Expansion/EXA1 -> /Expansion/A1
- J6 pad A13: /Expansion/EXA3 -> /Expansion/A3
- J6 pad A14: /Expansion/EXA5 -> /Expansion/A5
- J6 pad A15: /Expansion/EXA7 -> /Expansion/A7
- J6 pad A16: /Expansion/EXA9 -> /Expansion/A9
- J6 pad A17: /Expansion/EXA11 -> /Expansion/A11
- J6 pad A18: /Expansion/EXA13 -> /Expansion/A13
- J6 pad A19: /Expansion/EXA15 -> /Expansion/A15
- J6 pad A2: /Expansion/ExpansionSlot4/~{CFG_{IN}} -> unconnected-(J6-PadA2)
- J6 pad A20: /Expansion/EXA17 -> /Expansion/A17
- J6 pad A21: /Expansion/EXA19 -> /Expansion/A19
- J6 pad A24: +5V -> unconnected-(J6-PadA24)
- J6 pad A3: /Expansion/EXD0 -> /Expansion/D0
- J6 pad A31: +12V -> unconnected-(J6-PadA31)
- J6 pad A32: GND -> unconnected-(J6-PadA32)
- J6 pad A4: /Expansion/EXD2 -> /Expansion/D2
- J6 pad A5: /Expansion/EXD4 -> /Expansion/D4
- J6 pad A6: /Expansion/EXD6 -> /Expansion/D6
- J6 pad A7: /Expansion/EXD8 -> /Expansion/D8
- J6 pad A8: /Expansion/EXD10 -> /Expansion/D10
- J6 pad A9: /Expansion/EXD12 -> /Expansion/D12
- J6 pad B1: /Expansion/EXD16 -> /Expansion/D16
- J6 pad B10: /Expansion/EXD25 -> /Expansion/D25
- J6 pad B11: /Expansion/EXD26 -> /Expansion/D26
- J6 pad B12: /Expansion/EXD27 -> /Expansion/D27
- J6 pad B13: /Expansion/EXD28 -> /Expansion/D28
- J6 pad B14: /Expansion/EXD29 -> /Expansion/D29
- J6 pad B15: /Expansion/EXD30 -> /Expansion/D30
- J6 pad B16: /Expansion/EXD31 -> /Expansion/D31
- J6 pad B17: /Expansion/EXA0 -> /Expansion/A0
- J6 pad B18: /Expansion/EXA20 -> /Expansion/A20
- J6 pad B19: /Expansion/EXA21 -> /Expansion/A21
- J6 pad B2: /Expansion/EXD17 -> /Expansion/D17
- J6 pad B20: /Expansion/EXA22 -> /Expansion/A22
- J6 pad B21: /Expansion/EXA23 -> /Expansion/A23
- J6 pad B22: /Expansion/EXA24 -> /Expansion/A24
- J6 pad B23: /Expansion/EXA25 -> /Expansion/A25
- J6 pad B24: /Expansion/EXA26 -> /Expansion/A26
- J6 pad B25: /Expansion/EXA27 -> /Expansion/A27
- J6 pad B26: /Expansion/EXA28 -> /Expansion/A28
- J6 pad B27: /Expansion/EXA29 -> /Expansion/A29
- J6 pad B28: /Expansion/EXA30 -> /Expansion/A30
- J6 pad B29: /Expansion/EXA31 -> /Expansion/A31
- J6 pad B3: /Expansion/EXD18 -> /Expansion/D18
- J6 pad B31: /Expansion/ExpansionSlot4/BCLK -> unconnected-(J6-PadB31)
- J6 pad B32: GND -> unconnected-(J6-PadB32)
- J6 pad B4: /Expansion/EXD19 -> /Expansion/D19
- J6 pad B5: /Expansion/EXD20 -> /Expansion/D20
- J6 pad B6: /Expansion/EXD21 -> /Expansion/D21
- J6 pad B7: /Expansion/EXD22 -> /Expansion/D22
- J6 pad B8: /Expansion/EXD23 -> /Expansion/D23
- J6 pad B9: /Expansion/EXD24 -> /Expansion/D24
- J6 pad C1: +5V -> unconnected-(J6-PadC1)
- J6 pad C10: /Expansion/EXD15 -> /Expansion/D15
- J6 pad C11: GND -> unconnected-(J6-PadC11)
- J6 pad C12: /Expansion/EXA2 -> /Expansion/A2
- J6 pad C13: /Expansion/EXA4 -> /Expansion/A4
- J6 pad C14: /Expansion/EXA6 -> /Expansion/A6
- J6 pad C15: /Expansion/EXA8 -> /Expansion/A8
- J6 pad C16: /Expansion/EXA10 -> /Expansion/A10
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Routing:
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- removed copper zone on In2.Cu, net +3.3V
- removed copper zone on In1.Cu, net GND
- removed copper zone on In2.Cu, net GND
Other:
- board size 284.2 x 203.2 mm -> 221 x 243.8 mm
