File: hardware/memory.kicad_sch (KiCad schematic)
At the start: 23 parts, among them U10 74HC165, U15 SN74ALVC164245, U16 SN74ALVC164245, U17 SN74ALVC164245, U18 SN74ALVC164245, U2 ICE40HX4K-TQ144, U3 SN74ALVC164245, U4 SN74ALVC164245, U5 W25Q32JVSSIM, U9 74HC165

Commit message: begin work on a simpler first draft board
Parts:
- removed C17: 0.1u, Capacitor_SMD:C_0603_1608Metric, symbol UPduino_v3.0:Device_C
- removed D1: LTST-C191KGKT, LED_SMD:LED_0603_1608Metric, symbol UPduino_v3.0:Device_LED_ALT
- removed J10, J11, J12: ~, 68040:SIMM-72, symbol 68040:SIMM72_Socket
- removed R7: 2.2K, Resistor_SMD:R_0603_1608Metric, symbol UPduino_v3.0:Device_R
- removed R8, R9: 10K, Resistor_SMD:R_0603_1608Metric, symbol UPduino_v3.0:Device_R
- removed RN3, RN4, RN5, RN6: 10k, Resistor_THT:R_Array_SIP5, symbol Device:R_Network04_US
- removed U10, U9: 74HC165, Package_SO:SOIC-16_3.9x9.9mm_P1.27mm, symbol 74xx:74HC165
- removed U15, U16, U17, U18: SN74ALVC164245, Package_SO:TSSOP-48_6.1x12.5mm_P0.5mm, symbol 68040:SN74ALVC164245
- removed U2: ICE40HX4K-TQ144, Package_QFP:TQFP-144_20x20mm_P0.5mm, symbol FPGA_Lattice:ICE40HX4K-TQ144
- removed U5: W25Q32JVSSIM, Package_SO:SOIC-8_5.23x5.23mm_P1.27mm, symbol UPduino_v3.0:W25Q32JVSS-Memory_Flash
Connections:
- net D0: now also U4.2 (1B1); no longer U3.2 (1B1)
- net D1: now also U4.5 (1B3); no longer U3.3 (1B2)
- net D10: now also U3.8 (1B5); no longer U3.16 (2B3)
- net D11: now also U3.11 (1B7); no longer U3.17 (2B4)
- net D12: now also U3.13 (2B1); no longer U3.19 (2B5)
- net D13: now also U3.17 (2B4); no longer U3.20 (2B6)
- net D14: now also U3.20 (2B6); no longer U3.22 (2B7)
- net D16: now also U4.3 (1B2); no longer U4.2 (1B1)
- net D17: now also U4.6 (1B4); no longer U4.3 (1B2)
- net D18: now also U4.9 (1B6); no longer U4.5 (1B3)
- net D19: now also U4.12 (1B8); no longer U4.6 (1B4)
- net D2: now also U4.8 (1B5); no longer U3.5 (1B3)
- net D20: now also U4.14 (2B2); no longer U4.8 (1B5)
- net D21: now also U4.17 (2B4); no longer U4.9 (1B6)
- net D22: now also U4.20 (2B6); no longer U4.11 (1B7)
- net D23: now also U4.23 (2B8); no longer U4.12 (1B8)
- net D24: now also U3.3 (1B2); no longer U4.13 (2B1)
- net D25: now also U3.6 (1B4); no longer U4.14 (2B2)
- net D26: now also U3.9 (1B6); no longer U4.16 (2B3)
- net D27: now also U3.12 (1B8); no longer U4.17 (2B4)
- net D28: now also U3.14 (2B2); no longer U4.19 (2B5)
- net D29: now also U3.16 (2B3); no longer U4.20 (2B6)
- net D3: now also U4.11 (1B7); no longer U3.6 (1B4)
- net D30: now also U3.19 (2B5); no longer U4.22 (2B7)
- net D31: now also U3.22 (2B7); no longer U4.23 (2B8)
- net D4: now also U4.13 (2B1); no longer U3.8 (1B5)
- net D5: now also U4.16 (2B3); no longer U3.9 (1B6)
- net D6: now also U4.19 (2B5); no longer U3.11 (1B7)
- net D7: now also U4.22 (2B7); no longer U3.12 (1B8)
- net D8: now also U3.2 (1B1); no longer U3.13 (2B1)
- net D9: now also U3.5 (1B3); no longer U3.14 (2B2)
- net DRAM_D0: now also U4.47 (1A1); no longer U3.47 (1A1)
- net DRAM_D1: now also U4.44 (1A3); no longer U3.46 (1A2)
- net DRAM_D10: now also U3.41 (1A5); no longer U3.33 (2A3)
- net DRAM_D11: now also U3.38 (1A7); no longer U3.32 (2A4)
- net DRAM_D12: now also U3.36 (2A1); no longer U3.30 (2A5)
- net DRAM_D13: now also U3.32 (2A4); no longer U3.29 (2A6)
- net DRAM_D14: now also U3.29 (2A6); no longer U3.27 (2A7)
- net DRAM_D16: now also U4.46 (1A2); no longer U4.47 (1A1)
- net DRAM_D17: now also U4.43 (1A4); no longer U4.46 (1A2)
- net DRAM_D18: now also U4.40 (1A6); no longer U4.44 (1A3)
- net DRAM_D19: now also U4.37 (1A8); no longer U4.43 (1A4)
- net DRAM_D2: now also U4.41 (1A5); no longer U3.44 (1A3)
- net DRAM_D20: now also U4.35 (2A2); no longer U4.41 (1A5)
- net DRAM_D21: now also U4.32 (2A4); no longer U4.40 (1A6)
- net DRAM_D22: now also U4.29 (2A6); no longer U4.38 (1A7)
- net DRAM_D23: now also U4.26 (2A8); no longer U4.37 (1A8)
- net DRAM_D24: now also U3.46 (1A2); no longer U4.36 (2A1)
- net DRAM_D25: now also U3.43 (1A4); no longer U4.35 (2A2)
- net DRAM_D26: now also U3.40 (1A6); no longer U4.33 (2A3)
- net DRAM_D27: now also U3.37 (1A8); no longer U4.32 (2A4)
- net DRAM_D28: now also U3.35 (2A2); no longer U4.30 (2A5)
- net DRAM_D29: now also U3.33 (2A3); no longer U4.29 (2A6)
- net DRAM_D3: now also U4.38 (1A7); no longer U3.43 (1A4)
- net DRAM_D30: now also U3.30 (2A5); no longer U4.27 (2A7)
- net DRAM_D31: now also U3.27 (2A7); no longer U4.26 (2A8)
- net DRAM_D4: now also U4.36 (2A1); no longer U3.41 (1A5)
- net DRAM_D5: now also U4.33 (2A3); no longer U3.40 (1A6)
- net DRAM_D6: now also U4.30 (2A5); no longer U3.38 (1A7)
- net DRAM_D7: now also U4.27 (2A7); no longer U3.37 (1A8)
- net DRAM_D8: now also U3.47 (1A1); no longer U3.36 (2A1)
- net DRAM_D9: now also U3.44 (1A3); no longer U3.35 (2A2)
- no-connect marks 4 -> 0
Other:
- note removed: "Presence detect circuitry Should probably be HCT"
- moved on the sheet: J9, U3A, U3B, U4A, U4B
