File: hardware/memory.kicad_sch (KiCad schematic)
At the start: 3 parts, among them U3 SN74ALVC164245, U4 SN74ALVC164245

Commit message: update cpu symbol, topology
Changed lines of the file:
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@@
   (junction (at 76.2 172.72) (diameter 0) (color 0 0 0 0)
   )
+  (junction (at 106.68 35.56) (diameter 0) (color 0 0 0 0)
+  )
   (junction (at 76.2 175.26) (diameter 0) (color 0 0 0 0)
   )
@@
   (junction (at 76.2 182.88) (diameter 0) (color 0 0 0 0)
   )
+  (junction (at 124.46 109.22) (diameter 0) (color 0 0 0 0)
+  )
   (junction (at 40.64 152.4) (diameter 0) (color 0 0 0 0)
   )
@@
   (junction (at 76.2 180.34) (diameter 0) (color 0 0 0 0)
   )
-  (junction (at 124.46 109.22) (diameter 0) (color 0 0 0 0)
-  )
   (junction (at 40.64 170.18) (diameter 0) (color 0 0 0 0)
   )
@@
   (junction (at 246.38 134.62) (diameter 0) (color 0 0 0 0)
   )
+  (junction (at 109.22 40.64) (diameter 0) (color 0 0 0 0)
+  )
   (junction (at 66.04 160.02) (diameter 0) (color 0 0 0 0)
   )
@@
     (stroke (width 0) (type default))
   )
-  (wire (pts (xy 119.38 114.3) (xy 119.38 101.6))
-    (stroke (width 0) (type default))
-  )
   (bus (pts (xy 220.98 121.92) (xy 220.98 119.38))
     (stroke (width 0) (type default))
@@
     (stroke (width 0) (type default))
   )
-  (wire (pts (xy 124.46 114.3) (xy 119.38 114.3))
+  (wire (pts (xy 109.22 114.3) (xy 124.46 114.3))
     (stroke (width 0) (type default))
   )
@@
     (stroke (width 0) (type default))
   )
-  (wire (pts (xy 119.38 27.94) (xy 83.82 27.94))
-    (stroke (width 0) (type default))
-  )
   (wire (pts (xy 114.3 60.96) (xy 124.46 60.96))
     (stroke (width 0) (type default))
@@
     (stroke (width 0) (type default))
   )
+  (wire (pts (xy 106.68 35.56) (xy 124.46 35.56))
+    (stroke (width 0) (type default))
+  )
   (wire (pts (xy 220.98 63.5) (xy 231.14 63.5))
     (stroke (width 0) (type default))
@@
     (stroke (width 0) (type default))
   )
+  (wire (pts (xy 106.68 109.22) (xy 106.68 35.56))
+    (stroke (width 0) (type default))
+  )
   (wire (pts (xy 261.62 83.82) (xy 271.78 83.82))
     (stroke (width 0) (type default))
@@
     (stroke (width 0) (type default))
   )
+  (wire (pts (xy 109.22 40.64) (xy 124.46 40.64))
+    (stroke (width 0) (type default))
+  )
   (wire (pts (xy 261.62 109.22) (xy 271.78 109.22))
     (stroke (width 0) (type default))
@@
     (stroke (width 0) (type default))
   )
-  (wire (pts (xy 119.38 101.6) (xy 83.82 101.6))
-    (stroke (width 0) (type default))
-  )
-  (wire (pts (xy 83.82 96.52) (xy 124.46 96.52))
+  (wire (pts (xy 109.22 40.64) (xy 109.22 114.3))
     (stroke (width 0) (type default))
   )
@@
     (stroke (width 0) (type default))
   )
-  (wire (pts (xy 124.46 40.64) (xy 119.38 40.64))
+  (wire (pts (xy 83.82 40.64) (xy 109.22 40.64))
     (stroke (width 0) (type default))
   )
@@
     (stroke (width 0) (type default))
   )
-  (wire (pts (xy 119.38 40.64) (xy 119.38 27.94))
-    (stroke (width 0) (type default))
-  )
   (wire (pts (xy 165.1 38.1) (xy 175.26 38.1))
     (stroke (width 0) (type default))
@@
     (stroke (width 0) (type default))
   )
-  (wire (pts (xy 124.46 35.56) (xy 124.46 22.86))
-    (stroke (width 0) (type default))
-  )
   (wire (pts (xy 114.3 132.08) (xy 124.46 132.08))
     (stroke (width 0) (type default))
@@
     (stroke (width 0) (type default))
   )
+  (wire (pts (xy 124.46 109.22) (xy 106.68 109.22))
+    (stroke (width 0) (type default))
+  )
   (wire (pts (xy 76.2 185.42) (xy 76.2 190.5))
     (stroke (width 0) (type default))
@@
     (stroke (width 0) (type default))
   )
-  (wire (pts (xy 83.82 22.86) (xy 124.46 22.86))
+  (wire (pts (xy 83.82 35.56) (xy 106.68 35.56))
     (stroke (width 0) (type default))
   )
@@
     (stroke (width 0) (type default))
   )
-  (wire (pts (xy 124.46 109.22) (xy 124.46 96.52))
-    (stroke (width 0) (type default))
-  )
   (wire (pts (xy 261.62 58.42) (xy 271.78 58.42))
     (stroke (width 0) (type default))
@@
     (effects (font (size 1.27 1.27)) (justify right bottom))
   )
-  (label "DRAM_BUF_~{OE}" (at 83.82 96.52 0) (fields_autoplaced)
-    (effects (font (size 1.27 1.27)) (justify left bottom))
-  )
   (label "D19" (at 124.46 139.7 180) (fields_autoplaced)
     (effects (font (size 1.27 1.27)) (justify right bottom))
@@
     (effects (font (size 1.27 1.27)) (justify right bottom))
   )
-  (label "DRAM_BUF_DIR" (at 83.82 27.94 0) (fields_autoplaced)
-    (effects (font (size 1.27 1.27)) (justify left bottom))
-  )
   (label "DRAM_D10" (at 175.26 48.26 180) (fields_autoplaced)
     (effects (font (size 1.27 1.27)) (justify right bottom))
@@
     (effects (font (size 1.27 1.27)) (justify right bottom))
   )
-  (label "DRAM_BUF_~{OE}" (at 83.82 22.86 0) (fields_autoplaced)
-    (effects (font (size 1.27 1.27)) (justify left bottom))
-  )
-  (label "DRAM_BUF_DIR" (at 83.82 101.6 0) (fields_autoplaced)
-    (effects (font (size 1.27 1.27)) (justify left bottom))
-  )
   (label "DRAM_A2" (at 220.98 58.42 0) (fields_autoplaced)
     (effects (font (size 1.27 1.27)) (justify left bottom))
@@
     (effects (font (size 1.27 1.27)) (justify left bottom))
   )
+  (hierarchical_label "DRAM_BUF_DIR" (shape input) (at 83.82 40.64 180) (fields_autoplaced)
+    (effects (font (size 1.27 1.27)) (justify right))
+  )
+  (hierarchical_label "DRAM_BUF_~{OE}" (shape input) (at 83.82 35.56 180) (fields_autoplaced)
+    (effects (font (size 1.27 1.27)) (justify right))
+  )
   (hierarchical_label "D[0..31]" (shape bidirectional) (at 83.82 43.18 180) (fields_autoplaced)

Commit message: add interrupt logic, clean up modules
Parts:
- added C22, C23, C24, C25: 100nF, symbol Device:C
- added J10, J11, J8: ~, 68040:SIMM-72, symbol 68040:SIMM72_Socket
Connections:
- net +3V3: now also C24.1, C25.1, J10.10 (VCC), J10.30 (VCC), J10.59 (VCC), J11.10 (VCC), J11.30 (VCC), J11.59 (VCC), J8.10 (VCC), J8.30 (VCC), J8.59 (VCC)
- net +5V: now also C22.1, C23.1
- net DRAM_A0: now also J10.12 (A0), J11.12 (A0), J8.12 (A0)
- net DRAM_A1: now also J10.13 (A1), J11.13 (A1), J8.13 (A1)
- net DRAM_A10: now also J10.19 (A10), J11.19 (A10), J8.19 (A10)
- net DRAM_A11: now also J10.29 (A11), J11.29 (A11), J8.29 (A11)
- net DRAM_A2: now also J10.14 (A2), J11.14 (A2), J8.14 (A2)
- net DRAM_A3: now also J10.15 (A3), J11.15 (A3), J8.15 (A3)
- net DRAM_A4: now also J10.16 (A4), J11.16 (A4), J8.16 (A4)
- net DRAM_A5: now also J10.17 (A5), J11.17 (A5), J8.17 (A5)
- net DRAM_A6: now also J10.18 (A6), J11.18 (A6), J8.18 (A6)
- net DRAM_A7: now also J10.28 (A7), J11.28 (A7), J8.28 (A7)
- net DRAM_A8: now also J10.31 (A8), J11.31 (A8), J8.31 (A8)
- net DRAM_A9: now also J10.32 (A9), J11.32 (A9), J8.32 (A9)
- net DRAM_D0: now also J10.2 (DQ0), J11.2 (DQ0), J8.2 (DQ0)
- net DRAM_D1: now also J10.4 (DQ1), J11.4 (DQ1), J8.4 (DQ1)
- net DRAM_D10: now also J10.53 (DQ10), J11.53 (DQ10), J8.53 (DQ10)
- net DRAM_D11: now also J10.55 (DQ11), J11.55 (DQ11), J8.55 (DQ11)
- net DRAM_D12: now also J10.57 (DQ12), J11.57 (DQ12), J8.57 (DQ12)
- net DRAM_D13: now also J10.61 (DQ13), J11.61 (DQ13), J8.61 (DQ13)
- net DRAM_D14: now also J10.63 (DQ14), J11.63 (DQ14), J8.63 (DQ14)
- net DRAM_D15: now also J10.65 (DQ15), J11.65 (DQ15), J8.65 (DQ15)
- net DRAM_D16: now also J10.3 (DQ16), J11.3 (DQ16), J8.3 (DQ16)
- net DRAM_D17: now also J10.5 (DQ17), J11.5 (DQ17), J8.5 (DQ17)
- net DRAM_D18: now also J10.7 (DQ18), J11.7 (DQ18), J8.7 (DQ18)
- net DRAM_D19: now also J10.9 (DQ19), J11.9 (DQ19), J8.9 (DQ19)
- net DRAM_D2: now also J10.6 (DQ2), J11.6 (DQ2), J8.6 (DQ2)
- net DRAM_D20: now also J10.21 (DQ20), J11.21 (DQ20), J8.21 (DQ20)
- net DRAM_D21: now also J10.23 (DQ21), J11.23 (DQ21), J8.23 (DQ21)
- net DRAM_D22: now also J10.25 (DQ22), J11.25 (DQ22), J8.25 (DQ22)
- net DRAM_D23: now also J10.27 (DQ23), J11.27 (DQ23), J8.27 (DQ23)
- net DRAM_D24: now also J10.50 (DQ24), J11.50 (DQ24), J8.50 (DQ24)
- net DRAM_D25: now also J10.52 (DQ25), J11.52 (DQ25), J8.52 (DQ25)
- net DRAM_D26: now also J10.54 (DQ26), J11.54 (DQ26), J8.54 (DQ26)
- net DRAM_D27: now also J10.56 (DQ27), J11.56 (DQ27), J8.56 (DQ27)
- net DRAM_D28: now also J10.58 (DQ28), J11.58 (DQ28), J8.58 (DQ28)
- net DRAM_D29: now also J10.60 (DQ29), J11.60 (DQ29), J8.60 (DQ29)
- net DRAM_D3: now also J10.8 (DQ3), J11.8 (DQ3), J8.8 (DQ3)
- net DRAM_D30: now also J10.62 (DQ30), J11.62 (DQ30), J8.62 (DQ30)
- net DRAM_D31: now also J10.64 (DQ31), J11.64 (DQ31), J8.64 (DQ31)
- net DRAM_D4: now also J10.20 (DQ4), J11.20 (DQ4), J8.20 (DQ4)
- net DRAM_D5: now also J10.22 (DQ5), J11.22 (DQ5), J8.22 (DQ5)
- net DRAM_D6: now also J10.24 (DQ6), J11.24 (DQ6), J8.24 (DQ6)
- net DRAM_D7: now also J10.26 (DQ7), J11.26 (DQ7), J8.26 (DQ7)
- net DRAM_D8: now also J10.49 (DQ8), J11.49 (DQ8), J8.49 (DQ8)
- net DRAM_D9: now also J10.51 (DQ9), J11.51 (DQ9), J8.51 (DQ9)
- net DRAM_R/~{W}: now also J10.47 (R/~{W}), J11.47 (R/~{W}), J8.47 (R/~{W})
- net GND: now also C22.2, C23.2, C24.2, C25.2, J10.1 (GND), J10.39 (GND), J10.72 (GND), J11.1 (GND), J11.39 (GND), J11.72 (GND), J8.1 (GND), J8.39 (GND), J8.72 (GND)
- net ~{RAS0}: now also J10.44 (~{RAS0}), J11.44 (~{RAS0}), J8.44 (~{RAS0})
- net ~{RAS1}: now also J10.45 (~{RAS1}), J11.45 (~{RAS1}), J8.45 (~{RAS1})
- net ~{RAS2}: now also J10.34 (~{RAS2}), J11.34 (~{RAS2}), J8.34 (~{RAS2})
- net ~{RAS3}: now also J10.33 (~{RAS3}), J11.33 (~{RAS3}), J8.33 (~{RAS3})
- net PD_{A}1: no longer names the net of J9.67 (PD1)
- net PD_{A}2: no longer names the net of J9.68 (PD2)
- net PD_{A}3: no longer names the net of J9.69 (PD3)
- net PD_{A}4: no longer names the net of J9.70 (PD4)
- new net ~{CAS_B0}: J8.40 (~{CAS0})
- new net ~{CAS_B1}: J8.43 (~{CAS1})
- new net ~{CAS_B2}: J8.41 (~{CAS2})
- new net ~{CAS_B3}: J8.42 (~{CAS3})
- new net ~{CAS_C0}: J10.40 (~{CAS0})
- new net ~{CAS_C1}: J10.43 (~{CAS1})
- new net ~{CAS_C2}: J10.41 (~{CAS2})
- new net ~{CAS_C3}: J10.42 (~{CAS3})
- new net ~{CAS_D0}: J11.40 (~{CAS0})
- new net ~{CAS_D1}: J11.43 (~{CAS1})
- new net ~{CAS_D2}: J11.41 (~{CAS2})
- new net ~{CAS_D3}: J11.42 (~{CAS3})
- no-connect marks 0 -> 16
Other:
- note added: "DIR High: A -> B DIR Low: B -> A"
- moved on the sheet: J9, U3A, U3B, U4A, U4B

Commit message: getting closer
Parts:
- removed C24, C25: 100nF, symbol Device:C
- added C45, C46: 100nF, symbol Device:C
- U3, U4: value SN74ALVC164245 -> SN74AHCT164245; symbol 68040:SN74ALVC164245 -> 68040:SN74AHCT164245
Connections:
- net DRAM_BUF_DIR is gone; now on net DRAM_R/~{W}: U3.1 (1DIR), U3.24 (2DIR), U4.1 (1DIR), U4.24 (2DIR)
- net +3V3: no longer U3.31 (VCCA), U3.42 (VCCA), U4.31 (VCCA), U4.42 (VCCA)
- net +5V: now also U3.31 (VCC), U3.42 (VCC), U4.31 (VCC), U4.42 (VCC), C45.1, C46.1
- net GND: now also C45.2, C46.2
Other:
- moved on the sheet: C22, C23
