File: hardware/expansion.kicad_sch (KiCad schematic)
At the start: 1 part, among them J2 EXP

Commit message: add interrupt logic, clean up modules
Connections:
- net +3V3: no longer names the net of J2.C30
Changed lines of the file:
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@@
     (stroke (width 0) (type default))
   )
-  (wire (pts (xy 195.58 114.3) (xy 208.28 114.3))
-    (stroke (width 0) (type default))
-  )
   (label "EXA30" (at 121.92 109.22 0) (fields_autoplaced)
     (effects (font (size 1.27 1.27)) (justify left bottom))
@@
     (effects (font (size 1.27 1.27)) (justify left bottom))
   )
-  (hierarchical_label "~{TBI}" (shape bidirectional) (at 27.94 152.4 180) (fields_autoplaced)
-    (effects (font (size 1.27 1.27)) (justify right))
-  )
-  (hierarchical_label "R{slash}~{W}" (shape bidirectional) (at 27.94 170.18 180) (fields_autoplaced)
-    (effects (font (size 1.27 1.27)) (justify right))
-  )
-  (hierarchical_label "~{TEA}" (shape bidirectional) (at 27.94 154.94 180) (fields_autoplaced)
-    (effects (font (size 1.27 1.27)) (justify right))
-  )
-  (hierarchical_label "~{B_{BUSY}}" (shape output) (at 27.94 177.8 180) (fields_autoplaced)
+  (hierarchical_label "R{slash}~{W}" (shape bidirectional) (at 27.94 172.72 180) (fields_autoplaced)
+    (effects (font (size 1.27 1.27)) (justify right))
+  )
+  (hierarchical_label "~{TEA}" (shape bidirectional) (at 27.94 152.4 180) (fields_autoplaced)
+    (effects (font (size 1.27 1.27)) (justify right))
+  )
+  (hierarchical_label "~{B_{BUSY}}" (shape output) (at 27.94 180.34 180) (fields_autoplaced)
     (effects (font (size 1.27 1.27)) (justify right))
   )
@@
     (effects (font (size 1.27 1.27)) (justify left))
   )
-  (hierarchical_label "~{TCI}" (shape bidirectional) (at 27.94 149.86 180) (fields_autoplaced)
+  (hierarchical_label "~{TBI}{slash}~{TCI}" (shape bidirectional) (at 27.94 149.86 180) (fields_autoplaced)
     (effects (font (size 1.27 1.27)) (justify right))
   )
@@
     (effects (font (size 1.27 1.27)) (justify right))
   )
-  (hierarchical_label "~{B_{GRANT}}" (shape input) (at 27.94 175.26 180) (fields_autoplaced)
-    (effects (font (size 1.27 1.27)) (justify right))
-  )
-  (hierarchical_label "~{TS}" (shape bidirectional) (at 27.94 157.48 180) (fields_autoplaced)
+  (hierarchical_label "~{B_{GRANT}}" (shape input) (at 27.94 177.8 180) (fields_autoplaced)
+    (effects (font (size 1.27 1.27)) (justify right))
+  )
+  (hierarchical_label "~{SLAVE_{N}}" (shape output) (at 27.94 157.48 180) (fields_autoplaced)
+    (effects (font (size 1.27 1.27)) (justify right))
+  )
+  (hierarchical_label "BCLK" (shape input) (at 27.94 144.78 180) (fields_autoplaced)
+    (effects (font (size 1.27 1.27)) (justify right))
+  )
+  (hierarchical_label "~{TS}" (shape bidirectional) (at 27.94 154.94 180) (fields_autoplaced)
     (effects (font (size 1.27 1.27)) (justify right))
   )
@@
     (effects (font (size 1.27 1.27)) (justify right))
   )
-  (hierarchical_label "SIZ1" (shape bidirectional) (at 27.94 167.64 180) (fields_autoplaced)
-    (effects (font (size 1.27 1.27)) (justify right))
-  )
-  (hierarchical_label "SIZ0" (shape bidirectional) (at 27.94 165.1 180) (fields_autoplaced)
+  (hierarchical_label "SIZ1" (shape bidirectional) (at 27.94 170.18 180) (fields_autoplaced)
+    (effects (font (size 1.27 1.27)) (justify right))
+  )
+  (hierarchical_label "SIZ0" (shape bidirectional) (at 27.94 167.64 180) (fields_autoplaced)
     (effects (font (size 1.27 1.27)) (justify right))
   )
@@
     (effects (font (size 1.27 1.27)) (justify right))
   )
-  (hierarchical_label "~{B_{REQ}}" (shape output) (at 27.94 172.72 180) (fields_autoplaced)
+  (hierarchical_label "~{B_{REQ}}" (shape output) (at 27.94 175.26 180) (fields_autoplaced)
+    (effects (font (size 1.27 1.27)) (justify right))
+  )
+  (hierarchical_label "~{IACK}" (shape input) (at 27.94 165.1 180) (fields_autoplaced)
     (effects (font (size 1.27 1.27)) (justify right))
   )
@@
         )
       )
-    )
-  )
-  (symbol (lib_id "power:+3V3") (at 195.58 114.3 0) (unit 1)
-    (in_bom yes) (on_board yes) (dnp no) (fields_autoplaced)
-    (property "Reference" "#PWR0136" (at 195.58 118.11 0)
-      (effects (font (size 1.27 1.27)) hide)
-    )
-    (property "Value" "+3V3" (at 195.58 109.22 0)
-      (effects (font (size 1.27 1.27)))
-    )
-    (property "Footprint" "" (at 195.58 114.3 0)
-      (effects (font (size 1.27 1.27)) hide)
-    )
-    (property "Datasheet" "" (at 195.58 114.3 0)
-      (effects (font (size 1.27 1.27)) hide)
-    )
-    (pin "1")
-    (instances
-      (project "68040pc"
-        (path "/3006deba-2100-40f8-9f39-987a5c2c14c7/4c7887cb-c367-4b93-be02-0b485997fe7b/4a50b038-ddbb-45ef-83ad-890c6e7cc82c"
-          (reference "#PWR0136") (unit 1)
-        )
-        (path "/3006deba-2100-40f8-9f39-987a5c2c14c7/4c7887cb-c367-4b93-be02-0b485997fe7b/cb293a02-ab30-4c8a-a1c0-096525c507f2"
-          (reference "#PWR039") (unit 1)
-        )
-        (path "/3006deba-2100-40f8-9f39-987a5c2c14c7/4c7887cb-c367-4b93-be02-0b485997fe7b/0776ee06-ca6a-474b-8930-643fb1879758"
-          (reference "#PWR054") (unit 1)
-        )
-        (path "/3006deba-2100-40f8-9f39-987a5c2c14c7/4c7887cb-c367-4b93-be02-0b485997fe7b/e3fdc7e0-b0cd-4106-aa8e-240174c46b8d"
-          (reference "#PWR069") (unit 1)
-        )
-      )
