File: hardware/interrupts.kicad_sch (KiCad schematic)
At the start: 3 parts, among them U28 74HC00, U29 74HC138, U30 74LS348

Commit message: updates
Connections:
- net ~{IACK7} renamed ~{NMIACK}
- net ~{IRQ7} renamed ~{NMI}
Changed lines of the file:
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@@
     (effects (font (size 1.27 1.27)) (justify right))
   )
-  (hierarchical_label "~{IACK7}" (shape output) (at 137.16 55.88 0) (fields_autoplaced)
+  (hierarchical_label "~{NMIACK}" (shape output) (at 137.16 55.88 0) (fields_autoplaced)
     (effects (font (size 1.27 1.27)) (justify left))
   )
@@
     (effects (font (size 1.27 1.27)) (justify right))
   )
-  (hierarchical_label "~{IRQ7}" (shape input) (at 114.3 119.38 180) (fields_autoplaced)
+  (hierarchical_label "~{NMI}" (shape input) (at 114.3 119.38 180) (fields_autoplaced)
     (effects (font (size 1.27 1.27)) (justify right))
   )
