File: hardware/kbdmou.kicad_sch (KiCad schematic)
At the start: 17 parts, among them J13 DIN-5_180degree, J14 Mini-DIN-6, Q1 2N4403, Q2 FQP27P06, U21 ATmega8-16A

Commit message: getting closer
Connections:
- no-connect marks 3 -> 6
Other:
- moved on the sheet: C16, C17, C18, C19, L1, Q1, Q2, R7, R8
