File: hardware/processor.kicad_sch (KiCad schematic)
At the start: 1 part, among them U1 68LC040

Commit message: update cpu symbol, topology
Parts:
- added C10, C13: 0.22uF, symbol Device:C
- added C11, C15: 220pF, symbol Device:C
- added C12, C14: 22uF, symbol Device:C_Polarized_US
- added R6: 4.7k, symbol Device:R
- added RN3: 4.7k, Resistor_THT:R_Array_SIP6, symbol Device:R_Network05_Split
- added unit 2 of U1
Connections:
- net TMS is gone; now on an unnamed net: U1.S5 (TMS)
- net ~{MDIS} is gone; now on an unnamed net: U1.S6 (~{MDIS})
- net ~{TSRT} is gone; now on net GND: U1.T3 (~{TRST})
- net ~{BB}: now also R6.2
- net ~{RSTO}: now also RN3.5 (R4.2)
- net ~{TA}: now also U1.T14 (~{TA})
- net ~{TEA}: now also U1.S13 (~{TEA})
- net ~{TS}: now also RN3.6 (R5.2)
- net ~{TCI}/~{TBI}: now reaches U1.S11 (~{TBI})
- net ~{TCI}/~{TBI}: now also U1.T10 (~{TCI})
- net BCLK: no longer names the net of U1.R7 (BCLK)
- removed net GND_{L}: U1.C11 (GND), U1.C13 (GND), U1.C6 (GND), U1.C7 (GND), U1.C9 (GND), U1.K16 (GND), U1.K3 (GND), U1.L3 (GND), U1.M16 (GND), U1.R11 (GND), U1.R13 (GND), U1.R4 (GND), U1.S10 (GND), U1.T4 (GND)
- removed net GND_{O}: U1.B10 (GND), U1.B13 (GND), U1.B15 (GND), U1.B17 (GND), U1.B2 (GND), U1.B4 (GND), U1.B6 (GND), U1.B8 (GND), U1.D17 (GND), U1.D2 (GND), U1.F17 (GND), U1.F2 (GND), U1.H17 (GND), U1.H2 (GND), U1.L17 (GND), U1.L2 (GND), U1.N17 (GND), U1.N2 (GND), U1.Q17 (GND), U1.Q2 (GND), U1.S15 (GND), U1.S17 (GND), U1.S2 (GND)
- removed net GND_{P}: U1.R10 (GND), U1.R6 (GND), U1.S9 (GND)
- net JS0 renamed DLE
- net DLE: now also RN3.4 (R3.2)
- net PCLK: no longer names the net of U1.R9 (PCLK)
- net TCK renamed GND
- net GND: now also C10.2, C11.2, C12.2, C13.2, C14.2, C15.2, U1.B10 (GND), U1.B13 (GND), U1.B15 (GND), U1.B17 (GND), U1.B2 (GND), U1.B4 (GND), U1.B6 (GND), U1.B8 (GND), U1.C11 (GND), U1.C13 (GND), U1.C6 (GND), U1.C7 (GND), U1.C9 (GND), U1.D17 (GND), U1.D2 (GND), U1.F17 (GND), U1.F2 (GND), U1.H17 (GND), U1.H2 (GND), U1.K16 (GND), U1.K3 (GND), U1.L17 (GND), U1.L2 (GND), U1.L3 (GND), U1.M16 (GND), U1.N17 (GND), U1.N2 (GND), U1.Q17 (GND), U1.Q2 (GND), U1.R10 (GND), U1.R11 (GND), U1.R13 (GND), U1.R4 (GND), U1.R6 (GND), U1.S10 (GND), U1.S15 (GND), U1.S17 (GND), U1.S2 (GND), U1.S9 (GND), U1.T4 (GND)
- net TDI: no longer names the net of U1.S3 (TDI)
- net TDI: now also RN3.2 (R1.2)
- net TDO: no longer names the net of U1.T2 (TDO)
- net TLN0: no longer names the net of U1.Q18 (TLN0)
- net TLN1: no longer names the net of U1.P18 (TLN1)
- net UPA0: no longer names the net of U1.Q3 (UPA0)
- net UPA1: no longer names the net of U1.Q1 (UPA1)
- removed net V_{CC}_{L}: U1.C10 (V_{CC}), U1.C12 (V_{CC}), U1.C14 (V_{CC}), U1.C5 (V_{CC}), U1.C8 (V_{CC}), U1.H16 (V_{CC}), U1.H3 (V_{CC}), U1.J16 (V_{CC}), U1.J3 (V_{CC}), U1.L16 (V_{CC}), U1.M3 (V_{CC}), U1.R12 (V_{CC}), U1.R5 (V_{CC})
- removed net V_{CC}_{O}: U1.B14 (V_{CC}), U1.B5 (V_{CC}), U1.B9 (V_{CC}), U1.C17 (V_{CC}), U1.C2 (V_{CC}), U1.G17 (V_{CC}), U1.G2 (V_{CC}), U1.M17 (V_{CC}), U1.M2 (V_{CC}), U1.R17 (V_{CC}), U1.R2 (V_{CC}), U1.S16 (V_{CC})
- removed net V_{CC}_{P}: U1.R8 (V_{CC}), U1.S8 (V_{CC})
- net ~{CDIS}: no longer names the net of U1.T5 (~{CDIS})
- net ~{CDIS}: now also RN3.3 (R2.2)
- net ~{CIOUT}: no longer names the net of U1.R1 (~{CIOUT})
- net ~{IPEND}: no longer names the net of U1.S1 (~{IPEND})
- new net +5V: C10.1, C11.1, C12.1, C13.1, C14.1, C15.1, R6.1, RN3.1 (R1), RN3.1 (R1), RN3.1 (R1), RN3.1 (R1), RN3.1 (R1), U1.B14 (V_{CC}), U1.B5 (V_{CC}), U1.B9 (V_{CC}), U1.C10 (V_{CC}), U1.C12 (V_{CC}), U1.C14 (V_{CC}), U1.C17 (V_{CC}), U1.C2 (V_{CC}), U1.C5 (V_{CC}), U1.C8 (V_{CC}), U1.G17 (V_{CC}), U1.G2 (V_{CC}), U1.H16 (V_{CC}), U1.H3 (V_{CC}), U1.J16 (V_{CC}), U1.J3 (V_{CC}), U1.L16 (V_{CC}), U1.M17 (V_{CC}), U1.M2 (V_{CC}), U1.M3 (V_{CC}), U1.R12 (V_{CC}), U1.R17 (V_{CC}), U1.R2 (V_{CC}), U1.R5 (V_{CC}), U1.R8 (V_{CC}), U1.S16 (V_{CC}), U1.S8 (V_{CC})
- no-connect marks 0 -> 7

Commit message: add interrupt logic, clean up modules
Connections:
- net PST0: no longer names the net of U1.T15 (PST0)
- net PST1: no longer names the net of U1.S14 (PST1)
- net PST2: no longer names the net of U1.R14 (PST2)
- net PST3: no longer names the net of U1.T16 (PST3)
- no-connect marks 7 -> 11
Changed lines of the file:
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@@
   )
   (no_connect (at 198.12 88.9))
+  (no_connect (at 198.12 121.92))
   (no_connect (at 198.12 99.06))
   (no_connect (at 81.28 104.14))
+  (no_connect (at 198.12 119.38))
+  (no_connect (at 198.12 127))
+  (no_connect (at 198.12 124.46))
   (no_connect (at 198.12 86.36))
   (no_connect (at 198.12 66.04))
@@
     (stroke (width 0) (type default))
   )
-  (bus_entry (at 205.74 119.38) (size 2.54 2.54)
-    (stroke (width 0) (type default))
-  )
   (bus_entry (at 68.58 78.74) (size 2.54 2.54)
     (stroke (width 0) (type default))
@@
     (stroke (width 0) (type default))
   )
-  (bus_entry (at 205.74 121.92) (size 2.54 2.54)
-    (stroke (width 0) (type default))
-  )
   (bus_entry (at 116.84 139.7) (size 2.54 2.54)
     (stroke (width 0) (type default))
@@
     (stroke (width 0) (type default))
   )
-  (bus_entry (at 205.74 124.46) (size 2.54 2.54)
-    (stroke (width 0) (type default))
-  )
   (bus_entry (at 121.92 48.26) (size 2.54 -2.54)
     (stroke (width 0) (type default))
@@
     (stroke (width 0) (type default))
   )
-  (bus_entry (at 205.74 127) (size 2.54 2.54)
-    (stroke (width 0) (type default))
-  )
   (bus_entry (at 180.34 48.26) (size 2.54 -2.54)
     (stroke (width 0) (type default))
@@
     (stroke (width 0) (type default))
   )
-  (wire (pts (xy 205.74 124.46) (xy 198.12 124.46))
-    (stroke (width 0) (type default))
-  )
   (wire (pts (xy 144.78 53.34) (xy 144.78 48.26))
     (stroke (width 0) (type default))
@@
     (stroke (width 0) (type default))
   )
-  (wire (pts (xy 205.74 119.38) (xy 198.12 119.38))
-    (stroke (width 0) (type default))
-  )
   (bus (pts (xy 124.46 142.24) (xy 127 142.24))
     (stroke (width 0) (type default))
@@
     (stroke (width 0) (type default))
   )
-  (bus (pts (xy 208.28 124.46) (xy 208.28 127))
-    (stroke (width 0) (type default))
-  )
   (bus (pts (xy 210.82 76.2) (xy 208.28 76.2))
     (stroke (width 0) (type default))
@@
     (stroke (width 0) (type default))
   )
-  (bus (pts (xy 208.28 121.92) (xy 208.28 124.46))
-    (stroke (width 0) (type default))
-  )
   (wire (pts (xy 38.1 81.28) (xy 38.1 93.98))
     (stroke (width 0) (type default))
@@
     (stroke (width 0) (type default))
   )
-  (wire (pts (xy 205.74 127) (xy 198.12 127))
-    (stroke (width 0) (type default))
-  )
   (wire (pts (xy 78.74 99.06) (xy 66.04 99.06))
     (stroke (width 0) (type default))
@@
     (stroke (width 0) (type default))
   )
-  (bus (pts (xy 208.28 129.54) (xy 213.36 129.54))
-    (stroke (width 0) (type default))
-  )
   (wire (pts (xy 88.9 180.34) (xy 104.14 180.34))
     (stroke (width 0) (type default))
@@
     (stroke (width 0) (type default))
   )
-  (bus (pts (xy 208.28 127) (xy 208.28 129.54))
-    (stroke (width 0) (type default))
-  )
   (bus (pts (xy 132.08 45.72) (xy 134.62 45.72))
     (stroke (width 0) (type default))
@@
     (stroke (width 0) (type default))
   )
-  (wire (pts (xy 205.74 121.92) (xy 198.12 121.92))
-    (stroke (width 0) (type default))
-  )
   (bus (pts (xy 109.22 45.72) (xy 111.76 45.72))
     (stroke (width 0) (type default))
@@
     (effects (font (size 1.27 1.27)) (justify left bottom))
   )
-  (label "PST0" (at 205.74 119.38 180) (fields_autoplaced)
-    (effects (font (size 1.27 1.27)) (justify right bottom))
-  )
   (label "D12" (at 149.86 48.26 270) (fields_autoplaced)
     (effects (font (size 1.27 1.27)) (justify right bottom))
@@
     (effects (font (size 1.27 1.27)) (justify right bottom))
   )
-  (label "PST3" (at 205.74 127 180) (fields_autoplaced)
-    (effects (font (size 1.27 1.27)) (justify right bottom))
-  )
   (label "D22" (at 124.46 48.26 270) (fields_autoplaced)
     (effects (font (size 1.27 1.27)) (justify right bottom))
@@
     (effects (font (size 1.27 1.27)) (justify left bottom))
   )
-  (label "PST2" (at 205.74 124.46 180) (fields_autoplaced)
-    (effects (font (size 1.27 1.27)) (justify right bottom))
-  )
   (label "SIZ0" (at 205.74 68.58 180) (fields_autoplaced)
     (effects (font (size 1.27 1.27)) (justify right bottom))
@@
   (label "A30" (at 104.14 139.7 90) (fields_autoplaced)
     (effects (font (size 1.27 1.27)) (justify left bottom))
-  )
-  (label "PST1" (at 205.74 121.92 180) (fields_autoplaced)
-    (effects (font (size 1.27 1.27)) (justify right bottom))
   )
   (label "~{IPL0}" (at 73.66 66.04 0) (fields_autoplaced)
@@
     (effects (font (size 1.27 1.27)) (justify left))
   )
-  (hierarchical_label "~{AVEC}" (shape bidirectional) (at 76.2 73.66 180) (fields_autoplaced)
+  (hierarchical_label "~{AVEC}" (shape input) (at 76.2 73.66 180) (fields_autoplaced)
     (effects (font (size 1.27 1.27)) (justify right))
   )
@@
     (effects (font (size 1.27 1.27)) (justify left))
   )
-  (hierarchical_label "IPL[0..2]" (shape input) (at 68.58 63.5 180) (fields_autoplaced)
+  (hierarchical_label "~{IPL[0..2]}" (shape input) (at 68.58 63.5 180) (fields_autoplaced)
     (effects (font (size 1.27 1.27)) (justify right))
   )
@@
     (effects (font (size 1.27 1.27)) (justify left))
   )
-  (hierarchical_label "PST[0..3]" (shape bidirectional) (at 213.36 129.54 0) (fields_autoplaced)
-    (effects (font (size 1.27 1.27)) (justify left))
-  )

Commit message: updates
Parts:
- added R? (x14): 4.7k, symbol Device:R_Small_US
Connections:
- net +5V: now also R?.1, R?.1, R?.1, R?.1, R?.1, R?.1, R?.1, R?.1, R?.1, R?.1, R?.1, R?.1
- net GND: now also R?.2, R?.2
- net TT0: now also R?.1
- net TT1: now also R?.1
- net ~{IPL0}: now also R?.2
- net ~{IPL1}: now also R?.2
- net ~{IPL2}: now also R?.2

Commit message: getting closer
Parts:
- gave numbers to parts that had none: 14
Connections:
- net R/~{W}: now also R18.2
- net BCLK: now reaches U1.R7 (BCLK)
- net PCLK: now reaches U1.R9 (PCLK)
Changed lines of the file:
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@@
+    (stroke (width 0) (type default))
+  )
+  (wire (pts (xy 106.68 38.1) (xy 106.68 27.94))
     (stroke (width 0) (type default))
   )
@@
     (stroke (width 0) (type default))
   )
+  (wire (pts (xy 73.66 119.38) (xy 81.28 119.38))
+    (stroke (width 0) (type default))
+  )
   (wire (pts (xy 167.64 139.7) (xy 167.64 134.62))
     (stroke (width 0) (type default))
@@
     (stroke (width 0) (type default))
   )
+  (wire (pts (xy 38.1 38.1) (xy 106.68 38.1))
+    (stroke (width 0) (type default))
+  )
   (bus (pts (xy 137.16 142.24) (xy 139.7 142.24))
     (stroke (width 0) (type default))
@@
   )
   (wire (pts (xy 104.14 139.7) (xy 104.14 134.62))
+    (stroke (width 0) (type default))
+  )
+  (wire (pts (xy 73.66 116.84) (xy 81.28 116.84))
     (stroke (width 0) (type default))
   )
@@
     (effects (font (size 1.27 1.27)) (justify left))
   )
+  (hierarchical_label "R{slash}~{W}" (shape bidirectional) (at 38.1 38.1 180) (fields_autoplaced)
+    (effects (font (size 1.27 1.27)) (justify right))
+  )
   (hierarchical_label "~{AVEC}" (shape input) (at 76.2 73.66 180) (fields_autoplaced)
     (effects (font (size 1.27 1.27)) (justify right))
@@
     (effects (font (size 1.27 1.27)) (justify left))
   )
+  (hierarchical_label "PCLK" (shape input) (at 73.66 116.84 180) (fields_autoplaced)
+    (effects (font (size 1.27 1.27)) (justify right))
+  )
   (hierarchical_label "D[0..31]" (shape bidirectional) (at 187.96 45.72 0) (fields_autoplaced)
     (effects (font (size 1.27 1.27)) (justify left))
@@
   (hierarchical_label "TT[0..1]" (shape bidirectional) (at 215.9 15.24 0) (fields_autoplaced)
     (effects (font (size 1.27 1.27)) (justify left))
+  )
+  (hierarchical_label "BCLK" (shape input) (at 73.66 119.38 180) (fields_autoplaced)
+    (effects (font (size 1.27 1.27)) (justify right))
   )
   (hierarchical_label "~{IPL[0..2]}" (shape input) (at 68.58 63.5 180) (fields_autoplaced)
@@
   (symbol (lib_id "Device:R_Small_US") (at 106.68 25.4 0) (unit 1)
     (in_bom yes) (on_board yes) (dnp no) (fields_autoplaced)
-    (property "Reference" "R?" (at 109.22 24.13 0)
+    (property "Reference" "R18" (at 109.22 24.13 0)
       (effects (font (size 1.27 1.27)) (justify left))
     )
@@
       (project "68040pc"
         (path "/3006deba-2100-40f8-9f39-987a5c2c14c7/2a622311-cc5c-4b5f-b457-4d52db73c27a"
-          (reference "R?") (unit 1)
+          (reference "R18") (unit 1)
         )
       )
@@
   (symbol (lib_id "Device:R_Small_US") (at 76.2 25.4 0) (unit 1)
     (in_bom yes) (on_board yes) (dnp no) (fields_autoplaced)
-    (property "Reference" "R?" (at 78.74 24.13 0)
+    (property "Reference" "R14" (at 78.74 24.13 0)
       (effects (font (size 1.27 1.27)) (justify left))
     )
@@
       (project "68040pc"
         (path "/3006deba-2100-40f8-9f39-987a5c2c14c7/2a622311-cc5c-4b5f-b457-4d52db73c27a"
-          (reference "R?") (unit 1)
+          (reference "R14") (unit 1)
         )
       )
@@
   (symbol (lib_id "Device:R_Small_US") (at 45.72 25.4 0) (unit 1)
     (in_bom yes) (on_board yes) (dnp no) (fields_autoplaced)
-    (property "Reference" "R?" (at 48.26 24.13 0)
+    (property "Reference" "R10" (at 48.26 24.13 0)
       (effects (font (size 1.27 1.27)) (justify left))
     )
@@
       (project "68040pc"
         (path "/3006deba-2100-40f8-9f39-987a5c2c14c7/2a622311-cc5c-4b5f-b457-4d52db73c27a"
-          (reference "R?") (unit 1)
+          (reference "R10") (unit 1)
         )
       )
@@
   (symbol (lib_id "Device:R_Small_US") (at 53.34 25.4 0) (unit 1)
     (in_bom yes) (on_board yes) (dnp no) (fields_autoplaced)
-    (property "Reference" "R?" (at 55.88 24.13 0)
+    (property "Reference" "R11" (at 55.88 24.13 0)
       (effects (font (size 1.27 1.27)) (justify left))
     )
@@
       (project "68040pc"
         (path "/3006deba-2100-40f8-9f39-987a5c2c14c7/2a622311-cc5c-4b5f-b457-4d52db73c27a"
-          (reference "R?") (unit 1)
+          (reference "R11") (unit 1)
         )
       )
@@
   (symbol (lib_id "Device:R_Small_US") (at 83.82 25.4 0) (unit 1)
     (in_bom yes) (on_board yes) (dnp no) (fields_autoplaced)
-    (property "Reference" "R?" (at 86.36 24.13 0)
+    (property "Reference" "R15" (at 86.36 24.13 0)
       (effects (font (size 1.27 1.27)) (justify left))
     )
@@
       (project "68040pc"
         (path "/3006deba-2100-40f8-9f39-987a5c2c14c7/2a622311-cc5c-4b5f-b457-4d52db73c27a"
-          (reference "R?") (unit 1)
+          (reference "R15") (unit 1)
         )
       )
@@
   (symbol (lib_id "Device:R_Small_US") (at 60.96 25.4 0) (unit 1)
     (in_bom yes) (on_board yes) (dnp no) (fields_autoplaced)
-    (property "Reference" "R?" (at 63.5 24.13 0)
+    (property "Reference" "R12" (at 63.5 24.13 0)
       (effects (font (size 1.27 1.27)) (justify left))
     )
@@
       (project "68040pc"
         (path "/3006deba-2100-40f8-9f39-987a5c2c14c7/2a622311-cc5c-4b5f-b457-4d52db73c27a"
-          (reference "R?") (unit 1)
+          (reference "R12") (unit 1)
         )
       )
@@
   (symbol (lib_id "Device:R_Small_US") (at 200.66 25.4 0) (unit 1)
     (in_bom yes) (on_board yes) (dnp no) (fields_autoplaced)
-    (property "Reference" "R?" (at 203.2 24.13 0)
+    (property "Reference" "R23" (at 203.2 24.13 0)
       (effects (font (size 1.27 1.27)) (justify left))
     )
@@
       (project "68040pc"
         (path "/3006deba-2100-40f8-9f39-987a5c2c14c7/2a622311-cc5c-4b5f-b457-4d52db73c27a"
-          (reference "R?") (unit 1)
+          (reference "R23") (unit 1)
         )
       )
@@
   (symbol (lib_id "Device:R_Small_US") (at 114.3 25.4 0) (unit 1)
     (in_bom yes) (on_board yes) (dnp no) (fields_autoplaced)
-    (property "Reference" "R?" (at 116.84 24.13 0)
+    (property "Reference" "R19" (at 116.84 24.13 0)
       (effects (font (size 1.27 1.27)) (justify left))
     )
@@
       (project "68040pc"
         (path "/3006deba-2100-40f8-9f39-987a5c2c14c7/2a622311-cc5c-4b5f-b457-4d52db73c27a"
-          (reference "R?") (unit 1)
+          (reference "R19") (unit 1)
         )
       )
@@
   (symbol (lib_id "Device:R_Small_US") (at 121.92 25.4 0) (unit 1)
     (in_bom yes) (on_board yes) (dnp no) (fields_autoplaced)
-    (property "Reference" "R?" (at 124.46 24.13 0)
+    (property "Reference" "R20" (at 124.46 24.13 0)
       (effects (font (size 1.27 1.27)) (justify left))
     )
@@
       (project "68040pc"
         (path "/3006deba-2100-40f8-9f39-987a5c2c14c7/2a622311-cc5c-4b5f-b457-4d52db73c27a"
-          (reference "R?") (unit 1)
+          (reference "R20") (unit 1)
         )
       )
@@
   (symbol (lib_id "Device:R_Small_US") (at 193.04 25.4 0) (unit 1)
     (in_bom yes) (on_board yes) (dnp no) (fields_autoplaced)
-    (property "Reference" "R?" (at 195.58 24.13 0)
+    (property "Reference" "R22" (at 195.58 24.13 0)
       (effects (font (size 1.27 1.27)) (justify left))
     )
@@
       (project "68040pc"
         (path "/3006deba-2100-40f8-9f39-987a5c2c14c7/2a622311-cc5c-4b5f-b457-4d52db73c27a"
-          (reference "R?") (unit 1)
+          (reference "R22") (unit 1)
         )
       )
@@
   (symbol (lib_id "Device:R_Small_US") (at 91.44 25.4 0) (unit 1)
     (in_bom yes) (on_board yes) (dnp no) (fields_autoplaced)
-    (property "Reference" "R?" (at 93.98 24.13 0)
+    (property "Reference" "R16" (at 93.98 24.13 0)
       (effects (font (size 1.27 1.27)) (justify left))
     )
@@
       (project "68040pc"
         (path "/3006deba-2100-40f8-9f39-987a5c2c14c7/2a622311-cc5c-4b5f-b457-4d52db73c27a"
-          (reference "R?") (unit 1)
+          (reference "R16") (unit 1)
         )
       )
@@
   (symbol (lib_id "Device:R_Small_US") (at 68.58 25.4 0) (unit 1)
     (in_bom yes) (on_board yes) (dnp no) (fields_autoplaced)
-    (property "Reference" "R?" (at 71.12 24.13 0)
+    (property "Reference" "R13" (at 71.12 24.13 0)
       (effects (font (size 1.27 1.27)) (justify left))
     )
@@
       (project "68040pc"
         (path "/3006deba-2100-40f8-9f39-987a5c2c14c7/2a622311-cc5c-4b5f-b457-4d52db73c27a"
-          (reference "R?") (unit 1)
+          (reference "R13") (unit 1)
         )
       )
@@
   (symbol (lib_id "Device:R_Small_US") (at 129.54 25.4 0) (unit 1)
     (in_bom yes) (on_board yes) (dnp no) (fields_autoplaced)
-    (property "Reference" "R?" (at 132.08 24.13 0)
+    (property "Reference" "R21" (at 132.08 24.13 0)
       (effects (font (size 1.27 1.27)) (justify left))
     )
@@
       (project "68040pc"
         (path "/3006deba-2100-40f8-9f39-987a5c2c14c7/2a622311-cc5c-4b5f-b457-4d52db73c27a"
-          (reference "R?") (unit 1)
+          (reference "R21") (unit 1)
         )
       )
@@
   (symbol (lib_id "Device:R_Small_US") (at 99.06 25.4 0) (unit 1)
     (in_bom yes) (on_board yes) (dnp no) (fields_autoplaced)
-    (property "Reference" "R?" (at 101.6 24.13 0)
+    (property "Reference" "R17" (at 101.6 24.13 0)
       (effects (font (size 1.27 1.27)) (justify left))
     )
@@
       (project "68040pc"
         (path "/3006deba-2100-40f8-9f39-987a5c2c14c7/2a622311-cc5c-4b5f-b457-4d52db73c27a"
-          (reference "R?") (unit 1)
-        )
-      )
+          (reference "R17") (unit 1)
+        )
+      )
