File: hardware/68040pc.kicad_sch (KiCad schematic)
At the start: 6 parts, among them U1 68LC040, U23 PCF8584, U8 LTC6905xS5-133

Commit message: begin work on a simpler first draft board
Parts:
- removed U8: LTC6905xS5-133, Package_TO_SOT_SMD:TSOT-23-5, symbol Oscillator:LTC6905xS5-133
Other:
- added sheet FPGA (fpga.kicad_sch)
- sheet Memory ports: added DRAM_A[0..11], DRAM_R/~{W}, PD_{A}[1..4], ~{CAS_A[0..3]}, ~{RAS[0..3]}; removed A[0..31]
- moved on the sheet: R4, R5, U23

Commit message: updates
Parts:
- removed U1: 68LC040, 68040:PGA179, symbol 68040:68LC040
Other:
- added sheet Processor (processor.kicad_sch)
- added sheet SRAM (sram.kicad_sch)
- moved on the sheet: R4, R5, U23, U24

Commit message: update cpu symbol, topology
Connections:
- net D0: no longer U23.7 (D0)
- net D1: no longer U23.8 (D1)
- net D2: no longer U23.9 (D2)
- net D3: no longer U23.11 (D3)
- net D4: no longer U23.12 (D4)
- net D5: no longer U23.13 (D5)
- net D6: no longer U23.14 (D6)
- net D7: no longer U23.15 (D7)
- net +3.3V: now reaches R4.1
- net +3.3V: now also R5.1
- net PD16: now reaches U24.36 (PD16)
- net PD17: now reaches U24.37 (PD17)
- net PD18: now reaches U24.38 (PD18)
- net PD19: now reaches U24.39 (PD19)
- net PD20: now reaches U24.40 (PD20)
- net PD21: now reaches U24.41 (PD21)
- net PD22: now reaches U24.42 (PD22)
- net PD23: now reaches U24.43 (PD23)
- net PD24: now reaches U24.44 (PD24)
- net PD24: now also U23.7 (D0)
- net PD25: now reaches U24.45 (PD25)
- net PD25: now also U23.8 (D1)
- net PD26: now reaches U24.46 (PD26)
- net PD26: now also U23.9 (D2)
- net PD27: now reaches U24.47 (PD27)
- net PD27: now also U23.11 (D3)
- net PD28: now reaches U24.48 (PD28)
- net PD28: now also U23.12 (D4)
- net PD29: now reaches U24.49 (PD29)
- net PD29: now also U23.13 (D5)
- net PD30: now reaches U24.50 (PD30)
- net PD30: now also U23.14 (D6)
- net PD31: now reaches U24.51 (PD31)
- net PD31: now also U23.15 (D7)
Other:
- added sheet CPLD (cpld.kicad_sch)
- sheet FPGA ports: added none; removed DRAM_A[0..11], PD_{A}[1..4], ~{CAS_A[0..3]}, ~{RAS[0..3]}
- sheet Memory ports: added DRAM_BUF_DIR, DRAM_BUF_~{OE}; removed none
- sheet Processor ports: added IPL[0..2], PST[0..3], SC[0..1], ~{AVEC}, ~{LOCKE}, ~{LOCK}, ~{TA}, ~{TCI}/~{TBI}, ~{TEA}, ~{TIP}, ~{TS}; removed TLN[0..1], UPA[0..1]
- moved on the sheet: R5

Commit message: add interrupt logic, clean up modules
Parts:
- added C20: .01uF, symbol Device:C
- added C4: .1uF, symbol Device:C
- added U27: NB3N502, Package_SO:SOIC-8_3.9x4.9mm_P1.27mm, symbol 68040:NB3N502
- added U8: SN74ALVC164245, Package_SO:TSSOP-48_6.1x12.5mm_P0.5mm, symbol 68040:SN74ALVC164245
- added X1: 33MHz, Oscillator:Oscillator_DIP-8, symbol Oscillator:CXO_DIP8
Connections:
- net +3.3V: now also C20.1, C4.1, U27.2 (VDD), X1.1 (EN), X1.8 (Vcc)
- net BCLK: now also U27.4 (REF)
- net GND: now also C4.2, X1.4 (GND)
- net PCLK: now also U27.5 (CLKOUT)
- net ~{I2C_IACK}: now reaches U23.4 (~{IACK})
- net ~{I2C_IRQ}: now reaches U23.5 (~{INT})
- new net: U27.1 (X1/CLK), X1.5 (OUT)
- new net: C20.2, U27.3 (GND), U27.6 (S0), U27.7 (S1)
- no-connect marks 0 -> 1
Other:
- added sheet Interrupts (interrupts.kicad_sch)
- added sheet KbdMou (kbdmou.kicad_sch)
- sheet CPLD ports: added A[0..29], CLK, DRAM_A[0..11], DRAM_BUF_DIR, R/~{W}, SIZ[0..1], ~{CAS_A[0..3]}, ~{CAS_B[0..3]}, ~{CAS_C[0..3]}, ~{CAS_D[0..3]}, ~{DRAM_BUF_OE}, ~{DRAM_CS}, ~{MI}, ~{RAS[0..3]}, ~{RESET}, ~{TA}, ~{TS}; removed none
- sheet FPGA ports: added SC[0..1], ~{040_BG}, ~{040_BR}, ~{040_TCI}/~{040_TBI}, ~{68150_CS}, ~{DRAM_CS}, ~{DUART_CS}, ~{IDE_CS}, ~{PS/2_CS}, ~{SRAM_CS}, ~{TA}, ~{TEA}; removed PCLK
- sheet IO ports: added A[2..3], PA[0..1], PD[24..31], ~{CS}, ~{DTACK}, ~{IACK}, ~{IRQ}, ~{RESET}, ~{SWE}; removed none
- sheet Memory ports: added ~{CAS_B[0..3]}, ~{CAS_C[0..3]}, ~{CAS_D[0..3]}; removed PD_{A}[1..4]
- sheet Power ports: added PWR_GOOD; removed none
- sheet Processor ports: added ~{BB}, ~{BG}, ~{BR}, ~{IPL[0..2]}, ~{MI}, ~{RSTI}, ~{RSTO}; removed IPL[0..2]
- sheet SRAM ports: added A[2..19], PA1, PD[16..31], ~{LWE}, ~{UWE}; removed A[0..18], D[0..16], ~{WE}
- note added: "TT[0..1] = $3 means Acknowledge access, TM[0..2] then give interrupt level being acknowledged."

Commit message: updates
Parts:
- added C22 (x2), C23 (x2), C24 (x2), C25 (x2): 100nF, symbol Device:C
- added C? (x3): .1uF, symbol Device:C
- added R?: 4.7k, symbol Device:R_Small_US
- added U15, U16, U17, U18: SN74ALVC164245, Package_SO:TSSOP-48_6.1x12.5mm_P0.5mm, symbol 68040:SN74ALVC164245
- added X?: ASE-xxxMHz, Oscillator:Oscillator_SMD_Abracon_ASE-4Pin_3.2x2.5mm, symbol Oscillator:ASE-xxxMHz
Connections:
- net ~{I2C_DTACK} is gone; now on net ~{DSACK0}: U23.16 (~{RD})
- net +3.3V: now also C?.1, X?.1 (EN), X?.4 (Vdd); no longer R4.1, R5.1
- net +5V: now also R4.1, R5.1, U8.18 (VCCB), U8.7 (VCCB), C22.1, C22.1, C23.1, C23.1, C?.1, C?.1, U17.18 (VCCB), U17.7 (VCCB), U18.18 (VCCB), U18.7 (VCCB)
- net A0: now also U15.2 (1B1)
- net A1: now also U15.3 (1B2)
- net GND: now also U8.10 (GND), U8.15 (GND), U8.21 (GND), U8.28 (GND), U8.34 (GND), U8.39 (GND), U8.4 (GND), U8.45 (GND), C22.2, C22.2, C23.2, C23.2, C24.2, C24.2, C25.2, C25.2, C?.2, C?.2, C?.2, U17.10 (GND), U17.15 (GND), U17.21 (GND), U17.28 (GND), U17.34 (GND), U17.39 (GND), U17.4 (GND), U17.45 (GND), U18.10 (GND), U18.15 (GND), U18.21 (GND), U18.28 (GND), U18.34 (GND), U18.39 (GND), U18.4 (GND), U18.45 (GND), X?.2 (GND)
- net R/~{W}: now also U8.8 (1B5)
- net SIZ0: now also U8.2 (1B1)
- net SIZ1: now also U8.3 (1B2)
- net at U8.1 (1DIR): now also U8.24 (2DIR), U8.25 (*2OE), U8.48 (*1OE), R?.2
- net LV_R/~{W}: now reaches U8.41 (1A5)
- net LV_~{MI}: now reaches U8.43 (1A4)
- net LV_~{TS}: now reaches U8.44 (1A3)
- net LV_SIZ1: now reaches U8.46 (1A2)
- net LV_SIZ0: now reaches U8.47 (1A1)
- net ~{TS}: now reaches U8.5 (1B3)
- net ~{MI}: now reaches U8.6 (1B4)
- net at U23.1 (CLK): now also X?.3 (OUT)
- net +3V3: now reaches U8.31 (VCCA)
- net +3V3: now also U8.42 (VCCA), C24.1, C24.1, C25.1, C25.1, R?.1, U17.31 (VCCA), U17.42 (VCCA), U18.31 (VCCA), U18.42 (VCCA)
- new net A10: U15.16 (2B3)
- new net A11: U15.17 (2B4)
- new net A12: U15.19 (2B5)
- new net A13: U15.20 (2B6)
- new net A14: U15.22 (2B7)
- new net A15: U15.23 (2B8)
- new net A16: U16.23 (2B8)
- new net A17: U16.22 (2B7)
- new net A18: U16.20 (2B6)
- new net A19: U16.19 (2B5)
- new net A2: U15.5 (1B3)
- new net A20: U16.17 (2B4)
- new net A21: U16.16 (2B3)
- new net A22: U16.14 (2B2)
- new net A23: U16.13 (2B1)
- new net A24: U16.12 (1B8)
- new net A25: U16.11 (1B7)
- new net A26: U16.9 (1B6)
- new net A27: U16.8 (1B5)
- new net A28: U16.6 (1B4)
- new net A29: U16.5 (1B3)
- new net A3: U15.6 (1B4)
- new net A30: U16.3 (1B2)
- new net A31: U16.2 (1B1)
- new net A4: U15.8 (1B5)
- new net A5: U15.9 (1B6)
- new net A6: U15.11 (1B7)
- new net A7: U15.12 (1B8)
- new net A8: U15.13 (2B1)
- new net A9: U15.14 (2B2)
- new net LV.A0: U15.47 (1A1)
- new net LV.A1: U15.46 (1A2)
- new net LV.A10: U15.33 (2A3)
- new net LV.A11: U15.32 (2A4)
- new net LV.A12: U15.30 (2A5)
- new net LV.A13: U15.29 (2A6)
- new net LV.A14: U15.27 (2A7)
- new net LV.A15: U15.26 (2A8)
- new net LV.A16: U16.26 (2A8)
- new net LV.A17: U16.27 (2A7)
- new net LV.A18: U16.29 (2A6)
- new net LV.A19: U16.30 (2A5)
- new net LV.A2: U15.44 (1A3)
- new net LV.A20: U16.32 (2A4)
- new net LV.A21: U16.33 (2A3)
- new net LV.A22: U16.35 (2A2)
- new net LV.A23: U16.36 (2A1)
- new net LV.A24: U16.37 (1A8)
- new net LV.A25: U16.38 (1A7)
- new net LV.A26: U16.40 (1A6)
- new net LV.A27: U16.41 (1A5)
- new net LV.A28: U16.43 (1A4)
- new net LV.A29: U16.44 (1A3)
- new net LV.A3: U15.43 (1A4)
- new net LV.A30: U16.46 (1A2)
- new net LV.A31: U16.47 (1A1)
- new net LV.A4: U15.41 (1A5)
- new net LV.A5: U15.40 (1A6)
- new net LV.A6: U15.38 (1A7)
- new net LV.A7: U15.37 (1A8)
- new net LV.A8: U15.36 (2A1)
- new net LV.A9: U15.35 (2A2)
- new net LV_A_DIR: U15.1 (1DIR), U15.24 (2DIR), U16.1 (1DIR), U16.24 (2DIR)
- new net ~{LV_A_OE}: U15.25 (*2OE), U15.48 (*1OE), U16.25 (*2OE), U16.48 (*1OE)
Other:
- sheet CPLD ports: added {ABUS}; removed A[0..29]
- sheet FPGA ports: added ~{AVEC}, ~{DSACK[0..1]}; removed none
- sheet Interrupts ports: added ~{NMIACK}, ~{NMI}; removed ~{IACK7}, ~{IRQ7}
- moved on the sheet: U8A, U8B

Commit message: getting closer
Parts:
- added X2: ASE-12MHz, Oscillator:Oscillator_SMD_Abracon_ASE-4Pin_3.2x2.5mm, symbol Oscillator:ASE-xxxMHz
- added X3: 33MHz, Oscillator:Oscillator_DIP-14, symbol Oscillator:CXO_DIP8
- X4: renamed from X?; value ASE-xxxMHz -> ASE-12MHz
- gave numbers to parts that had none: 4
Connections:
- net +3.3V: now also C24.1, C25.1, U17.31 (VCCA), U17.42 (VCCA), X2.1 (EN), X2.4 (Vdd), X3.1 (EN), X3.8 (Vcc)
- net +3V3: no longer C24.1, C25.1, U17.31 (VCCA), U17.42 (VCCA)
- net GND: now also X2.2 (GND), X3.4 (GND)
- net ~{LOCKE}: now reaches U8.11 (1B7)
- net LV_~{LOCKE}: now reaches U8.38 (1A7)
- net LV_~{LOCK}: now reaches U8.40 (1A6)
- net ~{LOCK}: now reaches U8.9 (1B6)
- net at U27.1 (X1/CLK), X1.5 (OUT): now also X2.3 (OUT), X3.5 (OUT)
- net ~{SYS_RST}: now reaches U23.19 (~{RST})
Other:
- added sheet CF Card (cf.kicad_sch)
- sheet CPLD ports: added none; removed DRAM_BUF_DIR
- sheet FPGA ports: added LV{ABUS}, ~{LOCKE}, ~{LOCK}; removed A[0..31]
- sheet Memory ports: added none; removed DRAM_BUF_DIR
- sheet Processor ports: added none; removed PST[0..3]
- note added: "Only populate one"
- note added: "TT[0..1] = $3 means Acknowledge access, TM[0..2] then gives interrupt level being acknowledged."
- note removed: "TT[0..1] = $3 means Acknowledge access, TM[0..2] then give interrupt level being acknowledged."

Commit message: re-design level shifters
Parts:
- removed C20: .01uF, symbol Device:C
- removed C22 (x2), C23 (x2), C24 (x2), C25 (x2): 100nF, symbol Device:C
- removed C4: .1uF, symbol Device:C
- removed R9: 4.7k, symbol Device:R_Small_US
- removed U15, U16, U17, U18, U8: SN74ALVC164245, Package_SO:TSSOP-48_6.1x12.5mm_P0.5mm, symbol 68040:SN74ALVC164245
- removed U27: NB3N502, Package_SO:SOIC-8_3.9x4.9mm_P1.27mm, symbol 68040:NB3N502
- removed X1: 33MHz, Oscillator:Oscillator_DIP-8, symbol Oscillator:CXO_DIP8
- removed X2: ASE-12MHz, Oscillator:Oscillator_SMD_Abracon_ASE-4Pin_3.2x2.5mm, symbol Oscillator:ASE-xxxMHz
- removed X3: 33MHz, Oscillator:Oscillator_DIP-14, symbol Oscillator:CXO_DIP8
- added C22: 100nF, symbol Device:C
- added U33: 74LVC1G04, symbol 74xGxx:74LVC1G04
Connections:
- net +5V: now also C22.1, U33.5 (VCC)
- net GND: now also C22.2, U33.3 (GND)
- net R/~{W}: now also U33.2
- net ~{DSACK0}: now also U24.28 (~{DSACK0}); no longer U24.29 (~{DSACK1})
- net ~{DSACK1}: now also U24.29 (~{DSACK1}); no longer U24.28 (~{DSACK0})
- new net ~{R}/W: U33.4
- no-connect marks 1 -> 0
Other:
- added sheet Clock (clock.kicad_sch)
- sheet FPGA ports: added A[0..31], PA[0..1], PD[24..31], SIZ[0..1], ~{68150_DS}, ~{TS}; removed D[0..31], LV{ABUS}
- note added: "Higher Priority"
- note removed: "Only populate one"
