File: hardware/slots.kicad_sch (KiCad schematic)
At the start: 0 parts

Commit message: updates
Parts:
- added RN1, RN2: R_Network04_US, Resistor_THT:R_Array_SIP5, symbol Device:R_Network04_US
- added U11, U12, U13, U14: 74HC245, Package_SO:SOIC-20W_7.5x12.8mm_P1.27mm, symbol 74xx:74HC245
- added U6, U7: 74LS32, Package_SO:SOIC-14_3.9x8.7mm_P1.27mm, symbol 74xx:74LS32
Connections:
- new net +5V: U11.20 (VCC), U12.20 (VCC), U13.20 (VCC), U14.20 (VCC), U6.14 (VCC), U7.14 (VCC)
- new net A0: U11.2 (A0)
- new net A1: U11.3 (A1)
- new net A10: U12.4 (A2)
- new net A11: U12.5 (A3)
- new net A12: U12.6 (A4)
- new net A13: U12.7 (A5)
- new net A14: U12.8 (A6)
- new net A15: U12.9 (A7)
- new net A16: U13.2 (A0)
- new net A17: U13.3 (A1)
- new net A18: U13.4 (A2)
- new net A19: U13.5 (A3)
- new net A2: U11.4 (A2)
- new net A20: U13.6 (A4)
- new net A21: U13.7 (A5)
- new net A22: U13.8 (A6)
- new net A23: U13.9 (A7)
- new net A24: U14.2 (A0)
- new net A25: U14.3 (A1)
- new net A26: U14.4 (A2)
- new net A27: U14.5 (A3)
- new net A28: U14.6 (A4)
- new net A29: U14.7 (A5)
- new net A3: U11.5 (A3)
- new net A30: U14.8 (A6)
- new net A31: U14.9 (A7)
- new net A4: U11.6 (A4)
- new net A5: U11.7 (A5)
- new net A6: U11.8 (A6)
- new net A7: U11.9 (A7)
- new net A8: U12.2 (A0)
- new net A9: U12.3 (A1)
- new net EXA0: U11.18 (B0)
- new net EXA1: U11.17 (B1)
- new net EXA10: U12.16 (B2)
- new net EXA11: U12.15 (B3)
- new net EXA12: U12.14 (B4)
- new net EXA13: U12.13 (B5)
- new net EXA14: U12.12 (B6)
- new net EXA15: U12.11 (B7)
- new net EXA16: U13.18 (B0)
- new net EXA17: U13.17 (B1)
- new net EXA18: U13.16 (B2)
- new net EXA19: U13.15 (B3)
- new net EXA2: U11.16 (B2)
- new net EXA20: U13.14 (B4)
- new net EXA21: U13.13 (B5)
- new net EXA22: U13.12 (B6)
- new net EXA23: U13.11 (B7)
- new net EXA24: U14.18 (B0)
- new net EXA25: U14.17 (B1)
- new net EXA26: U14.16 (B2)
- new net EXA27: U14.15 (B3)
- new net EXA28: U14.14 (B4)
- new net EXA29: U14.13 (B5)
- new net EXA3: U11.15 (B3)
- new net EXA30: U14.12 (B6)
- new net EXA31: U14.11 (B7)
- new net EXA4: U11.14 (B4)
- new net EXA5: U11.13 (B5)
- new net EXA6: U11.12 (B6)
- new net EXA7: U11.11 (B7)
- new net EXA8: U12.18 (B0)
- new net EXA9: U12.17 (B1)
- new net EXDIR: U11.1 (A->B), U12.1 (A->B), U13.1 (A->B), U14.1 (A->B)
- new net ExpansionSlot1/~{CFG_{IN}}: U6.1
- new net ExpansionSlot1/~{CFG_{OUT}}: RN1.5 (R4), U6.2
- new net ExpansionSlot2/~{CFG_{IN}}: U6.3, U6.4
- new net ExpansionSlot2/~{CFG_{OUT}}: RN1.4 (R3), U6.5
- new net ExpansionSlot3/~{CFG_{IN}}: U6.6, U6.9
- new net ExpansionSlot3/~{CFG_{OUT}}: RN1.3 (R2), U6.10
- new net ExpansionSlot4/~{CFG_{IN}}: U6.12, U6.8
- new net ExpansionSlot4/~{CFG_{OUT}}: RN1.2 (R1), U6.13
- new net ExpansionSlot5/~{CFG_{IN}}: U6.11, U7.1
- new net ExpansionSlot5/~{CFG_{OUT}}: RN2.5 (R4), U7.2
- new net ExpansionSlot6/~{CFG_{IN}}: U7.3, U7.4
- new net ExpansionSlot6/~{CFG_{OUT}}: RN2.4 (R3), U7.5
- new net ExpansionSlot7/~{CFG_{IN}}: U7.6, U7.9
- new net ExpansionSlot7/~{CFG_{OUT}}: RN2.3 (R2), U7.10
- new net ExpansionSlot8/~{CFG_{IN}}: U7.12, U7.8
- new net ExpansionSlot8/~{CFG_{OUT}}: RN2.2 (R1), U7.13
- new net GND: RN1.1 (common), RN2.1 (common), U11.10 (GND), U12.10 (GND), U13.10 (GND), U14.10 (GND), U6.7 (GND), U7.7 (GND)
- new net ~{EXP_OE}: U11.19 (CE), U12.19 (CE), U13.19 (CE), U14.19 (CE)
Other:
- sheet ExpansionSlot1 ports: added ~{CFG_{IN}}, ~{CFG_{OUT}}; removed none
- sheet ExpansionSlot2 ports: added ~{CFG_{IN}}, ~{CFG_{OUT}}; removed none
- sheet ExpansionSlot3 ports: added ~{CFG_{IN}}, ~{CFG_{OUT}}; removed none
- sheet ExpansionSlot4 ports: added ~{CFG_{IN}}, ~{CFG_{OUT}}; removed none
- sheet ExpansionSlot5 ports: added ~{CFG_{IN}}, ~{CFG_{OUT}}; removed none
- sheet ExpansionSlot6 ports: added ~{CFG_{IN}}, ~{CFG_{OUT}}; removed none
- sheet ExpansionSlot7 ports: added ~{CFG_{IN}}, ~{CFG_{OUT}}; removed none
- sheet ExpansionSlot8 ports: added ~{CFG_{IN}}, ~{CFG_{OUT}}; removed none

Commit message: updates
Other:
- sheet ExpansionSlot1 ports: added EXA[0..31], EXD[0..31]; removed A[0..31], D[0..31]
Changed lines of the file:
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@@
+    (stroke (width 0) (type default))
+  )
+  (bus (pts (xy 27.94 25.4) (xy 38.1 25.4))
     (stroke (width 0) (type default))
   )
@@
   (label "A3" (at 302.26 35.56 0) (fields_autoplaced)
     (effects (font (size 1.27 1.27)) (justify left bottom))
+  )
+  (label "EXA[0..31]" (at 27.94 25.4 180) (fields_autoplaced)
+    (effects (font (size 1.27 1.27)) (justify right bottom))
   )
   (label "EXA2" (at 342.9 33.02 180) (fields_autoplaced)
@@
       (effects (font (size 1.27 1.27)) (justify left top))
     )
-    (pin "D[0..31]" bidirectional (at 38.1 25.4 180)
-      (effects (font (size 1.27 1.27)) (justify left))
-    )
-    (pin "A[0..31]" bidirectional (at 38.1 22.86 180)
-      (effects (font (size 1.27 1.27)) (justify left))
-    )
     (pin "~{CFG_{IN}}" input (at 38.1 27.94 180)
       (effects (font (size 1.27 1.27)) (justify left))
@@
       (effects (font (size 1.27 1.27)) (justify right))
     )
-    (instances
+    (pin "EXD[0..31]" bidirectional (at 38.1 22.86 180)
+      (effects (font (size 1.27 1.27)) (justify left))
+    )
+    (pin "EXA[0..31]" bidirectional (at 38.1 25.4 180)
+      (effects (font (size 1.27 1.27)) (justify left))
+    )
+    (instances

Commit message: updates
Parts:
- added U19, U20, U21, U22: 74HC245, Package_SO:SOIC-20W_7.5x12.8mm_P1.27mm, symbol 74xx:74HC245
Connections:
- net +5V: now also U19.20 (VCC), U20.20 (VCC), U21.20 (VCC), U22.20 (VCC)
- net GND: now also U19.10 (GND), U20.10 (GND), U21.10 (GND), U22.10 (GND)
- net ~{EXP_OE}: now also U19.19 (CE), U20.19 (CE), U21.19 (CE), U22.19 (CE)
- new net D0: U19.2 (A0)
- new net D1: U19.3 (A1)
- new net D10: U20.4 (A2)
- new net D11: U20.5 (A3)
- new net D12: U20.6 (A4)
- new net D13: U20.7 (A5)
- new net D14: U20.8 (A6)
- new net D15: U20.9 (A7)
- new net D16: U21.2 (A0)
- new net D17: U21.3 (A1)
- new net D18: U21.4 (A2)
- new net D19: U21.5 (A3)
- new net D2: U19.4 (A2)
- new net D20: U21.6 (A4)
- new net D21: U21.7 (A5)
- new net D22: U21.8 (A6)
- new net D23: U21.9 (A7)
- new net D24: U22.2 (A0)
- new net D25: U22.3 (A1)
- new net D26: U22.4 (A2)
- new net D27: U22.5 (A3)
- new net D28: U22.6 (A4)
- new net D29: U22.7 (A5)
- new net D3: U19.5 (A3)
- new net D30: U22.8 (A6)
- new net D31: U22.9 (A7)
- new net D4: U19.6 (A4)
- new net D5: U19.7 (A5)
- new net D6: U19.8 (A6)
- new net D7: U19.9 (A7)
- new net D8: U20.2 (A0)
- new net D9: U20.3 (A1)
- new net EXD0: U19.18 (B0)
- new net EXD1: U19.17 (B1)
- new net EXD10: U20.16 (B2)
- new net EXD11: U20.15 (B3)
- new net EXD12: U20.14 (B4)
- new net EXD13: U20.13 (B5)
- new net EXD14: U20.12 (B6)
- new net EXD15: U20.11 (B7)
- new net EXD16: U21.18 (B0)
- new net EXD17: U21.17 (B1)
- new net EXD18: U21.16 (B2)
- new net EXD19: U21.15 (B3)
- new net EXD2: U19.16 (B2)
- new net EXD20: U21.14 (B4)
- new net EXD21: U21.13 (B5)
- new net EXD22: U21.12 (B6)
- new net EXD23: U21.11 (B7)
- new net EXD24: U22.18 (B0)
- new net EXD25: U22.17 (B1)
- new net EXD26: U22.16 (B2)
- new net EXD27: U22.15 (B3)
- new net EXD28: U22.14 (B4)
- new net EXD29: U22.13 (B5)
- new net EXD3: U19.15 (B3)
- new net EXD30: U22.12 (B6)
- new net EXD31: U22.11 (B7)
- new net EXD4: U19.14 (B4)
- new net EXD5: U19.13 (B5)
- new net EXD6: U19.12 (B6)
- new net EXD7: U19.11 (B7)
- new net EXD8: U20.18 (B0)
- new net EXD9: U20.17 (B1)
Other:
- sheet ExpansionSlot2 ports: added EXA[0..31], EXD[0..31]; removed A[0..31], D[0..31]
- sheet ExpansionSlot3 ports: added EXA[0..31], EXD[0..31]; removed A[0..31], D[0..31]
- sheet ExpansionSlot4 ports: added EXA[0..31], EXD[0..31]; removed A[0..31], D[0..31]
- sheet ExpansionSlot5 ports: added EXA[0..31], EXD[0..31]; removed A[0..31], D[0..31]
- sheet ExpansionSlot6 ports: added EXA[0..31], EXD[0..31]; removed A[0..31], D[0..31]
- sheet ExpansionSlot7 ports: added EXA[0..31], EXD[0..31]; removed A[0..31], D[0..31]
- sheet ExpansionSlot8 ports: added EXA[0..31], EXD[0..31]; removed A[0..31], D[0..31]

Commit message: begin work on a simpler first draft board
Parts:
- removed RN2: R_Network04_US, Resistor_THT:R_Array_SIP5, symbol Device:R_Network04_US
- removed U7: 74LS32, Package_SO:SOIC-14_3.9x8.7mm_P1.27mm, symbol 74xx:74LS32
- renumbered U12 to U10, U20 to U11, U13 to U12, U21 to U13, U22 to U19, U11 to U6, U19 to U7, U6 to U9
Connections:
- net ExpansionSlot4/~{CFG_{IN}}: now also U9.13; no longer U9.12
- net ExpansionSlot4/~{CFG_{OUT}}: now also U9.12; no longer U9.13
- net ExpansionSlot5/~{CFG_{IN}}: no longer names the net of U9.11
Other:
- removed sheet ExpansionSlot5
- removed sheet ExpansionSlot6
- removed sheet ExpansionSlot7
- removed sheet ExpansionSlot8
- sheet ExpansionSlot1 ports: added R/~{W}, SIZ0, SIZ1, ~{B_{BUSY}}, ~{B_{GRANT}}, ~{B_{REQ}}, ~{IRQ}, ~{MI}, ~{TA}, ~{TBI}, ~{TCI}, ~{TEA}, ~{TS}; removed none
- sheet ExpansionSlot2 ports: added R/~{W}, SIZ0, SIZ1, ~{B_{BUSY}}, ~{B_{GRANT}}, ~{B_{REQ}}, ~{IRQ}, ~{MI}, ~{TA}, ~{TBI}, ~{TCI}, ~{TEA}, ~{TS}; removed none
- sheet ExpansionSlot3 ports: added R/~{W}, SIZ0, SIZ1, ~{B_{BUSY}}, ~{B_{GRANT}}, ~{B_{REQ}}, ~{IRQ}, ~{MI}, ~{TA}, ~{TBI}, ~{TCI}, ~{TEA}, ~{TS}; removed none
- sheet ExpansionSlot4 ports: added R/~{W}, SIZ0, SIZ1, ~{B_{BUSY}}, ~{B_{GRANT}}, ~{B_{REQ}}, ~{IRQ}, ~{MI}, ~{TA}, ~{TBI}, ~{TCI}, ~{TEA}, ~{TS}; removed none
- moved on the sheet: U9E

Commit message: add interrupt logic, clean up modules
Parts:
- added C? (x9): .1uF, symbol Device:C
Connections:
- net +5V: now also C?.1, C?.1, C?.1, C?.1, C?.1, C?.1, C?.1, C?.1, C?.1
- net GND: now also C?.2, C?.2, C?.2, C?.2, C?.2, C?.2, C?.2, C?.2, C?.2
- net EXD_DIR: now reaches U11.1 (A->B)
- net EXD_DIR: now also U13.1 (A->B), U19.1 (A->B), U7.1 (A->B)
- net EXDIR renamed EXA_DIR
- net ~{EXP_OE} renamed ~{EXA_OE}
- net ~{EXA_OE}: no longer U11.19 (CE), U13.19 (CE), U19.19 (CE), U7.19 (CE)
- new net ~{EXD_OE}: U11.19 (CE), U13.19 (CE), U19.19 (CE), U7.19 (CE)
Other:
- moved on the sheet: RN1, U10, U11, U12, U13, U14, U19, U6, U7, U9A, U9B, U9C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

Commit message: getting closer
Parts:
- gave numbers to parts that had none: 9
Changed lines of the file:
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@@
   (symbol (lib_id "Device:C") (at 43.18 257.81 0) (unit 1)
     (in_bom yes) (on_board yes) (dnp no) (fields_autoplaced)
-    (property "Reference" "C?" (at 46.99 256.54 0)
+    (property "Reference" "C48" (at 46.99 256.54 0)
       (effects (font (size 1.27 1.27)) (justify left))
     )
@@
       (project "68040pc"
         (path "/3006deba-2100-40f8-9f39-987a5c2c14c7/4c7887cb-c367-4b93-be02-0b485997fe7b"
-          (reference "C?") (unit 1)
+          (reference "C48") (unit 1)
         )
       )
@@
   (symbol (lib_id "Device:C") (at 93.98 257.81 0) (unit 1)
     (in_bom yes) (on_board yes) (dnp no) (fields_autoplaced)
-    (property "Reference" "C?" (at 97.79 256.54 0)
+    (property "Reference" "C52" (at 97.79 256.54 0)
       (effects (font (size 1.27 1.27)) (justify left))
     )
@@
       (project "68040pc"
         (path "/3006deba-2100-40f8-9f39-987a5c2c14c7/4c7887cb-c367-4b93-be02-0b485997fe7b"
-          (reference "C?") (unit 1)
+          (reference "C52") (unit 1)
         )
       )
@@
   (symbol (lib_id "Device:C") (at 55.88 257.81 0) (unit 1)
     (in_bom yes) (on_board yes) (dnp no) (fields_autoplaced)
-    (property "Reference" "C?" (at 59.69 256.54 0)
+    (property "Reference" "C49" (at 59.69 256.54 0)
       (effects (font (size 1.27 1.27)) (justify left))
     )
@@
       (project "68040pc"
         (path "/3006deba-2100-40f8-9f39-987a5c2c14c7/4c7887cb-c367-4b93-be02-0b485997fe7b"
-          (reference "C?") (unit 1)
+          (reference "C49") (unit 1)
         )
       )
@@
   (symbol (lib_id "Device:C") (at 68.58 257.81 0) (unit 1)
     (in_bom yes) (on_board yes) (dnp no) (fields_autoplaced)
-    (property "Reference" "C?" (at 72.39 256.54 0)
+    (property "Reference" "C50" (at 72.39 256.54 0)
       (effects (font (size 1.27 1.27)) (justify left))
     )
@@
       (project "68040pc"
         (path "/3006deba-2100-40f8-9f39-987a5c2c14c7/4c7887cb-c367-4b93-be02-0b485997fe7b"
-          (reference "C?") (unit 1)
+          (reference "C50") (unit 1)
         )
       )
@@
   (symbol (lib_id "Device:C") (at 81.28 257.81 0) (unit 1)
     (in_bom yes) (on_board yes) (dnp no) (fields_autoplaced)
-    (property "Reference" "C?" (at 85.09 256.54 0)
+    (property "Reference" "C51" (at 85.09 256.54 0)
       (effects (font (size 1.27 1.27)) (justify left))
     )
@@
       (project "68040pc"
         (path "/3006deba-2100-40f8-9f39-987a5c2c14c7/4c7887cb-c367-4b93-be02-0b485997fe7b"
-          (reference "C?") (unit 1)
+          (reference "C51") (unit 1)
         )
       )
@@
   (symbol (lib_id "Device:C") (at 320.04 143.51 0) (unit 1)
     (in_bom yes) (on_board yes) (dnp no) (fields_autoplaced)
-    (property "Reference" "C?" (at 323.85 142.24 0)
+    (property "Reference" "C47" (at 323.85 142.24 0)
       (effects (font (size 1.27 1.27)) (justify left))
     )
@@
       (project "68040pc"
         (path "/3006deba-2100-40f8-9f39-987a5c2c14c7/4c7887cb-c367-4b93-be02-0b485997fe7b"
-          (reference "C?") (unit 1)
+          (reference "C47") (unit 1)
         )
       )
@@
   (symbol (lib_id "Device:C") (at 132.08 257.81 0) (unit 1)
     (in_bom yes) (on_board yes) (dnp no) (fields_autoplaced)
-    (property "Reference" "C?" (at 135.89 256.54 0)
+    (property "Reference" "C55" (at 135.89 256.54 0)
       (effects (font (size 1.27 1.27)) (justify left))
     )
@@
       (project "68040pc"
         (path "/3006deba-2100-40f8-9f39-987a5c2c14c7/4c7887cb-c367-4b93-be02-0b485997fe7b"
-          (reference "C?") (unit 1)
+          (reference "C55") (unit 1)
         )
       )
@@
   (symbol (lib_id "Device:C") (at 106.68 257.81 0) (unit 1)
     (in_bom yes) (on_board yes) (dnp no) (fields_autoplaced)
-    (property "Reference" "C?" (at 110.49 256.54 0)
+    (property "Reference" "C53" (at 110.49 256.54 0)
       (effects (font (size 1.27 1.27)) (justify left))
     )
@@
       (project "68040pc"
         (path "/3006deba-2100-40f8-9f39-987a5c2c14c7/4c7887cb-c367-4b93-be02-0b485997fe7b"
-          (reference "C?") (unit 1)
+          (reference "C53") (unit 1)
         )
       )
@@
   (symbol (lib_id "Device:C") (at 119.38 257.81 0) (unit 1)
     (in_bom yes) (on_board yes) (dnp no) (fields_autoplaced)
-    (property "Reference" "C?" (at 123.19 256.54 0)
+    (property "Reference" "C54" (at 123.19 256.54 0)
       (effects (font (size 1.27 1.27)) (justify left))
     )
@@
       (project "68040pc"
         (path "/3006deba-2100-40f8-9f39-987a5c2c14c7/4c7887cb-c367-4b93-be02-0b485997fe7b"
-          (reference "C?") (unit 1)
-        )
-      )
+          (reference "C54") (unit 1)
+        )
+      )

Commit message: re-design level shifters
Connections:
- net ~{CFG_{OUT}}: now reaches U9.11
- net ExpansionSlot1/~{CFG_{IN}} renamed ~{CFG_{IN}}
Other:
- note added: "Use something other than LS logic"
- moved on the sheet: C47, U9E
Changed lines of the file:
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@@
   (junction (at 88.9 261.62) (diameter 0) (color 0 0 0 0)
   )
-  (junction (at 335.28 132.08) (diameter 0) (color 0 0 0 0)
+  (junction (at 373.38 88.9) (diameter 0) (color 0 0 0 0)
   )
   (junction (at 33.02 71.12) (diameter 0) (color 0 0 0 0)
@@
   (junction (at 33.02 124.46) (diameter 0) (color 0 0 0 0)
   )
-  (junction (at 335.28 157.48) (diameter 0) (color 0 0 0 0)
+  (junction (at 373.38 114.3) (diameter 0) (color 0 0 0 0)
   )
   (junction (at 99.06 73.66) (diameter 0) (color 0 0 0 0)
@@
   (junction (at 269.24 53.34) (diameter 0) (color 0 0 0 0)
   )
+  (junction (at 172.72 25.4) (diameter 0) (color 0 0 0 0)
+  )
   (junction (at 101.6 177.8) (diameter 0) (color 0 0 0 0)
   )
@@
     (stroke (width 0) (type default))
   )
-  (wire (pts (xy 320.04 132.08) (xy 320.04 139.7))
+  (wire (pts (xy 358.14 88.9) (xy 358.14 96.52))
     (stroke (width 0) (type default))
   )
@@
     (stroke (width 0) (type default))
   )
-  (wire (pts (xy 320.04 132.08) (xy 335.28 132.08))
+  (wire (pts (xy 358.14 88.9) (xy 373.38 88.9))
     (stroke (width 0) (type default))
   )
@@
     (stroke (width 0) (type default))
   )
+  (wire (pts (xy 170.18 25.4) (xy 172.72 25.4))
+    (stroke (width 0) (type default))
+  )
   (bus (pts (xy 152.4 157.48) (xy 152.4 160.02))
     (stroke (width 0) (type default))
@@
     (stroke (width 0) (type default))
   )
+  (wire (pts (xy 365.76 55.88) (xy 375.92 55.88))
+    (stroke (width 0) (type default))
+  )
   (bus (pts (xy 83.82 167.64) (xy 83.82 170.18))
     (stroke (width 0) (type default))
@@
     (stroke (width 0) (type default))
   )
-  (wire (pts (xy 320.04 157.48) (xy 335.28 157.48))
+  (wire (pts (xy 358.14 114.3) (xy 373.38 114.3))
     (stroke (width 0) (type default))
   )
@@
     (stroke (width 0) (type default))
   )
-  (wire (pts (xy 320.04 147.32) (xy 320.04 157.48))
+  (wire (pts (xy 358.14 104.14) (xy 358.14 114.3))
     (stroke (width 0) (type default))
   )
@@
   (bus (pts (xy 109.22 104.14) (xy 109.22 106.68))
     (stroke (width 0) (type default))
+  )
+  (text "Use something other\nthan LS logic" (at 375.92 91.44 0)
+    (effects (font (size 1.27 1.27)) (justify left bottom))
   )
   (label "A5" (at 40.64 60.96 0) (fields_autoplaced)
@@
     (effects (font (size 1.27 1.27)) (justify right))
   )
+  (hierarchical_label "~{CFG_{IN}}" (shape input) (at 170.18 25.4 180) (fields_autoplaced)
+    (effects (font (size 1.27 1.27)) (justify right))
+  )
   (hierarchical_label "A[0..31]" (shape bidirectional) (at 25.4 43.18 180) (fields_autoplaced)
     (effects (font (size 1.27 1.27)) (justify right))
@@
   (hierarchical_label "~{EXD_OE}" (shape input) (at 25.4 30.48 180) (fields_autoplaced)
     (effects (font (size 1.27 1.27)) (justify right))
+  )
+  (hierarchical_label "~{CFG_{OUT}}" (shape output) (at 375.92 55.88 0) (fields_autoplaced)
+    (effects (font (size 1.27 1.27)) (justify left))
   )
   (hierarchical_label "EXD_DIR" (shape input) (at 25.4 27.94 180) (fields_autoplaced)
@@
     )
   )
-  (symbol (lib_id "Device:C") (at 320.04 143.51 0) (unit 1)
+  (symbol (lib_id "Device:C") (at 358.14 100.33 0) (unit 1)
     (in_bom yes) (on_board yes) (dnp no) (fields_autoplaced)
-    (property "Reference" "C47" (at 323.85 142.24 0)
-      (effects (font (size 1.27 1.27)) (justify left))
-    )
-    (property "Value" ".1uF" (at 323.85 144.78 0)
-      (effects (font (size 1.27 1.27)) (justify left))
-    )
-    (property "Footprint" "" (at 321.0052 147.32 0)
-      (effects (font (size 1.27 1.27)) hide)
-    )
-    (property "Datasheet" "~" (at 320.04 143.51 0)
+    (property "Reference" "C47" (at 361.95 99.06 0)
+      (effects (font (size 1.27 1.27)) (justify left))
+    )
+    (property "Value" ".1uF" (at 361.95 101.6 0)
+      (effects (font (size 1.27 1.27)) (justify left))
+    )
+    (property "Footprint" "" (at 359.1052 104.14 0)
+      (effects (font (size 1.27 1.27)) hide)
+    )
+    (property "Datasheet" "~" (at 358.14 100.33 0)
       (effects (font (size 1.27 1.27)) hide)
     )
@@
     )
   )
-  (symbol (lib_id "power:GND") (at 335.28 157.48 0) (unit 1)
+  (symbol (lib_id "power:GND") (at 373.38 114.3 0) (unit 1)
     (in_bom yes) (on_board yes) (dnp no) (fields_autoplaced)
-    (property "Reference" "#PWR092" (at 335.28 163.83 0)
-      (effects (font (size 1.27 1.27)) hide)
-    )
-    (property "Value" "GND" (at 335.28 162.56 0)
+    (property "Reference" "#PWR092" (at 373.38 120.65 0)
+      (effects (font (size 1.27 1.27)) hide)
+    )
+    (property "Value" "GND" (at 373.38 119.38 0)
       (effects (font (size 1.27 1.27)))
     )
-    (property "Footprint" "" (at 335.28 157.48 0)
-      (effects (font (size 1.27 1.27)) hide)
-    )
-    (property "Datasheet" "" (at 335.28 157.48 0)
+    (property "Footprint" "" (at 373.38 114.3 0)
+      (effects (font (size 1.27 1.27)) hide)
+    )
+    (property "Datasheet" "" (at 373.38 114.3 0)
       (effects (font (size 1.27 1.27)) hide)
     )
@@
     )
   )
-  (symbol (lib_id "power:+5V") (at 335.28 132.08 0) (unit 1)
+  (symbol (lib_id "power:+5V") (at 373.38 88.9 0) (unit 1)
     (in_bom yes) (on_board yes) (dnp no) (fields_autoplaced)
-    (property "Reference" "#PWR090" (at 335.28 135.89 0)
-      (effects (font (size 1.27 1.27)) hide)
-    )
-    (property "Value" "+5V" (at 335.28 127 0)
+    (property "Reference" "#PWR090" (at 373.38 92.71 0)
+      (effects (font (size 1.27 1.27)) hide)
+    )
+    (property "Value" "+5V" (at 373.38 83.82 0)
       (effects (font (size 1.27 1.27)))
     )
-    (property "Footprint" "" (at 335.28 132.08 0)
-      (effects (font (size 1.27 1.27)) hide)
-    )
-    (property "Datasheet" "" (at 335.28 132.08 0)
+    (property "Footprint" "" (at 373.38 88.9 0)
+      (effects (font (size 1.27 1.27)) hide)
+    )
+    (property "Datasheet" "" (at 373.38 88.9 0)
       (effects (font (size 1.27 1.27)) hide)
     )
@@
     )
   )
-  (symbol (lib_id "74xx:74LS32") (at 335.28 144.78 0) (unit 5)
+  (symbol (lib_id "74xx:74LS32") (at 373.38 101.6 0) (unit 5)
     (in_bom yes) (on_board yes) (dnp no) (fields_autoplaced)
-    (property "Reference" "U9" (at 341.63 143.51 0)
-      (effects (font (size 1.27 1.27)) (justify left))
-    )
-    (property "Value" "74LS32" (at 341.63 146.05 0)
-      (effects (font (size 1.27 1.27)) (justify left))
-    )
-    (property "Footprint" "Package_SO:SOIC-14_3.9x8.7mm_P1.27mm" (at 335.28 144.78 0)
-      (effects (font (size 1.27 1.27)) hide)
-    )
-    (property "Datasheet" "http://www.ti.com/lit/gpn/sn74LS32" (at 335.28 144.78 0)
-      (effects (font (size 1.27 1.27)) hide)
-    )
+    (property "Reference" "U9" (at 379.73 100.33 0)
+      (effects (font (size 1.27 1.27)) (justify left))
+    )
+    (property "Value" "74LS32" (at 379.73 102.87 0)
+      (effects (font (size 1.27 1.27)) (justify left))
+    )
+    (property "Footprint" "Package_SO:SOIC-14_3.9x8.7mm_P1.27mm" (at 373.38 101.6 0)
+      (effects (font (size 1.27 1.27)) hide)
+    )
+    (property "Datasheet" "http://www.ti.com/lit/gpn/sn74LS32" (at 373.38 101.6 0)
+      (effects (font (size 1.27 1.27)) hide)
+    )
