File: hardware/motherboard/fpga.kicad_sch (KiCad schematic)
At the start: 17 parts, among them J5 Conn_01x06, U17 SN74ALVC164245, U18 SN74ALVC164245, U2 ICE40HX4K-TQ144, U34 74AHCT04, U35 74AHCT04, U5 W25Q32JVSSIM

Commit message: restructure, create minimum board project
Parts:
- C17: footprint Capacitor_SMD:C_0603_1608Metric -> (none); symbol UPduino_v3.0:Device_C -> Device:C
- D1: footprint LED_SMD:LED_0603_1608Metric -> (none); symbol UPduino_v3.0:Device_LED_ALT -> Device:LED
- R7, R8, R9: footprint Resistor_SMD:R_0603_1608Metric -> (none); symbol UPduino_v3.0:Device_R -> Device:R_Small_US
- U5: symbol UPduino_v3.0:W25Q32JVSS-Memory_Flash -> Memory_Flash:W25Q32JVSS
Connections:
- net +3V3 is gone; now on net +3.3V: D2.2 (A), R7.2, U2.100 (VCCIO_1), U2.123 (VCCIO_0), U2.131 (VCCIO_0), U2.30 (VCCIO_3), U2.6 (VCCIO_3), U2.72 (VCC_SPI), U2.89 (VCCIO_1)
- net LV.A0 is gone; now on net LV.A7: U2.93 (IOR_140_GBIN3)
- net LV.A1 is gone; now on net LV.A6: U2.94 (IOR_141_GBIN2)
- net LV.A19 is gone; now on net LV.A11: U2.87 (IOR_136)
- net LV.A20 is gone; now on net LV.A12: U2.85 (IOR_128)
- net LV.A21 is gone; now on net LV.A13: U2.84 (IOR_120)
- net LV.A22 is gone; now on net LV.A14: U2.83 (IOR_119)
- net LV.A23 is gone; now on net LV.A15: U2.82 (IOR_118)
- net LV.A24 is gone; now on net LV.A16: U2.81 (IOR_117)
- net LV.A25 is gone; now on net LV.A17: U2.80 (IOR_116)
- net LV.A26 is gone; now on net LV.A18: U2.79 (IOR_115)
- net ~{040_TCI}/~{040_TBI} is gone; now on net LV_~{LOCKE}: U2.17 (IOL_12A)
- net FLASH_IO2: now also U2.60 (IOB_95); no longer U2.61 (IOB_96)
- net FLASH_IO3: now also U2.61 (IOB_96); no longer U2.62 (IOB_102)
- net FLASH_SCK: now also R8.1; no longer R9.1
- net FLASH_SS: now also R9.1; no longer R8.1
- net FPGA_D0: now also U2.110 (IOT_168); no longer U2.114 (IOT_171)
- net FPGA_D1: now also U2.112 (IOT_169); no longer U2.115 (IOT_172)
- net FPGA_D2: now also U2.113 (IOT_170); no longer U2.116 (IOT_173)
- net FPGA_D3: now also U2.114 (IOT_171); no longer U2.117 (IOT_174)
- net FPGA_D4: now also U2.115 (IOT_172); no longer U2.118 (IOT_177)
- net FPGA_D5: now also U2.116 (IOT_173); no longer U2.119 (IOT_178)
- net FPGA_D6: now also U2.117 (IOT_174); no longer U2.120 (IOT_179)
- net FPGA_D7: now also U2.118 (IOT_177); no longer U2.121 (IOT_181)
- net FPGA_D_DIR: now also U2.63 (IOB_103_CBSEL0); no longer U2.64 (IOB_104_CBSEL1)
- net LV.A10: now also U2.88 (IOR_137); no longer U2.105 (IOR_165)
- net LV.A11: no longer U2.106 (IOR_166)
- net LV.A12: no longer U2.107 (IOR_167)
- net LV.A13: no longer U2.110 (IOT_168)
- net LV.A14: no longer U2.112 (IOT_169)
- net LV.A15: no longer U2.113 (IOT_170)
- net LV.A16: no longer U2.91 (IOR_139)
- net LV.A17: no longer U2.90 (IOR_138)
- net LV.A18: no longer U2.88 (IOR_137)
- net LV.A2: now also U2.98 (IOR_148); no longer U2.95 (IOR_144)
- net LV.A3: now also U2.97 (IOR_147); no longer U2.96 (IOR_146)
- net LV.A4: now also U2.96 (IOR_146); no longer U2.97 (IOR_147)
- net LV.A5: now also U2.95 (IOR_144); no longer U2.98 (IOR_148)
- net LV.A6: no longer U2.99 (IOR_152)
- net LV.A7: no longer U2.101 (IOR_160)
- net LV.A8: now also U2.91 (IOR_139); no longer U2.102 (IOR_161)
- net LV.A9: now also U2.90 (IOR_138); no longer U2.104 (IOR_164)
- net LV_68150_CS: now also U2.129 (IOT_198_GBIN0); no longer U2.33 (IOL_25A)
- net LV_AVEC: now also U2.62 (IOB_102); no longer U2.63 (IOB_103_CBSEL0)
- net LV_DRAM_CS: now also U2.124 (IOT_191); no longer U2.29 (IOL_23B)
- net LV_DUART_CS: now also U2.128 (IOT_197_GBIN1); no longer U2.32 (IOL_24B)
- net LV_PA0: now also U2.119 (IOT_178); no longer U2.122 (IOT_190)
- net LV_PA1: now also U2.120 (IOT_179); no longer U2.124 (IOT_191)
- net LV_PS/2_CS: now also U2.130 (IOT_206); no longer U2.34 (IOL_25B)
- net LV_R/~{W}: now also U2.19 (IOL_13A); no longer U2.26 (IOL_18B)
- net LV_SRAM_CS: now also U2.125 (IOT_192); no longer U2.31 (IOL_24A)
- net LV_~{040_BR}: now also U17.29 (2A6), U2.16 (IOL_10B); no longer U2.19 (IOL_13A)
- net LV_~{68150_DS}: now also U17.27 (2A7), U2.23 (IOL_17A); no longer U2.24 (IOL_17B)
- net LV_~{LOCKE}: now also U17.32 (2A4); no longer U2.20 (IOL_13B_GBIN7)
- net LV_~{LOCK}: now also U17.30 (2A5), U2.18 (IOL_12B); no longer U2.21 (IOL_14A_GBIN6)
- net LV_~{TS}: now also U2.20 (IOL_13B_GBIN7); no longer U2.23 (IOL_17A)
- net ~{040_BG}: now also U2.15 (IOL_10A); no longer U2.18 (IOL_12B)
- net ~{040_BR}: now also U17.20 (2B6)
- net ~{68150_DS}: now also U17.22 (2B7)
- net ~{LOCKE}: now also U17.17 (2B4)
- net ~{LOCK}: now also U17.19 (2B5)
- net ~{TA}: no longer U2.15 (IOL_10A)
- net ~{TEA}: no longer U2.16 (IOL_10B)
- net LV_I2C_CS: now reaches U2.134 (IOT_212)
- net LV_I2C_CS: now also U34.1
- net FPGA_A_DIR: now reaches U2.55 (IOB_91)
- net FPGA_A_~{OE}: now reaches U2.56 (IOB_94)
- net LV_IDE_CS: no longer names the net of U2.28 (IOL_23A)
- net LV_IDE_CS: no longer U34.1
- net ~{FPGA_D_OE} renamed FPGA_D_~{OE}
- net FPGA_D_~{OE}: now also U2.64 (IOB_104_CBSEL1); no longer U2.25 (IOL_18A)
- net ~{IDE_CS} renamed ~{I2C_CS}
- new net LV_SIZ0: U2.121 (IOT_181)
- new net LV_SIZ1: U2.122 (IOT_190)
- new net LV_~{TA}: U2.24 (IOL_17B)
- new net LV_~{TCI}/~{TBI}: U2.26 (IOL_18B)
- new net LV_~{TEA}: U2.25 (IOL_18A)
- new net LV_~{TIP}: U2.21 (IOL_14A_GBIN6)
Other:
- sheet AddressBuffer ports: added FPGA_ABUF_DIR, FPGA_ABUF_~{OE}; removed none
- sheet TransferBuffer ports: added LV_SIZ[0..1], LV_~{TA}, LV_~{TCI}/~{TBI}, LV_~{TEA}, LV_~{TIP}, ~{TA}, ~{TCI}/~{TBI}, ~{TEA}, ~{TIP}; removed LVSIZ[0..1], LV_~{040_BR}, LV_~{68150_DS}, LV_~{LOCKE}, LV_~{LOCK}, ~{040_BR}, ~{DS}, ~{LOCKE}, ~{LOCK}
- note added: "Bring interrupt processing here: - Route TT[1:0] and TM[2:0] through a 5v tolerant buffer and qualify with ~{040_BG}"
- moved on the sheet: C17, D2, U5

Commit message: work on testboard, move 3d models
Parts:
- renumbered U18 to U2, U17 to U2, U2 to U5
