File: hardware/testboard/datatrx.kicad_sch (KiCad schematic)
At the start: 11 parts, among them U14 SN74ALVC164245, U15 SN74ALVC164245

Commit message: root mostly finished
Parts:
- renumbered C32 to C40, C36 to C41, C33 to C42, C37 to C43, C34 to C44, C38 to C45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

Commit message: simpleboard nearly complete
Parts:
- C40, C41, C42, C43, C44, C45, C46, C47: footprint (none) -> Capacitor_SMD:C_0603_1608Metric
- R20: footprint (none) -> Resistor_SMD:R_0603_1608Metric
Other:
- moved on the sheet: C40, C41, C42, C43, C44, C45, C46, C47, R20, U16A, U16B, U17A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
