File: hardware/testboard/io.kicad_sch (KiCad schematic)
At the start: 20 parts, among them U2 MAX232, U3 MAX232, U4 68681, Y1 3.6864MHz

Commit message: root mostly finished
Changed lines of the file:
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@@
     (effects (font (size 1.27 1.27)) (justify right))
   )
-  (hierarchical_label "~{IACK}" (shape input) (at 71.12 172.72 180) (fields_autoplaced)
+  (hierarchical_label "~{IACK}" (shape output) (at 71.12 172.72 180) (fields_autoplaced)
     (effects (font (size 1.27 1.27)) (justify right))
   )

Commit message: work on testboard
Parts:
- added R2: 1k, symbol Device:R_Small_US
- Y1: symbol Device:Crystal_Small -> Device:Crystal
Connections:
- net +5V: now also R2.1
- net ~{IRQ}: now also R2.2
Changed lines of the file:
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@@
   (junction (at 60.96 101.6) (diameter 0) (color 0 0 0 0)
+  )
+  (junction (at 58.42 182.88) (diameter 0) (color 0 0 0 0)
   )
   (junction (at 251.46 58.42) (diameter 0) (color 0 0 0 0)
@@
     (stroke (width 0) (type default))
   )
-  (wire (pts (xy 41.91 128.27) (xy 44.45 128.27))
-    (stroke (width 0) (type default))
-  )
   (wire (pts (xy 96.52 76.2) (xy 81.28 76.2))
     (stroke (width 0) (type default))
@@
     (stroke (width 0) (type default))
   )
+  (wire (pts (xy 58.42 180.34) (xy 58.42 182.88))
+    (stroke (width 0) (type default))
+  )
   (bus (pts (xy 60.96 129.54) (xy 58.42 129.54))
     (stroke (width 0) (type default))
@@
     (stroke (width 0) (type default))
   )
+  (wire (pts (xy 45.72 124.46) (xy 45.72 121.92))
+    (stroke (width 0) (type default))
+  )
   (wire (pts (xy 40.64 86.36) (xy 30.48 86.36))
     (stroke (width 0) (type default))
   )
-  (wire (pts (xy 44.45 124.46) (xy 55.88 124.46))
-    (stroke (width 0) (type default))
-  )
   (wire (pts (xy 121.92 132.08) (xy 137.16 132.08))
     (stroke (width 0) (type default))
@@
     (stroke (width 0) (type default))
   )
-  (wire (pts (xy 44.45 123.19) (xy 44.45 124.46))
-    (stroke (width 0) (type default))
-  )
   (wire (pts (xy 63.5 144.78) (xy 71.12 144.78))
     (stroke (width 0) (type default))
@@
     (stroke (width 0) (type default))
   )
+  (wire (pts (xy 55.88 124.46) (xy 45.72 124.46))
+    (stroke (width 0) (type default))
+  )
   (wire (pts (xy 142.24 101.6) (xy 142.24 99.06))
     (stroke (width 0) (type default))
@@
     (stroke (width 0) (type default))
   )
-  (wire (pts (xy 44.45 128.27) (xy 44.45 127))
+  (wire (pts (xy 45.72 127) (xy 63.5 127))
     (stroke (width 0) (type default))
   )
@@
     (stroke (width 0) (type default))
   )
+  (wire (pts (xy 40.64 129.54) (xy 45.72 129.54))
+    (stroke (width 0) (type default))
+  )
+  (wire (pts (xy 45.72 121.92) (xy 40.64 121.92))
+    (stroke (width 0) (type default))
+  )
   (wire (pts (xy 96.52 190.5) (xy 121.92 190.5))
     (stroke (width 0) (type default))
@@
     (stroke (width 0) (type default))
   )
+  (wire (pts (xy 58.42 182.88) (xy 71.12 182.88))
+    (stroke (width 0) (type default))
+  )
   (wire (pts (xy 81.28 86.36) (xy 96.52 86.36))
     (stroke (width 0) (type default))
@@
     (stroke (width 0) (type default))
   )
+  (wire (pts (xy 48.26 182.88) (xy 58.42 182.88))
+    (stroke (width 0) (type default))
+  )
   (wire (pts (xy 40.64 81.28) (xy 30.48 81.28))
     (stroke (width 0) (type default))
@@
     (stroke (width 0) (type default))
   )
-  (wire (pts (xy 41.91 123.19) (xy 44.45 123.19))
-    (stroke (width 0) (type default))
-  )
   (wire (pts (xy 177.8 76.2) (xy 162.56 76.2))
     (stroke (width 0) (type default))
@@
     (stroke (width 0) (type default))
   )
+  (wire (pts (xy 45.72 129.54) (xy 45.72 127))
+    (stroke (width 0) (type default))
+  )
   (wire (pts (xy 66.04 154.94) (xy 71.12 154.94))
     (stroke (width 0) (type default))
@@
   )
   (wire (pts (xy 40.64 76.2) (xy 30.48 76.2))
-    (stroke (width 0) (type default))
-  )
-  (wire (pts (xy 44.45 127) (xy 63.5 127))
     (stroke (width 0) (type default))
   )
@@
     (effects (font (size 1.27 1.27)) (justify right))
   )
-  (hierarchical_label "~{IRQ}" (shape output) (at 71.12 182.88 180) (fields_autoplaced)
+  (hierarchical_label "~{IRQ}" (shape output) (at 48.26 182.88 180) (fields_autoplaced)
     (effects (font (size 1.27 1.27)) (justify right))
   )
@@
     )
   )
+  (symbol (lib_id "power:+5V") (at 58.42 175.26 0) (unit 1)
+    (in_bom yes) (on_board yes) (dnp no) (fields_autoplaced)
+    (property "Reference" "#PWR0119" (at 58.42 179.07 0)
+      (effects (font (size 1.27 1.27)) hide)
+    )
+    (property "Value" "+5V" (at 58.42 170.18 0)
+      (effects (font (size 1.27 1.27)))
+    )
+    (property "Footprint" "" (at 58.42 175.26 0)
+      (effects (font (size 1.27 1.27)) hide)
+    )
+    (property "Datasheet" "" (at 58.42 175.26 0)
+      (effects (font (size 1.27 1.27)) hide)
+    )
+    (pin "1")
+    (instances
+      (project "testboard"
+        (path "/a1ce156a-fb78-423b-b05a-d07384e5c8a7/2b8a05d0-742b-42f4-b29e-e8342ede593d"
+          (reference "#PWR0119") (unit 1)
+        )
+      )
+    )
+  )
   (symbol (lib_id "Device:C_Small") (at 58.42 124.46 90) (unit 1)
     (in_bom yes) (on_board yes) (dnp no) (fields_autoplaced)
@@
     )
   )
-  (symbol (lib_id "Device:Crystal_Small") (at 41.91 125.73 90) (mirror x) (unit 1)
+  (symbol (lib_id "Device:Crystal") (at 40.64 125.73 90) (mirror x) (unit 1)
     (in_bom yes) (on_board yes) (dnp no)
-    (property "Reference" "Y1" (at 39.37 124.46 90)
-      (effects (font (size 1.27 1.27)) (justify left))
-    )
-    (property "Value" "3.6864MHz" (at 39.37 127 90)
-      (effects (font (size 1.27 1.27)) (justify left))
-    )
-    (property "Footprint" "" (at 41.91 125.73 0)
-      (effects (font (size 1.27 1.27)) hide)
-    )
-    (property "Datasheet" "~" (at 41.91 125.73 0)
+    (property "Reference" "Y1" (at 38.1 124.46 90)
+      (effects (font (size 1.27 1.27)) (justify left))
+    )
+    (property "Value" "3.6864MHz" (at 38.1 127 90)
+      (effects (font (size 1.27 1.27)) (justify left))
+    )
+    (property "Footprint" "" (at 40.64 125.73 0)
+      (effects (font (size 1.27 1.27)) hide)
+    )
+    (property "Datasheet" "~" (at 40.64 125.73 0)
       (effects (font (size 1.27 1.27)) hide)
     )
@@
         )
       )
+    )
+  )
+  (symbol (lib_id "Device:R_Small_US") (at 58.42 177.8 0) (unit 1)
+    (in_bom yes) (on_board yes) (dnp no)
+    (property "Reference" "R2" (at 55.88 176.53 0)
+      (effects (font (size 1.27 1.27)) (justify right))
+    )
+    (property "Value" "1k" (at 55.88 179.07 0)
+      (effects (font (size 1.27 1.27)) (justify right))
+    )
+    (property "Footprint" "" (at 58.42 177.8 0)
+      (effects (font (size 1.27 1.27)) hide)
+    )
+    (property "Datasheet" "~" (at 58.42 177.8 0)
+      (effects (font (size 1.27 1.27)) hide)
+    )
+    (pin "2")
+    (pin "1")
+    (instances
+      (project "testboard"
+        (path "/a1ce156a-fb78-423b-b05a-d07384e5c8a7/2b8a05d0-742b-42f4-b29e-e8342ede593d"
+          (reference "R2") (unit 1)
+        )
+      )

Commit message: simpleboard nearly complete
Parts:
- C10, C11, C12, C13, C14, C25, C26, C7, C8, C9: footprint (none) -> Capacitor_SMD:C_0805_2012Metric
- C15, C16: footprint (none) -> Capacitor_SMD:C_0603_1608Metric
- C17: footprint (none) -> Capacitor_THT:CP_Radial_D5.0mm_P2.00mm
- C18: value .1uF -> 100nF; footprint (none) -> Capacitor_SMD:C_0603_1608Metric
- R2: footprint (none) -> Resistor_SMD:R_0603_1608Metric
- Y1: footprint (none) -> Crystal:Crystal_C38-LF_D3.0mm_L8.0mm_Vertical
Changed lines of the file:
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@@
       (effects (font (size 1.27 1.27)))
     )
-    (property "Footprint" "" (at 58.42 124.46 0)
+    (property "Footprint" "Capacitor_SMD:C_0603_1608Metric" (at 58.42 124.46 0)
       (effects (font (size 1.27 1.27)) hide)
     )
@@
       (effects (font (size 1.27 1.27)) (justify left))
     )
-    (property "Footprint" "" (at 147.32 182.88 0)
+    (property "Footprint" "Capacitor_THT:CP_Radial_D5.0mm_P2.00mm" (at 147.32 182.88 0)
       (effects (font (size 1.27 1.27)) hide)
     )
@@
       (effects (font (size 1.27 1.27)) (justify left))
     )
-    (property "Footprint" "" (at 120.9548 53.34 0)
+    (property "Footprint" "Capacitor_SMD:C_0805_2012Metric" (at 120.9548 53.34 0)
       (effects (font (size 1.27 1.27)) hide)
     )
@@
       (effects (font (size 1.27 1.27)) (justify left))
     )
-    (property "Footprint" "" (at 88.9 65.0748 0)
+    (property "Footprint" "Capacitor_SMD:C_0805_2012Metric" (at 88.9 65.0748 0)
       (effects (font (size 1.27 1.27)) hide)
     )
@@
       (effects (font (size 1.27 1.27)) (justify left))
     )
-    (property "Footprint" "" (at 120.9548 101.6 0)
+    (property "Footprint" "Capacitor_SMD:C_0805_2012Metric" (at 120.9548 101.6 0)
       (effects (font (size 1.27 1.27)) hide)
     )
@@
       (effects (font (size 1.27 1.27)) (justify left))
     )
-    (property "Footprint" "" (at 88.9 57.4548 0)
+    (property "Footprint" "Capacitor_SMD:C_0805_2012Metric" (at 88.9 57.4548 0)
       (effects (font (size 1.27 1.27)) hide)
     )
@@
       (effects (font (size 1.27 1.27)))
     )
-    (property "Footprint" "" (at 66.04 127 0)
+    (property "Footprint" "Capacitor_SMD:C_0603_1608Metric" (at 66.04 127 0)
       (effects (font (size 1.27 1.27)) hide)
     )
@@
       (effects (font (size 1.27 1.27)) (justify left))
     )
-    (property "Footprint" "" (at 82.2452 53.34 0)
+    (property "Footprint" "Capacitor_SMD:C_0805_2012Metric" (at 82.2452 53.34 0)
       (effects (font (size 1.27 1.27)) hide)
     )
@@
       (effects (font (size 1.27 1.27)) (justify left))
     )
-    (property "Footprint" "" (at 163.5252 53.34 0)
+    (property "Footprint" "Capacitor_SMD:C_0805_2012Metric" (at 163.5252 53.34 0)
       (effects (font (size 1.27 1.27)) hide)
     )
@@
       (effects (font (size 1.27 1.27)) (justify left))
     )
-    (property "Footprint" "" (at 40.64 125.73 0)
+    (property "Footprint" "Crystal:Crystal_C38-LF_D3.0mm_L8.0mm_Vertical" (at 40.64 125.73 0)
       (effects (font (size 1.27 1.27)) hide)
     )
@@
       (effects (font (size 1.27 1.27)) (justify right))
     )
-    (property "Footprint" "" (at 58.42 177.8 0)
+    (property "Footprint" "Resistor_SMD:R_0603_1608Metric" (at 58.42 177.8 0)
       (effects (font (size 1.27 1.27)) hide)
     )
@@
       (effects (font (size 1.27 1.27)) (justify left))
     )
-    (property "Value" ".1uF" (at 124.46 189.2363 0)
-      (effects (font (size 1.27 1.27)) (justify left))
-    )
-    (property "Footprint" "" (at 121.92 187.96 0)
+    (property "Value" "100nF" (at 124.46 189.2363 0)
+      (effects (font (size 1.27 1.27)) (justify left))
+    )
+    (property "Footprint" "Capacitor_SMD:C_0603_1608Metric" (at 121.92 187.96 0)
       (effects (font (size 1.27 1.27)) hide)
     )
@@
       (effects (font (size 1.27 1.27)) (justify left))
     )
-    (property "Footprint" "" (at 39.6748 101.6 0)
+    (property "Footprint" "Capacitor_SMD:C_0805_2012Metric" (at 39.6748 101.6 0)
       (effects (font (size 1.27 1.27)) hide)
     )
@@
       (effects (font (size 1.27 1.27)) (justify left))
     )
-    (property "Footprint" "" (at 170.18 65.0748 0)
+    (property "Footprint" "Capacitor_SMD:C_0805_2012Metric" (at 170.18 65.0748 0)
       (effects (font (size 1.27 1.27)) hide)
     )
@@
       (effects (font (size 1.27 1.27)) (justify left))
     )
-    (property "Footprint" "" (at 170.18 57.4548 0)
+    (property "Footprint" "Capacitor_SMD:C_0805_2012Metric" (at 170.18 57.4548 0)
       (effects (font (size 1.27 1.27)) hide)
     )
@@
       (effects (font (size 1.27 1.27)) (justify left))
     )
-    (property "Footprint" "" (at 39.6748 53.34 0)
-      (effects (font (size 1.27 1.27)) hide)
-    )
+    (property "Footprint" "Capacitor_SMD:C_0805_2012Metric" (at 39.6748 53.34 0)
+      (effects (font (size 1.27 1.27)) hide)
+    )

Commit message: pinouts
Parts:
- renumbered C7 to C501, C25 to C502, C15 to C503, C16 to C504, C8 to C505, C11 to C506, C13 to C507, C9 to C508, C26 to C509, C18 to C510, C17 to C511, C10 to C512, C12 to C513, C14 to C514, JS1 to JS501, JS2 to JS502, R2 to R501, U2 to U501, U4 to U502, U3 to U503, Y1 to Y501
