File: hardware/testboard/sram.kicad_sch (KiCad schematic)
At the start: 5 parts, among them U6 IS61C5128AS-25TLI, U7 IS61C5128AS-25TLI

Commit message: simpleboard nearly complete
Parts:
- removed C20: 1uF, symbol Device:C_Polarized_Small_US
- C21, C22: value .1uF -> 100nF; footprint (none) -> Capacitor_SMD:C_0603_1608Metric
Changed lines of the file:
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@@
-    )
-  )
-  (symbol (lib_id "power:GND") (at 33.02 30.48 0) (unit 1)
-    (in_bom yes) (on_board yes) (dnp no) (fields_autoplaced)
-    (property "Reference" "#PWR016" (at 33.02 36.83 0)
-      (effects (font (size 1.27 1.27)) hide)
-    )
-    (property "Value" "GND" (at 33.02 35.56 0)
-      (effects (font (size 1.27 1.27)))
-    )
-    (property "Footprint" "" (at 33.02 30.48 0)
-      (effects (font (size 1.27 1.27)) hide)
-    )
-    (property "Datasheet" "" (at 33.02 30.48 0)
-      (effects (font (size 1.27 1.27)) hide)
-    )
-    (pin "1")
-    (instances
-      (project "testboard"
-        (path "/a1ce156a-fb78-423b-b05a-d07384e5c8a7/e8f69379-7c84-47d9-8ed8-3fe10fcd197b"
-          (reference "#PWR016") (unit 1)
-        )
-      )
     )
   )
@@
       (effects (font (size 1.27 1.27)) (justify left))
     )
-    (property "Value" ".1uF" (at 124.46 100.3363 0)
-      (effects (font (size 1.27 1.27)) (justify left))
-    )
-    (property "Footprint" "" (at 121.92 99.06 0)
+    (property "Value" "100nF" (at 124.46 100.3363 0)
+      (effects (font (size 1.27 1.27)) (justify left))
+    )
+    (property "Footprint" "Capacitor_SMD:C_0603_1608Metric" (at 121.92 99.06 0)
       (effects (font (size 1.27 1.27)) hide)
     )
@@
         (path "/a1ce156a-fb78-423b-b05a-d07384e5c8a7/e8f69379-7c84-47d9-8ed8-3fe10fcd197b"
           (reference "C21") (unit 1)
-        )
-      )
-    )
-  )
-  (symbol (lib_id "power:+5V") (at 33.02 25.4 0) (unit 1)
-    (in_bom yes) (on_board yes) (dnp no) (fields_autoplaced)
-    (property "Reference" "#PWR015" (at 33.02 29.21 0)
-      (effects (font (size 1.27 1.27)) hide)
-    )
-    (property "Value" "+5V" (at 33.02 20.32 0)
-      (effects (font (size 1.27 1.27)))
-    )
-    (property "Footprint" "" (at 33.02 25.4 0)
-      (effects (font (size 1.27 1.27)) hide)
-    )
-    (property "Datasheet" "" (at 33.02 25.4 0)
-      (effects (font (size 1.27 1.27)) hide)
-    )
-    (pin "1")
-    (instances
-      (project "testboard"
-        (path "/a1ce156a-fb78-423b-b05a-d07384e5c8a7/e8f69379-7c84-47d9-8ed8-3fe10fcd197b"
-          (reference "#PWR015") (unit 1)
         )
       )
@@
     )
   )
-  (symbol (lib_id "Device:C_Polarized_Small_US") (at 33.02 27.94 0) (unit 1)
-    (in_bom yes) (on_board yes) (dnp no) (fields_autoplaced)
-    (property "Reference" "C20" (at 35.56 26.2382 0)
-      (effects (font (size 1.27 1.27)) (justify left))
-    )
-    (property "Value" "1uF" (at 35.56 28.7782 0)
-      (effects (font (size 1.27 1.27)) (justify left))
-    )
-    (property "Footprint" "" (at 33.02 27.94 0)
-      (effects (font (size 1.27 1.27)) hide)
-    )
-    (property "Datasheet" "~" (at 33.02 27.94 0)
-      (effects (font (size 1.27 1.27)) hide)
-    )
-    (pin "2")
-    (pin "1")
-    (instances
-      (project "testboard"
-        (path "/a1ce156a-fb78-423b-b05a-d07384e5c8a7/e8f69379-7c84-47d9-8ed8-3fe10fcd197b"
-          (reference "C20") (unit 1)
-        )
-      )
-    )
-  )
   (symbol (lib_id "Device:C_Small") (at 121.92 180.34 0) (unit 1)
     (in_bom yes) (on_board yes) (dnp no) (fields_autoplaced)
@@
       (effects (font (size 1.27 1.27)) (justify left))
     )
-    (property "Value" ".1uF" (at 124.46 181.6163 0)
-      (effects (font (size 1.27 1.27)) (justify left))
-    )
-    (property "Footprint" "" (at 121.92 180.34 0)
-      (effects (font (size 1.27 1.27)) hide)
-    )
+    (property "Value" "100nF" (at 124.46 181.6163 0)
+      (effects (font (size 1.27 1.27)) (justify left))
+    )
+    (property "Footprint" "Capacitor_SMD:C_0603_1608Metric" (at 121.92 180.34 0)
+      (effects (font (size 1.27 1.27)) hide)
+    )

Commit message: pinouts
Parts:
- renumbered C21 to C301, C22 to C302, U6 to U301, U7 to U302
Changed lines of the file:
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@@
   (symbol (lib_id "Memory_RAM:IS61C5128AS-25TLI") (at 104.14 68.58 0) (unit 1)
     (in_bom yes) (on_board yes) (dnp no) (fields_autoplaced)
-    (property "Reference" "U6" (at 106.3341 33.02 0)
+    (property "Reference" "U301" (at 106.3341 33.02 0)
       (effects (font (size 1.27 1.27)) (justify left))
     )
@@
       (project "testboard"
         (path "/a1ce156a-fb78-423b-b05a-d07384e5c8a7/e8f69379-7c84-47d9-8ed8-3fe10fcd197b"
-          (reference "U6") (unit 1)
+          (reference "U301") (unit 1)
         )
       )
@@
   (symbol (lib_id "power:GND") (at 104.14 182.88 0) (unit 1)
     (in_bom yes) (on_board yes) (dnp no) (fields_autoplaced)
-    (property "Reference" "#PWR022" (at 104.14 189.23 0)
+    (property "Reference" "#PWR0304" (at 104.14 189.23 0)
       (effects (font (size 1.27 1.27)) hide)
     )
@@
       (project "testboard"
         (path "/a1ce156a-fb78-423b-b05a-d07384e5c8a7/e8f69379-7c84-47d9-8ed8-3fe10fcd197b"
-          (reference "#PWR022") (unit 1)
+          (reference "#PWR0304") (unit 1)
         )
       )
@@
   (symbol (lib_id "power:+5V") (at 121.92 177.8 0) (unit 1)
     (in_bom yes) (on_board yes) (dnp no) (fields_autoplaced)
-    (property "Reference" "#PWR021" (at 121.92 181.61 0)
+    (property "Reference" "#PWR0306" (at 121.92 181.61 0)
       (effects (font (size 1.27 1.27)) hide)
     )
@@
       (project "testboard"
         (path "/a1ce156a-fb78-423b-b05a-d07384e5c8a7/e8f69379-7c84-47d9-8ed8-3fe10fcd197b"
-          (reference "#PWR021") (unit 1)
+          (reference "#PWR0306") (unit 1)
         )
       )
@@
   (symbol (lib_id "power:+5V") (at 121.92 96.52 0) (unit 1)
     (in_bom yes) (on_board yes) (dnp no) (fields_autoplaced)
-    (property "Reference" "#PWR018" (at 121.92 100.33 0)
+    (property "Reference" "#PWR0305" (at 121.92 100.33 0)
       (effects (font (size 1.27 1.27)) hide)
     )
@@
       (project "testboard"
         (path "/a1ce156a-fb78-423b-b05a-d07384e5c8a7/e8f69379-7c84-47d9-8ed8-3fe10fcd197b"
-          (reference "#PWR018") (unit 1)
+          (reference "#PWR0305") (unit 1)
         )
       )
@@
   (symbol (lib_id "power:+5V") (at 104.14 35.56 0) (unit 1)
     (in_bom yes) (on_board yes) (dnp no) (fields_autoplaced)
-    (property "Reference" "#PWR017" (at 104.14 39.37 0)
+    (property "Reference" "#PWR0301" (at 104.14 39.37 0)
       (effects (font (size 1.27 1.27)) hide)
     )
@@
       (project "testboard"
         (path "/a1ce156a-fb78-423b-b05a-d07384e5c8a7/e8f69379-7c84-47d9-8ed8-3fe10fcd197b"
-          (reference "#PWR017") (unit 1)
+          (reference "#PWR0301") (unit 1)
         )
       )
@@
   (symbol (lib_id "power:+5V") (at 104.14 116.84 0) (unit 1)
     (in_bom yes) (on_board yes) (dnp no) (fields_autoplaced)
-    (property "Reference" "#PWR020" (at 104.14 120.65 0)
+    (property "Reference" "#PWR0303" (at 104.14 120.65 0)
       (effects (font (size 1.27 1.27)) hide)
     )
@@
       (project "testboard"
         (path "/a1ce156a-fb78-423b-b05a-d07384e5c8a7/e8f69379-7c84-47d9-8ed8-3fe10fcd197b"
-          (reference "#PWR020") (unit 1)
+          (reference "#PWR0303") (unit 1)
         )
       )
@@
   (symbol (lib_id "Device:C_Small") (at 121.92 99.06 0) (unit 1)
     (in_bom yes) (on_board yes) (dnp no) (fields_autoplaced)
-    (property "Reference" "C21" (at 124.46 97.7963 0)
+    (property "Reference" "C301" (at 124.46 97.7963 0)
       (effects (font (size 1.27 1.27)) (justify left))
     )
@@
       (project "testboard"
         (path "/a1ce156a-fb78-423b-b05a-d07384e5c8a7/e8f69379-7c84-47d9-8ed8-3fe10fcd197b"
-          (reference "C21") (unit 1)
+          (reference "C301") (unit 1)
         )
       )
@@
   (symbol (lib_id "Memory_RAM:IS61C5128AS-25TLI") (at 104.14 149.86 0) (unit 1)
     (in_bom yes) (on_board yes) (dnp no) (fields_autoplaced)
-    (property "Reference" "U7" (at 106.3341 114.3 0)
+    (property "Reference" "U302" (at 106.3341 114.3 0)
       (effects (font (size 1.27 1.27)) (justify left))
     )
@@
       (project "testboard"
         (path "/a1ce156a-fb78-423b-b05a-d07384e5c8a7/e8f69379-7c84-47d9-8ed8-3fe10fcd197b"
-          (reference "U7") (unit 1)
+          (reference "U302") (unit 1)
         )
       )
@@
   (symbol (lib_id "power:GND") (at 104.14 101.6 0) (unit 1)
     (in_bom yes) (on_board yes) (dnp no) (fields_autoplaced)
-    (property "Reference" "#PWR019" (at 104.14 107.95 0)
+    (property "Reference" "#PWR0302" (at 104.14 107.95 0)
       (effects (font (size 1.27 1.27)) hide)
     )
@@
       (project "testboard"
         (path "/a1ce156a-fb78-423b-b05a-d07384e5c8a7/e8f69379-7c84-47d9-8ed8-3fe10fcd197b"
-          (reference "#PWR019") (unit 1)
+          (reference "#PWR0302") (unit 1)
         )
       )
@@
   (symbol (lib_id "Device:C_Small") (at 121.92 180.34 0) (unit 1)
     (in_bom yes) (on_board yes) (dnp no) (fields_autoplaced)
-    (property "Reference" "C22" (at 124.46 179.0763 0)
+    (property "Reference" "C302" (at 124.46 179.0763 0)
       (effects (font (size 1.27 1.27)) (justify left))
     )
@@
       (project "testboard"
         (path "/a1ce156a-fb78-423b-b05a-d07384e5c8a7/e8f69379-7c84-47d9-8ed8-3fe10fcd197b"
-          (reference "C22") (unit 1)
-        )
-      )
+          (reference "C302") (unit 1)
+        )
+      )
