File: hardware/testboard/fpga.kicad_sch (KiCad schematic)
At the start: 13 parts, among them J2 Conn_01x06, U10 SN74ALVC164245, U11 ICE40HX4K-TQ144, U12 74AHCT04, U13 SST26VF023BA

Commit message: work on testboard
Parts:
- removed R2: 4.7k, symbol Device:R_Small_US
Connections:
- net FPGA_A_DIR: now also U11.49 (IOB_81_GBIN5)
- net FPGA_A_~{OE}: now also U11.48 (IOB_80)
- net FPGA_D_DIR: no longer U10.1 (1DIR)
- net FPGA_D_~{OE}: no longer U10.48 (*1OE)
- net LV.A0: now also U11.1 (IOL_2A); no longer U11.73 (IOR_109)
- net LV.A1: now also U11.2 (IOL_2B); no longer U11.74 (IOR_110)
- net LV.A10: now also U11.15 (IOL_10A); no longer U11.84 (IOR_120)
- net LV.A11: now also U11.16 (IOL_10B); no longer U11.85 (IOR_128)
- net LV.A12: now also U11.17 (IOL_12A); no longer U11.87 (IOR_136)
- net LV.A13: now also U11.18 (IOL_12B); no longer U11.88 (IOR_137)
- net LV.A14: now also U11.19 (IOL_13A); no longer U11.90 (IOR_138)
- net LV.A15: now also U11.20 (IOL_13B_GBIN7); no longer U11.91 (IOR_139)
- net LV.A16: now also U11.73 (IOR_109); no longer U11.93 (IOR_140_GBIN3)
- net LV.A17: now also U11.74 (IOR_110); no longer U11.94 (IOR_141_GBIN2)
- net LV.A18: now also U11.75 (IOR_111); no longer U11.95 (IOR_144)
- net LV.A19: now also U11.76 (IOR_112); no longer U11.96 (IOR_146)
- net LV.A2: now also U11.3 (IOL_3A); no longer U11.75 (IOR_111)
- net LV.A20: now also U11.78 (IOR_114); no longer U11.97 (IOR_147)
- net LV.A21: now also U11.79 (IOR_115); no longer U11.98 (IOR_148)
- net LV.A22: now also U11.80 (IOR_116); no longer U11.99 (IOR_152)
- net LV.A23: now also U11.81 (IOR_117); no longer U11.101 (IOR_160)
- net LV.A24: now also U11.82 (IOR_118); no longer U11.102 (IOR_161)
- net LV.A25: now also U11.83 (IOR_119); no longer U11.104 (IOR_164)
- net LV.A26: now also U11.84 (IOR_120); no longer U11.105 (IOR_165)
- net LV.A27: now also U11.85 (IOR_128); no longer U11.106 (IOR_166)
- net LV.A28: now also U11.87 (IOR_136); no longer U11.107 (IOR_167)
- net LV.A29: now also U11.88 (IOR_137); no longer U11.110 (IOT_168)
- net LV.A3: now also U11.4 (IOL_3B); no longer U11.76 (IOR_112)
- net LV.A30: now also U11.90 (IOR_138); no longer U11.112 (IOT_169)
- net LV.A31: now also U11.91 (IOR_139); no longer U11.113 (IOT_170)
- net LV.A4: now also U11.7 (IOL_4A); no longer U11.78 (IOR_114)
- net LV.A5: now also U11.8 (IOL_4B); no longer U11.79 (IOR_115)
- net LV.A6: now also U11.9 (IOL_5A); no longer U11.80 (IOR_116)
- net LV.A7: now also U11.10 (IOL_5B); no longer U11.81 (IOR_117)
- net LV.A8: now also U11.11 (IOL_8A); no longer U11.82 (IOR_118)
- net LV.A9: now also U11.12 (IOL_8B); no longer U11.83 (IOR_119)
- net LV_68150_CS: now also U11.47 (IOB_79)
- net LV_COM_CS: now also U11.45 (IOB_73)
- net LV_RAM_CS: now also U11.44 (IOB_72)
- net ~{DSACK0}: now also U11.21 (IOL_14A_GBIN6); no longer U11.1 (IOL_2A)
- net ~{DSACK1}: now also U11.22 (IOL_14B); no longer U11.2 (IOL_2B)
- net LV_D24: now reaches U11.122 (IOT_190)
- net LV_D25: now reaches U11.124 (IOT_191)
- net LV_D26: now reaches U11.125 (IOT_192)
- net LV_D27: now reaches U11.128 (IOT_197_GBIN1)
- net LV_D28: now reaches U11.129 (IOT_198_GBIN0)
- net LV_D29: now reaches U11.130 (IOT_206)
- net LV_D30: now reaches U11.134 (IOT_212)
- net LV_D31: now reaches U11.135 (IOT_213)
- net SIZ0: now reaches U10.16 (2B3)
- net SIZ1: now reaches U10.17 (2B4)
- net ~{TS}: now reaches U10.19 (2B5)
- net ~{TIP}: now reaches U10.20 (2B6)
- net R/~{W}: now reaches U10.23 (2B8)
- net LV_R/~{W}: now reaches U10.26 (2A8)
- net LV_~{TIP}: now reaches U10.29 (2A6)
- net LV_~{TS}: now reaches U10.30 (2A5)
- net LV_SIZ1: now reaches U10.32 (2A4)
- net LV_SIZ0: now reaches U10.33 (2A3)
- net FPGA_D0: no longer names the net of U10.47 (1A1)
- net FPGA_D0: no longer U11.114 (IOT_171)
- net FPGA_D1: no longer names the net of U10.46 (1A2)
- net FPGA_D1: no longer U11.115 (IOT_172)
- net FPGA_D2: no longer names the net of U10.44 (1A3)
- net FPGA_D2: no longer U11.116 (IOT_173)
- net FPGA_D3: no longer names the net of U10.43 (1A4)
- net FPGA_D3: no longer U11.117 (IOT_174)
- net FPGA_D4: no longer names the net of U10.41 (1A5)
- net FPGA_D4: no longer U11.118 (IOT_177)
- net FPGA_D5: no longer names the net of U10.40 (1A6)
- net FPGA_D5: no longer U11.119 (IOT_178)
- net FPGA_D6: no longer names the net of U10.38 (1A7)
- net FPGA_D6: no longer U11.120 (IOT_179)
- net FPGA_D7: no longer names the net of U10.37 (1A8)
- net FPGA_D7: no longer U11.121 (IOT_181)
- net LV_PA0: no longer names the net of U10.36 (2A1)
- net LV_PA1: no longer names the net of U10.35 (2A2)
- net PA0: no longer names the net of U10.13 (2B1)
- net PA1: no longer names the net of U10.14 (2B2)
- net PD24 renamed IPL0
- net PD25 renamed IPL1
- net PD26 renamed IPL2
- net PD27: no longer names the net of U10.6 (1B4)
- net PD28: no longer names the net of U10.8 (1B5)
- net PD29: no longer names the net of U10.9 (1B6)
- net PD30: no longer names the net of U10.11 (1B7)
- net PD31: no longer names the net of U10.12 (1B8)
- new net LV_D0: U11.93 (IOR_140_GBIN3)
- new net LV_D1: U11.94 (IOR_141_GBIN2)
- new net LV_D10: U11.105 (IOR_165)
- new net LV_D11: U11.106 (IOR_166)
- new net LV_D12: U11.107 (IOR_167)
- new net LV_D13: U11.110 (IOT_168)
- new net LV_D14: U11.112 (IOT_169)
- new net LV_D15: U11.113 (IOT_170)
- new net LV_D16: U11.114 (IOT_171)
- new net LV_D17: U11.115 (IOT_172)
- new net LV_D18: U11.116 (IOT_173)
- new net LV_D19: U11.117 (IOT_174)
- new net LV_D2: U11.95 (IOR_144)
- new net LV_D20: U11.118 (IOT_177)
- new net LV_D21: U11.119 (IOT_178)
- new net LV_D22: U11.120 (IOT_179)
- new net LV_D23: U11.121 (IOT_181)
- new net LV_D3: U11.96 (IOR_146)
- new net LV_D4: U11.97 (IOR_147)
- new net LV_D5: U11.98 (IOR_148)
- new net LV_D6: U11.99 (IOR_152)
- new net LV_D7: U11.101 (IOR_160)
- new net LV_D8: U11.102 (IOR_161)
- new net LV_D9: U11.104 (IOR_164)
Other:
- added sheet DataTRX (datatrx.kicad_sch)
- moved on the sheet: U12B

Commit message: root mostly finished
Changed lines of the file:
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@@
+    (effects (font (size 1.27 1.27)) (justify right))
+  )
+  (hierarchical_label "~{COM_IRQ}" (shape input) (at 48.26 104.14 180) (fields_autoplaced)
     (effects (font (size 1.27 1.27)) (justify right))
   )
@@
     (effects (font (size 1.27 1.27)) (justify left))
   )
+  (hierarchical_label "~{COM_IACK}" (shape input) (at 48.26 106.68 180) (fields_autoplaced)
+    (effects (font (size 1.27 1.27)) (justify right))
+  )
   (hierarchical_label "~{TCI}" (shape output) (at 45.72 68.58 180) (fields_autoplaced)

Commit message: work on testboard
Parts:
- added C48, C49, C50, C51, C52, C53, C54, C55, C56, C57, C58, C59, C60, C61: 0.1u, symbol Device:C
- added C62, C63: .1uF, symbol Device:C_Small
- added U18, U19: SN74LVC07, symbol 68040:SN74LVC07
Connections:
- net +3.3V: now also C48.1, C49.1, C50.1, C53.1, C54.1, C55.1, C56.1, C57.1, C58.1, C59.1, C60.1, C61.1, C62.1, C63.1, U18.14 (VCC), U19.11, U19.13, U19.14 (VCC), U19.9
- net +5V: now also U10.17 (2B4), U12.13, C51.1, C52.1
- net FPGA_A_DIR: no longer U11.49 (IOB_81_GBIN5)
- net FPGA_A_~{OE}: no longer U11.48 (IOB_80)
- net FPGA_D_DIR: now also U11.49 (IOB_81_GBIN5)
- net FPGA_D_~{OE}: now also U11.48 (IOB_80)
- net GND: now also U10.1 (1DIR), U10.11 (1B7), U10.12 (1B8), U10.48 (*1OE), U10.9 (1B6), C48.2, C49.2, C50.2, C51.2, C52.2, C53.2, C54.2, C55.2, C56.2, C57.2, C58.2, C59.2, C60.2, C61.2, C62.2, C63.2, U18.7 (GND), U19.7 (GND)
- net LV_RAM_CS: now also U11.42 (IOB_64), U12.3; no longer U11.44 (IOB_72), U12.5
- net LV_R/~{W}: now also U11.144 (IOT_222)
- net LV_SIZ0: now also U10.36 (2A1), U11.138 (IOT_216); no longer U10.33 (2A3)
- net LV_SIZ1: now also U10.35 (2A2), U11.139 (IOT_217); no longer U10.32 (2A4)
- net LV_~{68150_DS}: now also U11.143 (IOT_221)
- net LV_~{TIP}: now also U11.142 (IOT_220)
- net LV_~{TS}: now also U11.141 (IOT_219)
- net SIZ0: now also U10.13 (2B1); no longer U10.16 (2B3)
- net SIZ1: now also U10.14 (2B2); no longer U10.17 (2B4)
- net ~{COM_IACK}: now also U12.6
- net ~{COM_IRQ}: now also U10.16 (2B3)
- net ~{DSACK0}: now also U18.8; no longer U11.21 (IOL_14A_GBIN6)
- net ~{DSACK1}: now also U18.10; no longer U11.22 (IOL_14B)
- net ~{RAM_CS}: now also U12.4; no longer U12.6
- net ~{TA}: now also U18.12
- net ~{TBI}: now also U19.2
- net ~{TCI}: now also U19.4
- net ~{TEA}: now also U19.6
- net LV_TT0: now reaches U11.136 (IOT_214)
- net LV_TT0: now also U10.47 (1A1)
- net LV_TT1: now reaches U11.137 (IOT_215)
- net LV_TT1: now also U10.46 (1A2)
- net LV_~{COM_IACK}: now reaches U11.43 (IOB_71)
- net LV_~{COM_IACK}: now also U12.5
- net LV_TM2: now reaches U10.41 (1A5)
- net LV_TM2: now also U11.25 (IOL_18A)
- net LV_TM1: now reaches U10.43 (1A4)
- net LV_TM1: now also U11.24 (IOL_17B)
- net LV_TM0: now reaches U10.44 (1A3)
- net LV_TM0: now also U11.23 (IOL_17A)
- net TM1: now reaches U10.6 (1B4)
- net TM2: now reaches U10.8 (1B5)
- net LV_~{TA}: now reaches U11.26 (IOL_18B)
- net LV_~{TA}: now also U18.13
- net LV_~{TEA}: now reaches U11.28 (IOL_23A)
- net LV_~{TEA}: now also U19.5
- net LV_~{TBI}: now reaches U11.29 (IOL_23B)
- net LV_~{TBI}: now also U19.1
- net LV_~{TCI}: now reaches U11.31 (IOL_24A)
- net LV_~{TCI}: now also U19.3
- net LV_~{IPL0}: now reaches U11.32 (IOL_24B)
- net LV_~{IPL0}: now also U18.1
- net LV_~{IPL1}: now reaches U11.33 (IOL_25A)
- net LV_~{IPL1}: now also U18.3
- net LV_~{IPL2}: now reaches U11.34 (IOL_25B)
- net LV_~{IPL2}: now also U18.5
- net IPL0 renamed TT0
- net IPL1 renamed TT1
- net IPL2 renamed TM0
- new net LV_~{COM_IRQ}: U10.33 (2A3), U11.44 (IOB_72)
- new net LV_~{DSACK0}: U11.21 (IOL_14A_GBIN6), U18.9
- new net LV_~{DSACK1}: U11.22 (IOL_14B), U18.11
- new net ~{IPL0}: U18.2
- new net ~{IPL1}: U18.4
- new net ~{IPL2}: U18.6
- no-connect marks 0 -> 8
Other:
- moved on the sheet: C30, J2, U11C, U12A, U12B, U12C, U12D, U12E, U12F, U12G

Commit message: simpleboard nearly complete
Parts:
- removed C60, C61: 0.1u, symbol Device:C
- added C60, C69, C72: 4.7uF, Capacitor_SMD:C_0603_1608Metric, symbol Device:C_Small
- added C61, C68, C70, C71: 100nF, Capacitor_SMD:C_0603_1608Metric, symbol Device:C_Small
- added D3: LED, LED_THT:LED_D3.0mm, symbol Device:LED
- added R10: 100, Resistor_SMD:R_0603_1608Metric, symbol Device:R_Small_US
- added R14, R19: 10k, Resistor_SMD:R_0603_1608Metric, symbol Device:R_Small_US
- added R15: 2.2K, Resistor_SMD:R_0603_1608Metric, symbol Device:R_Small_US
- added R23: 1k, Resistor_SMD:R_0603_1608Metric, symbol Device:R_Small_US
- added SW1: Button, Button_Switch_THT:SW_PUSH_6mm, symbol Switch:SW_Push
- C30, C62, C63: value .1uF -> 100nF; footprint (none) -> Capacitor_SMD:C_0603_1608Metric
- C31, C48, C49, C50, C51, C52, C53, C54, C55: value 0.1u -> 100nF; footprint (none) -> Capacitor_SMD:C_0603_1608Metric
- C56, C57, C58, C59: value 0.1u -> 4.7uF; footprint (none) -> Capacitor_SMD:C_0603_1608Metric
- D1: footprint (none) -> LED_SMD:LED_0603_1608Metric
- D2: footprint (none) -> Diode_SMD:D_0603_1608Metric
- J2: footprint (none) -> Connector_JST:JST_PH_B6B-PH-K_1x06_P2.00mm_Vertical
- R16, R17, R18: footprint (none) -> Resistor_SMD:R_0603_1608Metric
- U12, U18, U19: footprint (none) -> Package_SO:TSSOP-14_4.4x5mm_P0.65mm
Connections:
- net +3.3V: now also C60.1, C61.1, R14.1, R15.2, R19.1, R23.1; no longer U11.109 (VPP_FAST), U11.111 (VCC), U11.126 (VCCPLL1), U11.27 (VCC), U11.40 (VCC), U11.54 (VCCPLL0), U11.92 (VCC), U19.11, U19.13, U19.9
- net +5V: no longer U10.17 (2B4)
- net CDONE: now also U19.9, R19.2
- net FPGA_D_DIR: now also U11.48 (IOB_80); no longer U11.49 (IOB_81_GBIN5)
- net FPGA_D_~{OE}: now also U11.47 (IOB_79); no longer U11.48 (IOB_80)
- net GND: now also C60.2, C61.2, C68.2, C69.2, SW1.1; no longer U11.127 (GNDPLL1), U11.53 (GNDPLL0)
- net LV_68150_CS: now also U11.45 (IOB_73); no longer U11.47 (IOB_79)
- net LV_COM_CS: now also U11.44 (IOB_72); no longer U11.45 (IOB_73)
- net LV_RAM_CS: now also U11.41 (IOB_63); no longer U11.42 (IOB_64)
- net LV_~{COM_IRQ}: now also U11.43 (IOB_71); no longer U11.44 (IOB_72)
- net at U19.10: now also D3.1 (K)
- net at U11.66 (~{CRESET}): now also R14.2
- net LV_~{RST}: now reaches U10.32 (2A4)
- net LV_~{RST}: now also U11.49 (IOB_81_GBIN5)
- net ~{FPGA_RDY}: now reaches U19.8
- net FPGA_A_DIR renamed FPGA_LED
- net FPGA_LED: now also U19.11
- net FPGA_A_~{OE} renamed FPGA_BTN
- net FPGA_BTN: now also R23.2, SW1.2
- net LV_~{COM_IACK} renamed LV_COM_IACK
- net LV_COM_IACK: now also U11.42 (IOB_64); no longer U11.43 (IOB_71)
- new net: D3.2 (A), R15.1
- new net +1V2: C68.1, C69.1, R10.2, U11.111 (VCC), U11.27 (VCC), U11.40 (VCC), U11.92 (VCC)
- new net GND_PLL: C70.2, C71.2, C72.2, U11.127 (GNDPLL1), U11.53 (GNDPLL0)
- new net VCC_PLL: C70.1, C71.1, C72.1, R10.1, U11.126 (VCCPLL1), U11.54 (VCCPLL0)
- new net ~{RST}: U10.17 (2B4)
- no-connect marks 8 -> 5
Other:
- sheet AddressBuffer ports: added none; removed FPGA_ABUF_DIR, FPGA_ABUF_~{OE}
- note added: "From VCCIO_2"
- moved on the sheet: C50, U11A, U19E, U19F
