File: hardware/testboard/fpga.kicad_sch (KiCad schematic)
At the start: 66 parts, among them J801 Conn_01x06, SW801 Button, U801 SST26VF023BA, U802 SN74ALVC164245, U803 ICE40HX4K-TQ144, U804 SN74ALVC164245, U805 SN74ALVC164245, U806 SN74ALVC164245, U807 SN74ALVC164245, U808 SN74LVC07, U809 74AHCT04, U810 SN74LVC07

Commit message: layout
Connections:
- net FPGA_DBUF_DIR is gone; now on net FPGA_D_DIR: U804.1 (1DIR), U804.24 (2DIR), U805.1 (1DIR)
- net FPGA_DBUF_~{OE} is gone; now on net FPGA_D_~{OE}: R807.2, U804.25 (*2OE), U804.48 (*1OE), U805.48 (*1OE)
- net A0: now also U807.23 (2B8); no longer U805.23 (2B8)
- net A1: now also U807.22 (2B7); no longer U805.22 (2B7)
- net A2: now also U807.20 (2B6); no longer U805.20 (2B6)
- net A3: now also U807.19 (2B5); no longer U805.19 (2B5)
- net A4: now also U807.17 (2B4); no longer U805.17 (2B4)
- net A5: now also U807.16 (2B3); no longer U805.16 (2B3)
- net A6: now also U807.13 (2B1); no longer U805.14 (2B2)
- net A7: now also U807.14 (2B2); no longer U805.13 (2B1)
- net BCLK: now also U803.20 (IOL_13B_GBIN7); no longer U803.94 (IOR_141_GBIN2)
- net D0: now also U805.23 (2B8); no longer U807.13 (2B1)
- net D1: now also U805.22 (2B7); no longer U807.14 (2B2)
- net D10: now also U805.9 (1B6); no longer U804.5 (1B3)
- net D11: now also U805.8 (1B5); no longer U804.6 (1B4)
- net D12: now also U805.6 (1B4); no longer U804.8 (1B5)
- net D13: now also U805.5 (1B3); no longer U804.11 (1B7)
- net D14: now also U805.3 (1B2); no longer U804.13 (2B1)
- net D15: now also U805.2 (1B1); no longer U804.14 (2B2)
- net D16: now also U804.23 (2B8); no longer U804.9 (1B6)
- net D17: now also U804.22 (2B7); no longer U804.16 (2B3)
- net D18: now also U804.20 (2B6); no longer U804.12 (1B8)
- net D2: now also U805.20 (2B6); no longer U807.17 (2B4)
- net D20: now also U804.17 (2B4); no longer U804.22 (2B7)
- net D21: now also U804.16 (2B3); no longer U805.2 (1B1)
- net D22: now also U804.14 (2B2); no longer U804.20 (2B6)
- net D23: now also U804.13 (2B1); no longer U804.17 (2B4)
- net D24: now also U804.12 (1B8); no longer U805.3 (1B2)
- net D25: now also U804.11 (1B7); no longer U804.23 (2B8)
- net D26: now also U804.9 (1B6); no longer U805.5 (1B3)
- net D27: now also U804.8 (1B5); no longer U805.8 (1B5)
- net D28: now also U804.6 (1B4); no longer U805.6 (1B4)
- net D29: now also U804.5 (1B3); no longer U805.11 (1B7)
- net D3: now also U805.19 (2B5); no longer U807.16 (2B3)
- net D30: now also U804.3 (1B2); no longer U805.12 (1B8)
- net D31: now also U804.2 (1B1); no longer U805.9 (1B6)
- net D4: now also U805.17 (2B4); no longer U807.19 (2B5)
- net D5: now also U805.16 (2B3); no longer U807.20 (2B6)
- net D6: now also U805.14 (2B2); no longer U807.22 (2B7)
- net D7: now also U805.13 (2B1); no longer U807.23 (2B8)
- net D8: now also U805.12 (1B8); no longer U804.2 (1B1)
- net D9: now also U805.11 (1B7); no longer U804.3 (1B2)
- net FLASH_IO2: now also U803.64 (IOB_104_CBSEL1); no longer U803.56 (IOB_94)
- net FLASH_IO3: now also U803.63 (IOB_103_CBSEL0); no longer U803.60 (IOB_95)
- net FPGA_D_DIR: now also U803.110 (IOT_168), U805.24 (2DIR); no longer U803.47 (IOB_79), U803.62 (IOB_102)
- net FPGA_D_~{OE}: now also U803.112 (IOT_169), U805.25 (*2OE); no longer U803.45 (IOB_73), U803.63 (IOB_103_CBSEL0)
- net GND: now also U807.24 (2DIR), U807.25 (*2OE)
- net LV.A0: now also U803.91 (IOR_139), U807.26 (2A8); no longer U805.26 (2A8)
- net LV.A1: now also U803.90 (IOR_138), U807.27 (2A7); no longer U803.34 (IOL_25B), U805.27 (2A7)
- net LV.A10: now also U803.10 (IOL_5B); no longer U803.23 (IOL_17A)
- net LV.A11: now also U803.11 (IOL_8A); no longer U803.22 (IOL_14B)
- net LV.A12: now also U803.12 (IOL_8B); no longer U803.21 (IOL_14A_GBIN6)
- net LV.A13: now also U803.15 (IOL_10A); no longer U803.20 (IOL_13B_GBIN7)
- net LV.A14: now also U803.16 (IOL_10B); no longer U803.19 (IOL_13A)
- net LV.A16: now also U803.17 (IOL_12A); no longer U803.73 (IOR_109)
- net LV.A17: now also U803.19 (IOL_13A); no longer U803.74 (IOR_110)
- net LV.A18: now also U803.22 (IOL_14B); no longer U803.75 (IOR_111)
- net LV.A19: now also U803.21 (IOL_14A_GBIN6); no longer U803.76 (IOR_112)
- net LV.A2: now also U803.88 (IOR_137), U807.29 (2A6); no longer U803.33 (IOL_25A), U805.29 (2A6)
- net LV.A20: now also U803.24 (IOL_17B); no longer U803.78 (IOR_114)
- net LV.A21: now also U803.26 (IOL_18B); no longer U803.79 (IOR_115)
- net LV.A22: now also U803.81 (IOR_117); no longer U803.80 (IOR_116)
- net LV.A23: now also U803.23 (IOL_17A); no longer U803.81 (IOR_117)
- net LV.A24: now also U803.78 (IOR_114); no longer U803.82 (IOR_118)
- net LV.A25: now also U803.25 (IOL_18A); no longer U803.83 (IOR_119)
- net LV.A26: now also U803.80 (IOR_116); no longer U803.84 (IOR_120)
- net LV.A27: now also U803.75 (IOR_111); no longer U803.85 (IOR_128)
- net LV.A28: now also U803.79 (IOR_115); no longer U803.87 (IOR_136)
- net LV.A29: now also U803.74 (IOR_110); no longer U803.88 (IOR_137)
- net LV.A3: now also U803.87 (IOR_136), U807.30 (2A5); no longer U803.32 (IOL_24B), U805.30 (2A5)
- net LV.A30: now also U803.76 (IOR_112); no longer U803.90 (IOR_138)
- net LV.A31: now also U803.73 (IOR_109); no longer U803.91 (IOR_139)
- net LV.A4: now also U803.85 (IOR_128), U807.32 (2A4); no longer U803.31 (IOL_24A), U805.32 (2A4)
- net LV.A5: now also U803.84 (IOR_120), U807.33 (2A3); no longer U803.29 (IOL_23B), U805.33 (2A3)
- net LV.A6: now also U803.82 (IOR_118), U807.36 (2A1); no longer U803.28 (IOL_23A), U805.35 (2A2)
- net LV.A7: now also U803.83 (IOR_119), U807.35 (2A2); no longer U803.26 (IOL_18B), U805.36 (2A1)
- net LV.A8: now also U803.29 (IOL_23B); no longer U803.25 (IOL_18A)
- net LV.A9: now also U803.28 (IOL_23A); no longer U803.24 (IOL_17B)
- net LV_D0: now also U803.9 (IOL_5A), U805.26 (2A8); no longer U803.102 (IOR_161), U804.47 (1A1), U807.36 (2A1)
- net LV_D1: now also U803.8 (IOL_4B), U805.27 (2A7); no longer U803.104 (IOR_164), U804.46 (1A2), U807.35 (2A2)
- net LV_D10: now also U803.141 (IOT_219), U805.40 (1A6); no longer U803.116 (IOT_173), U804.33 (2A3)
- net LV_D11: now also U803.139 (IOT_217), U805.41 (1A5); no longer U803.117 (IOT_174), U804.32 (2A4)
- net LV_D12: now also U803.138 (IOT_216), U805.43 (1A4); no longer U803.118 (IOT_177), U804.30 (2A5)
- net LV_D13: now also U803.137 (IOT_215), U805.44 (1A3); no longer U803.119 (IOT_178), U804.29 (2A6)
- net LV_D14: now also U803.136 (IOT_214), U805.46 (1A2); no longer U803.120 (IOT_179), U804.27 (2A7)
- net LV_D15: now also U803.135 (IOT_213), U805.47 (1A1); no longer U803.121 (IOT_181), U804.26 (2A8)
- net LV_D16: now also U803.134 (IOT_212), U804.26 (2A8); no longer U803.1 (IOL_2A), U805.47 (1A1)
- net LV_D17: now also U803.130 (IOT_206), U804.27 (2A7); no longer U803.144 (IOT_222), U805.46 (1A2)
- net LV_D18: now also U803.129 (IOT_198_GBIN0), U804.29 (2A6); no longer U803.143 (IOT_221), U805.44 (1A3)
- net LV_D19: now also U803.128 (IOT_197_GBIN1), U804.30 (2A5); no longer U803.142 (IOT_220), U805.43 (1A4)
- net LV_D2: now also U803.7 (IOL_4A), U805.29 (2A6); no longer U803.105 (IOR_165), U804.44 (1A3), U807.32 (2A4)
- net LV_D20: now also U803.125 (IOT_192), U804.32 (2A4); no longer U803.141 (IOT_219), U805.41 (1A5)
- net LV_D21: now also U803.124 (IOT_191), U804.33 (2A3); no longer U803.139 (IOT_217), U805.40 (1A6)
- net LV_D22: now also U803.122 (IOT_190), U804.35 (2A2); no longer U803.138 (IOT_216), U805.38 (1A7)
- net LV_D23: now also U803.121 (IOT_181), U804.36 (2A1); no longer U803.137 (IOT_215), U805.37 (1A8)
- net LV_D24: now also U803.120 (IOT_179), U804.37 (1A8); no longer U803.136 (IOT_214)
- net LV_D25: now also U803.119 (IOT_178), U804.38 (1A7); no longer U803.135 (IOT_213)
- net LV_D26: now also U803.118 (IOT_177), U804.40 (1A6); no longer U803.134 (IOT_212)
- net LV_D27: now also U803.117 (IOT_174), U804.41 (1A5); no longer U803.130 (IOT_206)
- net LV_D28: now also U803.116 (IOT_173), U804.43 (1A4); no longer U803.129 (IOT_198_GBIN0)
- net LV_D29: now also U803.115 (IOT_172), U804.44 (1A3); no longer U803.128 (IOT_197_GBIN1)
- net LV_D3: now also U803.4 (IOL_3B), U805.30 (2A5); no longer U803.106 (IOR_166), U804.43 (1A4), U807.33 (2A3)
- net LV_D30: now also U803.114 (IOT_171), U804.46 (1A2); no longer U803.125 (IOT_192)
- net LV_D31: now also U803.113 (IOT_170), U804.47 (1A1); no longer U803.124 (IOT_191)
- net LV_D4: now also U803.3 (IOL_3A), U805.32 (2A4); no longer U803.107 (IOR_167), U804.41 (1A5), U807.30 (2A5)
- net LV_D5: now also U803.2 (IOL_2B), U805.33 (2A3); no longer U803.110 (IOT_168), U804.40 (1A6), U807.29 (2A6)
- net LV_D6: now also U803.1 (IOL_2A), U805.35 (2A2); no longer U803.112 (IOT_169), U804.38 (1A7), U807.27 (2A7)
- net LV_D7: now also U803.144 (IOT_222), U805.36 (2A1); no longer U803.113 (IOT_170), U804.37 (1A8), U807.26 (2A8)
- net LV_D8: now also U803.143 (IOT_221), U805.37 (1A8); no longer U803.114 (IOT_171), U804.36 (2A1)
- net LV_D9: now also U803.142 (IOT_220), U805.38 (1A7); no longer U803.115 (IOT_172), U804.35 (2A2)
- net LV_R/~{W}: no longer U803.122 (IOT_190)
- net LV_SIZ0: no longer U803.96 (IOR_146)
- net LV_SIZ1: no longer U803.97 (IOR_147)
- net LV_TM0: no longer U803.8 (IOL_4B)
- net LV_TM1: no longer U803.9 (IOL_5A)
- net LV_TM2: no longer U803.10 (IOL_5B)
- net LV_TT0: now also U802.35 (2A2); no longer U803.93 (IOR_140_GBIN3)
- net LV_TT1: now also U802.36 (2A1); no longer U803.95 (IOR_144)
- net LV_~{68150_DS}: now also U802.26 (2A8); no longer U803.101 (IOR_160)
- net LV_~{COM_IRQ}: now also U802.33 (2A3); no longer U803.64 (IOB_104_CBSEL1)
- net LV_~{DSACK0}: now also U803.101 (IOR_160); no longer U803.11 (IOL_8A)
- net LV_~{DSACK1}: now also U803.102 (IOR_161); no longer U803.12 (IOL_8B)
- net LV_~{IPL0}: now also U803.105 (IOR_165); no longer U803.2 (IOL_2B)
- net LV_~{IPL1}: now also U803.106 (IOR_166); no longer U803.3 (IOL_3A)
- net LV_~{IPL2}: now also U803.107 (IOR_167); no longer U803.4 (IOL_3B)
- net LV_~{RST}: now also U802.30 (2A5)
- net LV_~{TA}: now also U803.104 (IOR_164); no longer U803.7 (IOL_4A)
- net LV_~{TBI}: no longer U803.17 (IOL_12A)
- net LV_~{TCI}: no longer U803.16 (IOL_10B)
- net LV_~{TEA}: no longer U803.15 (IOL_10A)
- net LV_~{TIP}: no longer U803.99 (IOR_152)
- net LV_~{TS}: no longer U803.98 (IOR_148)
- net R/~{W}: now also U802.9 (1B6); no longer U802.6 (1B4)
- net SIZ1: now also U802.6 (1B4); no longer U802.9 (1B6)
- net TT0: now also U802.14 (2B2)
- net TT1: now also U802.13 (2B1)
- net ~{68150_DS}: now also U802.23 (2B8)
Other:
- moved on the sheet: C834, C835, C838, C839, C841, C842, U803B, U803C, U803D
