File: hardware/testboard/clock.kicad_sch (KiCad schematic)
At the start: 6 parts, among them U27 NB3N502, X1 ASE-33MHz, X2 33MHz, X3 33MHz

Commit message: work on testboard, move 3d models
Parts:
- removed C20: .01uF, symbol Device:C
- removed C4: .1uF, symbol Device:C
- removed U27: NB3N502, Package_SO:SOIC-8_3.9x4.9mm_P1.27mm, symbol 68040:NB3N502
- removed X2: 33MHz, Oscillator:Oscillator_DIP-14, symbol Oscillator:CXO_DIP8
- added C23: .1uF, symbol Device:C
- added C24: .01uF, symbol Device:C
- added U8: NB3N502, Package_SO:SOIC-8_3.9x4.9mm_P1.27mm, symbol 68040:NB3N502
- added X2: 33MHz, Oscillator:Oscillator_DIP-14, symbol Oscillator:CXO_DIP14
Connections:
- net +3.3V: now also C23.1, C24.1, U8.2 (VDD), X2.1 (EN), X2.14 (Vcc)
- net BCLK: now also U8.4 (REF)
- net GND: now also C23.2, C24.2, U8.3 (GND), U8.6 (S0), U8.7 (S1), X2.7 (GND)
- net PCLK: now also U8.5 (CLKOUT)
- net CLK33: now reaches X1.3 (OUT), X3.5 (OUT)
- net CLK33: now also U8.1 (X1/CLK), X2.8 (OUT)

Commit message: simpleboard nearly complete
Parts:
- C23: value .1uF -> 100nF; footprint (none) -> Capacitor_SMD:C_0603_1608Metric
- C24: value .01uF -> 100nF; footprint (none) -> Capacitor_SMD:C_0603_1608Metric
Changed lines of the file:
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@@
       (effects (font (size 1.27 1.27)) (justify left))
     )
-    (property "Value" ".01uF" (at 113.03 53.34 0)
+    (property "Value" "100nF" (at 113.03 53.34 0)
       (effects (font (size 1.27 1.27)) (justify left))
     )
-    (property "Footprint" "" (at 115.8748 55.88 0)
+    (property "Footprint" "Capacitor_SMD:C_0603_1608Metric" (at 115.8748 55.88 0)
       (effects (font (size 1.27 1.27)) hide)
     )
@@
       (effects (font (size 1.27 1.27)) (justify left))
     )
-    (property "Value" ".1uF" (at 85.09 40.64 0)
+    (property "Value" "100nF" (at 85.09 40.64 0)
       (effects (font (size 1.27 1.27)) (justify left))
     )
-    (property "Footprint" "" (at 82.2452 43.18 0)
+    (property "Footprint" "Capacitor_SMD:C_0603_1608Metric" (at 82.2452 43.18 0)
       (effects (font (size 1.27 1.27)) hide)
     )

Commit message: pinouts
Parts:
- renumbered C23 to C401, C24 to C402, U8 to U401, X1 to X401, X2 to X402, X3 to X403
Changed lines of the file:
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@@
   (symbol (lib_id "power:+3.3V") (at 99.06 33.02 0) (unit 1)
     (in_bom yes) (on_board yes) (dnp no) (fields_autoplaced)
-    (property "Reference" "#PWR023" (at 99.06 36.83 0)
+    (property "Reference" "#PWR0401" (at 99.06 36.83 0)
       (effects (font (size 1.27 1.27)) hide)
     )
@@
       (project "testboard"
         (path "/a1ce156a-fb78-423b-b05a-d07384e5c8a7/9c02df45-eefc-4cd9-a46c-364699428858"
-          (reference "#PWR023") (unit 1)
+          (reference "#PWR0401") (unit 1)
         )
       )
@@
   (symbol (lib_id "power:+3.3V") (at 134.62 35.56 0) (unit 1)
     (in_bom yes) (on_board yes) (dnp no) (fields_autoplaced)
-    (property "Reference" "#PWR024" (at 134.62 39.37 0)
+    (property "Reference" "#PWR0404" (at 134.62 39.37 0)
       (effects (font (size 1.27 1.27)) hide)
     )
@@
       (project "testboard"
         (path "/a1ce156a-fb78-423b-b05a-d07384e5c8a7/9c02df45-eefc-4cd9-a46c-364699428858"
-          (reference "#PWR024") (unit 1)
+          (reference "#PWR0404") (unit 1)
         )
       )
@@
   (symbol (lib_id "Oscillator:CXO_DIP14") (at 60.96 40.64 0) (unit 1)
     (in_bom yes) (on_board yes) (dnp no) (fields_autoplaced)
-    (property "Reference" "X2" (at 71.12 36.9921 0)
+    (property "Reference" "X402" (at 71.12 36.9921 0)
       (effects (font (size 1.27 1.27)))
     )
@@
       (project "testboard"
         (path "/a1ce156a-fb78-423b-b05a-d07384e5c8a7/9c02df45-eefc-4cd9-a46c-364699428858"
-          (reference "X2") (unit 1)
+          (reference "X402") (unit 1)
         )
       )
@@
   (symbol (lib_id "power:GND") (at 99.06 48.26 0) (unit 1)
     (in_bom yes) (on_board yes) (dnp no) (fields_autoplaced)
-    (property "Reference" "#PWR025" (at 99.06 54.61 0)
+    (property "Reference" "#PWR0402" (at 99.06 54.61 0)
       (effects (font (size 1.27 1.27)) hide)
     )
@@
       (project "testboard"
         (path "/a1ce156a-fb78-423b-b05a-d07384e5c8a7/9c02df45-eefc-4cd9-a46c-364699428858"
-          (reference "#PWR025") (unit 1)
+          (reference "#PWR0402") (unit 1)
         )
       )
@@
   (symbol (lib_id "Oscillator:ASE-xxxMHz") (at 33.02 40.64 0) (unit 1)
     (in_bom yes) (on_board yes) (dnp no) (fields_autoplaced)
-    (property "Reference" "X1" (at 45.72 36.9921 0)
+    (property "Reference" "X401" (at 45.72 36.9921 0)
       (effects (font (size 1.27 1.27)))
     )
@@
       (project "testboard"
         (path "/a1ce156a-fb78-423b-b05a-d07384e5c8a7/9c02df45-eefc-4cd9-a46c-364699428858"
-          (reference "X1") (unit 1)
+          (reference "X401") (unit 1)
         )
       )
@@
   (symbol (lib_id "Device:C") (at 116.84 52.07 0) (mirror y) (unit 1)
     (in_bom yes) (on_board yes) (dnp no)
-    (property "Reference" "C24" (at 113.03 50.8 0)
+    (property "Reference" "C402" (at 113.03 50.8 0)
       (effects (font (size 1.27 1.27)) (justify left))
     )
@@
       (project "testboard"
         (path "/a1ce156a-fb78-423b-b05a-d07384e5c8a7/9c02df45-eefc-4cd9-a46c-364699428858"
-          (reference "C24") (unit 1)
+          (reference "C402") (unit 1)
         )
       )
@@
   (symbol (lib_id "power:GND") (at 134.62 55.88 0) (unit 1)
     (in_bom yes) (on_board yes) (dnp no) (fields_autoplaced)
-    (property "Reference" "#PWR027" (at 134.62 62.23 0)
+    (property "Reference" "#PWR0405" (at 134.62 62.23 0)
       (effects (font (size 1.27 1.27)) hide)
     )
@@
       (project "testboard"
         (path "/a1ce156a-fb78-423b-b05a-d07384e5c8a7/9c02df45-eefc-4cd9-a46c-364699428858"
-          (reference "#PWR027") (unit 1)
+          (reference "#PWR0405") (unit 1)
         )
       )
@@
   (symbol (lib_id "power:+3.3V") (at 116.84 48.26 0) (unit 1)
     (in_bom yes) (on_board yes) (dnp no) (fields_autoplaced)
-    (property "Reference" "#PWR026" (at 116.84 52.07 0)
+    (property "Reference" "#PWR0403" (at 116.84 52.07 0)
       (effects (font (size 1.27 1.27)) hide)
     )
@@
       (project "testboard"
         (path "/a1ce156a-fb78-423b-b05a-d07384e5c8a7/9c02df45-eefc-4cd9-a46c-364699428858"
-          (reference "#PWR026") (unit 1)
+          (reference "#PWR0403") (unit 1)
         )
       )
@@
   (symbol (lib_id "Device:C") (at 81.28 39.37 0) (unit 1)
     (in_bom yes) (on_board yes) (dnp no) (fields_autoplaced)
-    (property "Reference" "C23" (at 85.09 38.1 0)
+    (property "Reference" "C401" (at 85.09 38.1 0)
       (effects (font (size 1.27 1.27)) (justify left))
     )
@@
       (project "testboard"
         (path "/a1ce156a-fb78-423b-b05a-d07384e5c8a7/9c02df45-eefc-4cd9-a46c-364699428858"
-          (reference "C23") (unit 1)
+          (reference "C401") (unit 1)
         )
       )
@@
   (symbol (lib_id "Oscillator:CXO_DIP8") (at 99.06 40.64 0) (unit 1)
     (in_bom yes) (on_board yes) (dnp no) (fields_autoplaced)
-    (property "Reference" "X3" (at 110.49 36.9921 0)
+    (property "Reference" "X403" (at 110.49 36.9921 0)
       (effects (font (size 1.27 1.27)))
     )
@@
       (project "testboard"
         (path "/a1ce156a-fb78-423b-b05a-d07384e5c8a7/9c02df45-eefc-4cd9-a46c-364699428858"
-          (reference "X3") (unit 1)
+          (reference "X403") (unit 1)
         )
       )
@@
   (symbol (lib_id "68040:NB3N502") (at 134.62 45.72 0) (unit 1)
     (in_bom yes) (on_board yes) (dnp no) (fields_autoplaced)
-    (property "Reference" "U8" (at 136.8141 33.02 0)
+    (property "Reference" "U401" (at 136.8141 33.02 0)
       (effects (font (size 1.27 1.27)) (justify left))
     )
@@
       (project "testboard"
         (path "/a1ce156a-fb78-423b-b05a-d07384e5c8a7/9c02df45-eefc-4cd9-a46c-364699428858"
-          (reference "U8") (unit 1)
-        )
-      )
+          (reference "U401") (unit 1)
+        )
+      )

Commit message: testboard - schematic and route done
Connections:
- net CLK33: no longer X402.8 (OUT)
- net GND: no longer X402.7 (GND)
- no-connect marks 1 -> 3
Changed lines of the file:
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@@
   (junction (at 91.44 33.02) (diameter 0) (color 0 0 0 0)
-  )
-  (junction (at 60.96 48.26) (diameter 0) (color 0 0 0 0)
   )
   (junction (at 121.92 55.88) (diameter 0) (color 0 0 0 0)
@@
   (junction (at 81.28 48.26) (diameter 0) (color 0 0 0 0)
   )
-  (junction (at 76.2 25.4) (diameter 0) (color 0 0 0 0)
-  )
   (junction (at 81.28 33.02) (diameter 0) (color 0 0 0 0)
   )
@@
   (junction (at 99.06 48.26) (diameter 0) (color 0 0 0 0)
   )
+  (no_connect (at 60.96 48.26))
+  (no_connect (at 68.58 40.64))
   (no_connect (at 124.46 43.18))
-  (wire (pts (xy 60.96 48.26) (xy 81.28 48.26))
+  (wire (pts (xy 33.02 50.8) (xy 81.28 50.8))
     (stroke (width 0) (type default))
   )
@@
     (stroke (width 0) (type default))
   )
-  (wire (pts (xy 76.2 25.4) (xy 119.38 25.4))
+  (wire (pts (xy 48.26 25.4) (xy 119.38 25.4))
+    (stroke (width 0) (type default))
+  )
+  (wire (pts (xy 81.28 50.8) (xy 81.28 48.26))
     (stroke (width 0) (type default))
   )
@@
     (stroke (width 0) (type default))
   )
-  (wire (pts (xy 33.02 48.26) (xy 60.96 48.26))
-    (stroke (width 0) (type default))
-  )
   (wire (pts (xy 121.92 50.8) (xy 121.92 55.88))
     (stroke (width 0) (type default))
   )
-  (wire (pts (xy 68.58 40.64) (xy 76.2 40.64))
+  (wire (pts (xy 33.02 50.8) (xy 33.02 48.26))
     (stroke (width 0) (type default))
   )
@@
     (stroke (width 0) (type default))
   )
-  (wire (pts (xy 76.2 40.64) (xy 76.2 25.4))
-    (stroke (width 0) (type default))
-  )
   (wire (pts (xy 91.44 33.02) (xy 91.44 40.64))
     (stroke (width 0) (type default))
@@
     (stroke (width 0) (type default))
   )
-  (wire (pts (xy 48.26 25.4) (xy 76.2 25.4))
-    (stroke (width 0) (type default))
-  )
