File: hardware/testboard/cpu.kicad_sch (KiCad schematic)
At the start: 23 parts, among them U1 68LC040

Commit message: work on testboard, move 3d models
Parts:
- removed R6: 4.7k, symbol Device:R
Connections:
- net SC0 is gone; now on net GND: U1.T12 (SC0)
- net SC1 is gone; now on net GND: U1.S12 (SC1)
- net ~{BG} is gone; now on net GND: U1.T13 (~{BG})
- net ~{BB}: now also R16.2
- net ~{MI}: now also R17.2
- net ~{BR}: no longer names the net of U1.T18 (~{BR})
- net ~{LOCKE}: no longer names the net of U1.R18 (~{LOCKE})
- net ~{LOCK}: no longer names the net of U1.S18 (~{LOCK})
- no-connect marks 11 -> 14

Commit message: work on testboard
Parts:
- added C19: 100nF, symbol Device:C
- added U5: 74LVC1G04, symbol 74xGxx:74LVC1G04
Connections:
- net +5V: now also C19.1, U5.5 (VCC)
- net GND: now also C19.2, U5.3 (GND)
- net R/~{W}: now also U5.2
- net ~{TA}: now also R14.2
- net ~{TEA}: now also R13.2
- net ~{TIP}: now also R15.2
- net ~{TCI}: now reaches R12.2
- net ~{TCI}: now also U1.T10 (~{TCI})
- net ~{TBI}: now reaches R11.2
- net ~{TBI}: now also U1.S11 (~{TBI})
- removed net ~{TCI}/~{TBI}: U1.S11 (~{TBI}), U1.T10 (~{TCI})
- new net ~{R}/W: U5.4

Commit message: simpleboard nearly complete
Parts:
- removed R18, R22, R23: 4.7k, symbol Device:R_Small_US
- removed RN3: 4.7k, Resistor_THT:R_Array_SIP6, symbol Device:R_Network05_Split
- added FB1: FerriteBead, Inductor_SMD:L_0805_2012Metric_Pad1.15x1.40mm_HandSolder, symbol Device:FerriteBead_Small
- added R26, R27, R28, R29: 4.7k, Resistor_SMD:R_0603_1608Metric, symbol Device:R_Small_US
- added RN2: 1k, Resistor_THT:R_Array_SIP10, symbol Device:R_Network09_US
- C10, C11, C13, C15, C19: footprint (none) -> Capacitor_SMD:C_0603_1608Metric
- C12, C14: footprint (none) -> Capacitor_THT:CP_Radial_D5.0mm_P2.00mm
- R10, R11, R12, R13, R14, R15, R16, R17, R19, R20, R21: footprint (none) -> Resistor_SMD:R_0603_1608Metric
- U5: footprint (none) -> Package_TO_SOT_SMD:SOT-23-5
Connections:
- net +5V: now also R26.1, R27.1, R28.1, R29.1, RN2.1 (common)
- net DLE: now also R29.2
- net R/~{W}: now also RN2.10 (R9)
- net SIZ0: now also RN2.8 (R7)
- net SIZ1: now also RN2.7 (R6)
- net TM0: now also RN2.6 (R5)
- net TM1: now also RN2.5 (R4)
- net TM2: now also RN2.4 (R3)
- net TT0: now also RN2.3 (R2)
- net TT1: now also RN2.2 (R1)
- net ~{RSTO}: now also R26.2
- net ~{TS}: now also FB1.2, R27.2; no longer U1.R16 (~{TS})
- net at U1.S6 (~{MDIS}), U1.T5 (~{CDIS}): now also R28.2
- net at U1.S3 (TDI), U1.S5 (TMS): now also R10.2
- new net: FB1.1, U1.R16 (~{TS})
- no-connect marks 14 -> 15
Other:
- moved on the sheet: R10

Commit message: pinouts
Parts:
- renumbered C19 to C207, FB1 to FB201, R26 to R201, R28 to R203, R27 to R214, R29 to R215, RN2 to RN201, U1 to U201, U5 to U202

Commit message: testboard - schematic and route done
Changed lines of the file:
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@@
     (effects (font (size 1.27 1.27)) (justify left bottom))
-  )
-  (label "~{SW_RST}" (at 81.28 99.06 180) (fields_autoplaced)
-    (effects (font (size 1.27 1.27)) (justify right bottom))
   )
   (label "R{slash}~{W}" (at 38.1 142.24 180) (fields_autoplaced)
@@
     (effects (font (size 1.27 1.27)) (justify left bottom))
   )
-  (label "~{HW_RST}" (at 81.28 101.6 180) (fields_autoplaced)
-    (effects (font (size 1.27 1.27)) (justify right bottom))
-  )
   (label "~{BB}" (at 35.56 48.26 0) (fields_autoplaced)
