File: hardware/testboard/testboard.kicad_pcb (KiCad board)
At the start: 4 copper layers, 143 parts, among them J1 Barrel_Jack, J2 Conn_01x06, SW1 Button, SW2 Button, U1 68LC040, U10 SN74ALVC164245, U11 ICE40HX4K-TQ144, U12 74AHCT04, U13 SST26VF023BA, U14 SN74ALVC164245, U15 SN74ALVC164245, U16 SN74ALVC164245, U17 SN74ALVC164245, U18 SN74LVC07, U19 SN74LVC07, U2 MAX232, U20 AP2112K-3.3, U21 AP2112K-1.2, U22 74LVC1G08, U23 TL7705A, U3 MAX232, U4 68681, U5 74LVC1G04, U6 IS61C5128AS-25TLI, U7 IS61C5128AS-25TLI, U8 NB3N502, X1 ASE-33MHz, X2 33MHz, X3 33MHz, Y1 3.6864MHz

Commit message: I ripped it all apart
Parts:
- moved R26 144.3 mm to (97.5, 149.7), turned to 90 degrees
- moved C6 143.2 mm to (89.9, 139.2), turned to 90 degrees
- moved R1 141.1 mm to (100.1, 149.7), turned to 90 degrees
- moved R28 138.1 mm to (102.6, 149.7), turned to 90 degrees
- moved R11 135.2 mm to (105.2, 149.7), turned to 90 degrees
- moved R12 132.5 mm to (107.7, 149.7), turned to 90 degrees
- moved R13 129.9 mm to (110.2, 149.7), turned to 90 degrees
- moved R29 127.4 mm to (112.8, 149.7), turned to 90 degrees
- moved R4 125.1 mm to (115.3, 149.7), turned to 90 degrees
- moved R3 123.0 mm to (117.9, 149.7), turned to 90 degrees
- moved R5 121.0 mm to (120.4, 149.7), turned to 90 degrees
- moved R6 119.2 mm to (122.9, 149.7), turned to 90 degrees
- moved R7 117.6 mm to (125.5, 149.7), turned to 90 degrees
- moved R9 116.2 mm to (128.0, 149.7), turned to 90 degrees
- moved FB1 115.4 mm to (130.6, 149.9), turned to -90 degrees
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Connections:
- C42 pad 1: +5V -> +3.3V
- C43 pad 1: +5V -> +3.3V
- C44 pad 1: +3.3V -> +5V
- C45 pad 1: +3.3V -> +5V
- U10 pad 11: GND -> /SIZ1
- U10 pad 12: GND -> /SIZ0
- U10 pad 13: /SIZ0 -> /R/~{W}
- U10 pad 14: /SIZ1 -> unconnected-(U10A-2B2-Pad14)
- U10 pad 17: /~{RST} -> unconnected-(U10A-2B4-Pad17)
- U10 pad 19: /~{TS} -> /~{RST}
- U10 pad 2: /TT0 -> /~{DS}
- U10 pad 22: /~{DS} -> /~{TS}
- U10 pad 23: /R/~{W} -> unconnected-(U10A-2B8-Pad23)
- U10 pad 26: /FPGA/LV_R/~{W} -> unconnected-(U10A-2A8-Pad26)
- U10 pad 27: /FPGA/LV_~{68150_DS} -> unconnected-(U10A-2A7-Pad27)
- U10 pad 29: /FPGA/LV_~{TIP} -> unconnected-(U10A-2A6-Pad29)
- U10 pad 30: /FPGA/LV_~{TS} -> unconnected-(U10A-2A5-Pad30)
- U10 pad 32: /FPGA/LV_~{RST} -> unconnected-(U10A-2A4-Pad32)
- U10 pad 33: /FPGA/LV_~{COM_IRQ} -> unconnected-(U10A-2A3-Pad33)
- U10 pad 35: /FPGA/LV_SIZ1 -> unconnected-(U10A-2A2-Pad35)
- U10 pad 36: /FPGA/LV_SIZ0 -> unconnected-(U10A-2A1-Pad36)
- U10 pad 41: /FPGA/LV_TM2 -> unconnected-(U10A-1A5-Pad41)
- U10 pad 43: /FPGA/LV_TM1 -> unconnected-(U10A-1A4-Pad43)
- U10 pad 44: /FPGA/LV_TM0 -> unconnected-(U10A-1A3-Pad44)
- U10 pad 46: /FPGA/LV_TT1 -> unconnected-(U10A-1A2-Pad46)
- U10 pad 47: /FPGA/LV_TT0 -> unconnected-(U10A-1A1-Pad47)
- U10 pad 5: /TM0 -> /TT0
- U10 pad 6: /TM1 -> /TM2
- U10 pad 8: /TM2 -> /TM1
- U10 pad 9: GND -> /TM0
- U11 pad 1: /FPGA/LV.A15 -> unconnected-(U11D-IOL_2A-Pad1)
- U11 pad 10: /FPGA/LV.A8 -> unconnected-(U11D-IOL_5B-Pad10)
- U11 pad 101: /FPGA/LV_D7 -> unconnected-(U11B-IOR_160-Pad101)
- U11 pad 102: /FPGA/LV_D8 -> unconnected-(U11B-IOR_161-Pad102)
- U11 pad 104: /FPGA/LV_D9 -> unconnected-(U11B-IOR_164-Pad104)
- U11 pad 105: /FPGA/LV_D10 -> unconnected-(U11B-IOR_165-Pad105)
- U11 pad 106: /FPGA/LV_D11 -> unconnected-(U11B-IOR_166-Pad106)
- U11 pad 107: /FPGA/LV_D12 -> unconnected-(U11B-IOR_167-Pad107)
- U11 pad 11: /FPGA/LV.A7 -> unconnected-(U11D-IOL_8A-Pad11)
- U11 pad 110: /FPGA/LV_D13 -> unconnected-(U11A-IOT_168-Pad110)
- U11 pad 112: /FPGA/LV_D14 -> unconnected-(U11A-IOT_169-Pad112)
- U11 pad 113: /FPGA/LV_D15 -> unconnected-(U11A-IOT_170-Pad113)
- U11 pad 114: /FPGA/LV_D16 -> unconnected-(U11A-IOT_171-Pad114)
- U11 pad 115: /FPGA/LV_D17 -> unconnected-(U11A-IOT_172-Pad115)
- U11 pad 116: /FPGA/LV_D18 -> unconnected-(U11A-IOT_173-Pad116)
- U11 pad 117: /FPGA/LV_D19 -> unconnected-(U11A-IOT_174-Pad117)
- U11 pad 118: /FPGA/LV_D20 -> unconnected-(U11A-IOT_177-Pad118)
- U11 pad 119: /FPGA/LV_D21 -> unconnected-(U11A-IOT_178-Pad119)
- U11 pad 12: /FPGA/LV.A6 -> unconnected-(U11D-IOL_8B-Pad12)
- U11 pad 120: /FPGA/LV_D22 -> unconnected-(U11A-IOT_179-Pad120)
- U11 pad 121: /FPGA/LV_D23 -> unconnected-(U11A-IOT_181-Pad121)
- U11 pad 122: /FPGA/LV_D24 -> unconnected-(U11A-IOT_190-Pad122)
- U11 pad 124: /FPGA/LV_D25 -> unconnected-(U11A-IOT_191-Pad124)
- U11 pad 125: /FPGA/LV_D26 -> unconnected-(U11A-IOT_192-Pad125)
- U11 pad 128: /FPGA/LV_D27 -> unconnected-(U11A-IOT_197_GBIN1-Pad128)
- U11 pad 129: /FPGA/LV_D28 -> unconnected-(U11A-IOT_198_GBIN0-Pad129)
- U11 pad 130: /FPGA/LV_D29 -> unconnected-(U11A-IOT_206-Pad130)
- U11 pad 134: /FPGA/LV_D30 -> unconnected-(U11A-IOT_212-Pad134)
- U11 pad 135: /FPGA/LV_D31 -> unconnected-(U11A-IOT_213-Pad135)
- U11 pad 136: /FPGA/LV_TT0 -> unconnected-(U11A-IOT_214-Pad136)
- U11 pad 137: /FPGA/LV_TT1 -> unconnected-(U11A-IOT_215-Pad137)
- U11 pad 138: /FPGA/LV_SIZ0 -> unconnected-(U11A-IOT_216-Pad138)
- U11 pad 139: /FPGA/LV_SIZ1 -> unconnected-(U11A-IOT_217-Pad139)
- U11 pad 141: /FPGA/LV_~{TS} -> unconnected-(U11A-IOT_219-Pad141)
- U11 pad 142: /FPGA/LV_~{TIP} -> unconnected-(U11A-IOT_220-Pad142)
- U11 pad 143: /FPGA/LV_~{68150_DS} -> unconnected-(U11A-IOT_221-Pad143)
- U11 pad 144: /FPGA/LV_R/~{W} -> unconnected-(U11A-IOT_222-Pad144)
- U11 pad 15: /FPGA/LV.A5 -> unconnected-(U11D-IOL_10A-Pad15)
- U11 pad 16: /FPGA/LV.A4 -> unconnected-(U11D-IOL_10B-Pad16)
- U11 pad 17: /FPGA/LV.A3 -> unconnected-(U11D-IOL_12A-Pad17)
- U11 pad 18: /FPGA/LV.A2 -> unconnected-(U11D-IOL_12B-Pad18)
- U11 pad 19: /FPGA/LV.A1 -> unconnected-(U11D-IOL_13A-Pad19)
- U11 pad 2: /FPGA/LV.A14 -> unconnected-(U11D-IOL_2B-Pad2)
- U11 pad 20: /FPGA/LV.A0 -> unconnected-(U11D-IOL_13B_GBIN7-Pad20)
- U11 pad 21: /BCLK -> unconnected-(U11D-IOL_14A_GBIN6-Pad21)
- U11 pad 23: /FPGA/LV_TM0 -> unconnected-(U11D-IOL_17A-Pad23)
- U11 pad 24: /FPGA/LV_TM1 -> unconnected-(U11D-IOL_17B-Pad24)
- U11 pad 25: /FPGA/LV_TM2 -> unconnected-(U11D-IOL_18A-Pad25)
- U11 pad 28: /FPGA/LV_~{IPL0} -> unconnected-(U11D-IOL_23A-Pad28)
- U11 pad 29: /FPGA/LV_~{IPL1} -> unconnected-(U11D-IOL_23B-Pad29)
- U11 pad 3: /FPGA/LV.A13 -> unconnected-(U11D-IOL_3A-Pad3)
- U11 pad 31: /FPGA/LV_~{IPL2} -> unconnected-(U11D-IOL_24A-Pad31)
- U11 pad 32: /FPGA/LV_~{DSACK0} -> unconnected-(U11D-IOL_24B-Pad32)
- U11 pad 33: /FPGA/LV_~{DSACK1} -> unconnected-(U11D-IOL_25A-Pad33)
- U11 pad 34: /FPGA/LV_~{TA} -> unconnected-(U11D-IOL_25B-Pad34)
- U11 pad 37: /FPGA/LV_~{TEA} -> unconnected-(U11C-IOB_56-Pad37)
- U11 pad 38: /FPGA/LV_~{TCI} -> unconnected-(U11C-IOB_57-Pad38)
- U11 pad 39: /FPGA/LV_~{TBI} -> unconnected-(U11C-IOB_61-Pad39)
- U11 pad 4: /FPGA/LV.A12 -> unconnected-(U11D-IOL_3B-Pad4)
- U11 pad 41: /FPGA/LV_COM_IACK -> unconnected-(U11C-IOB_63-Pad41)
- U11 pad 42: /FPGA/LV_RAM_CS -> unconnected-(U11C-IOB_64-Pad42)
- U11 pad 43: /FPGA/LV_AVEC -> unconnected-(U11C-IOB_71-Pad43)
- U11 pad 44: /FPGA/LV_COM_CS -> unconnected-(U11C-IOB_72-Pad44)
- U11 pad 45: /FPGA/LV_68150_CS -> unconnected-(U11C-IOB_73-Pad45)
- U11 pad 47: /FPGA/FPGA_D_~{OE} -> unconnected-(U11C-IOB_79-Pad47)
- U11 pad 48: /FPGA/FPGA_D_DIR -> unconnected-(U11C-IOB_80-Pad48)
- U11 pad 49: /FPGA/LV_~{RST} -> unconnected-(U11C-IOB_81_GBIN5-Pad49)
- U11 pad 55: /FPGA/FPGA_LED -> unconnected-(U11C-IOB_91-Pad55)
- U11 pad 56: /FPGA/FPGA_BTN -> unconnected-(U11C-IOB_94-Pad56)
- U11 pad 60: /FPGA/FLASH_IO2 -> unconnected-(U11C-IOB_95-Pad60)
- U11 pad 61: /FPGA/FLASH_IO3 -> unconnected-(U11C-IOB_96-Pad61)
- U11 pad 63: /FPGA/FPGA_D_DIR -> unconnected-(U11C-IOB_103_CBSEL0-Pad63)
- U11 pad 64: /FPGA/FPGA_D_~{OE} -> unconnected-(U11C-IOB_104_CBSEL1-Pad64)
- U11 pad 7: /FPGA/LV.A11 -> unconnected-(U11D-IOL_4A-Pad7)
- U11 pad 73: /FPGA/LV.A16 -> unconnected-(U11B-IOR_109-Pad73)
- U11 pad 74: /FPGA/LV.A17 -> unconnected-(U11B-IOR_110-Pad74)
- U11 pad 75: /FPGA/LV.A18 -> unconnected-(U11B-IOR_111-Pad75)
- U11 pad 76: /FPGA/LV.A19 -> unconnected-(U11B-IOR_112-Pad76)
- U11 pad 78: /FPGA/LV.A20 -> unconnected-(U11B-IOR_114-Pad78)
- U11 pad 79: /FPGA/LV.A21 -> unconnected-(U11B-IOR_115-Pad79)
- U11 pad 8: /FPGA/LV.A10 -> unconnected-(U11D-IOL_4B-Pad8)
- U11 pad 80: /FPGA/LV.A22 -> unconnected-(U11B-IOR_116-Pad80)
- U11 pad 81: /FPGA/LV.A23 -> unconnected-(U11B-IOR_117-Pad81)
- U11 pad 82: /FPGA/LV.A24 -> unconnected-(U11B-IOR_118-Pad82)
- U11 pad 83: /FPGA/LV.A25 -> unconnected-(U11B-IOR_119-Pad83)
- U11 pad 84: /FPGA/LV.A26 -> unconnected-(U11B-IOR_120-Pad84)
- U11 pad 85: /FPGA/LV.A27 -> unconnected-(U11B-IOR_128-Pad85)
- U11 pad 87: /FPGA/LV.A28 -> unconnected-(U11B-IOR_136-Pad87)
- U11 pad 88: /FPGA/LV.A29 -> unconnected-(U11B-IOR_137-Pad88)
- U11 pad 9: /FPGA/LV.A9 -> unconnected-(U11D-IOL_5A-Pad9)
- U11 pad 90: /FPGA/LV.A30 -> unconnected-(U11B-IOR_138-Pad90)
- U11 pad 91: /FPGA/LV.A31 -> unconnected-(U11B-IOR_139-Pad91)
- U11 pad 93: /FPGA/LV_D0 -> unconnected-(U11B-IOR_140_GBIN3-Pad93)
- U11 pad 94: /FPGA/LV_D1 -> unconnected-(U11B-IOR_141_GBIN2-Pad94)
- U11 pad 95: /FPGA/LV_D2 -> unconnected-(U11B-IOR_144-Pad95)
- U11 pad 96: /FPGA/LV_D3 -> unconnected-(U11B-IOR_146-Pad96)
- U11 pad 97: /FPGA/LV_D4 -> unconnected-(U11B-IOR_147-Pad97)
- U11 pad 98: /FPGA/LV_D5 -> unconnected-(U11B-IOR_148-Pad98)
- U11 pad 99: /FPGA/LV_D6 -> unconnected-(U11B-IOR_152-Pad99)
- U14 pad 11: /A9 -> /A6
- U14 pad 12: /A8 -> /A7
- U14 pad 13: /A7 -> /A8
- U14 pad 14: /A6 -> /A9
- U14 pad 16: /A5 -> /A10
- U14 pad 17: /A4 -> /A11
- U14 pad 19: /A3 -> /A12
- U14 pad 2: /A15 -> /A0
- U14 pad 20: /A2 -> /A13
- U14 pad 22: /A1 -> /A14
- U14 pad 23: /A0 -> /A15
- U14 pad 26: /FPGA/LV.A0 -> /FPGA/LV.A15
- U14 pad 27: /FPGA/LV.A1 -> /FPGA/LV.A14
- U14 pad 29: /FPGA/LV.A2 -> /FPGA/LV.A13
- U14 pad 3: /A14 -> /A1
- U14 pad 30: /FPGA/LV.A3 -> /FPGA/LV.A12
- U14 pad 32: /FPGA/LV.A4 -> /FPGA/LV.A11
- U14 pad 33: /FPGA/LV.A5 -> /FPGA/LV.A10
- U14 pad 35: /FPGA/LV.A6 -> /FPGA/LV.A9
- U14 pad 36: /FPGA/LV.A7 -> /FPGA/LV.A8
- U14 pad 37: /FPGA/LV.A8 -> /FPGA/LV.A7
- U14 pad 38: /FPGA/LV.A9 -> /FPGA/LV.A6
- U14 pad 40: /FPGA/LV.A10 -> /FPGA/LV.A5
- U14 pad 41: /FPGA/LV.A11 -> /FPGA/LV.A4
- U14 pad 43: /FPGA/LV.A12 -> /FPGA/LV.A3
- U14 pad 44: /FPGA/LV.A13 -> /FPGA/LV.A2
- U14 pad 46: /FPGA/LV.A14 -> /FPGA/LV.A1
- U14 pad 47: /FPGA/LV.A15 -> /FPGA/LV.A0
- U14 pad 5: /A13 -> /A2
- U14 pad 6: /A12 -> /A3
- U14 pad 8: /A11 -> /A4
- U14 pad 9: /A10 -> /A5

Commit message: pinouts
Parts:
- removed C32, C33, C34, C35, C36, C37, C38, C39, C40, C41, C42, C43, C44, C45, C46, C47: 100nF, Capacitor_SMD:C_0603_1608Metric
- removed R20: R_Small_US, Resistor_SMD:R_0603_1608Metric
- removed U14, U15, U16, U17: SN74ALVC164245, Package_SO:TSSOP-48_6.1x12.5mm_P0.5mm
- added C817: 100nF, Capacitor_SMD:C_0603_1608Metric, F.Cu at (210.6, -9.92)
- added C818: 100nF, Capacitor_SMD:C_0603_1608Metric, F.Cu at (210.6, -7.41)
- added C819: 100nF, Capacitor_SMD:C_0603_1608Metric, F.Cu at (210.6, -4.90)
- added C820: 100nF, Capacitor_SMD:C_0603_1608Metric, F.Cu at (210.6, -2.39)
- added C822: 100nF, Capacitor_SMD:C_0603_1608Metric, F.Cu at (210.6, 0.12)
- added C823: 100nF, Capacitor_SMD:C_0603_1608Metric, F.Cu at (210.6, 2.63)
- added C824: 100nF, Capacitor_SMD:C_0603_1608Metric, F.Cu at (214.6, -9.92)
- added C825: 100nF, Capacitor_SMD:C_0603_1608Metric, F.Cu at (214.6, -7.41)
- added C826: 100nF, Capacitor_SMD:C_0603_1608Metric, F.Cu at (214.6, -4.90)
- added C827: 100nF, Capacitor_SMD:C_0603_1608Metric, F.Cu at (214.6, -2.39)
- added C828: 100nF, Capacitor_SMD:C_0603_1608Metric, F.Cu at (214.6, 0.12)
- added C829: 100nF, Capacitor_SMD:C_0603_1608Metric, F.Cu at (214.6, 2.63)
- added C830: 100nF, Capacitor_SMD:C_0603_1608Metric, F.Cu at (218.7, -9.92)
- added C831: 100nF, Capacitor_SMD:C_0603_1608Metric, F.Cu at (218.7, -7.41)
- added C832: 100nF, Capacitor_SMD:C_0603_1608Metric, F.Cu at (218.7, -4.90)
- added C833: 100nF, Capacitor_SMD:C_0603_1608Metric, F.Cu at (218.7, -2.39)
- added R807: R_Small_US, Resistor_SMD:R_0603_1608Metric, F.Cu at (218.7, 0.12)
- added U804: SN74ALVC164245, Package_SO:TSSOP-48_6.1x12.5mm_P0.5mm, F.Cu at (216.3, 86.9)
- added U805: SN74ALVC164245, Package_SO:TSSOP-48_6.1x12.5mm_P0.5mm, F.Cu at (242.0, 56.8)
- added U806: SN74ALVC164245, Package_SO:TSSOP-48_6.1x12.5mm_P0.5mm, F.Cu at (247.4, 124.9)
- added U807: SN74ALVC164245, Package_SO:TSSOP-48_6.1x12.5mm_P0.5mm, F.Cu at (216.3, 108.2)
- moved C805 197.1 mm to (260.9, 54.8), turned to -90 degrees
- moved C807 194.4 mm to (255.9, 54.8), turned to -90 degrees
- moved U802 193.1 mm to (258.3, 56.8), turned to 90 degrees
- moved C803 190.9 mm to (260.9, 59.6), turned to 90 degrees
- moved C402 188.6 mm to (269.7, 125.1)
- moved U401 188.6 mm to (265.8, 125.2)
- moved C802 188.1 mm to (255.9, 59.6), turned to 90 degrees
- moved R201 182.1 mm to (275.4, 110.7), turned to 180 degrees
- moved R206 180.2 mm to (275.4, 108.2), turned to 180 degrees
- moved R203 178.3 mm to (275.4, 105.7), turned to 180 degrees
- moved R211 176.5 mm to (275.4, 103.1), turned to 180 degrees
- moved C206 176.3 mm to (264.9, 118.4), turned to 180 degrees
- moved R212 174.8 mm to (275.4, 100.6), turned to 180 degrees
- moved R213 173.1 mm to (275.4, 98.0), turned to 180 degrees
- moved R215 171.4 mm to (275.4, 95.5), turned to 180 degrees
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- renumbered C1 to C201, C2 to C202, C3 to C203, C4 to C204, C5 to C205, C6 to C206, C19 to C207, C21 to C301, C22 to C302, C23 to C401, C24 to C402, C7 to C501, C25 to C502, C15 to C503, C16 to C504, C8 to C505, C11 to C506, C13 to C507, C9 to C508, C26 to C509, C18 to C510, C17 to C511, C10 to C512, C12 to C513, C14 to C514, C27 to C601, C64 to C701, C66 to C702, C65 to C703, C67 to C704, C28 to C705, C31 to C801, C51 to C802, C52 to C803, C76 to C804, C53 to C805, C29 to C806, C54 to C807, C20 to C808, C60 to C809, C61 to C810, C68 to C811, C69 to C812, C70 to C813, C71 to C814, C72 to C815, C50 to C816, C56 to C821, C48 to C834, C57 to C835, C62 to C836, C30 to C837, C49 to C838, C58 to C839, C63 to C840, C55 to C841, C59 to C842, C74 to C901, C75 to C902, C73 to C903, D1 to D801, D2 to D802, D3 to D803, FB1 to FB201, J1 to J701, J2 to J801, JS1 to JS501, JS2 to JS502, R26 to R201, R3 to R202, R28 to R203, R4 to R204, R5 to R205, R1 to R206, R6 to R207, R7 to R208, R8 to R209, R9 to R210, R11 to R211, R12 to R212, R13 to R213, R27 to R214, R29 to R215, R2 to R501, R21 to R601, R22 to R602, R16 to R801, R23 to R802, R17 to R803, R18 to R804, R14 to R805, R19 to R806, R10 to R808, R15 to R809, R25 to R901, R24 to R902, RN2 to RN201, SW1 to SW801, SW2 to SW901, U1 to U201, U5 to U202, U6 to U301, U7 to U302, U8 to U401, U2 to U501, U4 to U502, U3 to U503, U9 to U601, U20 to U701, U21 to U702, U13 to U801, U10 to U802, U11 to U803, U18 to U808, U12 to U809, U19 to U810, U23 to U901, U22 to U902, X1 to X401, X2 to X402, X3 to X403, Y1 to Y501
Connections:
- U802 pad 11: /SIZ1 -> /~{TS}
- U802 pad 12: /SIZ0 -> /~{TIP}
- U802 pad 13: /R/~{W} -> unconnected-(U802A-2B1-Pad13)
- U802 pad 2: /~{DS} -> /TM2
- U802 pad 20: /~{TIP} -> unconnected-(U802A-2B6-Pad20)
- U802 pad 22: /~{TS} -> unconnected-(U802A-2B7-Pad22)
- U802 pad 3: /TT1 -> /TM1
- U802 pad 37: unconnected-(U10A-1A8-Pad37) -> /FPGA/LV_~{TIP}
- U802 pad 38: unconnected-(U10A-1A7-Pad38) -> /FPGA/LV_~{TS}
- U802 pad 40: unconnected-(U10A-1A6-Pad40) -> /FPGA/LV_SIZ1
- U802 pad 41: unconnected-(U10A-1A5-Pad41) -> /FPGA/LV_SIZ0
- U802 pad 43: unconnected-(U10A-1A4-Pad43) -> /FPGA/LV_R/~{W}
- U802 pad 44: unconnected-(U10A-1A3-Pad44) -> /FPGA/LV_TM0
- U802 pad 46: unconnected-(U10A-1A2-Pad46) -> /FPGA/LV_TM1
- U802 pad 47: unconnected-(U10A-1A1-Pad47) -> /FPGA/LV_TM2
- U802 pad 5: /TT0 -> /TM0
- U802 pad 6: /TM2 -> /R/~{W}
- U802 pad 8: /TM1 -> /SIZ0
- U802 pad 9: /TM0 -> /SIZ1
- U803 pad 1: unconnected-(U11D-IOL_2A-Pad1) -> /FPGA/LV_D16
- U803 pad 10: unconnected-(U11D-IOL_5B-Pad10) -> /FPGA/LV_TM2
- U803 pad 101: unconnected-(U11B-IOR_160-Pad101) -> /FPGA/LV_~{68150_DS}
- U803 pad 102: unconnected-(U11B-IOR_161-Pad102) -> /FPGA/LV_D0
- U803 pad 104: unconnected-(U11B-IOR_164-Pad104) -> /FPGA/LV_D1
- U803 pad 105: unconnected-(U11B-IOR_165-Pad105) -> /FPGA/LV_D2
- U803 pad 106: unconnected-(U11B-IOR_166-Pad106) -> /FPGA/LV_D3
- U803 pad 107: unconnected-(U11B-IOR_167-Pad107) -> /FPGA/LV_D4
- U803 pad 11: unconnected-(U11D-IOL_8A-Pad11) -> /FPGA/LV_~{DSACK0}
- U803 pad 110: unconnected-(U11A-IOT_168-Pad110) -> /FPGA/LV_D5
- U803 pad 112: unconnected-(U11A-IOT_169-Pad112) -> /FPGA/LV_D6
- U803 pad 113: unconnected-(U11A-IOT_170-Pad113) -> /FPGA/LV_D7
- U803 pad 114: unconnected-(U11A-IOT_171-Pad114) -> /FPGA/LV_D8
- U803 pad 115: unconnected-(U11A-IOT_172-Pad115) -> /FPGA/LV_D9
- U803 pad 116: unconnected-(U11A-IOT_173-Pad116) -> /FPGA/LV_D10
- U803 pad 117: unconnected-(U11A-IOT_174-Pad117) -> /FPGA/LV_D11
- U803 pad 118: unconnected-(U11A-IOT_177-Pad118) -> /FPGA/LV_D12
- U803 pad 119: unconnected-(U11A-IOT_178-Pad119) -> /FPGA/LV_D13
- U803 pad 12: unconnected-(U11D-IOL_8B-Pad12) -> /FPGA/LV_~{DSACK1}
- U803 pad 120: unconnected-(U11A-IOT_179-Pad120) -> /FPGA/LV_D14
- U803 pad 121: unconnected-(U11A-IOT_181-Pad121) -> /FPGA/LV_D15
- U803 pad 122: unconnected-(U11A-IOT_190-Pad122) -> /FPGA/LV_R/~{W}
- U803 pad 124: unconnected-(U11A-IOT_191-Pad124) -> /FPGA/LV_D31
- U803 pad 125: unconnected-(U11A-IOT_192-Pad125) -> /FPGA/LV_D30
- U803 pad 128: unconnected-(U11A-IOT_197_GBIN1-Pad128) -> /FPGA/LV_D29
- U803 pad 129: unconnected-(U11A-IOT_198_GBIN0-Pad129) -> /FPGA/LV_D28
- U803 pad 130: unconnected-(U11A-IOT_206-Pad130) -> /FPGA/LV_D27
- U803 pad 134: unconnected-(U11A-IOT_212-Pad134) -> /FPGA/LV_D26
- U803 pad 135: unconnected-(U11A-IOT_213-Pad135) -> /FPGA/LV_D25
- U803 pad 136: unconnected-(U11A-IOT_214-Pad136) -> /FPGA/LV_D24
- U803 pad 137: unconnected-(U11A-IOT_215-Pad137) -> /FPGA/LV_D23
- U803 pad 138: unconnected-(U11A-IOT_216-Pad138) -> /FPGA/LV_D22
- U803 pad 139: unconnected-(U11A-IOT_217-Pad139) -> /FPGA/LV_D21
- U803 pad 141: unconnected-(U11A-IOT_219-Pad141) -> /FPGA/LV_D20
- U803 pad 142: unconnected-(U11A-IOT_220-Pad142) -> /FPGA/LV_D19
- U803 pad 143: unconnected-(U11A-IOT_221-Pad143) -> /FPGA/LV_D18
- U803 pad 144: unconnected-(U11A-IOT_222-Pad144) -> /FPGA/LV_D17
- U803 pad 15: unconnected-(U11D-IOL_10A-Pad15) -> /FPGA/LV_~{TEA}
- U803 pad 16: unconnected-(U11D-IOL_10B-Pad16) -> /FPGA/LV_~{TCI}
- U803 pad 17: unconnected-(U11D-IOL_12A-Pad17) -> /FPGA/LV_~{TBI}
- U803 pad 18: unconnected-(U11D-IOL_12B-Pad18) -> /FPGA/LV.A15
- U803 pad 19: unconnected-(U11D-IOL_13A-Pad19) -> /FPGA/LV.A14
- U803 pad 2: unconnected-(U11D-IOL_2B-Pad2) -> /FPGA/LV_~{IPL0}
- U803 pad 20: unconnected-(U11D-IOL_13B_GBIN7-Pad20) -> /FPGA/LV.A13
- U803 pad 21: unconnected-(U11D-IOL_14A_GBIN6-Pad21) -> /FPGA/LV.A12
- U803 pad 22: unconnected-(U11D-IOL_14B-Pad22) -> /FPGA/LV.A11
- U803 pad 23: unconnected-(U11D-IOL_17A-Pad23) -> /FPGA/LV.A10
- U803 pad 24: unconnected-(U11D-IOL_17B-Pad24) -> /FPGA/LV.A9
- U803 pad 25: unconnected-(U11D-IOL_18A-Pad25) -> /FPGA/LV.A8
- U803 pad 26: unconnected-(U11D-IOL_18B-Pad26) -> /FPGA/LV.A7
- U803 pad 28: unconnected-(U11D-IOL_23A-Pad28) -> /FPGA/LV.A6
- U803 pad 29: unconnected-(U11D-IOL_23B-Pad29) -> /FPGA/LV.A5
- U803 pad 3: unconnected-(U11D-IOL_3A-Pad3) -> /FPGA/LV_~{IPL1}
- U803 pad 31: unconnected-(U11D-IOL_24A-Pad31) -> /FPGA/LV.A4
- U803 pad 32: unconnected-(U11D-IOL_24B-Pad32) -> /FPGA/LV.A3
- U803 pad 33: unconnected-(U11D-IOL_25A-Pad33) -> /FPGA/LV.A2
- U803 pad 34: unconnected-(U11D-IOL_25B-Pad34) -> /FPGA/LV.A1
- U803 pad 37: unconnected-(U11C-IOB_56-Pad37) -> /FPGA/LV.A0
- U803 pad 39: unconnected-(U11C-IOB_61-Pad39) -> /FPGA/LV_COM_IACK
- U803 pad 4: unconnected-(U11D-IOL_3B-Pad4) -> /FPGA/LV_~{IPL2}
- U803 pad 41: unconnected-(U11C-IOB_63-Pad41) -> /FPGA/LV_RAM_CS
- U803 pad 42: unconnected-(U11C-IOB_64-Pad42) -> /FPGA/LV_AVEC
- U803 pad 43: unconnected-(U11C-IOB_71-Pad43) -> /FPGA/LV_COM_CS
- U803 pad 44: unconnected-(U11C-IOB_72-Pad44) -> /FPGA/LV_68150_CS
- U803 pad 45: unconnected-(U11C-IOB_73-Pad45) -> /FPGA/FPGA_D_~{OE}
- U803 pad 47: unconnected-(U11C-IOB_79-Pad47) -> /FPGA/FPGA_D_DIR
- U803 pad 48: unconnected-(U11C-IOB_80-Pad48) -> /FPGA/LV_~{RST}
- U803 pad 52: unconnected-(U11C-IOB_82_GBIN4-Pad52) -> /FPGA/FPGA_LED
- U803 pad 55: unconnected-(U11C-IOB_91-Pad55) -> /FPGA/FPGA_BTN
- U803 pad 56: unconnected-(U11C-IOB_94-Pad56) -> /FPGA/FLASH_IO2
- U803 pad 60: unconnected-(U11C-IOB_95-Pad60) -> /FPGA/FLASH_IO3
- U803 pad 62: unconnected-(U11C-IOB_102-Pad62) -> /FPGA/FPGA_D_DIR
- U803 pad 63: unconnected-(U11C-IOB_103_CBSEL0-Pad63) -> /FPGA/FPGA_D_~{OE}
- U803 pad 64: unconnected-(U11C-IOB_104_CBSEL1-Pad64) -> /FPGA/LV_~{COM_IRQ}
- U803 pad 7: unconnected-(U11D-IOL_4A-Pad7) -> /FPGA/LV_~{TA}
- U803 pad 73: unconnected-(U11B-IOR_109-Pad73) -> /FPGA/LV.A16
- U803 pad 74: unconnected-(U11B-IOR_110-Pad74) -> /FPGA/LV.A17
- U803 pad 75: unconnected-(U11B-IOR_111-Pad75) -> /FPGA/LV.A18
- U803 pad 76: unconnected-(U11B-IOR_112-Pad76) -> /FPGA/LV.A19
- U803 pad 78: unconnected-(U11B-IOR_114-Pad78) -> /FPGA/LV.A20
- U803 pad 79: unconnected-(U11B-IOR_115-Pad79) -> /FPGA/LV.A21
- U803 pad 8: unconnected-(U11D-IOL_4B-Pad8) -> /FPGA/LV_TM0
- U803 pad 80: unconnected-(U11B-IOR_116-Pad80) -> /FPGA/LV.A22
- U803 pad 81: unconnected-(U11B-IOR_117-Pad81) -> /FPGA/LV.A23
- U803 pad 82: unconnected-(U11B-IOR_118-Pad82) -> /FPGA/LV.A24
- U803 pad 83: unconnected-(U11B-IOR_119-Pad83) -> /FPGA/LV.A25
- U803 pad 84: unconnected-(U11B-IOR_120-Pad84) -> /FPGA/LV.A26
- U803 pad 85: unconnected-(U11B-IOR_128-Pad85) -> /FPGA/LV.A27
- U803 pad 87: unconnected-(U11B-IOR_136-Pad87) -> /FPGA/LV.A28
- U803 pad 88: unconnected-(U11B-IOR_137-Pad88) -> /FPGA/LV.A29
- U803 pad 9: unconnected-(U11D-IOL_5A-Pad9) -> /FPGA/LV_TM1
- U803 pad 90: unconnected-(U11B-IOR_138-Pad90) -> /FPGA/LV.A30
- U803 pad 91: unconnected-(U11B-IOR_139-Pad91) -> /FPGA/LV.A31
- U803 pad 93: unconnected-(U11B-IOR_140_GBIN3-Pad93) -> /FPGA/LV_TT0
- U803 pad 94: unconnected-(U11B-IOR_141_GBIN2-Pad94) -> /BCLK
- U803 pad 95: unconnected-(U11B-IOR_144-Pad95) -> /FPGA/LV_TT1
- U803 pad 96: unconnected-(U11B-IOR_146-Pad96) -> /FPGA/LV_SIZ0
- U803 pad 97: unconnected-(U11B-IOR_147-Pad97) -> /FPGA/LV_SIZ1
- U803 pad 98: unconnected-(U11B-IOR_148-Pad98) -> /FPGA/LV_~{TS}
- U803 pad 99: unconnected-(U11B-IOR_152-Pad99) -> /FPGA/LV_~{TIP}

Commit message: layout
Parts:
- moved U805 122.9 mm to (126.4, 98.6)
- moved X402 117.1 mm to (147.0, 132.8), turned to 90 degrees
- moved U804 110.3 mm to (106.6, 98.6), turned to 90 degrees
- moved X403 109.3 mm to (147.0, 125.2), turned to 90 degrees
- moved R602 108.2 mm to (93.6, 138.7), turned to 90 degrees
- moved C401 106.0 mm to (147.0, 121.3), turned to 90 degrees
- moved C830 99.0 mm to (123.8, 18.2)
- moved C831 99.0 mm to (123.8, 20.8)
- moved C832 99.0 mm to (123.8, 23.3)
- moved C833 99.0 mm to (123.8, 25.8)
- moved R807 99.0 mm to (123.8, 28.3)
- moved C824 99.0 mm to (119.8, 18.2)
- moved C825 99.0 mm to (119.8, 20.8)
- moved C826 99.0 mm to (119.8, 23.3)
- moved C827 99.0 mm to (119.8, 25.8)
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Connections:
- R807 pad 2: /FPGA/FPGA_DBUF_~{OE} -> /FPGA/FPGA_D_~{OE}
- U802 pad 13: unconnected-(U802A-2B1-Pad13) -> /TT1
- U802 pad 14: unconnected-(U802A-2B2-Pad14) -> /TT0
- U802 pad 23: unconnected-(U802A-2B8-Pad23) -> /~{DS}
- U802 pad 26: unconnected-(U802A-2A8-Pad26) -> /FPGA/LV_~{68150_DS}
- U802 pad 30: unconnected-(U802A-2A5-Pad30) -> /FPGA/LV_~{RST}
- U802 pad 33: unconnected-(U802A-2A3-Pad33) -> /FPGA/LV_~{COM_IRQ}
- U802 pad 35: unconnected-(U802A-2A2-Pad35) -> /FPGA/LV_TT0
- U802 pad 36: unconnected-(U802A-2A1-Pad36) -> /FPGA/LV_TT1
- U802 pad 6: /R/~{W} -> /SIZ1
- U802 pad 9: /SIZ1 -> /R/~{W}
- U803 pad 1: /FPGA/LV_D16 -> /FPGA/LV_D6
- U803 pad 10: /FPGA/LV_TM2 -> /FPGA/LV.A10
- U803 pad 101: /FPGA/LV_~{68150_DS} -> /FPGA/LV_~{DSACK0}
- U803 pad 102: /FPGA/LV_D0 -> /FPGA/LV_~{DSACK1}
- U803 pad 104: /FPGA/LV_D1 -> /FPGA/LV_~{TA}
- U803 pad 105: /FPGA/LV_D2 -> /FPGA/LV_~{IPL0}
- U803 pad 106: /FPGA/LV_D3 -> /FPGA/LV_~{IPL1}
- U803 pad 107: /FPGA/LV_D4 -> /FPGA/LV_~{IPL2}
- U803 pad 11: /FPGA/LV_~{DSACK0} -> /FPGA/LV.A11
- U803 pad 110: /FPGA/LV_D5 -> /FPGA/FPGA_D_DIR
- U803 pad 112: /FPGA/LV_D6 -> /FPGA/FPGA_D_~{OE}
- U803 pad 113: /FPGA/LV_D7 -> /FPGA/LV_D31
- U803 pad 114: /FPGA/LV_D8 -> /FPGA/LV_D30
- U803 pad 115: /FPGA/LV_D9 -> /FPGA/LV_D29
- U803 pad 116: /FPGA/LV_D10 -> /FPGA/LV_D28
- U803 pad 117: /FPGA/LV_D11 -> /FPGA/LV_D27
- U803 pad 118: /FPGA/LV_D12 -> /FPGA/LV_D26
- U803 pad 119: /FPGA/LV_D13 -> /FPGA/LV_D25
- U803 pad 12: /FPGA/LV_~{DSACK1} -> /FPGA/LV.A12
- U803 pad 120: /FPGA/LV_D14 -> /FPGA/LV_D24
- U803 pad 121: /FPGA/LV_D15 -> /FPGA/LV_D23
- U803 pad 122: /FPGA/LV_R/~{W} -> /FPGA/LV_D22
- U803 pad 124: /FPGA/LV_D31 -> /FPGA/LV_D21
- U803 pad 125: /FPGA/LV_D30 -> /FPGA/LV_D20
- U803 pad 128: /FPGA/LV_D29 -> /FPGA/LV_D19
- U803 pad 129: /FPGA/LV_D28 -> /FPGA/LV_D18
- U803 pad 130: /FPGA/LV_D27 -> /FPGA/LV_D17
- U803 pad 134: /FPGA/LV_D26 -> /FPGA/LV_D16
- U803 pad 135: /FPGA/LV_D25 -> /FPGA/LV_D15
- U803 pad 136: /FPGA/LV_D24 -> /FPGA/LV_D14
- U803 pad 137: /FPGA/LV_D23 -> /FPGA/LV_D13
- U803 pad 138: /FPGA/LV_D22 -> /FPGA/LV_D12
- U803 pad 139: /FPGA/LV_D21 -> /FPGA/LV_D11
- U803 pad 141: /FPGA/LV_D20 -> /FPGA/LV_D10
- U803 pad 142: /FPGA/LV_D19 -> /FPGA/LV_D9
- U803 pad 143: /FPGA/LV_D18 -> /FPGA/LV_D8
- U803 pad 144: /FPGA/LV_D17 -> /FPGA/LV_D7
- U803 pad 15: /FPGA/LV_~{TEA} -> /FPGA/LV.A13
- U803 pad 16: /FPGA/LV_~{TCI} -> /FPGA/LV.A14
- U803 pad 17: /FPGA/LV_~{TBI} -> /FPGA/LV.A16
- U803 pad 19: /FPGA/LV.A14 -> /FPGA/LV.A17
- U803 pad 2: /FPGA/LV_~{IPL0} -> /FPGA/LV_D5
- U803 pad 20: /FPGA/LV.A13 -> /BCLK
- U803 pad 21: /FPGA/LV.A12 -> /FPGA/LV.A19
- U803 pad 22: /FPGA/LV.A11 -> /FPGA/LV.A18
- U803 pad 23: /FPGA/LV.A10 -> /FPGA/LV.A23
- U803 pad 24: /FPGA/LV.A9 -> /FPGA/LV.A20
- U803 pad 25: /FPGA/LV.A8 -> /FPGA/LV.A25
- U803 pad 26: /FPGA/LV.A7 -> /FPGA/LV.A21
- U803 pad 28: /FPGA/LV.A6 -> /FPGA/LV.A9
- U803 pad 29: /FPGA/LV.A5 -> /FPGA/LV.A8
- U803 pad 3: /FPGA/LV_~{IPL1} -> /FPGA/LV_D4
- U803 pad 31: /FPGA/LV.A4 -> unconnected-(U803D-IOL_24A-Pad31)
- U803 pad 32: /FPGA/LV.A3 -> unconnected-(U803D-IOL_24B-Pad32)
- U803 pad 33: /FPGA/LV.A2 -> unconnected-(U803D-IOL_25A-Pad33)
- U803 pad 34: /FPGA/LV.A1 -> unconnected-(U803D-IOL_25B-Pad34)
- U803 pad 4: /FPGA/LV_~{IPL2} -> /FPGA/LV_D3
- U803 pad 45: /FPGA/FPGA_D_~{OE} -> unconnected-(U803C-IOB_73-Pad45)
- U803 pad 47: /FPGA/FPGA_D_DIR -> unconnected-(U803C-IOB_79-Pad47)
- U803 pad 56: /FPGA/FLASH_IO2 -> unconnected-(U803C-IOB_94-Pad56)
- U803 pad 60: /FPGA/FLASH_IO3 -> unconnected-(U803C-IOB_95-Pad60)
- U803 pad 62: /FPGA/FPGA_D_DIR -> unconnected-(U803C-IOB_102-Pad62)
- U803 pad 63: /FPGA/FPGA_D_~{OE} -> /FPGA/FLASH_IO3
- U803 pad 64: /FPGA/LV_~{COM_IRQ} -> /FPGA/FLASH_IO2
- U803 pad 7: /FPGA/LV_~{TA} -> /FPGA/LV_D2
- U803 pad 73: /FPGA/LV.A16 -> /FPGA/LV.A31
- U803 pad 74: /FPGA/LV.A17 -> /FPGA/LV.A29
- U803 pad 75: /FPGA/LV.A18 -> /FPGA/LV.A27
- U803 pad 76: /FPGA/LV.A19 -> /FPGA/LV.A30
- U803 pad 78: /FPGA/LV.A20 -> /FPGA/LV.A24
- U803 pad 79: /FPGA/LV.A21 -> /FPGA/LV.A28
- U803 pad 8: /FPGA/LV_TM0 -> /FPGA/LV_D1
- U803 pad 80: /FPGA/LV.A22 -> /FPGA/LV.A26
- U803 pad 81: /FPGA/LV.A23 -> /FPGA/LV.A22
- U803 pad 82: /FPGA/LV.A24 -> /FPGA/LV.A6
- U803 pad 83: /FPGA/LV.A25 -> /FPGA/LV.A7
- U803 pad 84: /FPGA/LV.A26 -> /FPGA/LV.A5
- U803 pad 85: /FPGA/LV.A27 -> /FPGA/LV.A4
- U803 pad 87: /FPGA/LV.A28 -> /FPGA/LV.A3
- U803 pad 88: /FPGA/LV.A29 -> /FPGA/LV.A2
- U803 pad 9: /FPGA/LV_TM1 -> /FPGA/LV_D0
- U803 pad 90: /FPGA/LV.A30 -> /FPGA/LV.A1
- U803 pad 91: /FPGA/LV.A31 -> /FPGA/LV.A0
- U803 pad 93: /FPGA/LV_TT0 -> unconnected-(U803B-IOR_140_GBIN3-Pad93)
- U803 pad 94: /BCLK -> unconnected-(U803B-IOR_141_GBIN2-Pad94)
- U803 pad 95: /FPGA/LV_TT1 -> unconnected-(U803B-IOR_144-Pad95)
- U803 pad 96: /FPGA/LV_SIZ0 -> unconnected-(U803B-IOR_146-Pad96)
- U803 pad 97: /FPGA/LV_SIZ1 -> unconnected-(U803B-IOR_147-Pad97)
- U803 pad 98: /FPGA/LV_~{TS} -> unconnected-(U803B-IOR_148-Pad98)
- U803 pad 99: /FPGA/LV_~{TIP} -> unconnected-(U803B-IOR_152-Pad99)
- U804 pad 1: /FPGA/FPGA_DBUF_DIR -> /FPGA/FPGA_D_DIR
- U804 pad 11: /D13 -> /D25
- U804 pad 12: /D18 -> /D24
- U804 pad 13: /D14 -> /D23
- U804 pad 14: /D15 -> /D22
- U804 pad 16: /D17 -> /D21
- U804 pad 17: /D23 -> /D20
- U804 pad 2: /D8 -> /D31
- U804 pad 20: /D22 -> /D18
- U804 pad 22: /D20 -> /D17
- U804 pad 23: /D25 -> /D16
- U804 pad 24: /FPGA/FPGA_DBUF_DIR -> /FPGA/FPGA_D_DIR
- U804 pad 25: /FPGA/FPGA_DBUF_~{OE} -> /FPGA/FPGA_D_~{OE}
- U804 pad 26: /FPGA/LV_D15 -> /FPGA/LV_D16
- U804 pad 27: /FPGA/LV_D14 -> /FPGA/LV_D17
- U804 pad 29: /FPGA/LV_D13 -> /FPGA/LV_D18
- U804 pad 3: /D9 -> /D30
- U804 pad 30: /FPGA/LV_D12 -> /FPGA/LV_D19
- U804 pad 32: /FPGA/LV_D11 -> /FPGA/LV_D20
- U804 pad 33: /FPGA/LV_D10 -> /FPGA/LV_D21
- U804 pad 35: /FPGA/LV_D9 -> /FPGA/LV_D22
- U804 pad 36: /FPGA/LV_D8 -> /FPGA/LV_D23
- U804 pad 37: /FPGA/LV_D7 -> /FPGA/LV_D24
- U804 pad 38: /FPGA/LV_D6 -> /FPGA/LV_D25
- U804 pad 40: /FPGA/LV_D5 -> /FPGA/LV_D26
- U804 pad 41: /FPGA/LV_D4 -> /FPGA/LV_D27
- U804 pad 43: /FPGA/LV_D3 -> /FPGA/LV_D28
- U804 pad 44: /FPGA/LV_D2 -> /FPGA/LV_D29
- U804 pad 46: /FPGA/LV_D1 -> /FPGA/LV_D30
- U804 pad 47: /FPGA/LV_D0 -> /FPGA/LV_D31
- U804 pad 48: /FPGA/FPGA_DBUF_~{OE} -> /FPGA/FPGA_D_~{OE}
- U804 pad 5: /D10 -> /D29
- U804 pad 6: /D11 -> /D28
- U804 pad 8: /D12 -> /D27
- U804 pad 9: /D16 -> /D26
- U805 pad 1: /FPGA/FPGA_DBUF_DIR -> /FPGA/FPGA_D_DIR
- U805 pad 11: /D29 -> /D9
- U805 pad 12: /D30 -> /D8
- U805 pad 13: /A7 -> /D7
- U805 pad 14: /A6 -> /D6
- U805 pad 16: /A5 -> /D5
- U805 pad 17: /A4 -> /D4
- U805 pad 19: /A3 -> /D3
- U805 pad 2: /D21 -> /D15
- U805 pad 20: /A2 -> /D2
- U805 pad 22: /A1 -> /D1
- U805 pad 23: /A0 -> /D0
- U805 pad 24: unconnected-(U805A-2DIR-Pad24) -> /FPGA/FPGA_D_DIR
- U805 pad 25: unconnected-(U805A-*2OE-Pad25) -> /FPGA/FPGA_D_~{OE}
- U805 pad 26: /FPGA/LV.A0 -> /FPGA/LV_D0
- U805 pad 27: /FPGA/LV.A1 -> /FPGA/LV_D1
- U805 pad 29: /FPGA/LV.A2 -> /FPGA/LV_D2
- U805 pad 3: /D24 -> /D14
- U805 pad 30: /FPGA/LV.A3 -> /FPGA/LV_D3
- U805 pad 32: /FPGA/LV.A4 -> /FPGA/LV_D4
- U805 pad 33: /FPGA/LV.A5 -> /FPGA/LV_D5
- U805 pad 35: /FPGA/LV.A6 -> /FPGA/LV_D6
- U805 pad 36: /FPGA/LV.A7 -> /FPGA/LV_D7
- U805 pad 37: /FPGA/LV_D23 -> /FPGA/LV_D8
- U805 pad 38: /FPGA/LV_D22 -> /FPGA/LV_D9
- U805 pad 40: /FPGA/LV_D21 -> /FPGA/LV_D10
- U805 pad 41: /FPGA/LV_D20 -> /FPGA/LV_D11
- U805 pad 43: /FPGA/LV_D19 -> /FPGA/LV_D12
- U805 pad 44: /FPGA/LV_D18 -> /FPGA/LV_D13
- U805 pad 46: /FPGA/LV_D17 -> /FPGA/LV_D14
- U805 pad 47: /FPGA/LV_D16 -> /FPGA/LV_D15
- U805 pad 48: /FPGA/FPGA_DBUF_~{OE} -> /FPGA/FPGA_D_~{OE}
- U805 pad 5: /D26 -> /D13
- U805 pad 6: /D28 -> /D12
- U805 pad 8: /D27 -> /D11
- U805 pad 9: /D31 -> /D10
- U807 pad 13: /D0 -> /A6
- U807 pad 14: /D1 -> /A7
- U807 pad 16: /D3 -> /A5
- U807 pad 17: /D2 -> /A4
- U807 pad 19: /D4 -> /A3
- U807 pad 20: /D5 -> /A2
- U807 pad 22: /D6 -> /A1
- U807 pad 23: /D7 -> /A0
- U807 pad 24: unconnected-(U807A-2DIR-Pad24) -> GND
- U807 pad 25: unconnected-(U807A-*2OE-Pad25) -> GND
- U807 pad 26: /FPGA/LV_D7 -> /FPGA/LV.A0
- U807 pad 27: /FPGA/LV_D6 -> /FPGA/LV.A1
- U807 pad 29: /FPGA/LV_D5 -> /FPGA/LV.A2
- U807 pad 30: /FPGA/LV_D4 -> /FPGA/LV.A3
- U807 pad 32: /FPGA/LV_D2 -> /FPGA/LV.A4
- U807 pad 33: /FPGA/LV_D3 -> /FPGA/LV.A5
- U807 pad 35: /FPGA/LV_D1 -> /FPGA/LV.A7
- U807 pad 36: /FPGA/LV_D0 -> /FPGA/LV.A6
Routing:
- net /BCLK: track 0.00 -> 75.5 mm
- net GND: track 0.00 -> 65.7 mm, vias 1 -> 15
- net +3.3V: track 0.00 -> 61.9 mm, vias 0 -> 11
- net +1V2: track 0.00 -> 59.0 mm, vias 0 -> 4
- net /Clock/CLK33: track 0.00 -> 58.8 mm
- net /CPU/PCLK: track 0.00 -> 34.1 mm
- net /FPGA/VCC_PLL: track 0.00 -> 28.4 mm, vias 0 -> 3
- net /FPGA/FLASH_IO3: track 0.00 -> 24.2 mm
- net /FPGA/GND_PLL: track 0.00 -> 23.4 mm, vias 0 -> 3
- net +5V: track 0.00 -> 18.7 mm, vias 0 -> 2
- net /FPGA/FLASH_SCK: track 0.00 -> 18.4 mm
- net /FPGA/FLASH_MOSI: track 0.00 -> 16.0 mm
- net /FPGA/FLASH_IO2: track 0.00 -> 8.33 mm
- net /FPGA/FLASH_MISO: track 0.00 -> 8.03 mm
- net /FPGA/FLASH_SS: track 0.00 -> 7.93 mm
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- added copper zone on In2.Cu, net +3.3V
- added copper zone on In2.Cu, net +5V
- added copper zone on In1.Cu, net GND
